File: Hardware/Sensor.kicad_sch (KiCad schematic)
At the start: 6 parts, among them U5 BNO086, Y401 32.768 kHz

Commit message: Finished the schematic design.
Parts:
- added C401, C402: 100n, Capacitor_SMD:C_0402_1005Metric, symbol Device:C
- added R401, R402, R406, R407: 4k7, symbol Device:R
- added R403, R404, R405: 10k, symbol Device:R
- added U402: ICE40UL1K-CM36AI, Package_BGA:UCBGA-36_2.5x2.5mm_Layout6x6_P0.4mm, symbol Custom_VoxLink_Symbols:ICE40UL1K-CM36AI
- renumbered C401 to C404, C402 to C405, R401 to R408, U5 to U401
Connections:
- net +3V3: now also C401.1, C402.1, R401.1, R402.1, R403.1, R404.1, R405.1, R406.1, R407.1
- net BNO_SCL: now also R402.2, U402.B2 (IOT_24B)
- net BNO_SDA: now also R401.2, U402.A4 (IOT_19A)
- net GND: now also C401.2, C402.2
- net BNO_~{RST}: now reaches U401.11 (~{RST})
- net BNO_~{RST}: now also R405.2, U402.B5 (IOT_18B)
- net at U401.15 (ENV_SCL): now also R407.2
- net at U401.16 (ENV_SDA): now also R406.2
- net at U401.17 (SA0/H_MOSI): now also R404.2
- net at U401.4 (~{BOOT}): now also R403.2
- no-connect marks 0 -> 6
Other:
- note added: "For daisy-chaining temperatre/humidity sensors Needs to be teminated as I2C with pullup resistors"
- note added: "I2C Address Selection HIGH = 0x4B LOW = 0x4A"
- note added: "Interrupt to host device Only for SPI"
- note added: "Keep close to IC pads!"
- moved on the sheet: C403, C404, C405, R408, U401, Y401
