File: Hardware/System.kicad_sch (KiCad schematic)
At the start: 9 parts, among them SW301 Reset, U2 ICE40UL1K-CM36AI, U3 N25Q032A

Commit message: Finished the schematic design.
Parts:
- removed C1: 100n, Capacitor_SMD:C_0402_1005Metric, symbol Device:C
- removed unit 3 of U2
- added C301, C303, C304: 100n, Capacitor_SMD:C_0402_1005Metric, symbol Device:C
- added D301: TVS, Diode_SMD:D_0402_1005Metric, symbol Diode:1.5KExxA
- added D302, D303: LED, symbol Device:LED
- added D304: RX, symbol Device:LED
- added D305: TX, symbol Device:LED
- added J301: RJ45, rj45_molex_unshielded:CONN_855035-101_MOL, symbol rj45_molex_unshielded:RJ45_Molex_Unshielded
- added J302: TC2030, Connector:Tag-Connect_TC2030-IDC-FP_2x03_P1.27mm_Vertical, symbol Connector:Conn_ARM_SWD_TagConnect_TC2030
- added R301, R302, R304, R311: 22R, Resistor_SMD:R_0402_1005Metric, symbol Device:R
- added R305, R306, R307: 0R, symbol Device:R
- added R312, R313, R314: 500R, symbol Device:R
- added U301, U302, U303: TPD4E02B04, Package_SON:USON-10_2.5x1.0mm_P0.5mm, symbol Custom_VoxLink_Symbols:TPD4E02B04DQA
- added Y301: ASCO, Oscillator:Oscillator_SMD_Abracon_ASE-4Pin_3.2x2.5mm, symbol Oscillator:ASCO
- R303: value 10k -> 22R; footprint (none) -> Resistor_SMD:R_0402_1005Metric
- R310: renamed from R304; value 1k -> 500R
- renumbered C301 to C302, R301 to R308, R302 to R309, U3 to U304, U2 to U305, U2 to U306, U2 to U307
Connections:
- net CDONE: now also D302.2 (A)
- net FLASH_MISO: now also R303.1
- net FLASH_MOSI: now also R302.1
- net FLASH_SCK: now also R304.1
- net FLASH_~{CS}: now also R301.1
- net GND: now also C301.2, C303.2, C304.2, D301.2 (A2), D302.1 (K), J301.6 (GND), J302.5 (GND), R305.2, R306.2, R307.2, U301.3 (GND), U301.8 (NC), U302.3 (GND), U302.8 (NC), U303.3 (GND), U303.8 (NC), Y301.2 (GND)
- net VCCIO1: now also J302.1 (VCC); no longer R303.1
- net VCCIO2: now also C303.1, Y301.1 (Tri-State), Y301.4 (VDD)
- net ~{CRESET}: now also C304.1; no longer R303.2
- net at U307.A1 (RGB2): now also D305.1 (K)
- net at U307.A2 (RGB0): now also D303.1 (K)
- net at U307.B1 (RGB1): now also D304.1 (K)
- net ~{VOX_RX}_NOESD: now reaches U305.C1 (IOB_5B)
- net ~{VOX_RX}_NOESD: now also U302.5 (IN)
- net VOX_RX_NOESD: now reaches U305.D1 (IOB_4A)
- net VOX_RX_NOESD: now also U302.4 (IN)
- net 12MHZ_CLK: now reaches U305.D2 (IOB_8A_G4)
- net 12MHZ_CLK: now also R311.1
- net ~{VOX_CLK}_NOESD: now reaches U305.D6 (IOB_10A)
- net ~{VOX_CLK}_NOESD: now also U303.2 (IN)
- net ~{VOX_TX}_NOESD: now reaches U305.E1 (IOB_1B)
- net ~{VOX_TX}_NOESD: now also U302.2 (IN)
- net VOX_CLK_NOESD: now reaches U305.E2 (IOB_6A)
- net VOX_CLK_NOESD: now also U303.1 (IN)
- net VOX_TX_NOESD: now reaches U305.F1 (IOB_0A)
- net VOX_TX_NOESD: now also U302.1 (IN)
- new net: R303.2, U301.7 (NC)
- new net: D303.2 (A), R312.2
- new net: D305.2 (A), R314.2
- new net: R302.2, U301.9 (NC)
- new net: D304.2 (A), R313.2
- new net: R301.2, U301.10 (NC)
- new net: R304.2, U301.6 (NC)
- new net +3V3: C301.1, D301.1 (A1)
- new net FLASH_MISO_NOESD: J302.2 (SWDIO), U301.4 (IN)
- new net FLASH_MOSI_NOESD: J302.4 (SWCLK), U301.2 (IN)
- new net FLASH_SCK_NOESD: J302.6 (SWO), U301.5 (IN)
- new net FLASH_~{CS}_NOESD: J302.3 (~{RESET}), U301.1 (IN)
- new net OSC_OUT: R311.2, Y301.3 (OUT)
- new net VCC: J301.3 (VCC)
- new net VCCIO0: R312.1, R313.1, R314.1
- new net VOX_CLK: J301.4 (CLK), U303.10 (NC)
- new net VOX_RX: J301.1 (RX), U302.7 (NC)
- new net VOX_TX: J301.7 (TX), U302.10 (NC)
- new net ~{VOX_CLK}: J301.5 (~{CLK}), R306.1, U303.9 (NC)
- new net ~{VOX_RX}: J301.2 (~{RX}), R305.1, U302.6 (NC)
- new net ~{VOX_TX}: J301.8 (~{TX}), R307.1, U302.9 (NC)
- no-connect marks 0 -> 8
Other:
- note added: "CDONE is an Open-Drain Output which goes high after the device has been configured successfully"
- note added: "Chip is active when ~{CRESET} is LOW"
- note added: "ESD Protection IC"
- note added: "ESD Protection ICs"
- note added: "Ethernet Connector"
- note added: "FPGA Manual Reset"
- note added: "If LED shines, the device has not been configured properly!"
- note added: "No Placement (NOP) - Used in case a differential driver would not work -> ~{NEGATIVE} can be tied to GND"
- note added: "Used for LED driving"
- note added: "VCCIO0 = 3V3"
- moved on the sheet: C302, R308, R309, R310, U304
