File: Hardware/VoxLink.kicad_sch (KiCad schematic)
At the start: 0 parts

Commit message: Finished the schematic design.
Other:
- added sheet eFuse (efuse.kicad_sch)
- note added: "Technical Sheet Only! Please refer to the subsequent sheets for schematic"
Changed lines of the file:
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@@
 	(text "Root [1]"
 		(exclude_from_sim no)
-		(at 59.182 30.48 0)
+		(at 51.308 27.94 0)
 		(effects
 			(font
@@
 		)
 	)
+	(text "Technical Sheet Only!\nPlease refer to the subsequent sheets for schematic"
+		(exclude_from_sim no)
+		(at 141.732 58.674 0)
+		(effects
+			(font
+				(size 2.54 2.54)
+				(thickness 0.508)
+				(bold yes)
+			)
+		)
+	)
 	(sheet
-		(at 42.926 55.88)
+		(at 144.78 110.49)
+		(size 50.8 34.29)
+		(exclude_from_sim no)
+		(in_bom yes)
+		(on_board yes)
+		(dnp no)
+		(fields_autoplaced yes)
+		(stroke
+			(width 0.1524)
+			(type solid)
+		)
+		(fill
+			(color 0 0 0 0.0000)
+		)
+		(property "Sheetname" "eFuse"
+			(at 144.78 109.7784 0)
+			(effects
+				(font
+					(size 1.27 1.27)
+				)
+				(justify left bottom)
+			)
+		)
+		(property "Sheetfile" "efuse.kicad_sch"
+			(at 144.78 145.3646 0)
+			(effects
+				(font
+					(size 1.27 1.27)
+				)
+				(justify left top)
+			)
+		)
+		(instances
+			(project "VoxLink"
+				(path "/ded7c4da-7d9f-418d-838f-f5efc7d9c9cb"
+					(page "1")
+				)
+			)
+		)
+	)
+	(sheet
+		(at 88.011 69.215)
 		(size 51.054 34.29)
 		(exclude_from_sim no)
@@
 		)
 		(property "Sheetname" "Power"
-			(at 42.926 55.1684 0)
+			(at 88.011 68.5034 0)
 			(effects
 				(font
@@
 		)
 		(property "Sheetfile" "power.kicad_sch"
-			(at 42.926 90.7546 0)
+			(at 88.011 104.0896 0)
 			(effects
 				(font
@@
 	)
 	(sheet
-		(at 128.778 59.182)
-		(size 54.864 37.338)
+		(at 144.78 69.85)
+		(size 50.8 34.29)
 		(exclude_from_sim no)
 		(in_bom yes)
@@
 		)
 		(property "Sheetname" "Sensor"
-			(at 128.778 58.4704 0)
+			(at 144.78 69.1384 0)
 			(effects
 				(font
@@
 		)
 		(property "Sheetfile" "Sensor.kicad_sch"
-			(at 128.778 97.1046 0)
+			(at 144.78 104.7246 0)
 			(effects
 				(font
@@
 	)
 	(sheet
-		(at 43.18 99.06)
+		(at 88.265 111.125)
 		(size 51.054 35.052)
 		(exclude_from_sim no)
@@
 		)
 		(property "Sheetname" "System"
-			(at 43.18 98.3484 0)
+			(at 88.265 110.4134 0)
 			(effects
 				(font
@@
 		)
 		(property "Sheetfile" "System.kicad_sch"
-			(at 43.18 134.6966 0)
+			(at 88.265 146.7616 0)
 			(effects
 				(font
@@
 	(sheet_instances
 		(path "/"
-			(page "1")
+			(page "0")
 		)
 	)
