File: Hardware/Programmer_Board/ftdi.kicad_sch (KiCad schematic)
At the start: 27 parts, among them U201 FT2232HL, U202 93LC56B, Y201 16MHz

Commit message: Routed the programmer board
Parts:
- removed U201: FT2232HL, Package_QFP:LQFP-64_10x10mm_P0.5mm, symbol Interface_USB:FT2232HL
- added C12, C207: 4u7, Capacitor_SMD:C_0402_1005Metric, symbol Device:C
- added C210, C211, C213, C214, C215: 100n, Capacitor_SMD:C_0402_1005Metric, symbol Device:C
- added U201: FT2232HQ, Package_DFN_QFN:QFN-64-1EP_9x9mm_P0.5mm_EP4.35x4.35mm, symbol Interface_USB:FT2232HQ
- C208: value 10u -> 100n
- R202, R203, R204, R205, R206, R207, R208, R209, R210, R211, R212, R213: footprint (none) -> Resistor_SMD:R_0402_1005Metric
- U202: footprint Package_SO:SOIC-8_3.9x4.9mm_P1.27mm -> Package_DFN_QFN:TDFN-8-1EP_3x2mm_P0.5mm_EP1.3x1.4mm; Distributor Link https://www.mouser.sk/ProductDetail/Microchip-Technology/93LC56B-I-SN?qs=JhC4kYev1ubTO3jC60ECfA%3D%3D -> https://www.mouser.sk/ProductDetail/Microchip-Technology/93LC56BT-I-MC?qs=ZL7isbUZFInANak%2FIljUoQ%3D%3D
- renumbered C207 to C216
Connections:
- net +1V8: now also C12.1, C213.1, C214.1, C215.1, U201.12 (VCORE), U201.37 (VCORE), U201.49 (VREGOUT), U201.64 (VCORE); no longer C208.1, C209.1
- net +3V3: now also C208.1, C209.1, C207.1, C210.1, C211.1, U201.20 (VCCIO), U201.31 (VCCIO), U201.42 (VCCIO), U201.50 (VREGIN), U201.56 (VCCIO)
- net +3V3_VPHY: now also U201.4 (VPHY)
- net +3V3_VPLL: now also U201.9 (VPLL)
- net EECLK: now also U201.62 (EECLK)
- net EECS: now also U201.63 (EECS)
- net EEDATA: now also U201.61 (EEDATA)
- net FTDI_USB_D+: now also U201.8 (DP)
- net FTDI_USB_D-: now also U201.7 (DM)
- net GND: now also U202.9 (EP), C12.2, C207.2, C210.2, C211.2, C213.2, C214.2, C215.2, U201.1 (GND), U201.10 (AGND), U201.11 (GND), U201.13 (TEST), U201.15 (GND), U201.25 (GND), U201.35 (GND), U201.47 (GND), U201.5 (GND), U201.51 (GND), U201.65 (GND)
- net OSC_IN: now also U201.2 (OSCI)
- net OSC_OUT: now also U201.3 (OSCO)
- net at R210.1: now also U201.18 (ADBUS2)
- net at R213.1: now also U201.24 (ADBUS7)
- net at R211.1: now also U201.21 (ADBUS4)
- net at R206.2: now also U201.14 (~{RESET})
- net at R208.1: now also U201.16 (ADBUS0)
- net at R209.1: now also U201.17 (ADBUS1)
- net at R207.2: now also U201.6 (REF)
- net at R212.1: now also U201.23 (ADBUS6)

Commit message: Finished final PCB checks before manufacturing and uploaded the fabrication files
Parts:
- FB201, FB202: footprint Capacitor_SMD:C_0402_1005Metric -> Inductor_SMD:L_0402_1005Metric
Connections:
- net EEDATA: no longer R205.1
- net at R202.1, U202.4 (DO): now also R205.1
Other:
- moved on the sheet: R202, R203, R204, R205

Commit message: Added comments to the schematic, updated documentation with the board bringup, and wrote the VoxLink Verilog blink sketch.
Parts:
- Y201: value 16MHz -> 12MHz
Other:
- note added: "NEXT REVISION: Ref through 12k to GND! ~{RESET} through 1k to 3V3!"
Changed lines of the file:
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@@
 		(company "Czech Technical University in Prague")
 	)
+	(text "NEXT REVISION: \nRef through 12k to GND!\n~{RESET} through 1k to 3V3!"
+		(exclude_from_sim no)
+		(at 166.624 87.122 0)
+		(effects
+			(font
+				(size 1.27 1.27)
+				(thickness 0.254)
+				(bold yes)
+				(color 194 0 0 1)
+			)
+			(justify right)
+		)
+	)
 	(text "(10pF Load Capacitance - 5pF Stray Capacitance) * 2 = 10pF Load Capacitors"
 		(exclude_from_sim no)
@@
 			)
 		)
-		(property "Value" "16MHz"
+		(property "Value" "12MHz"
 			(at 46.99 154.94 0)
 			(effects
