File: Hardware/Sensor_Board/System.kicad_sch (KiCad schematic)
At the start: 34 parts, among them J301 RJ45, J302 TC2030, SW301 Reset, U301 TPD4E02B04, U302 TPD4E02B04, U303 TPD4E02B04, U304 N25Q032A, U305 ICE40UL1K-CM36AI, U306 ICE40UL1K-CM36AI, U307 ICE40UL1K-CM36AI, Y301 ASCO

Commit message: Cleared ERC errors and improved folder structure
Parts:
- removed U305, U306, U307: ICE40UL1K-CM36AI, Package_BGA:UCBGA-36_2.5x2.5mm_Layout6x6_P0.4mm, symbol Custom_VoxLink_Symbols:ICE40UL1K-CM36AI
- added U301: ICE40UL1K-CM36AI, Package_BGA:UCBGA-36_2.5x2.5mm_Layout6x6_P0.4mm, symbol Custom_VoxLink_Symbols:ICE40UL1K-CM36AI
- renumbered U301 to U302, U302 to U303, U303 to U304, U304 to U305
Connections:
- net 12MHZ_CLK: now also U301.D2 (IOB_8A_G4)
- net CDONE: now also U301.D5 (IOB_11B_CDONE)
- net FLASH_MISO: now also U301.E5 (IOB_15B_SI)
- net FLASH_MOSI: now also U301.F6 (IOB_14A_SO)
- net FLASH_SCK: now also U301.E6 (IOB_16A_SCK)
- net FLASH_~{CS}: now also U301.F5 (IOB_17B_SS)
- net VOX_CLK_NOESD: now also U301.E2 (IOB_6A)
- net VOX_RX_NOESD: now also U301.D1 (IOB_4A)
- net VOX_TX_NOESD: now also U301.F1 (IOB_0A)
- net ~{CRESET}: now also U301.F4 (~{CRESET})
- net ~{VOX_CLK}_NOESD: now also U301.D6 (IOB_10A)
- net ~{VOX_RX}_NOESD: now also U301.C1 (IOB_5B)
- net ~{VOX_TX}_NOESD: now also U301.E1 (IOB_1B)
- net at D303.1 (K): now also U301.A2 (RGB0)
- net at D305.1 (K): now also U301.A1 (RGB2)
- net at D304.1 (K): now also U301.B1 (RGB1)

Commit message: Fixed minor bugs in the schematic and updated the documentation.
Parts:
- U305: Distributor Link (none) -> https://eu.mouser.com/ProductDetail/Alliance-Memory/N25Q032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
Connections:
- net 12MHZ_CLK: now also U301.F2 (IOB_3B_G6); no longer U301.D2 (IOB_8A_G4)
- net ~{VOX_CLK}_NOESD: now also U301.F3 (IOB_7B_G5); no longer U301.D6 (IOB_10A)
Other:
- note added: "Table of differential comparator pin pairs"

Commit message: Added a programmer schematic
Parts:
- added D302, D303: TVS, Diode_SMD:D_0402_1005Metric, symbol Diode:1.5KExxA
- added J303: PicoBlade, Connector_Molex:Molex_PicoBlade_53048-0810_1x08_P1.25mm_Horizontal, symbol Connector_Generic:Conn_01x08
- renumbered D302 to D304, D303 to D305, D304 to D306, D305 to D307
Connections:
- net +3V3 is gone; now on net VCC: C301.1, D301.1 (A1)
- net CDONE: now also D302.1 (A1), J303.3 (Pin_3)
- net FLASH_MISO_NOESD: now also J303.5 (Pin_5)
- net FLASH_MOSI_NOESD: now also J303.6 (Pin_6)
- net FLASH_SCK_NOESD: now also J303.4 (Pin_4)
- net FLASH_~{CS}_NOESD: now also J303.7 (Pin_7)
- net GND: now also D302.2 (A2), D303.2 (A2), J303.1 (Pin_1)
- net VCC: now also J302.1 (VCC), J303.8 (Pin_8)
- net VCCIO1: no longer J302.1 (VCC)
- net ~{CRESET}: now also D303.1 (A1), J303.2 (Pin_2)
Other:
- note added: "WARNING: Connector is FLIPPED to match polarity!"

Commit message: Added documantation regarding the programmer board and updated the PDF schematics.
Parts:
- removed J301: RJ45, rj45_molex_unshielded:CONN_855035-101_MOL, symbol rj45_molex_unshielded:RJ45_Molex_Unshielded
- added J301: RJ45_Input, rj45_molex_unshielded:CONN_855035-101_MOL, symbol rj45_molex_unshielded:RJ45_Molex_Unshielded_Input
- added J304: RJ45_Output, rj45_molex_unshielded:CONN_855035-101_MOL, symbol rj45_molex_unshielded:RJ45_Molex_Unshielded_Output
- added R315, R316, R317: 0R, symbol Device:R
Connections:
- net GND: now also J301.6 (GND), J304.6 (GND), R315.2, R316.2, R317.2
- net VCC: now also J301.3 (VCC), J304.3 (VCC)
- net VOX_CLK: now also J301.4 (CLK), J304.4 (CLK)
- net VOX_RX: now also J301.1 (RX), J304.1 (RX)
- net VOX_TX: now also J301.7 (TX), J304.7 (TX)
- net ~{VOX_CLK}: now also J301.5 (~{CLK}), J304.5 (~{CLK}), R316.1
- net ~{VOX_RX}: now also J301.2 (~{RX}), J304.2 (~{RX}), R315.1
- net ~{VOX_TX}: now also J301.8 (~{TX}), J304.8 (~{TX}), R317.1
Other:
- note added: "Ethernet Connector Daisy Chain"
- note added: "Ethernet Connector Input"
- note removed: "Ethernet Connector"
- moved on the sheet: C301, C302, C303, C304, D301, D302, D303, D304, D305, D306, D307, J302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

Commit message: Pushing before updating KiCad
Parts:
- removed J301: RJ45_Input, rj45_molex_unshielded:CONN_855035-101_MOL, symbol rj45_molex_unshielded:RJ45_Molex_Unshielded_Input
- removed J304: RJ45_Output, rj45_molex_unshielded:CONN_855035-101_MOL, symbol rj45_molex_unshielded:RJ45_Molex_Unshielded_Output
- removed R305, R306, R307, R315, R316, R317: 0R, symbol Device:R
- removed unit 2 of U301
- removed U303, U304: TPD4E02B04, Package_SON:USON-10_2.5x1.0mm_P0.5mm, symbol Custom_VoxLink_Symbols:TPD4E02B04DQA
- D304, D305, D306, D307: footprint (none) -> LED_SMD:LED_0603_1608Metric
- R308, R309: footprint (none) -> Resistor_SMD:R_0402_1005Metric
- R310, R312, R313, R314: value 500R -> 510R; footprint (none) -> Resistor_SMD:R_0402_1005Metric
- SW301: footprint (none) -> Button_Switch_SMD:SW_Push_SPST_NO_Alps_SKRK
- U301: footprint Package_BGA:UCBGA-36_2.5x2.5mm_Layout6x6_P0.4mm -> Custom_VoxLink_Footprints:ICE40UL1K_UCBGA-36
- U305: footprint (none) -> Custom_VoxLink_Footprints:U-PDFN-8
Connections:
- net LED: now reaches D305.1 (K), U301.A2 (RGB0)
- net TX_LED: now reaches D307.1 (K), U301.A1 (RGB2)
- net RX_LED: now reaches D306.1 (K), U301.B1 (RGB1)
- no-connect marks 8 -> 2
Other:
- note removed: "ESD Protection ICs"
- note removed: "Ethernet Connector Daisy Chain"
- note removed: "Ethernet Connector Input"
- note removed: "No Placement (NOP) - Used in case a differential driver would not work -> ~{NEGATIVE} can be tied to GND"
- note removed: "Table of differential comparator pin pairs"
- moved on the sheet: C301, C302, C303, C304, D301, D302, D303, D304, D305, D306, D307, J302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

Commit message: Routing and Schematic update
Parts:
- removed J302: TC2030, Connector:Tag-Connect_TC2030-IDC-FP_2x03_P1.27mm_Vertical, symbol Connector:Conn_ARM_SWD_TagConnect_TC2030
- added D1: D_Schottky, Diode_SMD:D_0402_1005Metric, symbol Device:D_Schottky
- added J302: TC2030-NL, Connector:Tag-Connect_TC2030-IDC-NL_2x03_P1.27mm_Vertical, symbol Connector:Conn_ARM_SWD_TagConnect_TC2030-NL
- Y301: footprint Oscillator:Oscillator_SMD_Abracon_ASE-4Pin_3.2x2.5mm -> Oscillator:Oscillator_SMD_Abracon_ASCO-4Pin_1.6x1.2mm
Connections:
- net FLASH_MISO_NOESD: now also U302.2 (IN), J302.2 (SWDIO); no longer U302.4 (IN)
- net FLASH_MOSI_NOESD: now also U302.4 (IN), J302.4 (SWCLK); no longer U302.2 (IN)
- net FLASH_SCK_NOESD: now also U302.1 (IN), J302.6 (SWO); no longer U302.5 (IN)
- net FLASH_~{CS}_NOESD: now also U302.5 (IN), J302.3 (~{RESET}); no longer U302.1 (IN)
- net GND: now also J302.5 (GND)
- net VCC: now also D1.1 (K); no longer C301.1, D301.1 (A1), J303.8 (Pin_8)
- net at R303.2: now also U302.9 (NC); no longer U302.7 (NC)
- net at R302.2: now also U302.7 (NC); no longer U302.9 (NC)
- net FLASH_~{HOLD}: now reaches R309.2, U305.7 (~{HOLD})
- net FLASH_~{WP}: now reaches R308.2, U305.3 (~{WP})
- net at U302.10 (NC): now also R304.2; no longer R301.2
- net at U302.6 (NC): now also R301.2; no longer R304.2
- new net VCCD: C301.1, D1.2 (A), D301.1 (A1), J302.1 (VCC), J303.8 (Pin_8)
Other:
- moved on the sheet: R308

Commit message: Finised the design of the sensor board :)
Parts:
- removed R301, R302, R303, R304: 22R, Resistor_SMD:R_0402_1005Metric, symbol Device:R
- added R301: 4x22R, Custom_VoxLink_Footprints:EXBN8V101JX, symbol Custom_VoxLink_Symbols:4xResistor_Array
- D302: renamed from D1; value D_Schottky -> Schottky
- renumbered D302 to D303, D303 to D304, D304 to D308, J302 to J301, J303 to J302, R311 to R302, R310 to R303, R308 to R304, R309 to R305, R312 to R306, R313 to R307, R314 to R308
Connections:
- net FLASH_MISO: now also R301.3
- net FLASH_MISO_NOESD: now also U302.9 (NC), R301.6
- net FLASH_MOSI: now also R301.2
- net FLASH_MOSI_NOESD: now also U302.7 (NC), R301.7
- net FLASH_SCK: now also R301.4
- net FLASH_SCK_NOESD: now also U302.10 (NC), R301.5
- net FLASH_~{CS}: now also R301.1
- net FLASH_~{CS}_NOESD: now also U302.6 (NC), R301.8
Other:
- moved on the sheet: C301, D301, D302, D303, D304, J301, J302, U302

Commit message: Finished final PCB checks before manufacturing and uploaded the fabrication files
Parts:
- U302: footprint Package_SON:USON-10_2.5x1.0mm_P0.5mm -> Custom_VoxLink_Footprints:USON-10_2.5x1.0mm_P0.5mm__Reduced_Paste
Changed lines of the file:
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@@
 			)
 		)
-		(property "Datasheet" "https://eu.mouser.com/ProductDetail/Panasonic/EXB-N8V220JX?qs=bx0%2FPCyAc7556mtSQRzOoA%3D%3D"
+		(property "Datasheet" "https://www.mouser.sk/ProductDetail/Panasonic/EXB-N8V220JX?qs=bx0%2FPCyAc7556mtSQRzOoA%3D%3D"
 			(at 124.46 82.55 0)
 			(effects
@@
 			)
 		)
-		(property "Datasheet" "~"
+		(property "Datasheet" "https://www.mouser.sk/ProductDetail/Broadcom-Avago/HSMG-C190?qs=YDL0qNrpDT605sxOaps8VQ%3D%3D"
 			(at 269.24 147.32 0)
 			(effects
@@
 			)
 		)
-		(property "Footprint" "Package_SON:USON-10_2.5x1.0mm_P0.5mm"
+		(property "Footprint" "Custom_VoxLink_Footprints:USON-10_2.5x1.0mm_P0.5mm__Reduced_Paste"
 			(at 88.9 83.82 0)
 			(effects
