File: Hardware/Sensor_Board/System.kicad_sch (KiCad schematic)
At the start: 27 parts, among them J301 TC2030-NL, J302 PicoBlade, SW301 Reset, U301 ICE40UL1K-CM36AI, U302 TPD4E02B04, U305 N25Q032A, Y301 ASCO

Commit message: Updated documentation and finished first iteration of PCB rework based on manufacturer feedback.
Parts:
- U301: footprint Custom_VoxLink_Footprints:ICE40UL1K_UCBGA-36 -> Package_BGA:UCBGA-36_2.5x2.5mm_Layout6x6_P0.4mm
Changed lines of the file:
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@@
 			)
 		)
-		(property "Footprint" "Custom_VoxLink_Footprints:ICE40UL1K_UCBGA-36"
+		(property "Footprint" "Package_BGA:UCBGA-36_2.5x2.5mm_Layout6x6_P0.4mm"
 			(at 209.55 66.04 0)
 			(effects
@@
 	)
 	(symbol
+		(lib_name "ICE40UL1K-CM36AI_1")
 		(lib_id "Custom_VoxLink_Symbols:ICE40UL1K-CM36AI")
 		(at 193.04 120.65 0)
@@
 			)
 		)
-		(property "Footprint" "Custom_VoxLink_Footprints:ICE40UL1K_UCBGA-36"
+		(property "Footprint" "Package_BGA:UCBGA-36_2.5x2.5mm_Layout6x6_P0.4mm"
 			(at 193.04 120.65 0)
 			(effects

Commit message: Added comments to the schematic, updated documentation with the board bringup, and wrote the VoxLink Verilog blink sketch.
Parts:
- Y301: value ASCO -> 12MHz
Other:
- note added: "D302 is removed in the prototype version"
- note added: "If the LED shines, the device has been configured properly"
- note added: "NEXT REVISION: There is an imbalance of 22R resistors! No resistors on the CDONE and ~{CRESET}"
- note removed: "If LED shines, the device has not been configured properly!"
Changed lines of the file:
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@@
 		(company "Czech Technical University in Prague")
 	)
+	(text "D302 is removed in the \nprototype version"
+		(exclude_from_sim no)
+		(at 62.738 67.564 0)
+		(effects
+			(font
+				(size 1.27 1.27)
+				(thickness 0.254)
+				(bold yes)
+				(color 194 0 0 1)
+			)
+			(justify left)
+		)
+	)
 	(text "Used for LED driving"
 		(exclude_from_sim no)
@@
 		)
 	)
-	(text "If LED shines, the device has \nnot been configured properly!"
+	(text "If the LED shines, the device\nhas been configured properly"
 		(exclude_from_sim no)
 		(at 279.146 157.48 0)
@@
 		)
 	)
+	(text "NEXT REVISION:\nThere is an imbalance of 22R resistors!\nNo resistors on the CDONE and ~{CRESET}"
+		(exclude_from_sim no)
+		(at 146.304 37.084 0)
+		(effects
+			(font
+				(size 1.27 1.27)
+				(thickness 0.254)
+				(bold yes)
+				(color 194 0 0 1)
+			)
+			(justify right)
+		)
+	)
 	(text "System [3]"
 		(exclude_from_sim no)
@@
 			)
 		)
-		(property "Value" "ASCO"
+		(property "Value" "12MHz"
 			(at 128.27 132.0098 0)
 			(effects
