File: Hardware/Sensor_Board/Sensor.kicad_sch (KiCad schematic)
At the start: 16 parts, among them U401 BNO086, U402 ICE40UL1K-CM36AI, Y401 32.768 kHz

Commit message: Cleared ERC errors and improved folder structure
Parts:
- removed U402: ICE40UL1K-CM36AI, Package_BGA:UCBGA-36_2.5x2.5mm_Layout6x6_P0.4mm, symbol Custom_VoxLink_Symbols:ICE40UL1K-CM36AI
- added U301: ICE40UL1K-CM36AI, Package_BGA:UCBGA-36_2.5x2.5mm_Layout6x6_P0.4mm, symbol Custom_VoxLink_Symbols:ICE40UL1K-CM36AI
- U401: Distributor Link (none) -> https://eu.mouser.com/ProductDetail/CEVA/BNO086?qs=ulEaXIWI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
Connections:
- net BNO_SCL: now also U301.B2 (IOT_24B)
- net BNO_SDA: now also U301.A4 (IOT_19A)
- net BNO_~{RST}: now also U301.B5 (IOT_18B)
Changed lines of the file:
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@@
 	)
 	(symbol
-		(lib_name "+3.3VA_6")
 		(lib_id "power:+3.3VA")
 		(at 213.36 88.9 0)
@@
 			)
 		)
+		(property "Distributor Link" "https://eu.mouser.com/ProductDetail/CEVA/BNO086?qs=ulEaXIWI0c%2FqTo1scjodAw%3D%3D&srsltid=AfmBOop7Lm0NKSepOPNTaVnevCWe4BdpG9i9W3OMpkCwkAHHi0MmvZo2"
+			(at 147.32 91.44 0)
+			(effects
+				(font
+					(size 1.27 1.27)
+				)
+				(hide yes)
+			)
+		)
 		(pin "2"
 		)
@@
 	)
 	(symbol
-		(lib_name "+3.3VA_6")
 		(lib_id "power:+3.3VA")
 		(at 204.47 88.9 0)
@@
 	)
 	(symbol
-		(lib_name "+3.3VA_6")
 		(lib_id "power:+3.3VA")
 		(at 116.84 100.33 0)
@@
 					(reference "R408")
 					(unit 1)
+				)
+			)
+		)
+	)
+	(symbol
+		(lib_id "Custom_VoxLink_Symbols:ICE40UL1K-CM36AI")
+		(at 45.72 95.25 0)
+		(unit 3)
+		(exclude_from_sim no)
+		(in_bom yes)
+		(on_board yes)
+		(dnp no)
+		(fields_autoplaced yes)
+		(property "Reference" "U301"
+			(at 45.72 91.694 0)
+			(effects
+				(font
+					(size 1.27 1.27)
+				)
+				(hide yes)
+			)
+		)
+		(property "Value" "ICE40UL1K-CM36AI"
+			(at 45.72 93.472 0)
+			(effects
+				(font
+					(size 1.27 1.27)
+				)
+				(hide yes)
+			)
+		)
+		(property "Footprint" "Package_BGA:UCBGA-36_2.5x2.5mm_Layout6x6_P0.4mm"
+			(at 45.72 95.25 0)
+			(effects
+				(font
+					(size 1.27 1.27)
+				)
+				(hide yes)
+			)
+		)
+		(property "Datasheet" ""
+			(at 45.72 95.25 0)
+			(effects
+				(font
+					(size 1.27 1.27)
+				)
+				(hide yes)
+			)
+		)
+		(property "Description" ""
+			(at 45.72 95.25 0)
+			(effects
+				(font
+					(size 1.27 1.27)
+				)
+				(hide yes)
+			)
+		)
+		(property "Distributor Link" "https://eu.mouser.com/ProductDetail/Lattice/ICE40UL1K-CM36AI?qs=XJu%252BLGjWfSAZhGGFZ7EiQg%3D%3D"
+			(at 45.72 95.25 0)
+			(effects
+				(font
+					(size 1.27 1.27)
+				)
+				(hide yes)
+			)
+		)
+		(pin "E4"
+		)
+		(pin "A2"
+		)
+		(pin "D1"
+		)
+		(pin "F1"
+		)
+		(pin "D3"
+		)
+		(pin "A4"
+		)
+		(pin "C4"
+		)
+		(pin "D2"
+		)
+		(pin "B5"
+		)
+		(pin "B4"
+		)
+		(pin "E3"
+		)
+		(pin "B2"
+		)
+		(pin "E1"
+		)
+		(pin "D4"
+		)
+		(pin "B3"
+		)
+		(pin "F2"
+		)
+		(pin "C6"
+		)
+		(pin "E2"
+		)
+		(pin "C3"
+		)
+		(pin "C5"
+		)
+		(pin "C1"
+		)
+		(pin "F3"
+		)
+		(pin "D6"
+		)
+		(pin "A3"
+		)
+		(pin "C2"
+		)
+		(pin "B6"
+		)
+		(pin "D5"
+		)
+		(pin "F5"
+		)
+		(pin "E5"
+		)
+		(pin "A5"
+		)
+		(pin "F6"
+		)
+		(pin "E6"
+		)
+		(pin "A1"
+		)
+		(pin "A6"
+		)
+		(pin "B1"
+		)
+		(pin "F4"
+		)
+		(instances
+			(project "VoxSense"
+				(path "/ded7c4da-7d9f-418d-838f-f5efc7d9c9cb/9719f155-9a63-4412-a45f-eaa04d0e19ac"
+					(reference "U301")
+					(unit 3)
 				)
 			)
@@
 	)
 	(symbol
-		(lib_name "+3.3VA_6")
 		(lib_id "power:+3.3VA")
 		(at 140.97 80.01 0)
@@
 	)
 	(symbol
-		(lib_name "+3.3VA_6")
 		(lib_id "power:+3.3VA")
 		(at 97.79 80.01 0)
@@
 	)
 	(symbol
-		(lib_name "+3.3VA_6")
 		(lib_id "power:+3.3VA")
 		(at 106.68 80.01 0)
@@
 	)
 	(symbol
-		(lib_id "Custom_VoxLink_Symbols:ICE40UL1K-CM36AI")
-		(at 45.72 95.25 0)
-		(unit 3)
-		(exclude_from_sim no)
-		(in_bom yes)
-		(on_board yes)
-		(dnp no)
-		(fields_autoplaced yes)
-		(property "Reference" "U402"
-			(at 45.72 91.694 0)
-			(effects
-				(font
-					(size 1.27 1.27)
-				)
-				(hide yes)
-			)
-		)
-		(property "Value" "ICE40UL1K-CM36AI"
-			(at 45.72 93.472 0)
-			(effects
-				(font
-					(size 1.27 1.27)
-				)
-				(hide yes)
-			)
-		)
-		(property "Footprint" "Package_BGA:UCBGA-36_2.5x2.5mm_Layout6x6_P0.4mm"
-			(at 45.72 95.25 0)
-			(effects
-				(font
-					(size 1.27 1.27)
-				)
-				(hide yes)
-			)
-		)
-		(property "Datasheet" ""
-			(at 45.72 95.25 0)
-			(effects
-				(font
-					(size 1.27 1.27)
-				)
-				(hide yes)
-			)
-		)
-		(property "Description" ""
-			(at 45.72 95.25 0)
-			(effects
-				(font
-					(size 1.27 1.27)
-				)
-				(hide yes)
-			)
-		)
-		(property "Distributor Link" "https://eu.mouser.com/ProductDetail/Lattice/ICE40UL1K-CM36AI?qs=XJu%252BLGjWfSAZhGGFZ7EiQg%3D%3D"
-			(at 45.72 95.25 0)
-			(effects
-				(font
-					(size 1.27 1.27)
-				)
-				(hide yes)
-			)
-		)
-		(pin "D4"
-		)
-		(pin "D3"
-		)
-		(pin "D1"
-		)
-		(pin "B4"
-		)
-		(pin "B3"
-		)
-		(pin "E4"
-		)
-		(pin "C3"
-		)
-		(pin "C5"
-		)
-		(pin "A6"
-		)
-		(pin "F5"
-		)
-		(pin "C2"
-		)
-		(pin "E1"
-		)
-		(pin "E3"
-		)
-		(pin "F2"
-		)
-		(pin "F1"
-		)
-		(pin "C4"
-		)
-		(pin "D6"
-		)
-		(pin "F3"
-		)
-		(pin "D2"
-		)
-		(pin "A3"
-		)
-		(pin "B6"
-		)
-		(pin "C6"
-		)
-		(pin "A2"
-		)
-		(pin "B1"
-		)
-		(pin "A1"
-		)
-		(pin "B2"
-		)
-		(pin "A5"
-		)
-		(pin "F6"
-		)
-		(pin "C1"
-		)
-		(pin "B5"
-		)
-		(pin "E2"
-		)
-		(pin "A4"
-		)
-		(pin "E5"
-		)
-		(pin "E6"
-		)
-		(pin "F4"
-		)
-		(pin "D5"
-		)
-		(instances
-			(project "VoxLink"
-				(path "/ded7c4da-7d9f-418d-838f-f5efc7d9c9cb/9719f155-9a63-4412-a45f-eaa04d0e19ac"
-					(reference "U402")
-					(unit 3)
-				)
-			)
-		)
-	)
-	(symbol
 		(lib_id "Device:R")
 		(at 204.47 92.71 0)
@@
 	)
 	(symbol
-		(lib_name "+3.3VA_6")
 		(lib_id "power:+3.3VA")
 		(at 182.88 80.01 0)
@@
 	)
 	(symbol
-		(lib_name "+3.3VA_6")
 		(lib_id "power:+3.3VA")
 		(at 162.56 58.42 0)

Commit message: Fixed minor bugs in the schematic and updated the documentation.
Other:
- note added: "For daisy-chaining temperatre/humidity sensors. Even unused needs to be teminated with pullup resistors as per the I2C standard!"
- note removed: "For daisy-chaining temperatre/humidity sensors Needs to be teminated as I2C with pullup resistors"
Changed lines of the file:
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@@
 		)
 	)
-	(text "For daisy-chaining temperatre/humidity sensors\nNeeds to be teminated as I2C with pullup resistors"
+	(text "For daisy-chaining temperatre/humidity sensors.\nEven unused needs to be teminated with\npullup resistors as per the I2C standard!"
 		(exclude_from_sim no)
-		(at 178.816 104.14 0)
+		(at 180.594 104.648 0)
 		(effects
 			(font
@@
 		)
 	)
-	(text_box "BNO086 Crystal"
+	(text_box "BNO086"
 		(exclude_from_sim no)
 		(at 78.74 51.308 0)
-		(size 153.416 87.884)
+		(size 155.575 87.884)
 		(margins 1.5 1.5 1.5 1.5)
 		(stroke

Commit message: Pushing before updating KiCad
Parts:
- R401, R402, R403, R404, R405, R406, R407: footprint (none) -> Resistor_SMD:R_0402_1005Metric
- U301: footprint Package_BGA:UCBGA-36_2.5x2.5mm_Layout6x6_P0.4mm -> Custom_VoxLink_Footprints:ICE40UL1K_UCBGA-36
- U401: footprint (none) -> Package_LGA:LGA-28_5.2x3.8mm_P0.5mm
- Y401: footprint (none) -> Crystal:Crystal_SMD_MicroCrystal_CC8V-T1A-2Pin_2.0x1.2mm
Connections:
- net BNO_SCL: now also U301.C6 (IOT_22B_G0); no longer U301.B2 (IOT_24B)
- net BNO_SDA: no longer U301.A4 (IOT_19A)
- net BNO_~{RST}: now also U301.B6 (IOT_21A_G1); no longer U301.B5 (IOT_18B)
- net XOUT32_INT: now reaches C405.1, R408.2, Y401.1
- no-connect marks 6 -> 7
Changed lines of the file:
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@@
 	)
 	(no_connect
+		(at 144.78 102.87)
+	)
+	(no_connect
 		(at 54.61 96.52)
 	)
 	(no_connect
-		(at 54.61 106.68)
+		(at 54.61 99.06)
 	)
 	(no_connect
-		(at 144.78 102.87)
+		(at 144.78 100.33)
 	)
 	(no_connect
-		(at 54.61 99.06)
+		(at 54.61 93.98)
 	)
 	(no_connect
-		(at 54.61 104.14)
+		(at 54.61 88.9)
 	)
 	(no_connect
-		(at 144.78 100.33)
+		(at 54.61 91.44)
 	)
 	(wire
@@
 	(wire
 		(pts
-			(xy 54.61 88.9) (xy 58.42 88.9)
+			(xy 54.61 106.68) (xy 58.42 106.68)
 		)
 		(stroke
@@
 	(wire
 		(pts
-			(xy 54.61 93.98) (xy 58.42 93.98)
-		)
-		(stroke
-			(width 0)
-			(type default)
-		)
-	)
-	(wire
-		(pts
-			(xy 54.61 91.44) (xy 58.42 91.44)
+			(xy 54.61 104.14) (xy 58.42 104.14)
 		)
 		(stroke
@@
 		)
 	)
+	(label "XOUT32_INT"
+		(at 130.81 160.02 180)
+		(effects
+			(font
+				(size 1.27 1.27)
+			)
+			(justify right bottom)
+		)
+	)
 	(label "XIN32"
 		(at 189.23 113.03 180)
@@
 	(global_label "BNO_SCL"
 		(shape input)
-		(at 58.42 93.98 0)
+		(at 58.42 106.68 0)
 		(fields_autoplaced yes)
 		(effects
@@
 		)
 		(property "Intersheetrefs" "${INTERSHEET_REFS}"
-			(at 69.8114 93.98 0)
+			(at 69.8114 106.68 0)
 			(effects
 				(font
@@
 		)
 	)
-	(global_label "BNO_SDA"
-		(shape input)
-		(at 58.42 91.44 0)
-		(fields_autoplaced yes)
-		(effects
-			(font
-				(size 1.27 1.27)
-			)
-			(justify left)
-		)
-		(property "Intersheetrefs" "${INTERSHEET_REFS}"
-			(at 69.8719 91.44 0)
-			(effects
-				(font
-					(size 1.27 1.27)
-				)
-				(justify left)
-				(hide yes)
-			)
-		)
-	)
 	(global_label "BNO_~{RST}"
 		(shape input)
-		(at 58.42 88.9 0)
+		(at 58.42 104.14 0)
 		(fields_autoplaced yes)
 		(effects
@@
 		)
 		(property "Intersheetrefs" "${INTERSHEET_REFS}"
-			(at 69.7509 88.9 0)
+			(at 69.7509 104.14 0)
 			(effects
 				(font
@@
 			)
 		)
-		(property "Datasheet" "https://eu.mouser.com/ProductDetail/81-GCM1555G1H100JA6D"
+		(property "Datasheet" "https://www.mouser.sk/ProductDetail/Murata-Electronics/GRM1555C1H150FA01D?qs=ouTquLLW2S7neucAALMxaw%3D%3D"
 			(at 99.06 168.91 0)
 			(effects
@@
 			)
 		)
-		(property "Footprint" ""
+		(property "Footprint" "Package_LGA:LGA-28_5.2x3.8mm_P0.5mm"
 			(at 147.32 91.44 0)
 			(effects
@@
 			)
 		)
-		(property "Footprint" ""
+		(property "Footprint" "Resistor_SMD:R_0402_1005Metric"
 			(at 142.748 83.82 90)
 			(effects
@@
 			)
 		)
-		(property "Datasheet" ""
+		(property "Datasheet" "https://www.mouser.sk/ProductDetail/Vishay/CRCW040210K0JNED?qs=sGAEpiMZZMtlubZbdhIBIFsfWmIKznfcMCgOmcXe42g%3D"
 			(at 140.97 83.82 0)
 			(effects
@@
 			)
 		)
-		(property "Footprint" ""
+		(property "Footprint" "Resistor_SMD:R_0402_1005Metric"
 			(at 118.618 104.14 90)
 			(effects
@@
 			)
 		)
-		(property "Datasheet" ""
+		(property "Datasheet" "https://www.mouser.sk/ProductDetail/Vishay/CRCW040210K0JNED?qs=sGAEpiMZZMtlubZbdhIBIFsfWmIKznfcMCgOmcXe42g%3D"
 			(at 116.84 104.14 0)
 			(effects
@@
 			)
 		)
-		(property "Footprint" ""
+		(property "Footprint" "Resistor_SMD:R_0402_1005Metric"
 			(at 96.012 83.82 90)
 			(effects
@@
 			)
 		)
-		(property "Datasheet" ""
+		(property "Datasheet" "https://www.mouser.sk/ProductDetail/Vishay/CRCW04024K70JNED?qs=sGAEpiMZZMtlubZbdhIBIPcJW8E8ShybHI4602K%2FbXw%3D"
 			(at 97.79 83.82 0)
 			(effects
@@
 			)
 		)
-		(property "Footprint" "Package_BGA:UCBGA-36_2.5x2.5mm_Layout6x6_P0.4mm"
+		(property "Footprint" "Custom_VoxLink_Footprints:ICE40UL1K_UCBGA-36"
 			(at 45.72 95.25 0)
 			(effects
@@
 			)
 		)
-		(property "Footprint" ""
+		(property "Footprint" "Crystal:Crystal_SMD_MicroCrystal_CC8V-T1A-2Pin_2.0x1.2mm"
 			(at 107.95 160.02 0)
 			(effects
@@
 			)
 		)
-		(property "Footprint" ""
+		(property "Footprint" "Resistor_SMD:R_0402_1005Metric"
 			(at 104.902 83.82 90)
 			(effects
@@
 			)
 		)
-		(property "Datasheet" ""
+		(property "Datasheet" "https://www.mouser.sk/ProductDetail/Vishay/CRCW04024K70JNED?qs=sGAEpiMZZMtlubZbdhIBIPcJW8E8ShybHI4602K%2FbXw%3D"
 			(at 106.68 83.82 0)
 			(effects
@@
 			)
 		)
-		(property "Footprint" ""
+		(property "Footprint" "Resistor_SMD:R_0402_1005Metric"
 			(at 202.692 92.71 90)
 			(effects
@@
 			)
 		)
-		(property "Datasheet" ""
+		(property "Datasheet" "https://www.mouser.sk/ProductDetail/Vishay/CRCW04024K70JNED?qs=sGAEpiMZZMtlubZbdhIBIPcJW8E8ShybHI4602K%2FbXw%3D"
 			(at 204.47 92.71 0)
 			(effects
@@
 			)
 		)
-		(property "Footprint" ""
+		(property "Footprint" "Resistor_SMD:R_0402_1005Metric"
 			(at 211.582 92.71 90)
 			(effects
@@
 			)
 		)
-		(property "Datasheet" ""
+		(property "Datasheet" "https://www.mouser.sk/ProductDetail/Vishay/CRCW04024K70JNED?qs=sGAEpiMZZMtlubZbdhIBIPcJW8E8ShybHI4602K%2FbXw%3D"
 			(at 213.36 92.71 0)
 			(effects
@@
 			)
 		)
-		(property "Datasheet" ""
+		(property "Datasheet" "https://www.mouser.sk/ProductDetail/Murata-Electronics/GCM155R71H104KE02J?qs=hNud%2FORuBR1wlwGPFWBVDg%3D%3D"
 			(at 152.4 64.77 0)
 			(effects
@@
 			)
 		)
-		(property "Datasheet" "https://eu.mouser.com/ProductDetail/81-GCM1555G1H100JA6D"
+		(property "Datasheet" "https://www.mouser.sk/ProductDetail/Murata-Electronics/GCM155R71H104KE02J?qs=hNud%2FORuBR1wlwGPFWBVDg%3D%3D"
 			(at 181.61 128.27 0)
 			(effects
@@
 			)
 		)
-		(property "Datasheet" "https://eu.mouser.com/ProductDetail/81-GCM1555G1H100JA6D"
+		(property "Datasheet" "https://www.mouser.sk/ProductDetail/Murata-Electronics/GRM1555C1H150FA01D?qs=ouTquLLW2S7neucAALMxaw%3D%3D"
 			(at 116.84 168.91 0)
 			(effects
@@
 			)
 		)
-		(property "Footprint" ""
+		(property "Footprint" "Resistor_SMD:R_0402_1005Metric"
 			(at 181.102 83.82 90)
 			(effects
@@
 			)
 		)
-		(property "Datasheet" ""
+		(property "Datasheet" "https://www.mouser.sk/ProductDetail/Vishay/CRCW040210K0JNED?qs=sGAEpiMZZMtlubZbdhIBIFsfWmIKznfcMCgOmcXe42g%3D"
 			(at 182.88 83.82 0)
 			(effects
@@
 			)
 		)
-		(property "Datasheet" ""
+		(property "Datasheet" "https://www.mouser.sk/ProductDetail/Murata-Electronics/GCM155R71H104KE02J?qs=hNud%2FORuBR1wlwGPFWBVDg%3D%3D"
 			(at 140.97 64.77 0)
 			(effects

Commit message: Finised the design of the sensor board :)
Connections:
- net GND: now also U301.C2 (IOT_27A)
- no-connect marks 7 -> 6
Other:
- note added: "GND connected to C2 to allow BGA fanout"
Changed lines of the file:
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@@
 		)
 	)
+	(text "GND connected\nto C2 to allow \nBGA fanout"
+		(exclude_from_sim no)
+		(at 64.262 98.552 0)
+		(effects
+			(font
+				(size 1.27 1.27)
+				(color 255 0 0 1)
+			)
+		)
+	)
 	(text "CEVA recommends using a crystal with tolerance\n50ppm with 12.5pF capacitor loading."
 		(exclude_from_sim no)
@@
 	)
 	(no_connect
-		(at 54.61 99.06)
-	)
-	(no_connect
 		(at 144.78 100.33)
 	)
@@
 					(unit 1)
 				)
+			)
+		)
+	)
+	(symbol
+		(lib_id "power:GND")
+		(at 54.61 99.06 0)
+		(mirror y)
+		(unit 1)
+		(exclude_from_sim no)
+		(in_bom yes)
+		(on_board yes)
+		(dnp no)
+		(property "Reference" "#PWR0136"
+			(at 54.61 105.41 0)
+			(effects
+				(font
+					(size 1.27 1.27)
+				)
+				(hide yes)
+			)
+		)
+		(property "Value" "GND"
+			(at 54.61 102.87 0)
+			(effects
+				(font
+					(size 1.27 1.27)
+				)
+				(hide yes)
+			)
+		)
+		(property "Footprint" ""
+			(at 54.61 99.06 0)
+			(effects
+				(font
+					(size 1.27 1.27)
+				)
+				(hide yes)
+			)
+		)
+		(property "Datasheet" ""
+			(at 54.61 99.06 0)
+			(effects
+				(font
+					(size 1.27 1.27)
+				)
+				(hide yes)
+			)
+		)
+		(property "Description" ""
+			(at 54.61 99.06 0)
+			(effects
+				(font
+					(size 1.27 1.27)
+				)
+			)
+		)
+		(pin "1"
+		)
+		(instances
+			(project "VoxSense"
+				(path "/ded7c4da-7d9f-418d-838f-f5efc7d9c9cb/9719f155-9a63-4412-a45f-eaa04d0e19ac"
+					(reference "#PWR0136")
+					(unit 1)
+				)

Commit message: Updated documentation and finished first iteration of PCB rework based on manufacturer feedback.
Parts:
- U301: footprint Custom_VoxLink_Footprints:ICE40UL1K_UCBGA-36 -> Package_BGA:UCBGA-36_2.5x2.5mm_Layout6x6_P0.4mm
Connections:
- net GND: no longer U301.C2 (IOT_27A)
- no-connect marks 6 -> 7
Other:
- note removed: "GND connected to C2 to allow BGA fanout"
Changed lines of the file:
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@@
 		)
 	)
-	(text "GND connected\nto C2 to allow \nBGA fanout"
-		(exclude_from_sim no)
-		(at 64.262 98.552 0)
-		(effects
-			(font
-				(size 1.27 1.27)
-				(color 255 0 0 1)
-			)
-		)
-	)
 	(text "CEVA recommends using a crystal with tolerance\n50ppm with 12.5pF capacitor loading."
 		(exclude_from_sim no)
@@
 		(at 54.61 91.44)
 	)
+	(no_connect
+		(at 54.61 99.06)
+	)
 	(wire
 		(pts
@@
 			)
 		)
-		(property "Footprint" "Custom_VoxLink_Footprints:ICE40UL1K_UCBGA-36"
+		(property "Footprint" "Package_BGA:UCBGA-36_2.5x2.5mm_Layout6x6_P0.4mm"
 			(at 45.72 95.25 0)
 			(effects
@@
 					(unit 1)
 				)
-			)
-		)
-	)
-	(symbol
-		(lib_id "power:GND")
-		(at 54.61 99.06 0)
-		(mirror y)
-		(unit 1)
-		(exclude_from_sim no)
-		(in_bom yes)
-		(on_board yes)
-		(dnp no)
-		(property "Reference" "#PWR0136"
-			(at 54.61 105.41 0)
-			(effects
-				(font
-					(size 1.27 1.27)
-				)
-				(hide yes)
-			)
-		)
-		(property "Value" "GND"
-			(at 54.61 102.87 0)
-			(effects
-				(font
-					(size 1.27 1.27)
-				)
-				(hide yes)
-			)
-		)
-		(property "Footprint" ""
-			(at 54.61 99.06 0)
-			(effects
-				(font
-					(size 1.27 1.27)
-				)
-				(hide yes)
-			)
-		)
-		(property "Datasheet" ""
-			(at 54.61 99.06 0)
-			(effects
-				(font
-					(size 1.27 1.27)
-				)
-				(hide yes)
-			)
-		)
-		(property "Description" ""
-			(at 54.61 99.06 0)
-			(effects
-				(font
-					(size 1.27 1.27)
-				)
-			)
-		)
-		(pin "1"
-		)
-		(instances
-			(project "VoxSense"
-				(path "/ded7c4da-7d9f-418d-838f-f5efc7d9c9cb/9719f155-9a63-4412-a45f-eaa04d0e19ac"
-					(reference "#PWR0136")
-					(unit 1)
-				)

Commit message: * Created an I2C driver and a basic BNO protocol sequence implementation reading the advertisement message. * Created a Vivado project with simulation for the iCE40UL1K FPGA.
Other:
- note added: "NEXT REVISION: Connect ~{H_INT} to FPGA!"
Changed lines of the file:
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@@
+		)
+	)
+	(text "NEXT REVISION:\nConnect ~{H_INT} to FPGA!"
+		(exclude_from_sim no)
+		(at 143.256 97.536 0)
+		(effects
+			(font
+				(size 1.27 1.27)
+				(thickness 0.254)
+				(bold yes)
+				(color 194 0 0 1)
+			)
+			(justify right)
 		)
 	)
