File: Hardware/Sensor_Board/VoxSense.kicad_sch (KiCad schematic)
At the start: 0 parts

Commit message: Added a programmer schematic
Other:
- title: Root -> VoxSense Sensor Board - Root
Changed lines of the file:
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@@
 	(paper "A4")
 	(title_block
-		(title "Root")
+		(title "VoxSense Sensor Board - Root")
 		(date "2025-11-17")
 		(rev "1.0")

Commit message: Pushing before updating KiCad
Other:
- added sheet Connectivity (connectivity.kicad_sch)
Changed lines of the file:
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@@
 	(text "Technical Sheet Only!\nPlease refer to the subsequent sheets for schematic"
 		(exclude_from_sim no)
-		(at 141.732 58.674 0)
+		(at 146.177 56.896 0)
 		(effects
 			(font
@@
 	)
 	(sheet
-		(at 144.78 110.49)
+		(at 120.015 109.22)
 		(size 50.8 34.29)
 		(exclude_from_sim no)
@@
 		)
 		(property "Sheetname" "eFuse"
-			(at 144.78 109.7784 0)
+			(at 120.015 108.5084 0)
 			(effects
 				(font
@@
 		)
 		(property "Sheetfile" "efuse.kicad_sch"
-			(at 144.78 145.3646 0)
+			(at 120.015 144.0946 0)
 			(effects
 				(font
@@
 	)
 	(sheet
-		(at 88.011 69.215)
+		(at 176.53 87.63)
+		(size 50.8 34.29)
+		(exclude_from_sim no)
+		(in_bom yes)
+		(on_board yes)
+		(dnp no)
+		(fields_autoplaced yes)
+		(stroke
+			(width 0.1524)
+			(type solid)
+		)
+		(fill
+			(color 0 0 0 0.0000)
+		)
+		(property "Sheetname" "Connectivity"
+			(at 176.53 86.9184 0)
+			(effects
+				(font
+					(size 1.27 1.27)
+				)
+				(justify left bottom)
+			)
+		)
+		(property "Sheetfile" "connectivity.kicad_sch"
+			(at 176.53 122.5046 0)
+			(effects
+				(font
+					(size 1.27 1.27)
+				)
+				(justify left top)
+			)
+		)
+		(instances
+			(project "VoxSense"
+				(path "/ded7c4da-7d9f-418d-838f-f5efc7d9c9cb"
+					(page "5")
+				)
+			)
+		)
+	)
+	(sheet
+		(at 63.246 67.945)
 		(size 51.054 34.29)
 		(exclude_from_sim no)
@@
 		)
 		(property "Sheetname" "Power"
-			(at 88.011 68.5034 0)
+			(at 63.246 67.2334 0)
 			(effects
 				(font
@@
 		)
 		(property "Sheetfile" "power.kicad_sch"
-			(at 88.011 104.0896 0)
+			(at 63.246 102.8196 0)
 			(effects
 				(font
@@
 	)
 	(sheet
-		(at 144.78 69.85)
+		(at 120.015 68.58)
 		(size 50.8 34.29)
 		(exclude_from_sim no)
@@
 		)
 		(property "Sheetname" "Sensor"
-			(at 144.78 69.1384 0)
+			(at 120.015 67.8684 0)
 			(effects
 				(font
@@
 		)
 		(property "Sheetfile" "Sensor.kicad_sch"
-			(at 144.78 104.7246 0)
+			(at 120.015 103.4546 0)
 			(effects
 				(font
@@
 	)
 	(sheet
-		(at 88.265 111.125)
+		(at 63.5 109.855)
 		(size 51.054 35.052)
 		(exclude_from_sim no)
@@
 		)
 		(property "Sheetname" "System"
-			(at 88.265 110.4134 0)
+			(at 63.5 109.1434 0)
 			(effects
 				(font
@@
 		)
 		(property "Sheetfile" "System.kicad_sch"
-			(at 88.265 146.7616 0)
-			(effects
-				(font
+			(at 63.5 145.4916 0)
+			(effects
+				(font

Commit message: Finished final PCB checks before manufacturing and uploaded the fabrication files
Other:
- note added: "Root [0]"
- note removed: "Root [1]"
Changed lines of the file:
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@@
 		(company "Czech Technical University in Prague")
 	)
-	(text "Root [1]"
+	(text "Root [0]"
 		(exclude_from_sim no)
 		(at 51.308 27.94 0)
