File: Hardware/Sensor_Board/connectivity.kicad_sch (KiCad schematic)
At the start: 18 parts, among them J3 RJ45_Output, J4 RJ45_Input, SW1 Slide Switch, U10 TPD4E02B04, U11 CBTU02044, U3 TPD4E02B04, U301 ICE40UL1K-CM36AI, U4 TPD4E02B04, U9 TPD4E02B04

Commit message: Routing and Schematic update
Parts:
- removed R5: 10k, Resistor_SMD:R_0402_1005Metric, symbol Device:R
Connections:
- net ARCHITECTURE_SEL: now also SW1.2 (CNT)
- net VOX_CLK_N: now also U3.6 (NC); no longer U3.9 (NC)
- net VOX_CLK_P: now also U3.7 (NC); no longer U3.10 (NC)
- net VOX_RX_N: now also U10.7 (NC); no longer U10.9 (NC)
- net VOX_RX_P: now also U10.6 (NC); no longer U10.10 (NC)
- net VOX_TX_N: now also U3.10 (NC); no longer U3.6 (NC)
- net VOX_TX_NOESD_OUT: now also J3.8 (TX); no longer J3.7 (TX)
- net VOX_TX_P: now also U3.9 (NC); no longer U3.7 (NC)
- net ~{VOX_TX}_NOESD_OUT: now also J3.7 (~{TX}); no longer J3.8 (~{TX})
- net VOX_RX_NOESD_IN_N: now reaches U10.4 (IN)
- net VOX_RX_NOESD_IN_N: now also J4.2 (~{RX})
- net VOX_RX_NOESD_IN_P: now reaches U10.5 (IN)
- net VOX_RX_NOESD_IN_P: now also J4.1 (RX)
- net VOX_CLK_NOESD_IN renamed VOX_CLK_NOESD_IN_P
- net VOX_CLK_NOESD_IN_P: now also U3.4 (IN); no longer U3.1 (IN)
- net VOX_RX_NOESD_IN: no longer names the net of U10.1 (IN)
- net VOX_RX_NOESD_IN: no longer J4.1 (RX)
- net VOX_RX_OUT renamed VOX_RX_OUT_P
- net VOX_TX_NOESD_IN renamed VOX_TX_NOESD_IN_N
- net VOX_TX_NOESD_IN_N: now also U3.1 (IN); no longer U3.4 (IN)
- net ~{VOX_CLK}_NOESD_IN renamed VOX_CLK_NOESD_IN_N
- net VOX_CLK_NOESD_IN_N: now also U3.5 (IN); no longer U3.2 (IN)
- net ~{VOX_RX_OUT} renamed VOX_RX_OUT_N
- net ~{VOX_RX}_NOESD_IN: no longer names the net of U10.2 (IN)
- net ~{VOX_RX}_NOESD_IN: no longer J4.2 (~{RX})
- net ~{VOX_TX}_NOESD_IN renamed VOX_TX_NOESD_IN_P
- net VOX_TX_NOESD_IN_P: now also U3.2 (IN); no longer U3.5 (IN)
Other:
- note removed: "Cut-off frequency is 159 Hz"
Changed lines of the file:
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@@
 		)
 	)
-	(text "Cut-off frequency is 159 Hz"
-		(exclude_from_sim no)
-		(at 69.85 168.656 0)
-		(effects
-			(font
-				(size 1.27 1.27)
-				(thickness 0.1588)
-			)
-		)
-	)
 	(text_box "Architecture Selection"
 		(exclude_from_sim no)
@@
 	(wire
 		(pts
-			(xy 85.09 172.72) (xy 87.63 172.72)
-		)
-		(stroke
-			(width 0)
-			(type default)
-		)
-	)
-	(wire
-		(pts
 			(xy 233.68 60.96) (xy 256.54 60.96)
 		)
@@
 	(wire
 		(pts
-			(xy 74.93 172.72) (xy 77.47 172.72)
+			(xy 74.93 172.72) (xy 87.63 172.72)
 		)
 		(stroke
@@
 	)
 	(label "VOX_TX_N"
-		(at 185.42 100.33 180)
+		(at 176.53 100.33 0)
 		(effects
 			(font
 				(size 1.27 1.27)
 			)
-			(justify right bottom)
+			(justify left bottom)
 		)
 	)
@@
 		)
 	)
-	(label "VOX_CLK_NOESD_IN"
+	(label "VOX_CLK_NOESD_IN_P"
 		(at 58.42 60.96 180)
 		(effects
@@
 		)
 	)
-	(label "VOX_RX_OUT"
-		(at 187.96 110.49 180)
+	(label "VOX_RX_OUT_P"
+		(at 176.53 110.49 0)
 		(effects
 			(font
 				(size 1.27 1.27)
 			)
-			(justify right bottom)
+			(justify left bottom)
 		)
 	)
-	(label "~{VOX_CLK}_NOESD_IN"
+	(label "VOX_CLK_NOESD_IN_N"
 		(at 58.42 63.5 180)
 		(effects
@@
 		)
 	)
-	(label "VOX_TX_NOESD_IN"
+	(label "VOX_TX_NOESD_IN_P"
 		(at 58.42 72.39 180)
 		(effects
@@
 		)
 	)
-	(label "~{VOX_TX}_NOESD_IN"
+	(label "VOX_TX_NOESD_IN_N"
 		(at 58.42 74.93 180)
 		(effects
@@
 		)
 	)
-	(label "~{VOX_RX_OUT}"
-		(at 187.96 93.98 180)
+	(label "VOX_RX_OUT_N"
+		(at 176.53 93.98 0)
 		(effects
 			(font
 				(size 1.27 1.27)
 			)
-			(justify right bottom)
+			(justify left bottom)
 		)
 	)
@@
 		)
 	)
-	(label "~{VOX_RX_OUT}"
-		(at 187.96 113.03 180)
+	(label "VOX_RX_OUT_N"
+		(at 176.53 113.03 0)
 		(effects
 			(font
 				(size 1.27 1.27)
 			)
-			(justify right bottom)
+			(justify left bottom)
 		)
 	)
@@
 		)
 	)
-	(label "~{VOX_RX}_NOESD_IN"
+	(label "VOX_RX_NOESD_IN_N"
 		(at 58.42 100.33 180)
 		(effects
@@
 	)
 	(label "VOX_TX_P"
-		(at 185.42 97.79 180)
+		(at 176.53 97.79 0)
 		(effects
 			(font
 				(size 1.27 1.27)
 			)
-			(justify right bottom)
+			(justify left bottom)
 		)
 	)
@@
 		)
 	)
-	(label "VOX_RX_NOESD_IN"
+	(label "VOX_RX_NOESD_IN_P"
 		(at 58.42 97.79 180)
 		(effects
@@
 		)
 	)
-	(label "VOX_RX_OUT"
-		(at 187.96 91.44 180)
+	(label "VOX_RX_OUT_P"
+		(at 176.53 91.44 0)
 		(effects
 			(font
 				(size 1.27 1.27)
 			)
-			(justify right bottom)
+			(justify left bottom)
 		)
 	)
@@
 	)
 	(symbol
+		(lib_name "TPD4E02B04DQA_2")
 		(lib_id "Custom_VoxLink_Symbols:TPD4E02B04DQA")
-		(at 67.31 104.14 0)
+		(at 67.31 105.41 0)
+		(mirror x)
 		(unit 1)
 		(exclude_from_sim no)
@@
 		(dnp no)
 		(property "Reference" "U10"
-			(at 67.31 116.078 0)
+			(at 67.31 93.472 0)
 			(effects
 				(font
@@
 		)
 		(property "Value" "TPD4E02B04"
-			(at 67.31 118.618 0)
+			(at 67.31 90.932 0)
 			(effects
 				(font
@@
 		)
 		(property "Footprint" "Package_SON:USON-10_2.5x1.0mm_P0.5mm"
-			(at 67.31 104.14 0)
+			(at 67.31 105.41 0)
 			(effects
 				(font
@@
 		)
 		(property "Datasheet" ""
-			(at 67.31 104.14 0)
+			(at 67.31 105.41 0)
 			(effects
 				(font
@@
 		)
 		(property "Description" ""
-			(at 67.31 104.14 0)
+			(at 67.31 105.41 0)
 			(effects
 				(font
@@
 		)
 		(property "Distributor Link" "https://www.mouser.sk/ProductDetail/595-TPD4E02B04DQAR"
-			(at 67.31 104.14 0)
+			(at 67.31 105.41 0)
 			(effects
 				(font
@@
 	)
 	(symbol
-		(lib_id "Device:R")
-		(at 81.28 172.72 270)
-		(unit 1)
-		(exclude_from_sim no)
-		(in_bom yes)
-		(on_board yes)
-		(dnp no)
-		(property "Reference" "R5"
-			(at 81.28 177.8 90)
-			(effects
-				(font
-					(size 1.27 1.27)
-				)
-			)
-		)
-		(property "Value" "10k"
-			(at 81.28 175.26 90)
-			(effects
-				(font
-					(size 1.27 1.27)
-				)
-			)
-		)
-		(property "Footprint" "Resistor_SMD:R_0402_1005Metric"
-			(at 81.28 170.942 90)
-			(effects
-				(font
-					(size 1.27 1.27)
-				)
-				(hide yes)
-			)
-		)
-		(property "Datasheet" "https://www.mouser.sk/ProductDetail/Vishay/CRCW040210K0JNED?qs=sGAEpiMZZMtlubZbdhIBIFsfWmIKznfcMCgOmcXe42g%3D"
-			(at 81.28 172.72 0)
-			(effects
-				(font
-					(size 1.27 1.27)
-				)
-				(hide yes)
-			)
-		)
-		(property "Description" ""
-			(at 81.28 172.72 0)
-			(effects
-				(font
-					(size 1.27 1.27)
-				)
-			)
-		)
-		(pin "1"
-		)
-		(pin "2"
-		)
-		(instances
-			(project "VoxSense"
-				(path "/ded7c4da-7d9f-418d-838f-f5efc7d9c9cb/68ca1e05-bb71-451f-9769-47c16f9dd6da"
-					(reference "R5")
-					(unit 1)
-				)
-			)
-		)
-	)
-	(symbol
 		(lib_id "Device:C")
 		(at 74.93 177.8 0)
@@
 	)
 	(symbol
+		(lib_name "TPD4E02B04DQA_1")
 		(lib_id "Custom_VoxLink_Symbols:TPD4E02B04DQA")
-		(at 67.31 67.31 0)
+		(at 67.31 68.58 0)
+		(mirror x)
 		(unit 1)
 		(exclude_from_sim no)
@@
 		(dnp no)
 		(property "Reference" "U3"
-			(at 67.31 79.248 0)
+			(at 67.31 56.642 0)
 			(effects
 				(font
@@
 		)
 		(property "Value" "TPD4E02B04"
-			(at 67.31 81.788 0)
+			(at 67.31 54.102 0)
 			(effects
 				(font
@@
 		)
 		(property "Footprint" "Package_SON:USON-10_2.5x1.0mm_P0.5mm"
-			(at 67.31 67.31 0)
+			(at 67.31 68.58 0)
 			(effects
 				(font
@@
 		)
 		(property "Datasheet" ""
-			(at 67.31 67.31 0)
+			(at 67.31 68.58 0)
 			(effects
 				(font
@@
 		)
 		(property "Description" ""
-			(at 67.31 67.31 0)
+			(at 67.31 68.58 0)
 			(effects
 				(font
@@
 		)
 		(property "Distributor Link" "https://www.mouser.sk/ProductDetail/595-TPD4E02B04DQAR"
-			(at 67.31 67.31 0)
+			(at 67.31 68.58 0)
 			(effects
 				(font

Commit message: Finised the design of the sensor board :)
Parts:
- removed R2, R3: 0R, Resistor_SMD:R_0402_1005Metric, symbol Device:R
- added R503, R504: 0R, Resistor_SMD:R_0402_1005Metric, symbol Device:R
- added TP501, TP502: TestPoint, Custom_VoxLink_Footprints:Vox_Testpoint, symbol Connector:TestPoint
- renumbered C1 to C501, C3 to C502, D3 to D501, D4 to D502, J4 to J501, J3 to J502, R4 to R501, R1 to R502, SW1 to SW501, U3 to U501, U10 to U502, U4 to U503, U9 to U504, U11 to U505
Connections:
- net VOX_CLK_NOESD_IN_N is gone; now on net VOX_CLK_N: J501.5 (~{CLK}), U501.5 (IN)
- net VOX_CLK_NOESD_IN_P is gone; now on net VOX_CLK_P: J501.4 (CLK), U501.4 (IN)
- net VOX_RX_NOESD_IN_N is gone; now on net VOX_RX_N: J501.2 (~{RX}), U502.4 (IN)
- net VOX_RX_NOESD_IN_P is gone; now on net VOX_RX_P: J501.1 (RX), U502.5 (IN)
- net VOX_RX_NOESD_OUT is gone; now on net VOX_RX_OUT_P: J502.1 (RX), U504.1 (IN)
- net VOX_TX_NOESD_IN_N is gone; now on net VOX_TX_N: J501.7 (~{TX}), U501.1 (IN)
- net VOX_TX_NOESD_IN_P is gone; now on net VOX_TX_P: J501.8 (TX), U501.2 (IN)
- net VOX_TX_NOESD_OUT is gone; now on net VOX_TX_P: J502.8 (TX), U503.4 (IN)
- net ~{VOX_RX}_NOESD_OUT is gone; now on net VOX_RX_OUT_N: J502.2 (~{RX}), U504.2 (IN)
- net ~{VOX_TX}_NOESD_OUT is gone; now on net VOX_TX_N: J502.7 (~{TX}), U503.5 (IN)
- net GND: no longer R502.2
- net VOX_CLK_N: now also J502.5 (~{CLK}), R502.2, U503.1 (IN), U503.10 (NC); no longer U503.9 (NC)
- net VOX_CLK_P: now also J502.4 (CLK), R502.1, U503.2 (IN), U503.9 (NC); no longer U503.10 (NC)
- net VOX_RX_OUT_N: now also R504.1
- net VOX_RX_OUT_P: now also R504.2
- net VOX_TX_FPGA_N: now also TP502.1
- net VOX_TX_FPGA_P: now also TP501.1
- net VOX_TX_N: now also R503.1
- net VOX_TX_P: now also R503.2
- net VOX_RX_T_P: now reaches R501.1, U505.5 (C0_P)
- net VOX_RX_T_N: now reaches R501.2, U505.6 (C0_N)
- removed net VOX_CLK_NOESD_OUT: J502.4 (CLK), U503.1 (IN)
- removed net ~{VOX_CLK}_NOESD_OUT: J502.5 (~{CLK}), R502.1, U503.2 (IN)
Other:
- note added: "SEL = LOW -> A and B are conencted SEL = HIGH -> A and C are conencted"
- moved on the sheet: C502, R501, R502, SW501

Commit message: Finished final PCB checks before manufacturing and uploaded the fabrication files
Parts:
- U501, U502, U503, U504: footprint Package_SON:USON-10_2.5x1.0mm_P0.5mm -> Custom_VoxLink_Footprints:USON-10_2.5x1.0mm_P0.5mm__Reduced_Paste
Changed lines of the file:
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@@
 			)
 		)
-		(property "Footprint" "Package_SON:USON-10_2.5x1.0mm_P0.5mm"
+		(property "Footprint" "Custom_VoxLink_Footprints:USON-10_2.5x1.0mm_P0.5mm__Reduced_Paste"
 			(at 67.31 105.41 0)
 			(effects
@@
 			)
 		)
-		(property "Footprint" "Package_SON:USON-10_2.5x1.0mm_P0.5mm"
+		(property "Footprint" "Custom_VoxLink_Footprints:USON-10_2.5x1.0mm_P0.5mm__Reduced_Paste"
 			(at 226.06 97.79 0)
 			(effects
@@
 			)
 		)
-		(property "Footprint" "Package_SON:USON-10_2.5x1.0mm_P0.5mm"
+		(property "Footprint" "Custom_VoxLink_Footprints:USON-10_2.5x1.0mm_P0.5mm__Reduced_Paste"
 			(at 67.31 68.58 0)
 			(effects
@@
 			)
 		)
-		(property "Footprint" "Package_SON:USON-10_2.5x1.0mm_P0.5mm"
+		(property "Footprint" "Custom_VoxLink_Footprints:USON-10_2.5x1.0mm_P0.5mm__Reduced_Paste"
 			(at 226.06 67.31 0)
 			(effects

Commit message: Updated documentation and finished first iteration of PCB rework based on manufacturer feedback.
Parts:
- U301: footprint Custom_VoxLink_Footprints:ICE40UL1K_UCBGA-36 -> Package_BGA:UCBGA-36_2.5x2.5mm_Layout6x6_P0.4mm
Connections:
- net +1V2_CORE: no longer names the net of U301.D2 (IOB_8A_G4)
- no-connect marks 9 -> 10
Other:
- note removed: "1V2_CORE connected to D2 to allow BGA fanout"
Changed lines of the file:
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@@
 		)
 	)
-	(text "1V2_CORE connected to\nD2 to allow BGA fanout"
-		(exclude_from_sim no)
-		(at 130.81 119.38 0)
-		(effects
-			(font
-				(size 1.27 1.27)
-				(color 255 0 0 1)
-			)
-		)
-	)
 	(text "BUS"
 		(exclude_from_sim no)
@@
 	)
 	(no_connect
+		(at 124.46 133.35)
+	)
+	(no_connect
 		(at 233.68 105.41)
 	)
@@
 	(wire
 		(pts
-			(xy 130.81 128.27) (xy 130.81 127)
-		)
-		(stroke
-			(width 0)
-			(type default)
-		)
-	)
-	(wire
-		(pts
 			(xy 175.26 104.14) (xy 189.23 104.14)
 		)
@@
 	(wire
 		(pts
-			(xy 124.46 128.27) (xy 130.81 128.27)
-		)
-		(stroke
-			(width 0)
-			(type default)
-		)
-	)
-	(wire
-		(pts
 			(xy 233.68 63.5) (xy 256.54 63.5)
 		)
@@
 	(global_label "12MHZ_CLK"
 		(shape input)
-		(at 124.46 130.81 0)
+		(at 124.46 127 0)
 		(fields_autoplaced yes)
 		(effects
@@
 		)
 		(property "Intersheetrefs" "${INTERSHEET_REFS}"
-			(at 138.3913 130.81 0)
+			(at 138.3913 127 0)
 			(effects
 				(font
@@
 	(global_label "BNO_SDA"
 		(shape input)
-		(at 124.46 133.35 0)
+		(at 124.46 129.54 0)
 		(fields_autoplaced yes)
 		(effects
@@
 		)
 		(property "Intersheetrefs" "${INTERSHEET_REFS}"
-			(at 135.9119 133.35 0)
+			(at 135.9119 129.54 0)
 			(effects
 				(font
@@
 	)
 	(symbol
-		(lib_id "power:+3.3VA")
-		(at 130.81 127 0)
-		(unit 1)
-		(exclude_from_sim no)
-		(in_bom yes)
-		(on_board yes)
-		(dnp no)
-		(property "Reference" "#PWR0132"
-			(at 130.81 130.81 0)
-			(effects
-				(font
-					(size 1.27 1.27)
-				)
-				(hide yes)
-			)
-		)
-		(property "Value" "+1V2_CORE"
-			(at 125.222 122.936 0)
-			(effects
-				(font
-					(size 1.27 1.27)
-				)
-				(justify left)
-			)
-		)
-		(property "Footprint" ""
-			(at 130.81 127 0)
-			(effects
-				(font
-					(size 1.27 1.27)
-				)
-				(hide yes)
-			)
-		)
-		(property "Datasheet" ""
-			(at 130.81 127 0)
-			(effects
-				(font
-					(size 1.27 1.27)
-				)
-				(hide yes)
-			)
-		)
-		(property "Description" ""
-			(at 130.81 127 0)
-			(effects
-				(font
-					(size 1.27 1.27)
-				)
-			)
-		)
-		(pin "1"
-		)
-		(instances
-			(project "VoxSense"
-				(path "/ded7c4da-7d9f-418d-838f-f5efc7d9c9cb/68ca1e05-bb71-451f-9769-47c16f9dd6da"
-					(reference "#PWR0132")
-					(unit 1)
-				)
-			)
-		)
-	)
-	(symbol
 		(lib_id "power:GND")
 		(at 74.93 67.31 0)
@@
 			)
 		)
-		(property "Footprint" "Custom_VoxLink_Footprints:ICE40UL1K_UCBGA-36"
+		(property "Footprint" "Package_BGA:UCBGA-36_2.5x2.5mm_Layout6x6_P0.4mm"
 			(at 101.6 130.81 0)
 			(effects
