File: Hardware/Sensor_Board/efuse.kicad_sch (KiCad schematic)
At the start: 11 parts, among them U101 TPS25942ARVCR

Commit message: Cleared ERC errors and improved folder structure
Parts:
- removed U101: TPS25942ARVCR, TPS25942ARVCR:QFN50P300X400X80-21N, symbol TPS25942ARVCR:TPS25942ARVCR
- added U101: TPS25942ARVCR, TPS25942ARVCR:QFN50P300X400X80-21N, symbol Custom_VoxLink_Symbols:TPS25942ARVCR
Connections:
- net +5V: now also U101.3 (PGTH), U101.4 (OUT_1), U101.5 (OUT_2), U101.6 (OUT_3), U101.7 (OUT_4), U101.8 (OUT_5)
- net GND: now also U101.1 (DMODE), U101.16 (GND), U101.21 (EP)
- net OVP: now also U101.15 (OVP)
- net UVLO: now also U101.14 (EN)
- net VCC: now also U101.10 (IN_2), U101.11 (IN_3), U101.12 (IN_4), U101.13 (IN_5), U101.9 (IN_1)
- net at D101.2 (A), R105.1: now also U101.2 (PGOOD)
- net at C103.1: now also U101.18 (DVDT)
- net at R106.2: now also U101.17 (ILIM)
Changed lines of the file:
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@@
 	)
 	(junction
+		(at 180.34 88.9)
+		(diameter 0)
+		(color 0 0 0 0)
+	)
+	(junction
 		(at 107.95 76.2)
 		(diameter 0)
@@
 	(wire
 		(pts
-			(xy 180.34 86.36) (xy 180.34 96.52)
+			(xy 180.34 86.36) (xy 180.34 88.9)
 		)
 		(stroke
@@
 	(wire
 		(pts
-			(xy 180.34 86.36) (xy 190.5 86.36)
+			(xy 180.34 88.9) (xy 190.5 88.9)
 		)
 		(stroke
@@
 	(wire
 		(pts
+			(xy 180.34 88.9) (xy 180.34 96.52)
+		)
+		(stroke
+			(width 0)
+			(type default)
+		)
+	)
+	(wire
+		(pts
 			(xy 151.13 106.68) (xy 151.13 107.95)
 		)
@@
 	(wire
 		(pts
-			(xy 190.5 86.36) (xy 190.5 92.71)
+			(xy 190.5 88.9) (xy 190.5 92.71)
 		)
 		(stroke
@@
 	)
 	(symbol
+		(lib_id "Custom_VoxLink_Symbols:TPS25942ARVCR")
+		(at 165.1 90.17 0)
+		(unit 1)
+		(exclude_from_sim no)
+		(in_bom yes)
+		(on_board yes)
+		(dnp no)
+		(fields_autoplaced yes)
+		(property "Reference" "U101"
+			(at 165.735 67.31 0)
+			(effects
+				(font
+					(size 1.27 1.27)
+				)
+			)
+		)
+		(property "Value" "TPS25942ARVCR"
+			(at 165.735 69.85 0)
+			(effects
+				(font
+					(size 1.27 1.27)
+				)
+			)
+		)
+		(property "Footprint" "TPS25942ARVCR:QFN50P300X400X80-21N"
+			(at 165.1 90.17 0)
+			(effects
+				(font
+					(size 1.27 1.27)
+				)
+				(hide yes)
+			)
+		)
+		(property "Datasheet" ""
+			(at 165.1 90.17 0)
+			(effects
+				(font
+					(size 1.27 1.27)
+				)
+				(hide yes)
+			)
+		)
+		(property "Description" ""
+			(at 165.1 90.17 0)
+			(effects
+				(font
+					(size 1.27 1.27)
+				)
+				(hide yes)
+			)
+		)
+		(property "Distributor Link" "https://www.mouser.co.uk/ProductDetail/Texas-Instruments/TPS25942ARVCR?qs=1MXlzafEN39IodrvCe5%252B2w%3D%3D"
+			(at 165.1 90.17 0)
+			(effects
+				(font
+					(size 1.27 1.27)
+				)
+				(hide yes)
+			)
+		)
+		(pin "7"
+		)
+		(pin "6"
+		)
+		(pin "1"
+		)
+		(pin "11"
+		)
+		(pin "10"
+		)
+		(pin "21"
+		)
+		(pin "9"
+		)
+		(pin "18"
+		)
+		(pin "8"
+		)
+		(pin "2"
+		)
+		(pin "15"
+		)
+		(pin "20"
+		)
+		(pin "4"
+		)
+		(pin "12"
+		)
+		(pin "14"
+		)
+		(pin "5"
+		)
+		(pin "3"
+		)
+		(pin "16"
+		)
+		(pin "13"
+		)
+		(pin "19"
+		)
+		(pin "17"
+		)
+		(instances
+			(project ""
+				(path "/ded7c4da-7d9f-418d-838f-f5efc7d9c9cb/52ebae9c-e8b2-4352-947d-ab5ab95db8e1"
+					(reference "U101")
+					(unit 1)
+				)
+			)
+		)
+	)
+	(symbol
 		(lib_id "Device:R")
 		(at 130.81 86.36 180)
@@
 					(unit 1)
 				)
-			)
-		)
-	)
-	(symbol
-		(lib_id "TPS25942ARVCR:TPS25942ARVCR")
-		(at 152.4 82.55 0)
-		(unit 1)
-		(exclude_from_sim no)
-		(in_bom yes)
-		(on_board yes)
-		(dnp no)
-		(fields_autoplaced yes)
-		(property "Reference" "U101"
-			(at 165.735 67.31 0)
-			(effects
-				(font
-					(size 1.27 1.27)
-				)
-			)
-		)
-		(property "Value" "TPS25942ARVCR"
-			(at 165.735 69.85 0)
-			(effects
-				(font
-					(size 1.27 1.27)
-				)
-			)
-		)
-		(property "Footprint" "TPS25942ARVCR:QFN50P300X400X80-21N"
-			(at 179.07 169.85 0)
-			(effects
-				(font
-					(size 1.27 1.27)
-				)
-				(justify left top)
-				(hide yes)
-			)
-		)
-		(property "Datasheet" "https://eu.mouser.com/ProductDetail/Texas-Instruments/TPS25942ARVCR?qs=1MXlzafEN39IodrvCe5%252B2w%3D%3D"
-			(at 179.07 269.85 0)
-			(effects
-				(font
-					(size 1.27 1.27)
-				)
-				(justify left top)
-				(hide yes)
-			)
-		)
-		(property "Description" "18V, 5A, 42m Current Limiting Power MUX eFuse w/Integrated Reverse Current Protection, IMON & PG"
-			(at 152.4 82.55 0)
-			(effects
-				(font
-					(size 1.27 1.27)
-				)
-				(hide yes)
-			)
-		)
-		(property "Height" "0.8"
-			(at 179.07 469.85 0)
-			(effects
-				(font
-					(size 1.27 1.27)
-				)
-				(justify left top)
-				(hide yes)
-			)
-		)
-		(property "Mouser Part Number" "595-TPS25942ARVCR"
-			(at 179.07 569.85 0)
-			(effects
-				(font
-					(size 1.27 1.27)
-				)
-				(justify left top)
-				(hide yes)
-			)
-		)
-		(property "Mouser Price/Stock" "https://www.mouser.co.uk/ProductDetail/Texas-Instruments/TPS25942ARVCR?qs=1MXlzafEN39IodrvCe5%252B2w%3D%3D"
-			(at 179.07 669.85 0)
-			(effects
-				(font
-					(size 1.27 1.27)
-				)
-				(justify left top)
-				(hide yes)
-			)
-		)
-		(property "Manufacturer_Name" "Texas Instruments"
-			(at 179.07 769.85 0)
-			(effects
-				(font
-					(size 1.27 1.27)
-				)
-				(justify left top)
-				(hide yes)
-			)
-		)
-		(property "Manufacturer_Part_Number" "TPS25942ARVCR"
-			(at 179.07 869.85 0)
-			(effects
-				(font
-					(size 1.27 1.27)
-				)
-				(justify left top)
-				(hide yes)
-			)
-		)
-		(pin "2"
-		)
-		(pin "17"
-		)
-		(pin "16"
-		)
-		(pin "15"
-		)
-		(pin "21"
-		)
-		(pin "3"
-		)
-		(pin "6"
-		)
-		(pin "20"
-		)
-		(pin "13"
-		)
-		(pin "7"
-		)
-		(pin "5"
-		)
-		(pin "8"
-		)
-		(pin "1"
-		)
-		(pin "12"
-		)
-		(pin "14"
-		)
-		(pin "9"
-		)
-		(pin "10"
-		)
-		(pin "11"
-		)
-		(pin "18"
-		)
-		(pin "4"
-		)
-		(pin "19"
-		)
-		(instances
-			(project "VoxLink"
-				(path "/ded7c4da-7d9f-418d-838f-f5efc7d9c9cb/52ebae9c-e8b2-4352-947d-ab5ab95db8e1"
-					(reference "U101")
-					(unit 1)
-				)

Commit message: Pushing before updating KiCad
Other:
- moved on the sheet: C101, C102, C103, D101, R101, R102, R103, R104, R105, R106, U101

Commit message: Finished design of both programmer and sensor board PCBs
Parts:
- added D102, D103: Schottky, Diode_SMD:D_0402_1005Metric, symbol Device:D_Schottky
- R105: value 10k -> 1k
Connections:
- net +5V: now also D103.1 (K)
- net GND: now also D102.1 (K); no longer C103.2, R104.1, R106.1, U101.1 (DMODE), U101.16 (GND), U101.21 (EP)
- new net: C103.2, D102.2 (A), D103.2 (A), R104.1, R106.1, U101.1 (DMODE), U101.16 (GND), U101.21 (EP)
Other:
- note added: "Chip connected to GND via Schottky for reverse polarity protection"
