File: Hardware/Sensor_Board/power.kicad_sch (KiCad schematic)
At the start: 25 parts, among them U201 TPS7A20L_1V2, U202 TPS7A20L_2V2, U203 TPS7A20L_3V3, U204 TLV840, U205 ICE40UL1K-CM36AI

Commit message: Cleared ERC errors and improved folder structure
Parts:
- removed U205: ICE40UL1K-CM36AI, Package_BGA:UCBGA-36_2.5x2.5mm_Layout6x6_P0.4mm, symbol Custom_VoxLink_Symbols:ICE40UL1K-CM36AI
- added U301: ICE40UL1K-CM36AI, Package_BGA:UCBGA-36_2.5x2.5mm_Layout6x6_P0.4mm, symbol Custom_VoxLink_Symbols:ICE40UL1K-CM36AI
Connections:
- net +1V2_CORE: now also U301.D3 (VCC)
- net +1V2_PLL: now also U301.D4 (VCCPLL)
- net +2V5_NVCM: now also U301.B4 (VPP2V5)
- net +3V3: now also U301.B3 (VCCIO0), U301.E3 (VCCIO2), U301.E4 (SPI_VCCIO1)
- net GND: now also U301.C3 (GND), U301.C4 (GND), U301.C5 (GND_LED)
Other:
- moved on the sheet: C211, C212

Commit message: Fixed minor bugs in the schematic and updated the documentation.
Connections:
- net +1V2_CORE: now also U203.3 (EN)
- net +2V5_NVCM: no longer C201.1, U201.3 (EN), U201.4 (IN)
- net +3V3: now also U202.3 (EN)
- net +5V: now also C201.1, U201.3 (EN), U201.4 (IN); no longer U202.3 (EN), U203.3 (EN)
Other:
- note added: "C [uF] = (T_delay [uS] - 80uS) / 618937 32nF = (20,000us - 80uS) / 618937"
- note added: "EN_HIGH = 0.9V EN_LOW = 0.3V EN_MAX = 6.5V"
- note added: "Note that ~{CRESET} is active LOW, meaning the FPGA is active when ~{CRESET} is HIGH. This requires a ~{RESET} variant of the TLV840 chip which active LOW, meaning it is the correct reset logic."
- note added: "The FPGA wakes up after rougly 10us, however, the memory takes 150us to boot. We need to delay the FPGA startup, so that the flash memory is ready."
- note removed: "C [uF] = (T_delay - 80uS) / 618937 32nF = (20,000us - 80uS) / 618937"
- note removed: "The FPGA wakes up after rougly 10ms, however, the memory takes 20ms to boot. We need to delay the FPGA startup, so that the flash memory is ready."
- moved on the sheet: C203, C205

Commit message: Added a programmer schematic
Other:
- moved on the sheet: C201, C202, C203, C204, C205, C206, C207, C208, C209, C210, C211, C212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

Commit message: Pushing before updating KiCad
Parts:
- removed C218: 100n, Capacitor_SMD:C_0402_1005Metric, symbol Device:C
- C208: value 32n -> 33n
- C209, C213, C215: footprint (none) -> Capacitor_SMD:C_0603_1608Metric
- C211: footprint (none) -> Capacitor_SMD:C_0805_2012Metric; now not fitted; now left out of the parts list
- C212: now not fitted; now left out of the parts list
- R201: footprint (none) -> Resistor_SMD:R_0402_1005Metric
- R202: footprint (none) -> Resistor_SMD:R_0402_1005Metric; now not fitted; now left out of the parts list
- U301: footprint Package_BGA:UCBGA-36_2.5x2.5mm_Layout6x6_P0.4mm -> Custom_VoxLink_Footprints:ICE40UL1K_UCBGA-36
Connections:
- net +1V2_PLL is gone; now on net +1V2_CORE: C211.1, C212.1, R202.2, U301.D4 (VCCPLL)
- net CT: now reaches C208.1, U204.5 (CT)
Other:
- note added: "Due to tight BGA fanout, the 1V2_CORE and 1V2_PLL have to be connected together."

Commit message: Updated documentation and finished first iteration of PCB rework based on manufacturer feedback.
Parts:
- U301: footprint Custom_VoxLink_Footprints:ICE40UL1K_UCBGA-36 -> Package_BGA:UCBGA-36_2.5x2.5mm_Layout6x6_P0.4mm
Changed lines of the file:
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@@
 			)
 		)
-		(property "Footprint" "Custom_VoxLink_Footprints:ICE40UL1K_UCBGA-36"
+		(property "Footprint" "Package_BGA:UCBGA-36_2.5x2.5mm_Layout6x6_P0.4mm"
 			(at 255.27 82.55 0)
 			(effects

Commit message: Added comments to the schematic, updated documentation with the board bringup, and wrote the VoxLink Verilog blink sketch.
Parts:
- U204: value TLV840 -> TLV840MADL
Other:
- note added: "U204 is removed in the prototype version"
Changed lines of the file:
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@@
 		)
 	)
+	(text "U204 is removed in the \nprototype version"
+		(exclude_from_sim no)
+		(at 118.872 109.728 0)
+		(effects
+			(font
+				(size 1.27 1.27)
+				(thickness 0.254)
+				(bold yes)
+				(color 194 0 0 1)
+			)
+			(justify left)
+		)
+	)
 	(text_box "FPGA Power Input"
 		(exclude_from_sim no)
@@
 		(dnp no)
 		(property "Reference" "U204"
-			(at 115.062 92.71 0)
+			(at 117.348 90.678 0)
 			(effects
 				(font
@@
 			)
 		)
-		(property "Value" "TLV840"
-			(at 115.062 95.25 0)
+		(property "Value" "TLV840MADL"
+			(at 117.348 93.218 0)
 			(effects
 				(font
