File: Hardware/Controller_Board/ftdi.kicad_sch (KiCad schematic)
At the start: 0 parts

Commit message: Commited Schematic Changes
Other:
- company: (none) -> Czech Technical University in Prague
Changed lines of the file:
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@@
 	(generator_version "9.0")
 	(paper "A4")
+	(title_block
+		(rev "1.0")
+		(company "Czech Technical University in Prague")
+		(comment 1 "Designer: Michal Varsanyi")
+	)
 )

Commit message: Updated schematic diagram with configuration
Parts:
- added C201, C203, C207, C72: 4u7, Capacitor_SMD:C_0402_1005Metric, symbol Device:C
- added C202, C204, C208, C209, C210, C211, C213, C214, C215, C216: 100n, Capacitor_SMD:C_0402_1005Metric, symbol Device:C
- added C205, C206: 10p, Capacitor_SMD:C_0402_1005Metric, symbol Device:C
- added FB201, FB202: 600R, Inductor_SMD:L_0402_1005Metric, symbol Device:FerriteBead
- added R201: 22R, Resistor_SMD:R_0402_1005Metric, symbol Device:R
- added R202: 2k2, Resistor_SMD:R_0402_1005Metric, symbol Device:R
- added R203, R204, R205: 10k, Resistor_SMD:R_0402_1005Metric, symbol Device:R
- added R206: 12k, Resistor_SMD:R_0402_1005Metric, symbol Device:R
- added R207: 1k, Resistor_SMD:R_0402_1005Metric, symbol Device:R
- added U201: FT2232HQ, Package_DFN_QFN:QFN-64-1EP_9x9mm_P0.5mm_EP4.35x4.35mm, symbol Interface_USB:FT2232HQ
- added U202: 93LC56B, Package_DFN_QFN:TDFN-8-1EP_3x2mm_P0.5mm_EP1.3x1.4mm, symbol Custom_VoxLink_Symbols:93LC56B
- added Y201: 12MHz, Crystal:Crystal_SMD_2520-4Pin_2.5x2.0mm, symbol Device:Crystal_GND24
Connections:
- new net: R202.1, R205.1, U202.4 (DO)
- new net: R207.2, U201.14 (~{RESET})
- new net: R206.2, U201.6 (REF)
- new net: C206.1, R201.2, Y201.3
- new net +1V8_FTDI: C213.1, C214.1, C215.1, C72.1, U201.12 (VCORE), U201.37 (VCORE), U201.49 (VREGOUT), U201.64 (VCORE)
- new net +3V3: C207.1, C208.1, C209.1, C210.1, C211.1, C216.1, FB201.2, FB202.2, R203.2, R204.2, R205.2, R207.1, U201.20 (VCCIO), U201.31 (VCCIO), U201.42 (VCCIO), U201.50 (VREGIN), U201.56 (VCCIO), U202.6 (ORG), U202.8 (VCC)
- new net +3V3_VPHY: C201.1, C202.1, FB201.1, U201.4 (VPHY)
- new net +3V3_VPLL: C203.1, C204.1, FB202.1, U201.9 (VPLL)
- new net EECLK: R204.1, U201.62 (EECLK), U202.2 (CLK)
- new net EECS: R203.1, U201.63 (EECS), U202.1 (CS)
- new net EEDATA: R202.2, U201.61 (EEDATA), U202.3 (DI)
- new net FTDI_USB_D+: U201.8 (DP)
- new net FTDI_USB_D-: U201.7 (DM)
- new net GND: C201.2, C202.2, C203.2, C204.2, C205.2, C206.2, C207.2, C208.2, C209.2, C210.2, C211.2, C213.2, C214.2, C215.2, C216.2, C72.2, R206.1, U201.1 (GND), U201.10 (AGND), U201.11 (GND), U201.13 (TEST), U201.15 (GND), U201.25 (GND), U201.35 (GND), U201.47 (GND), U201.5 (GND), U201.51 (GND), U201.65 (GND), U202.5 (VSS), U202.9 (EP), Y201.2, Y201.4
- new net OSC_IN: C205.1, U201.2 (OSCI), Y201.1
- new net OSC_OUT: R201.1, U201.3 (OSCO)
- no-connect marks 0 -> 30
Other:
- note added: "(10pF Load Capacitance - 5pF Stray Capacitance) * 2 = 10pF Load Capacitors"
- note added: "FTDI [3]"
- note added: "Ferrite beads must be rated at least for 600mA"
- note added: "WE HAVE TO CHECK THE TDI/TDO CONNECTIONS!"
