File: Hardware/Controller_Board/Controller_Board.kicad_pcb (KiCad board)
At the start: 2 copper layers, 33 parts, among them U1 XC7A35T-CPG236, U2 TPS82084, U3 LT8645S, U4 TPS82084, U5 TPS82084, U6 XT30

Commit message: Updated the domcumentation
Parts:
- added D308: LED, LED_SMD:LED_0603_1608Metric, F.Cu at (133.3, 48.7)
- added Q1: DMN2400UFB-7, Package_DFN_QFN:Diodes_DFN1006-3, F.Cu at (135.8, 51.4)
- added R13: 280R, Resistor_SMD:R_0402_1005Metric, F.Cu at (132.7, 51.0)

Commit message: Commited Schematic Changes
Parts:
- removed U1: XC7A35T-CPG236, Package_BGA:Xilinx_CPG236
- added C14: 100n, Capacitor_SMD:C_0402_1005Metric, F.Cu at (165.7, 31.5)
- added C15: 10p, Capacitor_SMD:C_0402_1005Metric, F.Cu at (165.7, 33.4)
- added C16: 10u, Capacitor_SMD:C_0805_2012Metric, F.Cu at (162.0, 32.0)
- added C17: 1u, Capacitor_SMD:C_0402_1005Metric, F.Cu at (165.7, 35.4)
- added C18: 100n, Capacitor_SMD:C_0402_1005Metric, F.Cu at (165.7, 37.4)
- added C19: 100n, Capacitor_SMD:C_0402_1005Metric, F.Cu at (165.7, 39.3)
- added C20: 100n, Capacitor_SMD:C_0402_1005Metric, F.Cu at (165.7, 41.3)
- added C21: 100n, Capacitor_SMD:C_0402_1005Metric, F.Cu at (165.7, 43.3)
- added C22: 100n, Capacitor_SMD:C_0402_1005Metric, F.Cu at (165.7, 45.2)
- added C23: 100n, Capacitor_SMD:C_0402_1005Metric, F.Cu at (168.5, 31.5)
- added C24: 100n, Capacitor_SMD:C_0402_1005Metric, F.Cu at (168.5, 33.4)
- added C25: 100n, Capacitor_SMD:C_0402_1005Metric, F.Cu at (168.5, 35.4)
- added C26: 100n, Capacitor_SMD:C_0402_1005Metric, F.Cu at (168.5, 37.4)
- added C27: 100n, Capacitor_SMD:C_0402_1005Metric, F.Cu at (168.5, 39.3)
- added C28: 100n, Capacitor_SMD:C_0402_1005Metric, F.Cu at (168.5, 41.3)
- added C29: 100n, Capacitor_SMD:C_0402_1005Metric, F.Cu at (168.5, 43.3)
- added C30: 100n, Capacitor_SMD:C_0402_1005Metric, F.Cu at (168.5, 45.2)
- added C31: 100n, Capacitor_SMD:C_0402_1005Metric, F.Cu at (171.4, 31.5)
- added C32: 1u, Capacitor_SMD:C_0402_1005Metric, F.Cu at (171.4, 33.4)
- added C33: 100n, Capacitor_SMD:C_0402_1005Metric, F.Cu at (171.4, 35.4)
- added C34: 100n, Capacitor_SMD:C_0402_1005Metric, F.Cu at (171.4, 37.4)
- added C35: 100n, Capacitor_SMD:C_0402_1005Metric, F.Cu at (171.4, 39.3)
- added C36: 100n, Capacitor_SMD:C_0402_1005Metric, F.Cu at (171.4, 41.3)
- added C37: 100n, Capacitor_SMD:C_0402_1005Metric, F.Cu at (171.4, 43.3)
- added C38: 100n, Capacitor_SMD:C_0402_1005Metric, F.Cu at (171.4, 45.2)
- added C39: 1u, Capacitor_SMD:C_0402_1005Metric, F.Cu at (174.3, 31.5)
- added C40: 10u, Capacitor_SMD:C_0805_2012Metric, F.Cu at (162.0, 35.0)
- added C41: 100n, Capacitor_SMD:C_0402_1005Metric, F.Cu at (174.3, 33.4)
- added C42: 100n, Capacitor_SMD:C_0402_1005Metric, F.Cu at (174.3, 35.4)
- added C43: 100n, Capacitor_SMD:C_0402_1005Metric, F.Cu at (174.3, 37.4)
- added C44: 100n, Capacitor_SMD:C_0402_1005Metric, F.Cu at (174.3, 39.3)
- added C45: 1u, Capacitor_SMD:C_0402_1005Metric, F.Cu at (174.3, 41.3)
- added C46: 100n, Capacitor_SMD:C_0402_1005Metric, F.Cu at (174.3, 43.3)
- added C47: 100n, Capacitor_SMD:C_0402_1005Metric, F.Cu at (174.3, 45.2)
- added C48: 100n, Capacitor_SMD:C_0402_1005Metric, F.Cu at (177.1, 31.5)
- added C49: 100n, Capacitor_SMD:C_0402_1005Metric, F.Cu at (177.1, 33.4)
- added C50: 100n, Capacitor_SMD:C_0402_1005Metric, F.Cu at (177.1, 35.4)
- added C51: 100n, Capacitor_SMD:C_0402_1005Metric, F.Cu at (177.1, 37.4)
- added C52: 100n, Capacitor_SMD:C_0402_1005Metric, F.Cu at (177.1, 39.3)
- added C53: 100n, Capacitor_SMD:C_0402_1005Metric, F.Cu at (177.1, 41.3)
- added C54: 1u, Capacitor_SMD:C_0402_1005Metric, F.Cu at (177.1, 43.3)
- added C55: 10u, Capacitor_SMD:C_0805_2012Metric, F.Cu at (162.0, 38.0)
- added C56: 1u, Capacitor_SMD:C_0402_1005Metric, F.Cu at (177.1, 45.2)
- added C57: 10u, Capacitor_SMD:C_0805_2012Metric, F.Cu at (162.0, 41.0)
- added C58: 1u, Capacitor_SMD:C_0402_1005Metric, F.Cu at (180.0, 31.5)
- added C59: 1u, Capacitor_SMD:C_0402_1005Metric, F.Cu at (180.0, 33.4)
- added C60: 10u, Capacitor_SMD:C_0805_2012Metric, F.Cu at (162.0, 44.0)
- added C61: 100n, Capacitor_SMD:C_0402_1005Metric, F.Cu at (180.0, 35.4)
- added C62: 100n, Capacitor_SMD:C_0402_1005Metric, F.Cu at (180.0, 37.4)
- added C63: 1u, Capacitor_SMD:C_0402_1005Metric, F.Cu at (180.0, 39.3)
- added C64: 10u, Capacitor_SMD:C_0805_2012Metric, F.Cu at (162.0, 47.0)
- added C65: 1u, Capacitor_SMD:C_0402_1005Metric, F.Cu at (180.0, 41.3)
- added C66: 1u, Capacitor_SMD:C_0402_1005Metric, F.Cu at (180.0, 43.3)
- added C67: 1u, Capacitor_SMD:C_0402_1005Metric, F.Cu at (180.0, 45.2)
- added C68: 10u, Capacitor_SMD:C_0805_2012Metric, F.Cu at (162.0, 50.0)
- added C69: 100u, Capacitor_SMD:CP_Elec_8x6.5, F.Cu at (151.9, 35.4)
- added C70: 100u, Capacitor_SMD:CP_Elec_8x6.5, F.Cu at (151.9, 45.2)
- added C71: 100u, Capacitor_SMD:CP_Elec_8x6.5, F.Cu at (151.9, 55.1)
- added C77: 10u, Capacitor_SMD:C_0805_2012Metric, F.Cu at (162.0, 53.0)
- C11, C12: value 0.47u -> 470n

Commit message: Commited Schematic Changes
Parts:
- removed D301: TVS, Diode_SMD:D_0402_1005Metric
- added U1: XC7A35T-CPG236, Package_BGA:Xilinx_CPG236, F.Cu at (135.8, 37.4)

Commit message: Updated schematic diagram with configuration
Parts:
- added C201: 4u7, Capacitor_SMD:C_0402_1005Metric, F.Cu at (167.4, 64.1)
- added C202: 100n, Capacitor_SMD:C_0402_1005Metric, F.Cu at (167.4, 66.1)
- added C203: 4u7, Capacitor_SMD:C_0402_1005Metric, F.Cu at (167.4, 68.1)
- added C204: 100n, Capacitor_SMD:C_0402_1005Metric, F.Cu at (170.2, 62.2)
- added C205: 10p, Capacitor_SMD:C_0402_1005Metric, F.Cu at (170.2, 64.1)
- added C206: 10p, Capacitor_SMD:C_0402_1005Metric, F.Cu at (170.2, 66.1)
- added C207: 4u7, Capacitor_SMD:C_0402_1005Metric, F.Cu at (170.2, 68.1)
- added C208: 100n, Capacitor_SMD:C_0402_1005Metric, F.Cu at (173.1, 62.2)
- added C209: 100n, Capacitor_SMD:C_0402_1005Metric, F.Cu at (173.1, 64.1)
- added C210: 100n, Capacitor_SMD:C_0402_1005Metric, F.Cu at (173.1, 66.1)
- added C211: 100n, Capacitor_SMD:C_0402_1005Metric, F.Cu at (173.1, 68.1)
- added C213: 100n, Capacitor_SMD:C_0402_1005Metric, F.Cu at (176.0, 62.2)
- added C214: 100n, Capacitor_SMD:C_0402_1005Metric, F.Cu at (176.0, 64.1)
- added C215: 100n, Capacitor_SMD:C_0402_1005Metric, F.Cu at (176.0, 66.1)
- added C216: 100n, Capacitor_SMD:C_0402_1005Metric, F.Cu at (176.0, 68.1)
- added C72: 4u7, Capacitor_SMD:C_0402_1005Metric, F.Cu at (167.4, 62.2)
- added C73: 100n, Capacitor_SMD:C_0402_1005Metric, F.Cu at (167.4, 79.6)
- added FB201: 600R, Inductor_SMD:L_0402_1005Metric, F.Cu at (178.9, 62.2)
- added FB202: 600R, Inductor_SMD:L_0402_1005Metric, F.Cu at (178.9, 64.2)
- added R201: 22R, Resistor_SMD:R_0402_1005Metric, F.Cu at (178.9, 66.2)
- added R202: 2k2, Resistor_SMD:R_0402_1005Metric, F.Cu at (181.8, 62.2)
- added R203: 10k, Resistor_SMD:R_0402_1005Metric, F.Cu at (181.8, 64.2)
- added R204: 10k, Resistor_SMD:R_0402_1005Metric, F.Cu at (181.8, 66.2)
- added R205: 10k, Resistor_SMD:R_0402_1005Metric, F.Cu at (184.7, 62.2)
- added R206: 12k, Resistor_SMD:R_0402_1005Metric, F.Cu at (184.7, 64.2)
- added R207: 1k, Resistor_SMD:R_0402_1005Metric, F.Cu at (184.7, 66.2)
- added U201: FT2232HQ, Package_DFN_QFN:QFN-64-1EP_9x9mm_P0.5mm_EP4.35x4.35mm, F.Cu at (171.9, 55.6)
- added U202: 93LC56B, Package_DFN_QFN:TDFN-8-1EP_3x2mm_P0.5mm_EP1.3x1.4mm, F.Cu at (180.2, 51.8)
- added U7: IS25LP256D, Package_SON:WSON-8-1EP_8x6mm_P1.27mm_EP3.4x4.3mm, F.Cu at (188.9, 46.9)
- added Y201: 12MHz, Crystal:Crystal_SMD_2520-4Pin_2.5x2.0mm, F.Cu at (179.8, 55.6)
- L4: footprint Inductor_SMD:L_Coilcraft_XAL6060-XXX -> Inductor_SMD:L_Coilcraft_XAL6030-XXX

Commit message: Added USB hub symbol
Parts:
- removed C213, C214: 100n, Capacitor_SMD:C_0402_1005Metric
- removed the C72 at (167.4, 62.2)
- removed U201: FT2232HQ, Package_DFN_QFN:QFN-64-1EP_9x9mm_P0.5mm_EP4.35x4.35mm
- added C100: 4u7, Capacitor_SMD:C_0402_1005Metric, F.Cu at (121.4, 68.7)
- added C101: 100n, Capacitor_SMD:C_0402_1005Metric, F.Cu at (121.4, 70.6)
- added C102: 100n, Capacitor_SMD:C_0402_1005Metric, F.Cu at (124.2, 60.8)
- added C103: 10p, Capacitor_SMD:C_0402_1005Metric, F.Cu at (124.2, 62.8)
- added C104: 10p, Capacitor_SMD:C_0402_1005Metric, F.Cu at (124.2, 64.7)
- added C74: 1u, Capacitor_SMD:C_0402_1005Metric, F.Cu at (134.0, 89.3)
- added C80: 100n, Capacitor_SMD:C_0402_1005Metric, F.Cu at (129.1, 82.3)
- added C82: 100n, Capacitor_SMD:C_0402_1005Metric, F.Cu at (129.1, 84.3)
- added C90: 4u7, Capacitor_SMD:C_0402_1005Metric, F.Cu at (118.5, 60.8)
- added C91: 100n, Capacitor_SMD:C_0402_1005Metric, F.Cu at (118.5, 62.8)
- added C92: 100n, Capacitor_SMD:C_0402_1005Metric, F.Cu at (118.5, 64.7)
- added C93: 100n, Capacitor_SMD:C_0402_1005Metric, F.Cu at (118.5, 66.7)
- added C94: 100n, Capacitor_SMD:C_0402_1005Metric, F.Cu at (118.5, 68.7)
- added C95: 100n, Capacitor_SMD:C_0402_1005Metric, F.Cu at (118.5, 70.6)
- added C96: 100n, Capacitor_SMD:C_0402_1005Metric, F.Cu at (121.4, 60.8)
- added C97: 100n, Capacitor_SMD:C_0402_1005Metric, F.Cu at (121.4, 62.8)
- added C98: 4u7, Capacitor_SMD:C_0402_1005Metric, F.Cu at (121.4, 64.7)
- added C99: 100n, Capacitor_SMD:C_0402_1005Metric, F.Cu at (121.4, 66.7)
- added D3: LED, LED_SMD:LED_0603_1608Metric, F.Cu at (134.6, 87.1)
- added FB4: 600R, Inductor_SMD:L_0402_1005Metric, F.Cu at (127.1, 71.0)
- added FB5: 600R, Inductor_SMD:L_0402_1005Metric, F.Cu at (127.1, 73.0)
- added R14: 200R, Resistor_SMD:R_0402_1005Metric, F.Cu at (138.1, 86.8)
- added R17: 200R, Resistor_SMD:R_0402_1005Metric, F.Cu at (138.1, 88.8)
- added R33: 1k, Resistor_SMD:R_0402_1005Metric, F.Cu at (127.1, 75.0)
- added R34: 12k, Resistor_SMD:R_0402_1005Metric, F.Cu at (130.1, 71.0)
- added R35: 10k, Resistor_SMD:R_0402_1005Metric, F.Cu at (130.1, 73.0)
- added R36: 10k, Resistor_SMD:R_0402_1005Metric, F.Cu at (130.1, 75.0)
- added R37: 10k, Resistor_SMD:R_0402_1005Metric, F.Cu at (133.0, 71.0)
- added R38: 2k2, Resistor_SMD:R_0402_1005Metric, F.Cu at (133.0, 73.0)
- added R39: 22R, Resistor_SMD:R_0402_1005Metric, F.Cu at (133.0, 75.0)
- added SW1: Reset, Button_Switch_SMD:SW_Push_SPST_NO_Alps_SKRK, F.Cu at (135.8, 83.5)
- added U10: FT232H, Package_DFN_QFN:QFN-48-1EP_8x8mm_P0.5mm_EP6.2x6.2mm, F.Cu at (131.2, 64.9)
- added U11: 93LC56B, Package_DFN_QFN:TDFN-8-1EP_3x2mm_P0.5mm_EP1.3x1.4mm, F.Cu at (119.7, 73.5)
- added U8: FT232H, Package_DFN_QFN:QFN-48-1EP_8x8mm_P0.5mm_EP6.2x6.2mm, F.Cu at (122.6, 86.5)
- added Y2: 12MHz, Crystal:Crystal_SMD_2520-4Pin_2.5x2.0mm, F.Cu at (119.3, 77.3)
- renumbered C13 to C1, C1 to C10, C4 to C11, C5 to C12, C70 to C13, C6 to C14, C7 to C15, C71 to C16, C14 to C17, C15 to C18, C46 to C19, C12 to C2, C47 to C20, C59 to C21, C60 to C22, C48 to C23, C49 to C24, C50 to C25, C51 to C26, C52 to C27, C53 to C28, C56 to C29, C11 to C3, C58 to C30, C54 to C31, C55 to C32, C68 to C33, C67 to C34, C66 to C35, C65 to C36, C25 to C37, C24 to C38, C23 to C39, C10 to C4, C22 to C40, C21 to C41, C20 to C42, C16 to C43, C17 to C44, C18 to C45, C19 to C46, C41 to C47, C42 to C48, C43 to C49, C9 to C5, C44 to C50, C45 to C51, C57 to C52, C33 to C53, C34 to C54, C35 to C55, C36 to C56, C37 to C57, C38 to C58, C39 to C59, C8 to C6, C40 to C60, C64 to C61, C63 to C62, C62 to C63, C61 to C64, C26 to C65, C27 to C66, C28 to C67, C29 to C68, C30 to C69, C2 to C7, C31 to C70, C32 to C71, C77 to C72, C207 to C75, C208 to C76, C209 to C77, C210 to C78, C211 to C79, C3 to C8, C215 to C81, C201 to C83, C202 to C84, C203 to C85, C204 to C86, C216 to C87, C205 to C88, C206 to C89, C69 to C9, D308 to D1, FB201 to FB2, FB202 to FB3, L4 to L1, R7 to R1, R207 to R26, R206 to R27, R205 to R28, R203 to R29, R1 to R3, R204 to R30, R202 to R31, R201 to R32, R8 to R4, R3 to R5, R9 to R6, R4 to R7, R5 to R8, R6 to R9, U2 to U1, U3 to U2, U4 to U3, U5 to U4, U6 to U5, U1 to U6, U202 to U9, Y201 to Y1
Connections:
- net /FTDI/EECLK renamed /JTAG/EECLK
- net /FTDI/EECS renamed /JTAG/EECS
- net /FTDI/EEDATA renamed /JTAG/EEDATA
- net /FTDI/OSC_IN renamed /JTAG/OSC_IN
- C18 pad 2: AGND -> GND
- C81 pad 1: +1V8_FTDI -> Net-(U8-VCCCORE)
- R32 pad 1: /FTDI/OSC_OUT -> /JTAG/OSC_OUT
- U6 pad A11: (no net) -> GND
- U6 pad A12: (no net) -> GND
- U6 pad A13: (no net) -> GND
- U6 pad B11: (no net) -> GND
- U6 pad B12: (no net) -> GND
- U6 pad B13: (no net) -> GND
- U6 pad C11: (no net) -> /FPGA_Config/SCK_FPGA
- U6 pad C12: AGND -> GND
- U6 pad C8: (no net) -> /FPGA_Config/TDO_FPGA
- U6 pad D18: (no net) -> /FPGA_Config/SDI_FPGA
- U6 pad D19: (no net) -> /FPGA_Config/SDO_FPGA
- U6 pad F18: (no net) -> /FPGA_Config/NHL_FPGA
- U6 pad G18: (no net) -> /FPGA_Config/NWP_FPGA
- U6 pad K19: (no net) -> /FPGA_Config/NCS_FPGA
- U6 pad U10: (no net) -> /FPGA_Config/MODE2
- U6 pad U11: (no net) -> /FPGA_Config/FPGA_INIT
- U6 pad U12: (no net) -> /FPGA_Config/FPGA_DONE
- U6 pad V10: (no net) -> /FPGA_Config/FPGA_RST
- U6 pad V11: (no net) -> Net-(U6B-CFGBVS_0)
- U6 pad V12: (no net) -> /FPGA_Config/MODE0
- U6 pad W10: (no net) -> /FPGA_Config/TMS
- U6 pad W11: (no net) -> /FPGA_Config/MODE1
- U6 pad W8: (no net) -> /FPGA_Config/TCK
- U6 pad W9: (no net) -> /FPGA_Config/TDI_FPGA
- U7 pad 1: unconnected-(U7-NCS-Pad1) -> /FPGA_Config/NCS_FPGA
- U7 pad 2: unconnected-(U7-SDO-Pad2) -> /FPGA_Config/SDO_FLASH
- U7 pad 3: unconnected-(U7-NWP-Pad3) -> /FPGA_Config/NWP_FLASH
- U7 pad 5: unconnected-(U7-SDI-Pad5) -> /FPGA_Config/SDI_FLASH
- U7 pad 6: unconnected-(U7-SCK-Pad6) -> /FPGA_Config/SCK_FLASH
- U7 pad 7: unconnected-(U7-NHOLD-Pad7) -> /FPGA_Config/NHL_FLASH
- U7 pad 9: (no net) -> GND

Commit message: Updated the schematic design - Fix the XC7A35T-CPG236 outline issue
Parts:
- added C105: 10p, Capacitor_SMD:C_0402_1005Metric, F.Cu at (132.7, 94.0)
- added C106: 10p, Capacitor_SMD:C_0402_1005Metric, F.Cu at (132.7, 95.9)
- added C107: 4u7, Capacitor_SMD:C_0402_1005Metric, F.Cu at (132.7, 97.9)
- added C108: 100n, Capacitor_SMD:C_0402_1005Metric, F.Cu at (132.7, 99.9)
- added C109: 100n, Capacitor_SMD:C_0402_1005Metric, F.Cu at (135.6, 80.2)
- added C110: 100n, Capacitor_SMD:C_0402_1005Metric, F.Cu at (135.6, 82.1)
- added C111: 100n, Capacitor_SMD:C_0402_1005Metric, F.Cu at (135.6, 84.1)
- added C112: 100n, Capacitor_SMD:C_0402_1005Metric, F.Cu at (135.6, 86.1)
- added C113: 100n, Capacitor_SMD:C_0402_1005Metric, F.Cu at (135.6, 88.0)
- added C114: 10n, Capacitor_SMD:C_0402_1005Metric, F.Cu at (135.6, 90.0)
- added C115: 100n, Capacitor_SMD:C_0402_1005Metric, F.Cu at (135.6, 92.0)
- added C116: 10n, Capacitor_SMD:C_0402_1005Metric, F.Cu at (135.6, 94.0)
- added C117: 100n, Capacitor_SMD:C_0402_1005Metric, F.Cu at (135.6, 95.9)
- added D104: TVS, Diode_SMD:D_0402_1005Metric, F.Cu at (119.8, 129.3)
- added D105: LED, LED_SMD:LED_0603_1608Metric, F.Cu at (113.2, 127.8)
- added J103: USB_C_USB2.0, Connector_USB:USB_C_Receptacle_GCT_USB4105-xx-A_16P_TopMnt_Horizontal, F.Cu at (118.0, 62.1)
- added R104: 5k1, Resistor_SMD:R_0402_1005Metric, F.Cu at (150.1, 84.2)
- added R105: 5k1, Resistor_SMD:R_0402_1005Metric, F.Cu at (150.1, 86.1)
- added R107: 1k, Resistor_SMD:R_0402_1005Metric, F.Cu at (150.1, 88.1)
- added R40: 22R, Resistor_SMD:R_0402_1005Metric, F.Cu at (147.2, 86.1)
- added R41: 12k, Resistor_SMD:R_0402_1005Metric, F.Cu at (147.2, 88.1)
- added R42: 100k, Resistor_SMD:R_0402_1005Metric, F.Cu at (147.2, 90.1)
- added R43: 100k, Resistor_SMD:R_0402_1005Metric, F.Cu at (147.2, 92.1)
- added R44: 100k, Resistor_SMD:R_0402_1005Metric, F.Cu at (147.2, 94.1)
- added R45: 100k, Resistor_SMD:R_0402_1005Metric, F.Cu at (147.2, 96.1)
- added R46: 100k, Resistor_SMD:R_0402_1005Metric, F.Cu at (147.2, 98.1)
- added R47: 100k, Resistor_SMD:R_0402_1005Metric, F.Cu at (150.1, 80.2)
- added R48: 1k, Resistor_SMD:R_0402_1005Metric, F.Cu at (150.1, 82.2)
- added U12: USB2512B, Package_DFN_QFN:QFN-36-1EP_6x6mm_P0.5mm_EP3.7x3.7mm, F.Cu at (136.7, 125.6)
- added U14: RJ45, Custom_VoxLink_Footprints:TE_RJ45, F.Cu at (102.9, 146.0)
- added U15: TPD4E02B04, Package_SON:USON-10_2.5x1.0mm_P0.5mm, F.Cu at (186.1, 81.3)
- added U16: RJ45, Custom_VoxLink_Footprints:TE_RJ45, F.Cu at (86.7, 80.0)
- added U17: RJ45, Custom_VoxLink_Footprints:TE_RJ45, F.Cu at (164.5, 124.1)
- added U18: TPD4E02B04, Package_SON:USON-10_2.5x1.0mm_P0.5mm, F.Cu at (189.0, 81.3)
- added U19: TPD4E02B04, Package_SON:USON-10_2.5x1.0mm_P0.5mm, F.Cu at (191.9, 81.3)
- added U20: TPD4E02B04, Package_SON:USON-10_2.5x1.0mm_P0.5mm, F.Cu at (194.8, 81.3)
- added U21: TPD4E02B04, Package_SON:USON-10_2.5x1.0mm_P0.5mm, F.Cu at (197.7, 81.3)
- added U22: RJ45, Custom_VoxLink_Footprints:TE_RJ45, F.Cu at (124.7, 146.0)
- added U23: TPD4E02B04, Package_SON:USON-10_2.5x1.0mm_P0.5mm, F.Cu at (186.1, 85.6)
- added U24: TPD4E02B04, Package_SON:USON-10_2.5x1.0mm_P0.5mm, F.Cu at (189.0, 85.6)
- added U25: RJ45, Custom_VoxLink_Footprints:TE_RJ45, F.Cu at (86.7, 101.8)
- added U26: TPD4E02B04, Package_SON:USON-10_2.5x1.0mm_P0.5mm, F.Cu at (191.9, 85.6)
- added U27: TPD4E02B04, Package_SON:USON-10_2.5x1.0mm_P0.5mm, F.Cu at (194.8, 85.6)
- added U28: RJ45, Custom_VoxLink_Footprints:TE_RJ45, F.Cu at (164.5, 102.2)
- added U29: TPD4E02B04, Package_SON:USON-10_2.5x1.0mm_P0.5mm, F.Cu at (197.7, 85.6)
- added U30: TPD4E02B04, Package_SON:USON-10_2.5x1.0mm_P0.5mm, F.Cu at (186.1, 89.9)
- added U31: RJ45, Custom_VoxLink_Footprints:TE_RJ45, F.Cu at (146.6, 146.0)
- added U32: TPD4E02B04, Package_SON:USON-10_2.5x1.0mm_P0.5mm, F.Cu at (189.0, 89.9)
- added U33: TPD4E02B04, Package_SON:USON-10_2.5x1.0mm_P0.5mm, F.Cu at (191.9, 89.9)
- added U34: RJ45, Custom_VoxLink_Footprints:TE_RJ45, F.Cu at (86.7, 123.6)
- added U37: RJ45, Custom_VoxLink_Footprints:TE_RJ45, F.Cu at (164.5, 80.4)
- added U39: TPD4E02B04, Package_SON:USON-10_2.5x1.0mm_P0.5mm, F.Cu at (194.8, 89.9)
- added U501: TPD4E02B04, Package_SON:USON-10_2.5x1.0mm_P0.5mm, F.Cu at (116.7, 128.0)
- added Y3: 24MHz, Crystal:Crystal_SMD_2520-4Pin_2.5x2.0mm, F.Cu at (101.5, 128.7)
- moved Y1 101.7 mm to (101.5, 120.6)
- moved C23 92.6 mm to (112.6, 97.9)
- moved C24 92.6 mm to (112.6, 99.9)
- moved C21 91.9 mm to (112.6, 95.9)
- moved C15 89.3 mm to (124.6, 128.8)
- moved C12 89.3 mm to (124.6, 124.5)
- moved C8 89.3 mm to (124.6, 120.3)
- moved U7 87.5 mm to (137.4, 117.7)
- moved C30 87.1 mm to (115.5, 90.0)
- moved C36 85.8 mm to (115.5, 97.9)
- moved C63 85.8 mm to (121.2, 99.9)
- moved U1 85.2 mm to (130.0, 116.2)
- moved U3 85.2 mm to (130.0, 120.7)
- moved U4 85.2 mm to (130.0, 125.3)
- moved C47 83.9 mm to (118.3, 95.9)
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Connections:
- U10 pad 6: FTDI_USB_D- -> SERIAL_D-
- U10 pad 7: FTDI_USB_D+ -> SERIAL_D+
- U8 pad 6: FTDI_USB_D- -> JTAG_D-
- U8 pad 7: FTDI_USB_D+ -> JTAG_D+
