File: Hardware/Controller_Board/Controller_Board.kicad_pcb (KiCad board)
At the start: 8 copper layers, 211 parts, among them J103 USB_C_USB2.0, Q1 DMN2400UFB-7, SW1 Reset, U1 TPS82084, U10 FT232H, U11 93LC56B, U12 USB2512B, U14 RJ45, U15 TPD4E02B04, U16 RJ45, U17 RJ45, U18 TPD4E02B04, U19 TPD4E02B04, U2 LT8645S, U20 TPD4E02B04, U21 TPD4E02B04, U22 RJ45, U23 TPD4E02B04, U24 TPD4E02B04, U25 RJ45, U26 TPD4E02B04, U27 TPD4E02B04, U28 RJ45, U29 TPD4E02B04, U3 TPS82084, U30 TPD4E02B04, U31 RJ45, U32 TPD4E02B04, U33 TPD4E02B04, U34 RJ45, U37 RJ45, U39 TPD4E02B04, U4 TPS82084, U5 XT30, U501 TPD4E02B04, U6 XC7A35T-CPG236, U7 IS25LP256D, U8 FT232H, U9 93LC56B, Y1 12MHz, Y2 12MHz, Y3 24MHz, Y301 12MHz

Commit message: Finished the schematic review
Parts:
- removed C1, C11, C14, C22, C32, C33, C43, C52, C60, C61, C7, C72: 10u, Capacitor_SMD:C_0805_2012Metric
- removed C10, C17, C19, C20, C23, C24, C25, C26, C27, C28, C37, C38, C39, C40, C41, C42, C45, C46, C47, C48, C49, C50, C53, C54, C55, C56, C57, C58, C63, C64, C65, C66, C67, C68, C69, C70, C73, C76, C77, C78, C79, C80, C81, C82, C84, C86, C87, C91, C92, C93, C94, C95, C96, C97, C99: 100n, Capacitor_SMD:C_0402_1005Metric
- removed C100, C75, C83, C85, C90, C98: 4u7, Capacitor_SMD:C_0402_1005Metric
- removed C12, C15, C4, C8: 22u, Capacitor_SMD:C_1210_3225Metric
- removed C13, C16, C5, C9: 100u, Capacitor_SMD:CP_Elec_8x6.5
- removed C18, C88, C89: 10p, Capacitor_SMD:C_0402_1005Metric
- removed C2, C3: 470n, Capacitor_SMD:C_0402_1005Metric
- removed C21, C29, C30, C31, C34, C35, C36, C44, C51, C59, C62, C71, C74: 1u, Capacitor_SMD:C_0402_1005Metric
- removed C6: 2.2p, Capacitor_SMD:C_0402_1005Metric
- removed D1, D105, D3: LED, LED_SMD:LED_0603_1608Metric
- removed FB2, FB3, FB4, FB5: 600R, Inductor_SMD:L_0402_1005Metric
- removed J103: USB_C_USB2.0, Connector_USB:USB_C_Receptacle_GCT_USB4105-xx-A_16P_TopMnt_Horizontal
- removed L1: 2u2, Inductor_SMD:L_Coilcraft_XAL6030-XXX
- removed Q1: DMN2400UFB-7, Package_DFN_QFN:Diodes_DFN1006-3
- removed R1: 1Meg, Resistor_SMD:R_0402_1005Metric
- removed R10, R2, R7: 499k, Resistor_SMD:R_0402_1005Metric
- removed R11: 156.3k, Resistor_SMD:R_0402_1005Metric
- removed R12, R5, R9: 50k, Resistor_SMD:R_0402_1005Metric
- removed R13: 280R, Resistor_SMD:R_0402_1005Metric
- removed R14, R17: 200R, Resistor_SMD:R_0402_1005Metric
- removed R26, R33, R48: 1k, Resistor_SMD:R_0402_1005Metric
- removed R27, R34, R41: 12k, Resistor_SMD:R_0402_1005Metric
- removed R28, R29, R30, R35, R36, R37: 10k, Resistor_SMD:R_0402_1005Metric
- removed R3: 12.5k, Resistor_SMD:R_0402_1005Metric
- removed R31, R38: 2k2, Resistor_SMD:R_0402_1005Metric
- removed R32, R39, R40: 22R, Resistor_SMD:R_0402_1005Metric
- removed R4: 243k, Resistor_SMD:R_0402_1005Metric
- removed R42, R43, R44, R45, R46, R47: 100k, Resistor_SMD:R_0402_1005Metric
- removed R6: 41.2k, Resistor_SMD:R_0402_1005Metric
- removed R8: 62.5k, Resistor_SMD:R_0402_1005Metric
- removed SW1: Reset, Button_Switch_SMD:SW_Push_SPST_NO_Alps_SKRK
- removed U1, U3, U4: TPS82084, Package_LGA:Texas_SIL0008C_MicroSiP-8-1EP_2.8x3mm_P0.65mm_EP1.1x1.9mm
- removed U10, U8: FT232H, Package_DFN_QFN:QFN-48-1EP_8x8mm_P0.5mm_EP6.2x6.2mm
- removed U11, U9: 93LC56B, Package_DFN_QFN:TDFN-8-1EP_3x2mm_P0.5mm_EP1.3x1.4mm
- removed U12: USB2512B, Package_DFN_QFN:QFN-36-1EP_6x6mm_P0.5mm_EP3.7x3.7mm
- removed U14, U16, U17, U22, U25, U28, U31, U34, U37: RJ45, Custom_VoxLink_Footprints:TE_RJ45
- removed U15, U18, U19, U20, U21, U23, U24, U26, U27, U29, U30, U32, U33, U39: TPD4E02B04, Package_SON:USON-10_2.5x1.0mm_P0.5mm
- removed U2: LT8645S, Custom_VoxLink_Footprints:LT8645S
- removed U5: XT30, Connector_AMASS:AMASS_XT30PW-M_1x02_P2.50mm_Horizontal
- removed U6: XC7A35T-CPG236, Package_BGA:Xilinx_CPG236
- removed U7: IS25LP256D, Package_SON:WSON-8-1EP_8x6mm_P1.27mm_EP3.4x4.3mm
- removed Y1, Y2: 12MHz, Crystal:Crystal_SMD_2520-4Pin_2.5x2.0mm
- removed Y3: 24MHz, Crystal:Crystal_SMD_2520-4Pin_2.5x2.0mm
- added C201: 100n, Capacitor_SMD:C_0402_1005Metric, F.Cu at (160.2, 121.0)
- added C202: 10p, Capacitor_SMD:C_0402_1005Metric, F.Cu at (160.2, 122.9)
- added C203: 100n, Capacitor_SMD:C_0201_0603Metric, F.Cu at (147.8, 120.8)
- added C204: 100n, Capacitor_SMD:C_0201_0603Metric, F.Cu at (147.8, 122.6)
- added C205: 1u, Capacitor_SMD:C_0402_1005Metric, F.Cu at (160.2, 124.9)
- added C206: 10u, Capacitor_SMD:C_0805_2012Metric, F.Cu at (144.3, 108.4)
- added C207: 100n, Capacitor_SMD:C_0201_0603Metric, F.Cu at (147.8, 124.3)
- added C208: 100n, Capacitor_SMD:C_0201_0603Metric, F.Cu at (147.8, 126.1)
- added C209: 100n, Capacitor_SMD:C_0201_0603Metric, F.Cu at (147.8, 127.8)
- added C210: 100n, Capacitor_SMD:C_0201_0603Metric, F.Cu at (147.8, 129.6)
- added C211: 100n, Capacitor_SMD:C_0201_0603Metric, F.Cu at (147.8, 131.3)
- added C212: 100n, Capacitor_SMD:C_0201_0603Metric, F.Cu at (150.2, 120.8)
- added C213: 1u, Capacitor_SMD:C_0402_1005Metric, F.Cu at (160.2, 126.9)
- added C214: 1u, Capacitor_SMD:C_0402_1005Metric, F.Cu at (160.2, 128.8)
- added C215: 1u, Capacitor_SMD:C_0402_1005Metric, F.Cu at (163.1, 121.0)
- added C216: 10u, Capacitor_SMD:C_0805_2012Metric, F.Cu at (144.3, 111.4)
- added C217: 10u, Capacitor_SMD:C_0805_2012Metric, F.Cu at (144.3, 114.5)
- added C218: 1u, Capacitor_SMD:C_0402_1005Metric, F.Cu at (163.1, 122.9)
- added C219: 1u, Capacitor_SMD:C_0402_1005Metric, F.Cu at (163.1, 124.9)
- added C220: 1u, Capacitor_SMD:C_0402_1005Metric, F.Cu at (163.1, 126.9)
- added C221: 100n, Capacitor_SMD:C_0201_0603Metric, F.Cu at (150.2, 122.6)
- added C222: 100n, Capacitor_SMD:C_0201_0603Metric, F.Cu at (150.2, 124.3)
- added C223: 100n, Capacitor_SMD:C_0201_0603Metric, F.Cu at (150.2, 126.1)
- added C224: 100n, Capacitor_SMD:C_0201_0603Metric, F.Cu at (150.2, 127.8)
- added C225: 100n, Capacitor_SMD:C_0201_0603Metric, F.Cu at (150.2, 129.6)
- added C226: 100n, Capacitor_SMD:C_0201_0603Metric, F.Cu at (150.2, 131.3)
- added C227: 10u, Capacitor_SMD:C_0805_2012Metric, F.Cu at (144.3, 117.5)
- added C228: 1u, Capacitor_SMD:C_0402_1005Metric, F.Cu at (163.1, 128.8)
- added C229: 100n, Capacitor_SMD:C_0201_0603Metric, F.Cu at (152.7, 120.8)
- added C230: 100n, Capacitor_SMD:C_0201_0603Metric, F.Cu at (152.7, 122.6)
- added C231: 100n, Capacitor_SMD:C_0201_0603Metric, F.Cu at (152.7, 124.3)
- added C232: 100n, Capacitor_SMD:C_0201_0603Metric, F.Cu at (152.7, 126.1)
- added C233: 100n, Capacitor_SMD:C_0201_0603Metric, F.Cu at (152.7, 127.8)
- added C234: 100n, Capacitor_SMD:C_0201_0603Metric, F.Cu at (152.7, 129.6)
- added C235: 1u, Capacitor_SMD:C_0402_1005Metric, F.Cu at (166.0, 121.0)
- added C236: 10u, Capacitor_SMD:C_0805_2012Metric, F.Cu at (144.3, 120.5)
- added C237: 100n, Capacitor_SMD:C_0201_0603Metric, F.Cu at (152.7, 131.3)
- added C238: 100n, Capacitor_SMD:C_0201_0603Metric, F.Cu at (155.1, 120.8)
- added C239: 100n, Capacitor_SMD:C_0201_0603Metric, F.Cu at (155.1, 122.6)
- added C240: 100n, Capacitor_SMD:C_0201_0603Metric, F.Cu at (155.1, 124.3)
- added C241: 100n, Capacitor_SMD:C_0201_0603Metric, F.Cu at (155.1, 126.1)
- added C242: 100n, Capacitor_SMD:C_0201_0603Metric, F.Cu at (155.1, 127.8)
- added C243: 1u, Capacitor_SMD:C_0402_1005Metric, F.Cu at (166.0, 122.9)
- added C244: 10u, Capacitor_SMD:C_0805_2012Metric, F.Cu at (144.3, 123.5)
- added C245: 10u, Capacitor_SMD:C_0805_2012Metric, F.Cu at (144.3, 126.5)
- added C246: 1u, Capacitor_SMD:C_0402_1005Metric, F.Cu at (166.0, 124.9)
- added C247: 100n, Capacitor_SMD:C_0201_0603Metric, F.Cu at (155.1, 129.6)
- added C248: 100n, Capacitor_SMD:C_0201_0603Metric, F.Cu at (155.1, 131.3)
- added C249: 100n, Capacitor_SMD:C_0201_0603Metric, F.Cu at (157.6, 120.8)
- added C250: 100n, Capacitor_SMD:C_0201_0603Metric, F.Cu at (157.6, 122.6)
- added C251: 100n, Capacitor_SMD:C_0201_0603Metric, F.Cu at (157.6, 124.3)
- added C252: 100n, Capacitor_SMD:C_0201_0603Metric, F.Cu at (157.6, 126.1)
- added C253: 100n, Capacitor_SMD:C_0201_0603Metric, F.Cu at (157.6, 127.8)
- added C254: 100n, Capacitor_SMD:C_0201_0603Metric, F.Cu at (157.6, 129.6)
- added C255: 1u, Capacitor_SMD:C_0402_1005Metric, F.Cu at (166.0, 126.9)
- added C256: 10u, Capacitor_SMD:C_0805_2012Metric, F.Cu at (144.3, 129.5)
- added C301: 1u, Capacitor_SMD:C_0402_1005Metric, F.Cu at (127.2, 111.3)
- added C302: 100n, Capacitor_SMD:C_0402_1005Metric, F.Cu at (127.2, 113.3)
- added C401: 4u7, Capacitor_SMD:C_0402_1005Metric, F.Cu at (97.3, 103.8)
- added C402: 100n, Capacitor_SMD:C_0402_1005Metric, F.Cu at (97.3, 105.8)
- added C403: 100n, Capacitor_SMD:C_0402_1005Metric, F.Cu at (97.3, 107.7)
- added C404: 100n, Capacitor_SMD:C_0402_1005Metric, F.Cu at (97.3, 109.7)
- added C405: 100n, Capacitor_SMD:C_0402_1005Metric, F.Cu at (97.3, 111.7)
- added C406: 100n, Capacitor_SMD:C_0402_1005Metric, F.Cu at (97.3, 113.6)
- added C407: 100n, Capacitor_SMD:C_0402_1005Metric, F.Cu at (100.1, 103.8)
- added C408: 100n, Capacitor_SMD:C_0402_1005Metric, F.Cu at (100.1, 105.8)
- added C409: 4u7, Capacitor_SMD:C_0402_1005Metric, F.Cu at (100.1, 107.7)
- added C410: 100n, Capacitor_SMD:C_0402_1005Metric, F.Cu at (100.1, 109.7)
- added C411: 4u7, Capacitor_SMD:C_0402_1005Metric, F.Cu at (100.1, 111.7)
- added C412: 100n, Capacitor_SMD:C_0402_1005Metric, F.Cu at (100.1, 113.6)
- added C413: 100n, Capacitor_SMD:C_0402_1005Metric, F.Cu at (103.0, 103.8)
- added C414: 10p, Capacitor_SMD:C_0402_1005Metric, F.Cu at (103.0, 105.8)
- added C415: 10p, Capacitor_SMD:C_0402_1005Metric, F.Cu at (103.0, 107.7)
- added C501: 4u7, Capacitor_SMD:C_0402_1005Metric, F.Cu at (76.0, 103.8)
- added C502: 100n, Capacitor_SMD:C_0402_1005Metric, F.Cu at (76.0, 105.8)
- added C503: 100n, Capacitor_SMD:C_0402_1005Metric, F.Cu at (76.0, 107.7)
- added C504: 100n, Capacitor_SMD:C_0402_1005Metric, F.Cu at (76.0, 109.7)
- added C505: 100n, Capacitor_SMD:C_0402_1005Metric, F.Cu at (76.0, 111.7)
- added C506: 100n, Capacitor_SMD:C_0402_1005Metric, F.Cu at (76.0, 113.6)
- added C507: 100n, Capacitor_SMD:C_0402_1005Metric, F.Cu at (78.9, 103.8)
- added C508: 100n, Capacitor_SMD:C_0402_1005Metric, F.Cu at (78.9, 105.8)
- added C509: 4u7, Capacitor_SMD:C_0402_1005Metric, F.Cu at (78.9, 107.7)
- added C510: 100n, Capacitor_SMD:C_0402_1005Metric, F.Cu at (78.9, 109.7)
- added C511: 4u7, Capacitor_SMD:C_0402_1005Metric, F.Cu at (78.9, 111.7)
- added C512: 100n, Capacitor_SMD:C_0402_1005Metric, F.Cu at (78.9, 113.6)
- added C513: 100n, Capacitor_SMD:C_0402_1005Metric, F.Cu at (81.8, 103.8)
- added C514: 10p, Capacitor_SMD:C_0402_1005Metric, F.Cu at (81.8, 105.8)
- added C515: 10p, Capacitor_SMD:C_0402_1005Metric, F.Cu at (81.8, 107.7)
- added C601: 4u7, Capacitor_SMD:C_0402_1005Metric, F.Cu at (155.2, 95.9)
- added C602: 100n, Capacitor_SMD:C_0402_1005Metric, F.Cu at (155.2, 97.9)
- added C603: 100n, Capacitor_SMD:C_0402_1005Metric, F.Cu at (155.2, 99.9)
- added C604: 100n, Capacitor_SMD:C_0402_1005Metric, F.Cu at (155.2, 101.8)
- added C605: 100n, Capacitor_SMD:C_0402_1005Metric, F.Cu at (155.2, 103.8)
- added C606: 100n, Capacitor_SMD:C_0402_1005Metric, F.Cu at (158.1, 95.9)
- added C607: 100n, Capacitor_SMD:C_0402_1005Metric, F.Cu at (158.1, 97.9)
- added C608: 10n, Capacitor_SMD:C_0402_1005Metric, F.Cu at (158.1, 99.9)
- added C609: 100n, Capacitor_SMD:C_0402_1005Metric, F.Cu at (158.1, 101.8)
- added C610: 10n, Capacitor_SMD:C_0402_1005Metric, F.Cu at (158.1, 103.8)
- added C611: 100n, Capacitor_SMD:C_0402_1005Metric, F.Cu at (161.0, 95.9)
- added C612: 10p, Capacitor_SMD:C_0402_1005Metric, F.Cu at (161.0, 97.9)
- added C613: 10p, Capacitor_SMD:C_0402_1005Metric, F.Cu at (161.0, 99.9)
- added D101: LED, LED_SMD:LED_0603_1608Metric, F.Cu at (172.3, 63.5)
- added D102: TVS, Diode_THT:D_DO-201AE_P15.24mm_Horizontal, F.Cu at (158.8, 33.7)
- added D103: TVS/Zener, Diode_SMD:D_0603_1608Metric, F.Cu at (172.3, 66.0)
- added D301: LED, LED_SMD:LED_0603_1608Metric, F.Cu at (122.0, 116.0)
- added D601: TVS, Diode_THT:D_DO-201AE_P15.24mm_Horizontal, F.Cu at (144.2, 91.5)
- added D602: LED, LED_SMD:LED_0603_1608Metric, F.Cu at (164.4, 100.3)
- added FB201: 600R/100MHz, Inductor_SMD:L_0402_1005Metric, F.Cu at (160.3, 130.8)
- added FB401: 600R, Inductor_SMD:L_0402_1005Metric, F.Cu at (105.9, 114.0)
- added FB402: 600R, Inductor_SMD:L_0402_1005Metric, F.Cu at (105.9, 116.0)
- added FB501: 600R, Inductor_SMD:L_0402_1005Metric, F.Cu at (84.7, 114.0)
- added FB502: 600R, Inductor_SMD:L_0402_1005Metric, F.Cu at (84.7, 116.0)
- added J601: USB-C, Connector_USB:USB_C_Receptacle_GCT_USB4105-xx-A_16P_TopMnt_Horizontal, F.Cu at (147.9, 100.2)
- added L101: 2u2, Inductor_SMD:L_Coilcraft_XAL6030-XXX, F.Cu at (146.2, 61.9)
- added Q101: DMN2400UFB-7, Package_DFN_QFN:Diodes_DFN1006-3, F.Cu at (163.1, 65.4)
- added R101: 499k, Resistor_SMD:R_0402_1005Metric, F.Cu at (162.9, 55.1)
- added R102: 12.5k, Resistor_SMD:R_0402_1005Metric, F.Cu at (162.9, 57.0)
- added R103: 50k, Resistor_SMD:R_0402_1005Metric, F.Cu at (162.9, 59.0)
- added R106: 243k, Resistor_SMD:R_0402_1005Metric, F.Cu at (162.9, 63.0)
- added R108: 499k, Resistor_SMD:R_0402_1005Metric, F.Cu at (165.8, 57.0)
- added R109: 62.5k, Resistor_SMD:R_0402_1005Metric, F.Cu at (165.8, 59.0)
- added R110: 50k, Resistor_SMD:R_0402_1005Metric, F.Cu at (165.8, 61.0)
- added R111: 280R, Resistor_SMD:R_0402_1005Metric, F.Cu at (165.8, 63.0)
- added R112: 499k, Resistor_SMD:R_0402_1005Metric, F.Cu at (168.8, 55.1)
- added R113: 156.3k, Resistor_SMD:R_0402_1005Metric, F.Cu at (168.8, 57.0)
- added R114: 50k, Resistor_SMD:R_0402_1005Metric, F.Cu at (168.8, 59.0)
- added R301: 200R, Resistor_SMD:R_0402_1005Metric, F.Cu at (118.5, 103.8)
- added R303: 200R, Resistor_SMD:R_0402_1005Metric, F.Cu at (118.5, 107.8)
- added R304: 1k, Resistor_SMD:R_0402_1005Metric, F.Cu at (118.5, 109.8)
- added R305: 4.7k, Resistor_SMD:R_0402_1005Metric, F.Cu at (118.5, 111.8)
- added R306: 4.7k, Resistor_SMD:R_0402_1005Metric, F.Cu at (118.5, 113.7)
- added R307: 4.7k, Resistor_SMD:R_0402_1005Metric, F.Cu at (121.4, 103.8)
- added R308: 100R, Resistor_SMD:R_0402_1005Metric, F.Cu at (121.4, 105.8)
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Connections:
- C101 pad 1: +3V3_VPLL -> +5V
- C102 pad 1: +3V3 -> +1V0
- C103 pad 1: /Serial/OSC_IN -> +1V0
- C104 pad 1: Net-(C104-Pad1) -> VIN
- C104 pad 2: GND -> Net-(C104-Pad2)
- C105 pad 1: /USB/OSC_IN -> VIN
- C106 pad 1: Net-(C106-Pad1) -> VIN
- C107 pad 1: +3V3 -> VIN
- C108 pad 1: +3V3 -> +5V
- C109 pad 1: +3V3 -> +5V
- C110 pad 1: +3V3 -> +5V
- C110 pad 2: GND -> /Power/FB_5V0
- C111 pad 1: +3V3 -> /Power/TR/SS
- C112 pad 1: +3V3 -> +5V
- C113 pad 1: +3V3 -> +1V8
- C114 pad 1: Net-(U12-PLLFILT) -> +1V8
- C115 pad 1: Net-(U12-PLLFILT) -> +5V
- C116 pad 1: Net-(U12-CRFILT) -> +3V3
- C117 pad 1: Net-(U12-CRFILT) -> +3V3
- C303 pad 1: VCCIO2 -> +3V3
- R104 pad 1: GND -> +5V
- R104 pad 2: Net-(J103-CC1) -> /Power/FB_5V0
- R105 pad 1: GND -> Net-(C104-Pad2)
- R105 pad 2: Net-(J103-CC2) -> GND
- R107 pad 2: VBUS -> GND
- R302 pad 1: 12MHZ_CLK -> +3V3
- R302 pad 2: /FPGA_Config/OSC_OUT -> Net-(U201B-CFGBVS_0)
- U501 pad 1: /Connectivity/P1_TX_N -> /Serial/OSC_IN
- U501 pad 10: /Connectivity/P1_TX_N -> GND
- U501 pad 2: /Connectivity/P1_TX_P -> /Serial/OSC_OUT
- U501 pad 3: GND -> +3V3_VPHY
- U501 pad 4: /Connectivity/P1_CLK_N -> GND
- U501 pad 5: /Connectivity/P1_CLK_P -> Net-(U501-REF)
- U501 pad 6: /Connectivity/P1_CLK_P -> SERIAL_D-
- U501 pad 7: /Connectivity/P1_CLK_N -> SERIAL_D+
- U501 pad 8: GND -> +3V3_VPLL
- U501 pad 9: /Connectivity/P1_TX_P -> GND
- Y301 pad 1: VCCIO2 -> +3V3
- Y301 pad 4: VCCIO2 -> +3V3

Commit message: Started schematic rework and the PCB design
Parts:
- removed R312: 100R, Resistor_SMD:R_0402_1005Metric
- removed R313: 22R, Resistor_SMD:R_0402_1005Metric
- added C416: 10p, Capacitor_SMD:C_0402_1005Metric, F.Cu at (48.2, 145.8)
- added C516: 10p, Capacitor_SMD:C_0402_1005Metric, F.Cu at (19.6, 116.8)
- added C614: 10p, Capacitor_SMD:C_0402_1005Metric, F.Cu at (94.2, 81.4)
- added D603: LED, LED_SMD:LED_0603_1608Metric, F.Cu at (89.1, 103.8)
- added TP301: N3, TestPoint:TestPoint_Pad_D1.0mm, F.Cu at (46.3, 113.3)
- added TP302: M2, TestPoint:TestPoint_Pad_D1.0mm, F.Cu at (46.3, 116.3)
- added TP303: M3, TestPoint:TestPoint_Pad_D1.0mm, F.Cu at (46.3, 119.4)
- added TP304: L3, TestPoint:TestPoint_Pad_D1.0mm, F.Cu at (46.3, 122.5)
- added TP305: K3, TestPoint:TestPoint_Pad_D1.0mm, F.Cu at (46.3, 125.5)
- C203, C204, C207, C208, C209, C210, C211, C212, C221, C222, C223, C224, C225, C226, C229, C230, C231, C232, C233, C234, C237, C238, C239, C240, C241, C242, C247, C248, C249, C250, C251, C252, C253, C254: moved to B.Cu
- C401, C409, C501, C509, C601: value 4u7 -> 10u; footprint Capacitor_SMD:C_0402_1005Metric -> Capacitor_SMD:C_0805_2012Metric
- C411, C511: value 4u7 -> 100n
- C412, C512: value 100n -> 10u; footprint Capacitor_SMD:C_0402_1005Metric -> Capacitor_SMD:C_0805_2012Metric
- C414, C514, C612: value 10p -> 100n
- C608, C610: value 10n -> 100n
- C609, C611: value 100n -> 10n
- D101: value LED -> TVS/Zener; footprint LED_SMD:LED_0603_1608Metric -> Diode_SMD:D_0603_1608Metric
- D102: value TVS -> LED; footprint Diode_THT:D_DO-201AE_P15.24mm_Horizontal -> LED_SMD:LED_0603_1608Metric
- D103: value TVS/Zener -> TVS; footprint Diode_SMD:D_0603_1608Metric -> Diode_SMD:D_0402_1005Metric
- D601: value TVS -> Schottky; footprint Diode_THT:D_DO-201AE_P15.24mm_Horizontal -> Diode_SMD:D_SOD-323F
- D602: value LED -> TVS; footprint LED_SMD:LED_0603_1608Metric -> Diode_SMD:D_0402_1005Metric
- R302: value 4.7k -> 100R
- R303: value 200R -> 4.7k
- R304, Re301, Re302: value 1k -> 4.7k
- R308, R309, R310: value 100R -> 4.7k
- R311: value 100R -> 22R
- R403, R404, R405, R503, R504, R505: value 10k -> 12k
- U601: footprint Amass_XT60:CONN_XT60PW-M_AMA -> Custom_VoxLink_Footprints:X2SON-3
- moved U702 106.2 mm to (156.2, 140.4)
- moved U710 106.1 mm to (195.9, 100.7), turned to 90 degrees
- moved U711 104.6 mm to (175.7, 140.4)
- moved U716 102.5 mm to (195.9, 120.2), turned to 90 degrees
- moved D103 91.8 mm to (80.5, 69.7)
- moved U701 83.8 mm to (116.5, 120.2), turned to -90 degrees
- moved Q101 82.9 mm to (80.4, 72.1)
- moved C409 82.8 mm to (32.6, 155.7)
- moved C412 81.2 mm to (32.6, 158.7)
- moved C401 81.1 mm to (32.6, 152.7)
- moved Y601 80.9 mm to (83.8, 96.8)
- moved U301 79.7 mm to (51.8, 97.8)
- moved U717 79.6 mm to (136.7, 140.4)
- moved R402 79.4 mm to (39.2, 152.2)
- moved R403 79.4 mm to (39.2, 154.2)
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Connections:
- C409 pad 1: +3V3_VPHY -> +3V3_VPHY_JTAG
- C410 pad 1: +3V3_VPHY -> +3V3_VPHY_JTAG
- C411 pad 1: +3V3_VPLL -> Net-(U401-~{RESET})
- C412 pad 1: +3V3_VPLL -> +3V3_VPLL_JTAG
- C413 pad 1: +3V3 -> +3V3_VPLL_JTAG
- C414 pad 1: /JTAG/OSC_IN -> +3V3
- C415 pad 1: Net-(C415-Pad1) -> /JTAG/OSC_IN
- C509 pad 1: +3V3_VPHY -> +3V3_VPHY_SER
- C510 pad 1: +3V3_VPHY -> +3V3_VPHY_SER
- C511 pad 1: +3V3_VPLL -> Net-(U501-~{RESET})
- C512 pad 1: +3V3_VPLL -> +3V3_VPLL_SER
- C513 pad 1: +3V3 -> +3V3_VPLL_SER
- C514 pad 1: /Serial/OSC_IN -> +3V3
- C515 pad 1: Net-(C515-Pad1) -> /Serial/OSC_IN
- C608 pad 1: Net-(U602-PLLFILT) -> Net-(U602-NRESET)
- C610 pad 1: Net-(U602-CRFILT) -> Net-(U602-PLLFILT)
- C612 pad 1: /USB/OSC_IN -> Net-(U602-CRFILT)
- C613 pad 1: Net-(C613-Pad1) -> /USB/OSC_IN
- D101 pad 1: Net-(D101-K) -> VIN
- D101 pad 2: Net-(D101-A) -> GND
- D102 pad 1: VIN -> Net-(D102-K)
- D102 pad 2: GND -> Net-(D102-A)
- D103 pad 1: VIN -> GND
- D103 pad 2: GND -> VIN
- D301 pad 1: Net-(D301-K) -> GND
- D301 pad 2: /FPGA_Config/FPGA_DONE -> Net-(D301-A)
- D601 pad 1: VBUS -> +5V
- D601 pad 2: GND -> VBUS
- D602 pad 2: Net-(D602-A) -> VBUS
- FB401 pad 1: +3V3_VPHY -> +3V3_VPHY_JTAG
- FB402 pad 1: +3V3_VPLL -> +3V3_VPLL_JTAG
- FB501 pad 1: +3V3_VPHY -> +3V3_VPHY_SER
- FB502 pad 1: +3V3_VPLL -> +3V3_VPLL_SER
- Q101 pad 3: Net-(D101-K) -> Net-(D102-K)
- R111 pad 2: Net-(D101-A) -> Net-(D102-A)
- R302 pad 1: +3V3 -> /FPGA_Config/FPGA_DONE
- R302 pad 2: Net-(U201B-CFGBVS_0) -> Net-(D301-A)
- R303 pad 1: Net-(D301-K) -> +3V3
- R303 pad 2: GND -> Net-(U201B-CFGBVS_0)
- R304 pad 1: /FPGA_Config/MODE0 -> +3V3
- R304 pad 2: +3V3 -> Net-(U201B-IO_L3P_T0_DQS_PUDC_B_14)
- R305 pad 1: +3V3 -> /FPGA_Config/MODE0
- R305 pad 2: /FPGA_Config/FPGA_INIT -> +3V3
- R306 pad 2: /FPGA_Config/FPGA_RST -> /FPGA_Config/FPGA_INIT
- R307 pad 2: /FPGA_Config/NCS_FPGA -> /FPGA_Config/FPGA_RST
- R308 pad 1: /FPGA_Config/SCK_FPGA -> +3V3
- R308 pad 2: /FPGA_Config/SCK_FLASH -> /FPGA_Config/NHL_FPGA
- R309 pad 1: /FPGA_Config/SDI_FPGA -> +3V3
- R309 pad 2: /FPGA_Config/SDI_FLASH -> /FPGA_Config/NWP_FPGA
- R310 pad 1: /FPGA_Config/SDO_FPGA -> +3V3
- R310 pad 2: /FPGA_Config/SDO_FLASH -> /FPGA_Config/NCS_FPGA
- R311 pad 1: /FPGA_Config/NWP_FPGA -> 12MHZ_CLK
- R311 pad 2: /FPGA_Config/NWP_FLASH -> /FPGA_Config/OSC_OUT
- R407 pad 2: Net-(C415-Pad1) -> Net-(C416-Pad1)
- R507 pad 2: Net-(C515-Pad1) -> Net-(C516-Pad1)
- R601 pad 1: Net-(D602-A) -> Net-(D603-A)
- R611 pad 2: Net-(C613-Pad1) -> Net-(C614-Pad1)
- U102 pad 39: (no net) -> GND
- U102 pad 40: (no net) -> GND
- U102 pad 41: (no net) -> GND
- U102 pad 42: (no net) -> GND
- U201 pad A14: /Connectivity/P8_CLK_P -> /Connectivity/P3_CLK_P
- U201 pad A15: /Connectivity/P8_CLK_N -> /Connectivity/P3_CLK_N
- U201 pad A16: /Connectivity/P8_RX_P -> /Connectivity/P3_RX_P
- U201 pad A17: /Connectivity/P8_RX_N -> /Connectivity/P3_RX_N
- U201 pad B15: /Connectivity/P8_TX_N -> /Connectivity/P3_TX_N
- U201 pad C15: /Connectivity/P8_TX_P -> /Connectivity/P3_TX_P
- U201 pad E18: /Connectivity/P1_CLK_P -> Net-(U201B-IO_L3P_T0_DQS_PUDC_B_14)
- U201 pad E19: /Connectivity/P1_CLK_N -> /FPGA_Config/SCK_FPGA
- U201 pad G17: /Connectivity/P1_RX_N -> P6_L2
- U201 pad G19: /Connectivity/P1_TX_N -> P5_L2
- U201 pad G2: P5_L2 -> /Connectivity/P7_CLK_N
- U201 pad G3: P5_L1 -> /Connectivity/P7_CLK_P
- U201 pad H1: P7_L1 -> /Connectivity/P7_RX_P
- U201 pad H17: /Connectivity/P1_RX_P -> P6_L1
- U201 pad H19: /Connectivity/P1_TX_P -> P5_L1
- U201 pad H2: P6_L1 -> /Connectivity/P7_TX_P
- U201 pad J1: P7_L2 -> /Connectivity/P7_RX_N
- U201 pad J2: P6_L2 -> /Connectivity/P7_TX_N
- U201 pad J3: P9_L2 -> P8_L2
- U201 pad K17: /Connectivity/P3_RX_N -> /Connectivity/P5_RX_N
- U201 pad K2: P8_L1 -> P7_L1
- U201 pad K3: unconnected-(U201G-IO_L7N_T1_AD6N_35-PadK3) -> P9_L1
- U201 pad L1: P9_L1 -> P8_L1
- U201 pad L17: /Connectivity/P3_RX_P -> /Connectivity/P5_RX_P
- U201 pad L2: P8_L2 -> P7_L2
- U201 pad L3: unconnected-(U201G-IO_L8P_T1_AD14P_35-PadL3) -> P9_L2
- U201 pad M1: unconnected-(U201G-IO_L9N_T1_DQS_AD7N_35-PadM1) -> Net-(U201G-IO_L9N_T1_DQS_AD7N_35)
- U201 pad M18: /Connectivity/P3_TX_P -> /Connectivity/P5_TX_P
- U201 pad M19: /Connectivity/P3_TX_N -> /Connectivity/P5_TX_N
- U201 pad M2: unconnected-(U201G-IO_L9P_T1_DQS_AD7P_35-PadM2) -> Net-(U201G-IO_L9P_T1_DQS_AD7P_35)
- U201 pad M3: unconnected-(U201G-IO_L8N_T1_AD14N_35-PadM3) -> Net-(U201G-IO_L8N_T1_AD14N_35)
- U201 pad N1: unconnected-(U201G-IO_L10N_T1_AD15N_35-PadN1) -> Net-(U201G-IO_L10N_T1_AD15N_35)
- U201 pad N2: unconnected-(U201G-IO_L10P_T1_AD15P_35-PadN2) -> Net-(U201G-IO_L10P_T1_AD15P_35)
- U201 pad P19: /Connectivity/P3_CLK_P -> /Connectivity/P5_CLK_P
- U201 pad R19: /Connectivity/P3_CLK_N -> /Connectivity/P5_CLK_N
- U201 pad T17: /Connectivity/P5_TX_P -> /Connectivity/P6_TX_P
- U201 pad T18: /Connectivity/P5_TX_N -> /Connectivity/P6_TX_N
- U201 pad U15: /Connectivity/P7_TX_P -> /Connectivity/P8_RX_P
- U201 pad U16: /Connectivity/P7_TX_N -> /Connectivity/P8_RX_N
- U201 pad U17: /Connectivity/P5_RX_P -> /Connectivity/P6_RX_P
- U201 pad U18: /Connectivity/P5_RX_N -> /Connectivity/P6_RX_N
- U201 pad V13: /Connectivity/P7_RX_P -> /Connectivity/P8_TX_P
- U201 pad V14: /Connectivity/P7_RX_N -> /Connectivity/P8_TX_N
- U201 pad V15: /Connectivity/P6_RX_P -> /Connectivity/P1_TX_P
- U201 pad V16: /Connectivity/P6_CLK_P -> /Connectivity/P1_RX_P
- U201 pad V17: /Connectivity/P6_CLK_N -> /Connectivity/P1_RX_N
- U201 pad V4: /Serial/SERIAL_IO -> /Serial/SERIAL_PWR#
- U201 pad W13: /Connectivity/P7_CLK_P -> /Connectivity/P8_CLK_P
- U201 pad W14: /Connectivity/P7_CLK_N -> /Connectivity/P8_CLK_N
- U201 pad W15: /Connectivity/P6_RX_N -> /Connectivity/P1_TX_N
- U201 pad W16: /Connectivity/P6_TX_P -> /Connectivity/P1_CLK_P
- U201 pad W17: /Connectivity/P6_TX_N -> /Connectivity/P1_CLK_N
- U201 pad W18: /Connectivity/P5_CLK_P -> /Connectivity/P6_CLK_P
- U201 pad W19: /Connectivity/P5_CLK_N -> /Connectivity/P6_CLK_N
- U201 pad W4: /Serial/SERIAL_OE# -> /Serial/SERIAL_CLK
- U201 pad W5: /Serial/SERIAL_CLK -> /Serial/SERIAL_OE#
- U301 pad 2: /FPGA_Config/SDO_FLASH -> /FPGA_Config/SDO_FPGA
- U301 pad 3: /FPGA_Config/NWP_FLASH -> /FPGA_Config/NWP_FPGA
- U301 pad 5: /FPGA_Config/SDI_FLASH -> /FPGA_Config/SDI_FPGA
- U301 pad 6: /FPGA_Config/SCK_FLASH -> /FPGA_Config/SCK_FPGA
- U301 pad 7: /FPGA_Config/NHL_FLASH -> /FPGA_Config/NHL_FPGA
- U401 pad 3: +3V3_VPHY -> +3V3_VPHY_JTAG
- U401 pad 8: +3V3_VPLL -> +3V3_VPLL_JTAG
- U501 pad 29: /Serial/SERIAL_IO -> /Serial/SERIAL_CLK
- U501 pad 3: +3V3_VPHY -> +3V3_VPHY_SER
- U501 pad 30: /Serial/SERIAL_CLK -> /Serial/SERIAL_OE#
- U501 pad 31: /Serial/SERIAL_OE# -> /Serial/SERIAL_PWR#
- U501 pad 8: +3V3_VPLL -> +3V3_VPLL_SER
- Y401 pad 3: Net-(C415-Pad1) -> Net-(C416-Pad1)
- Y501 pad 3: Net-(C515-Pad1) -> Net-(C516-Pad1)
- Y601 pad 3: Net-(C613-Pad1) -> Net-(C614-Pad1)
Routing:
- net /Connectivity/P2_TX_N: track 0.00 -> 61.0 mm
- net /Connectivity/P3_TX_N: track 0.00 -> 59.2 mm
- net /Connectivity/P2_TX_P: track 0.00 -> 58.6 mm
- net /Connectivity/P3_TX_P: track 0.00 -> 56.3 mm
- net /Connectivity/P7_CLK_N: track 0.00 -> 51.3 mm
- net /Connectivity/P3_CLK_N: track 0.00 -> 49.9 mm
- net /Connectivity/P6_TX_N: track 0.00 -> 49.2 mm
- net /Connectivity/P7_CLK_P: track 0.00 -> 49.1 mm
- net /Connectivity/P3_RX_P: track 0.00 -> 49.0 mm
- net /Connectivity/P6_TX_P: track 0.00 -> 48.4 mm
- net /Connectivity/P3_CLK_P: track 0.00 -> 48.4 mm
- net /Connectivity/P3_RX_N: track 0.00 -> 46.2 mm
- net /Connectivity/P4_TX_N: track 0.00 -> 44.1 mm
- net /Connectivity/P4_TX_P: track 0.00 -> 43.1 mm
- net /Connectivity/P7_TX_N: track 0.00 -> 39.8 mm
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- added copper zone on In1.Cu, net GND
- added copper zone on In4.Cu, net GND
Other:
- board outline added: 85 x 85 mm
- copper layers 8 -> 6
- board text added: "BANK35 K2 - L3 : U703"
- board text added: "Bank43 One RJ45"

Commit message: Commit before upgrading to KiCad 10.0
Parts:
- added C257: 100n, Capacitor_SMD:C_0201_0603Metric, F.Cu at (102.9, 137.6)
- added C258: 10u, Capacitor_SMD:C_0603_1608Metric, F.Cu at (85.0, 148.2)
- C203, C204, C229, C230, C231, C232, C233, C242, C247, C252, C253, C254: moved to F.Cu
- C205, C219: value 1u -> 10u; footprint Capacitor_SMD:C_0402_1005Metric -> Capacitor_SMD:C_0603_1608Metric
- C206: footprint Capacitor_SMD:C_0805_2012Metric -> Capacitor_SMD:C_0603_1608Metric; moved to B.Cu
- C213, C214, C215, C218, C228, C235, C243, C246, C255: value 1u -> 100n; footprint Capacitor_SMD:C_0402_1005Metric -> Capacitor_SMD:C_0201_0603Metric
- C216, C217, C244, C245, C256: value 10u -> 100n; footprint Capacitor_SMD:C_0805_2012Metric -> Capacitor_SMD:C_0201_0603Metric
- C220: value 1u -> 100n; footprint Capacitor_SMD:C_0402_1005Metric -> Capacitor_SMD:C_0201_0603Metric; moved to B.Cu
- C227: value 10u -> 100n; footprint Capacitor_SMD:C_0805_2012Metric -> Capacitor_SMD:C_0201_0603Metric; moved to B.Cu
- C234, C248: value 100n -> 10u; footprint Capacitor_SMD:C_0201_0603Metric -> Capacitor_SMD:C_0603_1608Metric; moved to F.Cu
- C237, C249: value 100n -> 10u; footprint Capacitor_SMD:C_0201_0603Metric -> Capacitor_SMD:C_0603_1608Metric
- U201: value XC7A35T-CPG236 -> XC7A35T-CSG324; footprint Package_BGA:Xilinx_CPG236 -> Package_BGA:Xilinx_CSG324
- moved U301 104.4 mm to (156.2, 98.0)
- moved C237 80.2 mm to (159.4, 110.7), turned to 90 degrees
- moved C251 79.5 mm to (157.0, 107.9), turned to 0 degrees
- moved C250 78.0 mm to (157.0, 108.7)
- moved C241 76.5 mm to (158.2, 113.1), turned to -90 degrees
- moved C240 76.3 mm to (157.8, 111.1)
- moved C238 76.2 mm to (158.2, 108.3), turned to -90 degrees
- moved C239 76.2 mm to (157.8, 109.5)
- moved C226 75.3 mm to (157.4, 113.1), turned to 90 degrees
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Connections:
- C206 pad 1: +3V3 -> +1V0
- C207 pad 1: +3V3 -> +1V0
- C208 pad 1: +3V3 -> +1V0
- C209 pad 1: +3V3 -> +1V0
- C210 pad 1: +3V3 -> +1V0
- C211 pad 1: +3V3 -> +1V0
- C212 pad 1: +3V3 -> +1V0
- C217 pad 1: +1V0 -> +3V3
- C218 pad 1: +1V0 -> +3V3
- C219 pad 1: +1V0 -> +3V3
- C227 pad 1: +1V8 -> +1V0
- C228 pad 1: +1V8 -> +3V3
- C229 pad 1: +1V8 -> +3V3
- C230 pad 1: +1V8 -> +3V3
- C237 pad 1: +3V3 -> +1V8
- C238 pad 1: +3V3 -> +1V8
- C239 pad 1: +3V3 -> +1V8
- C240 pad 1: +3V3 -> +1V8
- C241 pad 1: +3V3 -> +1V8
- C245 pad 1: +1V0 -> +3V3
- C246 pad 1: +1V0 -> +3V3
- C247 pad 1: +1V0 -> +3V3
- C248 pad 1: +1V0 -> +3V3
- C249 pad 1: +3V3 -> +1V0
- C250 pad 1: +3V3 -> +1V0
- C251 pad 1: +3V3 -> +1V0
- TP301 pad 1: Net-(U201G-IO_L10N_T1_AD15N_35) -> Net-(U201E-IO_L12N_T1_MRCC_16)
- TP302 pad 1: Net-(U201G-IO_L10P_T1_AD15P_35) -> Net-(U201E-IO_L12P_T1_MRCC_16)
- TP303 pad 1: Net-(U201G-IO_L9N_T1_DQS_AD7N_35) -> Net-(U201E-IO_L11N_T1_SRCC_16)
- TP304 pad 1: Net-(U201G-IO_L9P_T1_DQS_AD7P_35) -> Net-(U201E-IO_L11P_T1_SRCC_16)
- TP305 pad 1: Net-(U201G-IO_L8N_T1_AD14N_35) -> Net-(U201E-IO_L6N_T0_VREF_16)
- U201 pad A1: GND -> unconnected-(U201G-IO_L9N_T1_DQS_AD7N_35-PadA1)
- U201 pad A11: GND -> unconnected-(U201D-IO_L4N_T0_15-PadA11)
- U201 pad A13: GND -> unconnected-(U201D-IO_L9P_T1_DQS_AD3P_15-PadA13)
- U201 pad A14: /Connectivity/P3_CLK_P -> unconnected-(U201D-IO_L9N_T1_DQS_AD3N_15-PadA14)
- U201 pad A15: /Connectivity/P3_CLK_N -> unconnected-(U201D-IO_L8P_T1_AD10P_15-PadA15)
- U201 pad A16: /Connectivity/P3_RX_P -> unconnected-(U201D-IO_L8N_T1_AD10N_15-PadA16)
- U201 pad A17: /Connectivity/P3_RX_N -> +3V3
- U201 pad A18: /Connectivity/P9_RX_N -> unconnected-(U201D-IO_L10N_T1_AD11N_15-PadA18)
- U201 pad A2: unconnected-(U201C-MGTPTXN1_216-PadA2) -> GND
- U201 pad A3: GND -> unconnected-(U201G-IO_L8N_T1_AD14N_35-PadA3)
- U201 pad A4: GND -> unconnected-(U201G-IO_L8P_T1_AD14P_35-PadA4)
- U201 pad A5: GND -> unconnected-(U201G-IO_L3N_T0_DQS_AD5N_35-PadA5)
- U201 pad A6: GND -> unconnected-(U201G-IO_L3P_T0_DQS_AD5P_35-PadA6)
- U201 pad A7: GND -> +3V3
- U201 pad A8: unconnected-(U201C-MGTREFCLK0N_216-PadA8) -> Net-(U201E-IO_L12N_T1_MRCC_16)
- U201 pad A9: GND -> unconnected-(U201E-IO_L14N_T2_SRCC_16-PadA9)
- U201 pad B1: GND -> unconnected-(U201G-IO_L9P_T1_DQS_AD7P_35-PadB1)
- U201 pad B10: unconnected-(U201C-MGTREFCLK1P_216-PadB10) -> +3V3
- U201 pad B11: GND -> unconnected-(U201D-IO_L4P_T0_15-PadB11)
- U201 pad B12: GND -> unconnected-(U201D-IO_L3N_T0_DQS_AD1N_15-PadB12)
- U201 pad B13: GND -> unconnected-(U201D-IO_L2P_T0_AD8P_15-PadB13)
- U201 pad B14: GND -> unconnected-(U201D-IO_L2N_T0_AD8N_15-PadB14)
- U201 pad B15: /Connectivity/P3_TX_N -> GND
- U201 pad B16: /Connectivity/P9_CLK_N -> unconnected-(U201D-IO_L7P_T1_AD2P_15-PadB16)
- U201 pad B17: /Connectivity/P9_TX_N -> unconnected-(U201D-IO_L7N_T1_AD2N_15-PadB17)
- U201 pad B18: /Connectivity/P9_RX_P -> unconnected-(U201D-IO_L10P_T1_AD11P_15-PadB18)
- U201 pad B3: GND -> unconnected-(U201G-IO_L10P_T1_AD15P_35-PadB3)
- U201 pad B4: GND -> unconnected-(U201G-IO_L7N_T1_AD6N_35-PadB4)
- U201 pad B6: GND -> unconnected-(U201G-IO_L2N_T0_AD12N_35-PadB6)
- U201 pad B7: GND -> unconnected-(U201G-IO_L2P_T0_AD12P_35-PadB7)
- U201 pad B8: unconnected-(U201C-MGTREFCLK0P_216-PadB8) -> Net-(U201E-IO_L12P_T1_MRCC_16)
- U201 pad B9: GND -> Net-(U201E-IO_L11N_T1_SRCC_16)
- U201 pad C1: GND -> unconnected-(U201G-IO_L16N_T2_35-PadC1)
- U201 pad C10: GND -> 12MHZ_CLK
- U201 pad C11: /FPGA_Config/SCK_FPGA -> unconnected-(U201E-IO_L13P_T2_MRCC_16-PadC11)
- U201 pad C12: GND -> unconnected-(U201D-IO_L3P_T0_DQS_AD1P_15-PadC12)
- U201 pad C13: Net-(U201A-VCCADC_0) -> +3V3
- U201 pad C14: +3V3 -> unconnected-(U201D-IO_L1N_T0_AD0N_15-PadC14)
- U201 pad C15: /Connectivity/P3_TX_P -> unconnected-(U201D-IO_L12N_T1_MRCC_15-PadC15)
- U201 pad C16: /Connectivity/P9_CLK_P -> unconnected-(U201D-IO_L20P_T3_A20_15-PadC16)
- U201 pad C17: /Connectivity/P9_TX_P -> unconnected-(U201D-IO_L20N_T3_A19_15-PadC17)
- U201 pad C18: +3V3 -> GND
- U201 pad C2: GND -> unconnected-(U201G-IO_L16P_T2_35-PadC2)
- U201 pad C3: GND -> +3V3
- U201 pad C4: GND -> unconnected-(U201G-IO_L7P_T1_AD6P_35-PadC4)
- U201 pad C5: GND -> unconnected-(U201G-IO_L1N_T0_AD4N_35-PadC5)
- U201 pad C6: GND -> unconnected-(U201G-IO_L1P_T0_AD4P_35-PadC6)
- U201 pad C7: GND -> unconnected-(U201G-IO_L4N_T0_35-PadC7)
- U201 pad C8: TCK -> GND
- U201 pad C9: +1V8 -> Net-(U201E-IO_L11P_T1_SRCC_16)
- U201 pad D1: unconnected-(U201C-MGTPTXN0_216-PadD1) -> GND
- U201 pad D18: /FPGA_Config/SDI_FPGA -> unconnected-(U201D-IO_L21N_T3_DQS_A18_15-PadD18)
- U201 pad D3: GND -> unconnected-(U201G-IO_L12N_T1_MRCC_35-PadD3)
- U201 pad E1: GND -> unconnected-(U201G-IO_L18N_T2_35-PadE1)
- U201 pad E17: GND -> unconnected-(U201D-IO_L16P_T2_A28_15-PadE17)
- U201 pad E18: Net-(U201B-IO_L3P_T0_DQS_PUDC_B_14) -> unconnected-(U201D-IO_L21P_T3_DQS_15-PadE18)
- U201 pad E2: GND -> unconnected-(U201G-IO_L14P_T2_SRCC_35-PadE2)
- U201 pad E3: GND -> unconnected-(U201G-IO_L12P_T1_MRCC_35-PadE3)
- U201 pad F1: GND -> unconnected-(U201G-IO_L18P_T2_35-PadF1)
- U201 pad F17: +3V3 -> GND
- U201 pad F18: /FPGA_Config/NHL_FPGA -> unconnected-(U201D-IO_L22N_T3_A16_15-PadF18)
- U201 pad F2: GND -> +3V3
- U201 pad F3: GND -> unconnected-(U201G-IO_L13N_T2_MRCC_35-PadF3)
- U201 pad G1: GND -> unconnected-(U201G-IO_L17N_T2_35-PadG1)
- U201 pad G10: +1V0 -> GND
- U201 pad G11: GND -> +1V0
- U201 pad G12: +3V3 -> GND
- U201 pad G13: +3V3 -> unconnected-(U201D-IO_0_15-PadG13)
- U201 pad G17: P6_L2 -> unconnected-(U201D-IO_L18N_T2_A23_15-PadG17)
- U201 pad G18: /FPGA_Config/NWP_FPGA -> unconnected-(U201D-IO_L22P_T3_A17_15-PadG18)
- U201 pad G2: /Connectivity/P7_CLK_N -> unconnected-(U201G-IO_L15N_T2_DQS_35-PadG2)
- U201 pad G3: /Connectivity/P7_CLK_P -> unconnected-(U201G-IO_L20N_T3_35-PadG3)
- U201 pad G7: GND -> +1V0
- U201 pad G9: GND -> +1V0
- U201 pad H1: /Connectivity/P7_RX_P -> unconnected-(U201G-IO_L17P_T2_35-PadH1)
- U201 pad H10: +1V0 -> Net-(U201A-VCCADC_0)
- U201 pad H12: GND -> +1V8
- U201 pad H13: +1V8 -> GND
- U201 pad H17: P6_L1 -> unconnected-(U201D-IO_L18P_T2_A24_15-PadH17)
- U201 pad H18: GND -> +3V3
- U201 pad H2: /Connectivity/P7_TX_P -> unconnected-(U201G-IO_L15P_T2_DQS_35-PadH2)
- U201 pad H3: +3V3 -> GND
- U201 pad H8: GND -> +1V0
- U201 pad J1: /Connectivity/P7_RX_N -> +3V3
- U201 pad J10: +1V0 -> GND
- U201 pad J11: GND -> +1V0
- U201 pad J13: +1V8 -> unconnected-(U201D-IO_L17N_T2_A25_15-PadJ13)
- U201 pad J17: /Connectivity/P2_CLK_P -> unconnected-(U201D-IO_L23P_T3_FOE_B_15-PadJ17)
- U201 pad J18: /Connectivity/P2_CLK_N -> unconnected-(U201D-IO_L23N_T3_FWE_B_15-PadJ18)
- U201 pad J2: /Connectivity/P7_TX_N -> unconnected-(U201G-IO_L22N_T3_35-PadJ2)
- U201 pad J3: P8_L2 -> unconnected-(U201G-IO_L22P_T3_35-PadJ3)
- U201 pad J7: +3V3 -> +1V0
- U201 pad K1: +3V3 -> unconnected-(U201G-IO_L23N_T3_35-PadK1)
- U201 pad K12: +3V3 -> +1V8
- U201 pad K13: +3V3 -> unconnected-(U201D-IO_L17P_T2_A26_15-PadK13)
- U201 pad K17: /Connectivity/P5_RX_N -> /FPGA_Config/SDI_FPGA
- U201 pad K18: /Connectivity/P2_TX_N -> /FPGA_Config/SDO_FPGA
- U201 pad K2: P7_L1 -> unconnected-(U201G-IO_L23P_T3_35-PadK2)
- U201 pad K3: P9_L1 -> unconnected-(U201F-IO_L2P_T0_34-PadK3)
- U201 pad K7: +3V3 -> GND
- U201 pad K8: GND -> +1V0
- U201 pad L1: P8_L1 -> unconnected-(U201F-IO_L1P_T0_34-PadL1)
- U201 pad L10: +1V0 -> GND
- U201 pad L11: GND -> +1V0
- U201 pad L12: +3V3 -> GND
- U201 pad L13: +3V3 -> /FPGA_Config/NCS_FPGA
- U201 pad L17: /Connectivity/P5_RX_P -> +3V3
- U201 pad L18: /Connectivity/P2_TX_P -> unconnected-(U201C-IO_L4P_T0_D04_14-PadL18)
- U201 pad L2: P7_L2 -> GND
- U201 pad L3: P9_L2 -> unconnected-(U201F-IO_L2N_T0_34-PadL3)
- U201 pad L7: +3V3 -> +1V0
- U201 pad M1: Net-(U201G-IO_L9N_T1_DQS_AD7N_35) -> unconnected-(U201F-IO_L1N_T0_34-PadM1)
- U201 pad M11: +1V0 -> GND
- U201 pad M12: +3V3 -> +1V8
- U201 pad M13: GND -> unconnected-(U201C-IO_L6N_T0_D08_VREF_14-PadM13)
- U201 pad M17: +3V3 -> unconnected-(U201C-IO_L10N_T1_D15_14-PadM17)
- U201 pad M18: /Connectivity/P5_TX_P -> unconnected-(U201C-IO_L4N_T0_D05_14-PadM18)
- U201 pad M2: Net-(U201G-IO_L9P_T1_DQS_AD7P_35) -> unconnected-(U201F-IO_L4N_T0_34-PadM2)
- U201 pad M3: Net-(U201G-IO_L8N_T1_AD14N_35) -> unconnected-(U201F-IO_L4P_T0_34-PadM3)
- U201 pad M7: +3V3 -> GND
- U201 pad M8: +3V3 -> +1V0
- U201 pad N1: Net-(U201G-IO_L10N_T1_AD15N_35) -> unconnected-(U201F-IO_L3N_T0_DQS_34-PadN1)
- U201 pad N10: +1V0 -> GND
- U201 pad N13: GND -> +3V3
- U201 pad N17: /Connectivity/P4_CLK_P -> unconnected-(U201C-IO_L9P_T1_DQS_14-PadN17)
- U201 pad N18: /Connectivity/P2_RX_P -> GND
- U201 pad N2: Net-(U201G-IO_L10P_T1_AD15P_35) -> unconnected-(U201F-IO_L3P_T0_DQS_34-PadN2)
- U201 pad N3: unconnected-(U201G-IO_L12P_T1_MRCC_35-PadN3) -> +3V3
- U201 pad N7: +3V3 -> +1V0
- U201 pad N8: +3V3 -> GND
- U201 pad N9: GND -> +1V0
- U201 pad P1: unconnected-(U201G-IO_L19N_T3_VREF_35-PadP1) -> GND
- U201 pad P17: /Connectivity/P4_CLK_N -> unconnected-(U201C-IO_L12P_T1_MRCC_14-PadP17)
- U201 pad P18: /Connectivity/P4_TX_P -> unconnected-(U201C-IO_L9N_T1_DQS_D13_14-PadP18)
- U201 pad P2: GND -> unconnected-(U201F-IO_L15P_T2_DQS_34-PadP2)
- U201 pad P3: 12MHZ_CLK -> unconnected-(U201F-IO_L14N_T2_SRCC_34-PadP3)
- U201 pad R1: +3V3 -> unconnected-(U201F-IO_L17P_T2_34-PadR1)
- U201 pad R17: +3V3 -> unconnected-(U201C-IO_L12N_T1_MRCC_14-PadR17)
- U201 pad R18: /Connectivity/P4_TX_N -> /Connectivity/P3_RX_P
- U201 pad R2: /Serial/SERIAL_D1 -> unconnected-(U201F-IO_L15N_T2_DQS_34-PadR2)
- U201 pad R3: /Serial/SERIAL_D3 -> unconnected-(U201F-IO_L11P_T1_SRCC_34-PadR3)
- U201 pad T1: /Serial/SERIAL_D5 -> unconnected-(U201F-IO_L17N_T2_34-PadT1)
- U201 pad T17: /Connectivity/P6_TX_P -> GND
- U201 pad T18: /Connectivity/P6_TX_N -> /Connectivity/P3_RX_N
- U201 pad T2: /Serial/SERIAL_D2 -> +3V3
- U201 pad T3: /Serial/SERIAL_D4 -> unconnected-(U201F-IO_L11N_T1_SRCC_34-PadT3)
- U201 pad U1: /Serial/SERIAL_D6 -> unconnected-(U201F-IO_L7P_T1_34-PadU1)
- U201 pad U10: /FPGA_Config/MODE2 -> GND
- U201 pad U11: /FPGA_Config/FPGA_INIT -> unconnected-(U201C-IO_L19N_T3_A09_D25_VREF_14-PadU11)
- U201 pad U12: /FPGA_Config/FPGA_DONE -> /Connectivity/P4_RX_P
- U201 pad U13: +3V3 -> /Connectivity/P5_TX_N
- U201 pad U14: unconnected-(U201D-IO_25_14-PadU14) -> /Connectivity/P5_CLK_P
- U201 pad U15: /Connectivity/P8_RX_P -> +3V3
- U201 pad U16: /Connectivity/P8_RX_N -> /Connectivity/P3_TX_P
- U201 pad U17: /Connectivity/P6_RX_P -> /Connectivity/P3_CLK_P
- U201 pad U18: /Connectivity/P6_RX_N -> /Connectivity/P3_CLK_N
- U201 pad U2: /Serial/SERIAL_WR# -> unconnected-(U201F-IO_L9P_T1_DQS_34-PadU2)
- U201 pad U3: /Serial/SERIAL_RD# -> unconnected-(U201F-IO_L8N_T1_34-PadU3)
- U201 pad U4: /Serial/SERIAL_SIWU# -> unconnected-(U201F-IO_L8P_T1_34-PadU4)
- U201 pad U5: P3_L1 -> +3V3
- U201 pad U6: GND -> unconnected-(U201F-IO_L22N_T3_34-PadU6)
- U201 pad U7: P4_L1 -> unconnected-(U201F-IO_L22P_T3_34-PadU7)
- U201 pad U8: P2_L1 -> unconnected-(U201F-IO_25_34-PadU8)
- U201 pad U9: GND -> /Connectivity/P4_TX_P
- U201 pad V1: +3V3 -> unconnected-(U201F-IO_L7N_T1_34-PadV1)
- U201 pad V10: /FPGA_Config/FPGA_RST -> /Connectivity/P4_CLK_P
- U201 pad V11: Net-(U201B-CFGBVS_0) -> /Connectivity/P4_CLK_N
- U201 pad V12: /FPGA_Config/MODE0 -> /Connectivity/P4_RX_N
- U201 pad V13: /Connectivity/P8_TX_P -> GND
- U201 pad V14: /Connectivity/P8_TX_N -> /Connectivity/P5_CLK_N
- U201 pad V15: /Connectivity/P1_TX_P -> /Connectivity/P5_RX_P
- U201 pad V16: /Connectivity/P1_RX_P -> /Connectivity/P5_RX_N
- U201 pad V17: /Connectivity/P1_RX_N -> /Connectivity/P3_TX_N
- U201 pad V18: GND -> +3V3
- U201 pad V2: /Serial/SERIAL_D7 -> unconnected-(U201F-IO_L9N_T1_DQS_34-PadV2)
- U201 pad V3: /Serial/SERIAL_RXF# -> GND
- U201 pad V4: /Serial/SERIAL_PWR# -> unconnected-(U201F-IO_L10N_T1_34-PadV4)
- U201 pad V5: P3_L2 -> unconnected-(U201F-IO_L10P_T1_34-PadV5)
- U201 pad V6: +3V3 -> unconnected-(U201F-IO_L20N_T3_34-PadV6)
- U201 pad V7: P4_L2 -> unconnected-(U201F-IO_L20P_T3_34-PadV7)
- U201 pad V8: P2_L2 -> +3V3
- U201 pad V9: +3V3 -> /Connectivity/P4_TX_N
Routing:
- net /Connectivity/P7_CLK_N: track 51.3 -> 0.00 mm
- net /Connectivity/P6_TX_N: track 49.2 -> 0.00 mm
- net /Connectivity/P7_CLK_P: track 49.1 -> 0.00 mm
- net /Connectivity/P6_TX_P: track 48.4 -> 0.00 mm
- net /Connectivity/P7_TX_N: track 39.8 -> 0.00 mm
- net /Connectivity/P7_TX_P: track 38.8 -> 0.00 mm
- net /Connectivity/P7_RX_P: track 37.9 -> 0.00 mm
- net /Connectivity/P8_CLK_N: track 37.2 -> 0.00 mm
- net /Connectivity/P7_RX_N: track 37.0 -> 0.00 mm
- net /Connectivity/P1_RX_P: track 36.8 -> 0.00 mm
- net /Connectivity/P6_CLK_N: track 36.8 -> 0.00 mm
- net /Connectivity/P6_RX_P: track 35.5 -> 0.00 mm
- net /Connectivity/P1_RX_N: track 35.4 -> 0.00 mm
- net /Connectivity/P6_CLK_P: track 35.3 -> 0.00 mm
- net /Connectivity/P8_TX_N: track 35.3 -> 0.00 mm
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Other:
- board text removed: "BANK35 K2 - L3 : U703"
- board text removed: "Bank43 One RJ45"
