File: Hardware/Controller_Board/Controller_Board.kicad_pcb (KiCad board)
At the start: 6 copper layers, 85 x 85 mm, 258 parts, among them J601 USB-C, Q101 DMN2400UFB-7, SW301 Reset, U101 TPS82084, U102 LT8645S, U103 TDS5311P, U104 TPS82084, U105 TPS82084, U106 XT30, U201 XC7A35T-CSG324, U301 IS25LP256D, U401 FT232H, U402 93LC56B, U501 FT232H, U502 93LC56B, U601 ESD122, U602 USB2512B, U701 RJ45, U702 RJ45, U703 RJ45, U704 TPD4E02B04, U705 TPD4E02B04, U706 TPD4E02B04, U707 TPD4E02B04, U708 TPD4E02B04, U709 TPD4E02B04, U710 RJ45, U711 RJ45, U712 RJ45, U713 TPD4E02B04, U714 TPD4E02B04, U715 TPD4E02B04, U716 RJ45, U717 RJ45, U718 RJ45, U719 TPD4E02B04, U720 TPD4E02B04, U721 TPD4E02B04, U722 TPD4E02B04, U723 TPD4E02B04, U724 TPD4E02B04, Y301 12MHz, Y401 12MHz, Y501 12MHz, Y601 24MHz

Commit message: Converted to 10.0 KiCad schematic + Began BGA fan
Parts:
- added Y1: 24MHz, Crystal:Crystal_SMD_2520-4Pin_2.5x2.0mm, F.Cu at (75.6, 119.9)
- added Y2: 12MHz, Crystal:Crystal_SMD_2520-4Pin_2.5x2.0mm, F.Cu at (75.6, 113.8)
- added Y3: 12MHz, Crystal:Crystal_SMD_2520-4Pin_2.5x2.0mm, F.Cu at (82.1, 113.8)
- C213, C214, C215, C216, C217: moved to B.Cu
- moved U713 219.9 mm to (223.4, 114.3)
- moved U722 208.6 mm to (211.8, 122.9)
- moved U723 208.6 mm to (214.7, 122.9)
- moved U724 208.6 mm to (217.6, 122.9)
- moved U705 205.8 mm to (211.8, 114.3)
- moved U706 205.8 mm to (214.7, 114.3)
- moved U714 205.8 mm to (211.8, 118.6)
- moved U715 205.8 mm to (214.7, 118.6)
- moved U719 205.8 mm to (217.6, 118.6)
- moved U721 205.8 mm to (223.4, 118.6)
- moved U720 205.8 mm to (220.5, 118.6)
- moved U708 202.9 mm to (217.6, 114.3)
- moved U709 202.9 mm to (220.5, 114.3)
- moved C213 20.5 mm to (80.4, 121.5), turned to 180 degrees
- moved C214 15.2 mm to (80.4, 123.2)
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Connections:
- U201 pad A18: unconnected-(U201D-IO_L10N_T1_AD11N_15-PadA18) -> /Connectivity/P9_RX_N
- U201 pad B18: unconnected-(U201D-IO_L10P_T1_AD11P_15-PadB18) -> /Connectivity/P9_RX_P
- U201 pad C1: unconnected-(U201G-IO_L16N_T2_35-PadC1) -> /Connectivity/P7_TX_N
- U201 pad C16: unconnected-(U201D-IO_L20P_T3_A20_15-PadC16) -> /Connectivity/P9_CLK_P
- U201 pad C17: unconnected-(U201D-IO_L20N_T3_A19_15-PadC17) -> /Connectivity/P9_CLK_N
- U201 pad C2: unconnected-(U201G-IO_L16P_T2_35-PadC2) -> /Connectivity/P7_TX_P
- U201 pad D18: unconnected-(U201D-IO_L21N_T3_DQS_A18_15-PadD18) -> /Connectivity/P9_TX_N
- U201 pad E1: unconnected-(U201G-IO_L18N_T2_35-PadE1) -> /Connectivity/P7_CLK_N
- U201 pad E18: unconnected-(U201D-IO_L21P_T3_DQS_15-PadE18) -> /Connectivity/P9_TX_P
- U201 pad F1: unconnected-(U201G-IO_L18P_T2_35-PadF1) -> /Connectivity/P7_CLK_P
- U201 pad F18: unconnected-(U201D-IO_L22N_T3_A16_15-PadF18) -> /Connectivity/P2_RX_N
- U201 pad G1: unconnected-(U201G-IO_L17N_T2_35-PadG1) -> /Connectivity/P7_RX_N
- U201 pad G17: unconnected-(U201D-IO_L18N_T2_A23_15-PadG17) -> /Connectivity/P2_CLK_N
- U201 pad G18: unconnected-(U201D-IO_L22P_T3_A17_15-PadG18) -> /Connectivity/P2_RX_P
- U201 pad H1: unconnected-(U201G-IO_L17P_T2_35-PadH1) -> /Connectivity/P7_RX_P
- U201 pad H17: unconnected-(U201D-IO_L18P_T2_A24_15-PadH17) -> /Connectivity/P2_CLK_P
- U201 pad J17: unconnected-(U201D-IO_L23P_T3_FOE_B_15-PadJ17) -> /Connectivity/P2_TX_P
- U201 pad J18: unconnected-(U201D-IO_L23N_T3_FWE_B_15-PadJ18) -> /Connectivity/P2_TX_N
- U201 pad J2: unconnected-(U201G-IO_L22N_T3_35-PadJ2) -> /Connectivity/P8_TX_N
- U201 pad J3: unconnected-(U201G-IO_L22P_T3_35-PadJ3) -> /Connectivity/P8_TX_P
- U201 pad K1: unconnected-(U201G-IO_L23N_T3_35-PadK1) -> /Connectivity/P8_CLK_N
- U201 pad K2: unconnected-(U201G-IO_L23P_T3_35-PadK2) -> /Connectivity/P8_CLK_P
- U201 pad L18: unconnected-(U201C-IO_L4P_T0_D04_14-PadL18) -> /Connectivity/P3_RX_P
- U201 pad M18: unconnected-(U201C-IO_L4N_T0_D05_14-PadM18) -> /Connectivity/P3_RX_N
- U201 pad M2: unconnected-(U201F-IO_L4N_T0_34-PadM2) -> /Connectivity/P8_RX_N
- U201 pad M3: unconnected-(U201F-IO_L4P_T0_34-PadM3) -> /Connectivity/P8_RX_P
- U201 pad N17: unconnected-(U201C-IO_L9P_T1_DQS_14-PadN17) -> /Connectivity/P3_CLK_P
- U201 pad P18: unconnected-(U201C-IO_L9N_T1_DQS_D13_14-PadP18) -> /Connectivity/P3_CLK_N
- U201 pad R1: unconnected-(U201F-IO_L17P_T2_34-PadR1) -> /Connectivity/P1_TX_P
- U201 pad R18: /Connectivity/P3_RX_P -> /Connectivity/P3_TX_P
- U201 pad T1: unconnected-(U201F-IO_L17N_T2_34-PadT1) -> /Connectivity/P1_TX_N
- U201 pad T13: /Connectivity/P5_TX_P -> unconnected-(U201C-IO_L23P_T3_A03_D19_14-PadT13)
- U201 pad T18: /Connectivity/P3_RX_N -> /Connectivity/P3_TX_N
- U201 pad U1: unconnected-(U201F-IO_L7P_T1_34-PadU1) -> /Connectivity/P1_CLK_P
- U201 pad U12: /Connectivity/P4_RX_P -> /Connectivity/P4_CLK_P
- U201 pad U13: /Connectivity/P5_TX_N -> unconnected-(U201C-IO_L23N_T3_A02_D18_14-PadU13)
- U201 pad U14: /Connectivity/P5_CLK_P -> /Connectivity/P4_RX_P
- U201 pad U16: /Connectivity/P3_TX_P -> /Connectivity/P5_CLK_P
- U201 pad U17: /Connectivity/P3_CLK_P -> /Connectivity/P5_RX_P
- U201 pad U18: /Connectivity/P3_CLK_N -> /Connectivity/P5_RX_N
- U201 pad U2: unconnected-(U201F-IO_L9P_T1_DQS_34-PadU2) -> /Connectivity/P1_RX_P
- U201 pad U9: /Connectivity/P4_TX_P -> /Connectivity/P6_RX_P
- U201 pad V1: unconnected-(U201F-IO_L7N_T1_34-PadV1) -> /Connectivity/P1_CLK_N
- U201 pad V10: /Connectivity/P4_CLK_P -> /Connectivity/P4_TX_P
- U201 pad V11: /Connectivity/P4_CLK_N -> /Connectivity/P4_TX_N
- U201 pad V12: /Connectivity/P4_RX_N -> /Connectivity/P4_CLK_N
- U201 pad V14: /Connectivity/P5_CLK_N -> /Connectivity/P4_RX_N
- U201 pad V15: /Connectivity/P5_RX_P -> /Connectivity/P5_TX_P
- U201 pad V16: /Connectivity/P5_RX_N -> /Connectivity/P5_TX_N
- U201 pad V17: /Connectivity/P3_TX_N -> /Connectivity/P5_CLK_N
- U201 pad V2: unconnected-(U201F-IO_L9N_T1_DQS_34-PadV2) -> /Connectivity/P1_RX_N
- U201 pad V4: unconnected-(U201F-IO_L10N_T1_34-PadV4) -> /Connectivity/P6_TX_N
- U201 pad V5: unconnected-(U201F-IO_L10P_T1_34-PadV5) -> /Connectivity/P6_TX_P
- U201 pad V6: unconnected-(U201F-IO_L20N_T3_34-PadV6) -> /Connectivity/P6_CLK_N
- U201 pad V7: unconnected-(U201F-IO_L20P_T3_34-PadV7) -> /Connectivity/P6_CLK_P
- U201 pad V9: /Connectivity/P4_TX_N -> /Connectivity/P6_RX_N
Routing:
- net /Connectivity/P9_CLK_N: track 0.00 -> 52.5 mm
- net /Connectivity/P9_TX_N: track 0.00 -> 52.0 mm
- net /Connectivity/P9_CLK_P: track 0.00 -> 52.0 mm
- net /Connectivity/P9_RX_P: track 0.00 -> 50.7 mm
- net /Connectivity/P9_TX_P: track 0.00 -> 50.5 mm
- net /Connectivity/P2_CLK_N: track 0.00 -> 50.1 mm
- net /Connectivity/P9_RX_N: track 0.00 -> 47.5 mm
- net /Connectivity/P2_CLK_P: track 0.00 -> 45.3 mm
- net /Connectivity/P7_RX_P: track 0.00 -> 41.6 mm
- net /Connectivity/P7_CLK_N: track 0.00 -> 40.2 mm
- net /Connectivity/P7_TX_P: track 0.00 -> 40.2 mm
- net /Connectivity/P2_RX_P: track 0.00 -> 40.1 mm
- net /Connectivity/P7_RX_N: track 0.00 -> 39.9 mm
- net /Connectivity/P7_CLK_P: track 0.00 -> 39.1 mm
- net /Connectivity/P7_TX_N: track 0.00 -> 38.7 mm
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- added copper zone on In2.Cu, net +3V3

Commit message: Advanced PCB routing and reorganized FPGA traces
Parts:
- removed U707, U708, U709: TPD4E02B04, Package_SON:USON-10_2.5x1.0mm_P0.5mm
- removed Y401, Y501: 12MHz, Crystal:Crystal_SMD_2520-4Pin_2.5x2.0mm
- removed Y601: 24MHz, Crystal:Crystal_SMD_2520-4Pin_2.5x2.0mm
- added U725: TPD4E02B04, Package_SON:USON-10_2.5x1.0mm_P0.5mm, F.Cu at (129.0, 121.8)
- added U726: TPD4E02B04, Package_SON:USON-10_2.5x1.0mm_P0.5mm, F.Cu at (183.4, 99.1)
- added U727: TPD4E02B04, Package_SON:USON-10_2.5x1.0mm_P0.5mm, F.Cu at (157.8, 127.9)
- added U728: TPD4E02B04, Package_SON:USON-10_2.5x1.0mm_P0.5mm, F.Cu at (177.3, 127.9)
- added U729: TPD4E02B04, Package_SON:USON-10_2.5x1.0mm_P0.5mm, F.Cu at (129.0, 92.9)
- added U730: TPD4E02B04, Package_SON:USON-10_2.5x1.0mm_P0.5mm, F.Cu at (129.0, 99.1)
- moved U706 89.3 mm to (129.0, 89.4)
- moved U715 87.3 mm to (129.0, 102.3)
- moved U720 85.9 mm to (135.1, 127.9), turned to 90 degrees
- moved U723 76.6 mm to (138.3, 127.9), turned to -90 degrees
- moved U705 58.8 mm to (154.6, 127.9), turned to 90 degrees
- moved U724 47.9 mm to (183.4, 89.4)
- moved U721 47.3 mm to (183.4, 93.4)
- moved U713 41.8 mm to (183.4, 102.3)
- moved U714 38.9 mm to (174.1, 127.9), turned to 90 degrees
- moved U704 35.2 mm to (129.0, 118.6)
- moved U719 34.4 mm to (183.4, 121.8), turned to 180 degrees
- moved U722 28.7 mm to (183.4, 118.6)
- moved C206 2.50 mm to (153.0, 113.2)
- moved C207 2.50 mm to (154.6, 112.0)
- moved C208 2.50 mm to (154.6, 110.4)
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Connections:
- U201 pad F18: /Connectivity/P2_RX_N -> unconnected-(U201D-IO_L22N_T3_A16_15-PadF18)
- U201 pad G17: /Connectivity/P2_CLK_N -> /Connectivity/P2_RX_N
- U201 pad G18: /Connectivity/P2_RX_P -> unconnected-(U201D-IO_L22P_T3_A17_15-PadG18)
- U201 pad H17: /Connectivity/P2_CLK_P -> /Connectivity/P2_RX_P
- U201 pad J17: /Connectivity/P2_TX_P -> /Connectivity/P2_CLK_P
- U201 pad J18: /Connectivity/P2_TX_N -> /Connectivity/P2_CLK_N
- U201 pad L18: /Connectivity/P3_RX_P -> /Connectivity/P2_TX_P
- U201 pad M18: /Connectivity/P3_RX_N -> /Connectivity/P2_TX_N
- U201 pad N1: unconnected-(U201F-IO_L3N_T0_DQS_34-PadN1) -> /Connectivity/P1_TX_N
- U201 pad N17: /Connectivity/P3_CLK_P -> /Connectivity/P3_RX_P
- U201 pad N2: unconnected-(U201F-IO_L3P_T0_DQS_34-PadN2) -> /Connectivity/P1_TX_P
- U201 pad P18: /Connectivity/P3_CLK_N -> /Connectivity/P3_RX_N
- U201 pad P2: unconnected-(U201F-IO_L15P_T2_DQS_34-PadP2) -> /Connectivity/P1_CLK_P
- U201 pad R1: /Connectivity/P1_TX_P -> unconnected-(U201F-IO_L17P_T2_34-PadR1)
- U201 pad R18: /Connectivity/P3_TX_P -> /Connectivity/P3_CLK_P
- U201 pad R2: unconnected-(U201F-IO_L15N_T2_DQS_34-PadR2) -> /Connectivity/P1_CLK_N
- U201 pad T1: /Connectivity/P1_TX_N -> unconnected-(U201F-IO_L17N_T2_34-PadT1)
- U201 pad T11: unconnected-(U201C-IO_L19P_T3_A10_D26_14-PadT11) -> /Connectivity/P4_CLK_P
- U201 pad T18: /Connectivity/P3_TX_N -> /Connectivity/P3_CLK_N
- U201 pad U1: /Connectivity/P1_CLK_P -> /Connectivity/P1_RX_P
- U201 pad U11: unconnected-(U201C-IO_L19N_T3_A09_D25_VREF_14-PadU11) -> /Connectivity/P4_CLK_N
- U201 pad U12: /Connectivity/P4_CLK_P -> /Connectivity/P4_RX_P
- U201 pad U14: /Connectivity/P4_RX_P -> /Connectivity/P5_TX_P
- U201 pad U16: /Connectivity/P5_CLK_P -> /Connectivity/P5_RX_P
- U201 pad U17: /Connectivity/P5_RX_P -> /Connectivity/P3_TX_P
- U201 pad U18: /Connectivity/P5_RX_N -> /Connectivity/P3_TX_N
- U201 pad U2: /Connectivity/P1_RX_P -> /Connectivity/P6_TX_P
- U201 pad U9: /Connectivity/P6_RX_P -> /Connectivity/P4_TX_P
- U201 pad V1: /Connectivity/P1_CLK_N -> /Connectivity/P1_RX_N
- U201 pad V10: /Connectivity/P4_TX_P -> unconnected-(U201C-IO_L21P_T3_DQS_14-PadV10)
- U201 pad V11: /Connectivity/P4_TX_N -> unconnected-(U201C-IO_L21N_T3_DQS_A06_D22_14-PadV11)
- U201 pad V12: /Connectivity/P4_CLK_N -> /Connectivity/P4_RX_N
- U201 pad V14: /Connectivity/P4_RX_N -> /Connectivity/P5_TX_N
- U201 pad V15: /Connectivity/P5_TX_P -> /Connectivity/P5_CLK_P
- U201 pad V16: /Connectivity/P5_TX_N -> /Connectivity/P5_CLK_N
- U201 pad V17: /Connectivity/P5_CLK_N -> /Connectivity/P5_RX_N
- U201 pad V2: /Connectivity/P1_RX_N -> /Connectivity/P6_TX_N
- U201 pad V4: /Connectivity/P6_TX_N -> /Connectivity/P6_CLK_N
- U201 pad V5: /Connectivity/P6_TX_P -> /Connectivity/P6_CLK_P
- U201 pad V6: /Connectivity/P6_CLK_N -> /Connectivity/P6_RX_N
- U201 pad V7: /Connectivity/P6_CLK_P -> /Connectivity/P6_RX_P
- U201 pad V9: /Connectivity/P6_RX_N -> /Connectivity/P4_TX_N
- U720 pad 1: /Connectivity/P6_TX_N -> /Connectivity/P6_TX_P
- U720 pad 10: /Connectivity/P6_TX_N -> /Connectivity/P6_TX_P
- U720 pad 2: /Connectivity/P6_TX_P -> /Connectivity/P6_TX_N
- U720 pad 9: /Connectivity/P6_TX_P -> /Connectivity/P6_TX_N
- U723 pad 4: /Connectivity/P6_RX_N -> /Connectivity/P6_RX_P
- U723 pad 5: /Connectivity/P6_RX_P -> /Connectivity/P6_RX_N
- U723 pad 6: /Connectivity/P6_RX_P -> /Connectivity/P6_RX_N
- U723 pad 7: /Connectivity/P6_RX_N -> /Connectivity/P6_RX_P
Routing:
- net /Connectivity/P1_TX_P: track 19.6 -> 46.7 mm
- net /Connectivity/P1_CLK_N: track 13.7 -> 39.8 mm
- net /Connectivity/P1_CLK_P: track 13.6 -> 38.3 mm
- net /Connectivity/P1_TX_N: track 20.9 -> 45.5 mm
- net /Connectivity/P7_TX_N: track 38.7 -> 58.7 mm
- net /Connectivity/P7_TX_P: track 40.2 -> 59.9 mm
- net /Connectivity/P1_RX_N: track 14.0 -> 29.6 mm
- net /Connectivity/P7_CLK_N: track 40.2 -> 53.4 mm
- net /Connectivity/P7_CLK_P: track 39.1 -> 51.9 mm
- net /Connectivity/P1_RX_P: track 16.7 -> 29.2 mm
- net unconnected-(U201F-IO_L3P_T0_DQS_34-PadN2): track 9.51 -> 0.00 mm
- net /Connectivity/P2_CLK_N: track 50.1 -> 41.0 mm
- net /Connectivity/P7_RX_N: track 39.9 -> 49.0 mm
- net unconnected-(U201F-IO_L3N_T0_DQS_34-PadN1): track 8.38 -> 0.00 mm
- net /Connectivity/P7_RX_P: track 41.6 -> 49.9 mm
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Other:
- board text added: "Modify the ESD pinout!"

Commit message: Commiting PCB design with 45 degree tracks
Parts:
- moved U706 0.90 mm to (129.0, 90.3)
- moved U724 0.90 mm to (183.4, 90.3)
- moved U729 0.60 mm to (129.0, 93.5)
- moved U721 0.10 mm to (183.4, 93.5)
- turned U719 to 0 degrees
- turned U723 to 90 degrees
- turned U725 to 0 degrees
- turned U727 to 90 degrees
Connections:
- U713 pad 1: /Connectivity/P2_RX_N -> /Connectivity/P2_CLK_P
- U713 pad 10: /Connectivity/P2_RX_N -> /Connectivity/P2_CLK_P
- U713 pad 2: /Connectivity/P2_RX_P -> /Connectivity/P2_CLK_N
- U713 pad 4: /Connectivity/P2_TX_N -> /Connectivity/P2_TX_P
- U713 pad 5: /Connectivity/P2_TX_P -> /Connectivity/P2_TX_N
- U713 pad 6: /Connectivity/P2_TX_P -> /Connectivity/P2_TX_N
- U713 pad 7: /Connectivity/P2_TX_N -> /Connectivity/P2_TX_P
- U713 pad 9: /Connectivity/P2_RX_P -> /Connectivity/P2_CLK_N
- U714 pad 1: /Connectivity/P5_RX_N -> /Connectivity/P5_TX_P
- U714 pad 10: /Connectivity/P5_RX_N -> /Connectivity/P5_TX_P
- U714 pad 2: /Connectivity/P5_RX_P -> /Connectivity/P5_TX_N
- U714 pad 4: /Connectivity/P5_TX_N -> /Connectivity/P5_CLK_N
- U714 pad 5: /Connectivity/P5_TX_P -> /Connectivity/P5_CLK_P
- U714 pad 6: /Connectivity/P5_TX_P -> /Connectivity/P5_CLK_P
- U714 pad 7: /Connectivity/P5_TX_N -> /Connectivity/P5_CLK_N
- U714 pad 9: /Connectivity/P5_RX_P -> /Connectivity/P5_TX_N
- U715 pad 4: /Connectivity/P8_TX_N -> unconnected-(U715-IN-Pad4)
- U715 pad 5: /Connectivity/P8_TX_P -> unconnected-(U715-IN-Pad5)
- U715 pad 6: /Connectivity/P8_TX_P -> unconnected-(U715-NC-Pad6)
- U715 pad 7: /Connectivity/P8_TX_N -> unconnected-(U715-NC-Pad7)
- U719 pad 1: /Connectivity/P3_TX_N -> /Connectivity/P3_CLK_P
- U719 pad 10: /Connectivity/P3_TX_N -> /Connectivity/P3_CLK_P
- U719 pad 2: /Connectivity/P3_TX_P -> /Connectivity/P3_CLK_N
- U719 pad 4: /Connectivity/P3_CLK_N -> /Connectivity/P3_TX_P
- U719 pad 5: /Connectivity/P3_CLK_P -> /Connectivity/P3_TX_N
- U719 pad 6: /Connectivity/P3_CLK_P -> /Connectivity/P3_TX_N
- U719 pad 7: /Connectivity/P3_CLK_N -> /Connectivity/P3_TX_P
- U719 pad 9: /Connectivity/P3_TX_P -> /Connectivity/P3_CLK_N
- U720 pad 1: /Connectivity/P6_TX_P -> /Connectivity/P6_TX_N
- U720 pad 10: /Connectivity/P6_TX_P -> /Connectivity/P6_TX_N
- U720 pad 2: /Connectivity/P6_TX_N -> /Connectivity/P6_TX_P
- U720 pad 9: /Connectivity/P6_TX_N -> /Connectivity/P6_TX_P
- U721 pad 4: /Connectivity/P9_CLK_N -> unconnected-(U721-IN-Pad4)
- U721 pad 5: /Connectivity/P9_CLK_P -> unconnected-(U721-IN-Pad5)
- U721 pad 6: /Connectivity/P9_CLK_P -> unconnected-(U721-NC-Pad6)
- U721 pad 7: /Connectivity/P9_CLK_N -> unconnected-(U721-NC-Pad7)
- U722 pad 4: /Connectivity/P3_RX_N -> /Connectivity/P3_RX_P
- U722 pad 5: /Connectivity/P3_RX_P -> /Connectivity/P3_RX_N
- U722 pad 6: /Connectivity/P3_RX_P -> /Connectivity/P3_RX_N
- U722 pad 7: /Connectivity/P3_RX_N -> /Connectivity/P3_RX_P
- U723 pad 1: unconnected-(U723-IN-Pad1) -> /Connectivity/P6_RX_N
- U723 pad 10: unconnected-(U723-NC-Pad10) -> /Connectivity/P6_RX_N
- U723 pad 2: unconnected-(U723-IN-Pad2) -> /Connectivity/P6_RX_P
- U723 pad 4: /Connectivity/P6_RX_P -> unconnected-(U723-IN-Pad4)
- U723 pad 5: /Connectivity/P6_RX_N -> unconnected-(U723-IN-Pad5)
- U723 pad 6: /Connectivity/P6_RX_N -> unconnected-(U723-NC-Pad6)
- U723 pad 7: /Connectivity/P6_RX_P -> unconnected-(U723-NC-Pad7)
- U723 pad 9: unconnected-(U723-NC-Pad9) -> /Connectivity/P6_RX_P
- U724 pad 1: unconnected-(U724-IN-Pad1) -> /Connectivity/P9_RX_P
- U724 pad 10: unconnected-(U724-NC-Pad10) -> /Connectivity/P9_RX_P
- U724 pad 2: unconnected-(U724-IN-Pad2) -> /Connectivity/P9_RX_N
- U724 pad 4: /Connectivity/P9_RX_N -> /Connectivity/P9_CLK_P
- U724 pad 5: /Connectivity/P9_RX_P -> /Connectivity/P9_CLK_N
- U724 pad 6: /Connectivity/P9_RX_P -> /Connectivity/P9_CLK_N
- U724 pad 7: /Connectivity/P9_RX_N -> /Connectivity/P9_CLK_P
- U724 pad 9: unconnected-(U724-NC-Pad9) -> /Connectivity/P9_RX_N
- U725 pad 1: unconnected-(U725-IN-Pad1) -> /Connectivity/P1_RX_N
- U725 pad 10: unconnected-(U725-NC-Pad10) -> /Connectivity/P1_RX_N
- U725 pad 2: unconnected-(U725-IN-Pad2) -> /Connectivity/P1_RX_P
- U725 pad 4: /Connectivity/P1_RX_P -> unconnected-(U725-IN-Pad4)
- U725 pad 5: /Connectivity/P1_RX_N -> unconnected-(U725-IN-Pad5)
- U725 pad 6: /Connectivity/P1_RX_N -> unconnected-(U725-NC-Pad6)
- U725 pad 7: /Connectivity/P1_RX_P -> unconnected-(U725-NC-Pad7)
- U725 pad 9: unconnected-(U725-NC-Pad9) -> /Connectivity/P1_RX_P
- U726 pad 1: /Connectivity/P2_CLK_N -> unconnected-(U726-IN-Pad1)
- U726 pad 10: /Connectivity/P2_CLK_N -> unconnected-(U726-NC-Pad10)
- U726 pad 2: /Connectivity/P2_CLK_P -> unconnected-(U726-IN-Pad2)
- U726 pad 4: unconnected-(U726-IN-Pad4) -> /Connectivity/P2_RX_P
- U726 pad 5: unconnected-(U726-IN-Pad5) -> /Connectivity/P2_RX_N
- U726 pad 6: unconnected-(U726-NC-Pad6) -> /Connectivity/P2_RX_N
- U726 pad 7: unconnected-(U726-NC-Pad7) -> /Connectivity/P2_RX_P
- U726 pad 9: /Connectivity/P2_CLK_P -> unconnected-(U726-NC-Pad9)
- U727 pad 1: unconnected-(U727-IN-Pad1) -> /Connectivity/P4_RX_N
- U727 pad 10: unconnected-(U727-NC-Pad10) -> /Connectivity/P4_RX_N
- U727 pad 2: unconnected-(U727-IN-Pad2) -> /Connectivity/P4_RX_P
- U727 pad 4: /Connectivity/P4_RX_P -> unconnected-(U727-IN-Pad4)
- U727 pad 5: /Connectivity/P4_RX_N -> unconnected-(U727-IN-Pad5)
- U727 pad 6: /Connectivity/P4_RX_N -> unconnected-(U727-NC-Pad6)
- U727 pad 7: /Connectivity/P4_RX_P -> unconnected-(U727-NC-Pad7)
- U727 pad 9: unconnected-(U727-NC-Pad9) -> /Connectivity/P4_RX_P
- U728 pad 1: /Connectivity/P5_CLK_N -> /Connectivity/P5_RX_N
- U728 pad 10: /Connectivity/P5_CLK_N -> /Connectivity/P5_RX_N
- U728 pad 2: /Connectivity/P5_CLK_P -> /Connectivity/P5_RX_P
- U728 pad 9: /Connectivity/P5_CLK_P -> /Connectivity/P5_RX_P
- U729 pad 1: unconnected-(U729-IN-Pad1) -> /Connectivity/P7_RX_N
- U729 pad 10: unconnected-(U729-NC-Pad10) -> /Connectivity/P7_RX_N
- U729 pad 2: unconnected-(U729-IN-Pad2) -> /Connectivity/P7_RX_P
- U729 pad 4: /Connectivity/P7_RX_N -> unconnected-(U729-IN-Pad4)
- U729 pad 5: /Connectivity/P7_RX_P -> unconnected-(U729-IN-Pad5)
- U729 pad 6: /Connectivity/P7_RX_P -> unconnected-(U729-NC-Pad6)
- U729 pad 7: /Connectivity/P7_RX_N -> unconnected-(U729-NC-Pad7)
- U729 pad 9: unconnected-(U729-NC-Pad9) -> /Connectivity/P7_RX_P
- U730 pad 1: /Connectivity/P8_CLK_N -> /Connectivity/P8_TX_N
- U730 pad 10: /Connectivity/P8_CLK_N -> /Connectivity/P8_TX_N
- U730 pad 2: /Connectivity/P8_CLK_P -> /Connectivity/P8_TX_P
- U730 pad 4: unconnected-(U730-IN-Pad4) -> /Connectivity/P8_CLK_N
- U730 pad 5: unconnected-(U730-IN-Pad5) -> /Connectivity/P8_CLK_P
- U730 pad 6: unconnected-(U730-NC-Pad6) -> /Connectivity/P8_CLK_P
- U730 pad 7: unconnected-(U730-NC-Pad7) -> /Connectivity/P8_CLK_N
- U730 pad 9: /Connectivity/P8_CLK_P -> /Connectivity/P8_TX_P
Routing:
- net /Connectivity/P8_TX_P: track 19.2 -> 47.1 mm
- net /Connectivity/P8_TX_N: track 18.3 -> 46.0 mm
- net /Connectivity/P8_CLK_N: track 17.4 -> 41.1 mm
- net /Connectivity/P8_CLK_P: track 18.5 -> 40.7 mm
- net /Connectivity/P6_TX_N: track 18.4 -> 35.2 mm
- net /Connectivity/P6_TX_P: track 19.9 -> 36.3 mm
- net /Connectivity/P6_CLK_N: track 16.7 -> 31.9 mm
- net /Connectivity/P6_CLK_P: track 15.5 -> 30.4 mm
- net /Connectivity/P6_RX_N: track 17.5 -> 31.4 mm
- net /Connectivity/P9_RX_P: track 47.8 -> 61.7 mm
- net /Connectivity/P9_RX_N: track 44.6 -> 58.5 mm
- net /Connectivity/P6_RX_P: track 19.3 -> 33.0 mm
- net /Connectivity/P8_RX_N: track 28.3 -> 41.5 mm
- net /Connectivity/P8_RX_P: track 30.7 -> 43.8 mm
- net /Connectivity/P1_TX_P: track 46.7 -> 36.1 mm
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Other:
- board text removed: "Modify the ESD pinout!"

Commit message: Advanced PCB design: Routed FTDIs + SPI Flash
Parts:
- removed C228: 100n, Capacitor_SMD:C_0201_0603Metric
- C203, C218, C229, C230, C231, C232, C233, C235, C242, C243, C244, C245, C246, C247, C252, C253, C254, C255, C256, C257: moved to B.Cu
- R303, R304, R305, R306, Re301, Re302: footprint Resistor_SMD:R_0402_1005Metric -> Resistor_SMD:R_0201_0603Metric; moved to B.Cu
- moved R304 112.4 mm to (161.0, 113.6), turned to 180 degrees
- moved R311 112.4 mm to (166.1, 102.3)
- moved Y301 111.4 mm to (166.0, 100.7)
- moved R308 111.4 mm to (161.2, 100.9), turned to -90 degrees
- moved R305 109.4 mm to (158.2, 117.2), turned to -90 degrees
- moved C303 106.4 mm to (164.6, 100.7), turned to -90 degrees
- moved R303 105.9 mm to (155.0, 117.1), turned to 90 degrees
- moved Re301 104.0 mm to (159.0, 117.2), turned to -90 degrees
- moved R310 103.0 mm to (151.3, 100.0), turned to 90 degrees
- moved C302 103.0 mm to (161.2, 99.0), turned to 90 degrees
- moved Re302 102.5 mm to (157.4, 117.2), turned to -90 degrees
- moved R309 101.9 mm to (151.3, 102.5), turned to 90 degrees
- moved R306 101.6 mm to (153.8, 116.8)
- moved C113 100.8 mm to (181.4, 44.6)
- moved C116 100.8 mm to (181.4, 48.8)
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Connections:
- U201 pad A1: unconnected-(U201G-IO_L9N_T1_DQS_AD7N_35-PadA1) -> SERIAL_D2
- U201 pad A3: unconnected-(U201G-IO_L8N_T1_AD14N_35-PadA3) -> SERIAL_D5
- U201 pad A4: unconnected-(U201G-IO_L8P_T1_AD14P_35-PadA4) -> SERIAL_D7
- U201 pad A5: unconnected-(U201G-IO_L3N_T0_DQS_AD5N_35-PadA5) -> SERIAL_D8
- U201 pad A6: unconnected-(U201G-IO_L3P_T0_DQS_AD5P_35-PadA6) -> SERIAL_PWR#
- U201 pad B1: unconnected-(U201G-IO_L9P_T1_DQS_AD7P_35-PadB1) -> SERIAL_D1
- U201 pad B2: unconnected-(U201G-IO_L10N_T1_AD15N_35-PadB2) -> SERIAL_D3
- U201 pad B3: unconnected-(U201G-IO_L10P_T1_AD15P_35-PadB3) -> SERIAL_D4
- U201 pad B4: unconnected-(U201G-IO_L7N_T1_AD6N_35-PadB4) -> SERIAL_D6
- U201 pad B7: unconnected-(U201G-IO_L2P_T0_AD12P_35-PadB7) -> SERIAL_OE#
- U201 pad C4: unconnected-(U201G-IO_L7P_T1_AD6P_35-PadC4) -> SERIAL_SIWU#
- U201 pad D2: unconnected-(U201G-IO_L14N_T2_SRCC_35-PadD2) -> SERIAL_TXE#
- U201 pad D3: unconnected-(U201G-IO_L12N_T1_MRCC_35-PadD3) -> SERIAL_RXF#
- U201 pad D5: unconnected-(U201G-IO_L11P_T1_SRCC_35-PadD5) -> SERIAL_WR#
- U201 pad E2: unconnected-(U201G-IO_L14P_T2_SRCC_35-PadE2) -> SERIAL_RD#
- U201 pad E3: unconnected-(U201G-IO_L12P_T1_MRCC_35-PadE3) -> SERIAL_CLK
- U501 pad 13: /Serial/SERIAL_D1 -> SERIAL_D1
- U501 pad 14: /Serial/SERIAL_D2 -> SERIAL_D2
- U501 pad 15: /Serial/SERIAL_D3 -> SERIAL_D3
- U501 pad 16: /Serial/SERIAL_D4 -> SERIAL_D4
- U501 pad 17: /Serial/SERIAL_D5 -> SERIAL_D5
- U501 pad 18: /Serial/SERIAL_D6 -> SERIAL_D6
- U501 pad 19: /Serial/SERIAL_D7 -> SERIAL_D7
- U501 pad 20: /Serial/SERIAL_D8 -> SERIAL_D8
- U501 pad 21: /Serial/SERIAL_RXF# -> SERIAL_RXF#
- U501 pad 25: /Serial/SERIAL_TXE# -> SERIAL_TXE#
- U501 pad 26: /Serial/SERIAL_RD# -> SERIAL_RD#
- U501 pad 27: /Serial/SERIAL_WR# -> SERIAL_WR#
- U501 pad 28: /Serial/SERIAL_SIWU# -> SERIAL_SIWU#
- U501 pad 29: /Serial/SERIAL_CLK -> SERIAL_CLK
- U501 pad 30: /Serial/SERIAL_OE# -> SERIAL_OE#
- U501 pad 31: /Serial/SERIAL_PWR# -> SERIAL_PWR#
Routing:
- net SERIAL_CLK: track 0.00 -> 39.0 mm, vias 0 -> 2
- net SERIAL_OE#: track 0.00 -> 34.3 mm, vias 0 -> 2
- net SERIAL_D1: track 0.00 -> 33.2 mm
- net SERIAL_D3: track 0.00 -> 33.1 mm
- net SERIAL_D4: track 0.00 -> 33.1 mm
- net SERIAL_PWR#: track 0.00 -> 33.1 mm, vias 0 -> 2
- net SERIAL_WR#: track 0.00 -> 33.0 mm, vias 0 -> 2
- net SERIAL_RXF#: track 0.00 -> 32.9 mm, vias 0 -> 2
- net SERIAL_D6: track 0.00 -> 32.8 mm
- net SERIAL_SIWU#: track 0.00 -> 32.2 mm, vias 0 -> 2
- net SERIAL_D2: track 0.00 -> 32.2 mm
- net SERIAL_D5: track 0.00 -> 32.0 mm
- net SERIAL_D8: track 0.00 -> 31.7 mm
- net SERIAL_D7: track 0.00 -> 31.7 mm
- net SERIAL_TXE#: track 0.00 -> 31.5 mm, vias 0 -> 2
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- added copper zone on In2.Cu, net +5V
