File: Hardware/Controller_Board/Controller_Board.kicad_pcb (KiCad board)
At the start: 6 copper layers, 85 x 85 mm, 260 parts, among them J601 USB-C, Q101 DMN2400UFB-7, SW301 Reset, U101 TPS82084, U102 LT8645S, U103 TDS5311P, U104 TPS82084, U105 TPS82084, U106 XT30, U201 XC7A35T-CSG324, U301 IS25LP256D, U401 FT232H, U402 93LC56B, U501 FT232H, U502 93LC56B, U601 ESD122, U602 USB2512B, U701 RJ45, U702 RJ45, U703 RJ45, U704 TPD4E02B04, U705 TPD4E02B04, U706 TPD4E02B04, U710 RJ45, U711 RJ45, U712 RJ45, U713 TPD4E02B04, U714 TPD4E02B04, U715 TPD4E02B04, U716 RJ45, U717 RJ45, U718 RJ45, U719 TPD4E02B04, U720 TPD4E02B04, U721 TPD4E02B04, U722 TPD4E02B04, U723 TPD4E02B04, U724 TPD4E02B04, U725 TPD4E02B04, U726 TPD4E02B04, U727 TPD4E02B04, U728 TPD4E02B04, U729 TPD4E02B04, U730 TPD4E02B04, Y1 24MHz, Y2 12MHz, Y3 12MHz, Y301 12MHz

Commit message: Advanced PCB design - Routed FTDI chips + USB HUB
Parts:
- removed C202: 10p, Capacitor_SMD:C_0402_1005Metric
- removed C406, C506: 100n, Capacitor_SMD:C_0402_1005Metric
- added D604: TVS, Diode_SMD:D_0402_1005Metric, B.Cu at (143.4, 65.4)
- added H1: M3, MountingHole:MountingHole_3.2mm_M3_Pad_Via, F.Cu at (120.7, 65.2)
- added H2: M3, MountingHole:MountingHole_3.2mm_M3_Pad_Via, F.Cu at (191.7, 65.2)
- added H3: M3, MountingHole:MountingHole_3.2mm_M3_Pad_Via, F.Cu at (120.7, 136.2)
- added H4: M3, MountingHole:MountingHole_3.2mm_M3_Pad_Via, F.Cu at (191.7, 136.2)
- C201: footprint Capacitor_SMD:C_0402_1005Metric -> Capacitor_SMD:C_0201_0603Metric; moved to B.Cu
- C205, C219, C234, C248, C258, C404, C405, C407, C408, C410, C413, C502, C503, C507, C508, C510, C511, C513, C605, C609, C610, C611, C612, C613, C614, D602, FB401, FB402, FB501, FB502, R403, R405, R406, R501, R503, R505, R506, R610, R611, R612, R701, R702, R703, R704, R705, R706, R707, R708, R709, R710, R711, R712, R713, R714, R715, R716, R717, R718, Y1: moved to B.Cu
- C409, C412, C509, C512: footprint Capacitor_SMD:C_0805_2012Metric -> Capacitor_SMD:C_0603_1608Metric; moved to B.Cu
- FB201: footprint Inductor_SMD:L_0402_1005Metric -> Inductor_SMD:L_0201_0603Metric; moved to B.Cu
- U301: footprint Package_SON:WSON-8-1EP_8x6mm_P1.27mm_EP3.4x4.3mm -> Custom_VoxLink_Footprints:WSON-8-1EP_8.0x6.0mm_P1.27mm_EP4.7x4.6mm
- moved R707 163.6 mm to (184.8, 107.6)
- moved R713 161.9 mm to (184.8, 127.1)
- moved R710 160.7 mm to (184.8, 96.4)
- moved R718 159.9 mm to (184.8, 76.9)
- moved R716 158.7 mm to (184.8, 115.9)
- moved R711 158.2 mm to (180.0, 129.3), turned to -90 degrees
- moved R715 158.0 mm to (184.8, 88.1)
- moved R708 148.3 mm to (168.8, 129.3), turned to -90 degrees
- moved C501 143.6 mm to (138.7, 73.8)
- moved C401 142.6 mm to (151.4, 73.8)
- moved R501 142.4 mm to (141.8, 79.5), turned to -90 degrees
- moved R705 141.5 mm to (160.5, 129.3), turned to -90 degrees
- moved R401 141.1 mm to (154.7, 79.3), turned to 180 degrees
- moved R404 137.4 mm to (149.2, 73.8), turned to 90 degrees
- moved R504 136.6 mm to (136.4, 73.8), turned to 90 degrees
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Connections:
- U201 pad A15: unconnected-(U201D-IO_L8P_T1_AD10P_15-PadA15) -> P9_L2
- U201 pad A16: unconnected-(U201D-IO_L8N_T1_AD10N_15-PadA16) -> P9_L1
- U201 pad K3: unconnected-(U201F-IO_L2P_T0_34-PadK3) -> P7_L2
- U201 pad L3: unconnected-(U201F-IO_L2N_T0_34-PadL3) -> P7_L1
- U201 pad P17: unconnected-(U201C-IO_L12P_T1_MRCC_14-PadP17) -> P2_L2
- U201 pad P4: unconnected-(U201F-IO_L14P_T2_SRCC_34-PadP4) -> P8_L1
- U201 pad P5: unconnected-(U201F-IO_L13N_T2_MRCC_34-PadP5) -> P8_L2
- U201 pad R15: unconnected-(U201C-IO_L13N_T2_MRCC_14-PadR15) -> P3_L1
- U201 pad R16: unconnected-(U201C-IO_L15P_T2_DQS_RDWR_B_14-PadR16) -> P3_L2
- U201 pad R17: unconnected-(U201C-IO_L12N_T1_MRCC_14-PadR17) -> P2_L1
- U201 pad T10: unconnected-(U201C-IO_L24N_T3_A00_D16_14-PadT10) -> P4_L2
- U201 pad T14: unconnected-(U201C-IO_L14P_T2_SRCC_14-PadT14) -> P5_L1
- U201 pad T15: unconnected-(U201C-IO_L14N_T2_SRCC_14-PadT15) -> P5_L2
- U201 pad T9: unconnected-(U201C-IO_L24P_T3_A01_D17_14-PadT9) -> P4_L1
- U201 pad U3: unconnected-(U201F-IO_L8N_T1_34-PadU3) -> P1_L1
- U201 pad U4: unconnected-(U201F-IO_L8P_T1_34-PadU4) -> P1_L2
- U201 pad U6: unconnected-(U201F-IO_L22N_T3_34-PadU6) -> P6_L1
- U201 pad U7: unconnected-(U201F-IO_L22P_T3_34-PadU7) -> P6_L2
- U602 pad 1: JTAG_D- -> SERIAL_D-
- U602 pad 2: JTAG_D+ -> SERIAL_D+
- U602 pad 3: SERIAL_D- -> JTAG_D-
- U602 pad 4: SERIAL_D+ -> JTAG_D+
Routing:
- net /FPGA_Config/FPGA_DONE: track 0.00 -> 108.2 mm, vias 0 -> 2
- net /FPGA_Config/FPGA_RST: track 0.00 -> 105.8 mm, vias 0 -> 2
- net P7_L1: track 0.00 -> 66.3 mm, vias 0 -> 1
- net P9_L2: track 0.00 -> 50.7 mm, vias 0 -> 1
- net P7_L2: track 0.00 -> 46.7 mm, vias 0 -> 1
- net P8_L1: track 0.00 -> 41.1 mm, vias 0 -> 1
- net P9_L1: track 0.00 -> 39.2 mm, vias 0 -> 1
- net GND: track 33.4 -> 71.8 mm, vias 97 -> 164
- net P2_L2: track 0.00 -> 38.1 mm, vias 0 -> 1
- net P3_L1: track 0.00 -> 32.1 mm, vias 0 -> 1
- net P8_L2: track 0.00 -> 32.1 mm, vias 0 -> 1
- net +3V3: track 21.4 -> 52.8 mm, vias 29 -> 50
- net P6_L1: track 0.00 -> 30.3 mm, vias 0 -> 1
- net P2_L1: track 0.00 -> 28.0 mm, vias 0 -> 1
- net P5_L2: track 0.00 -> 26.7 mm, vias 0 -> 1
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