File: Hardware/Controller_Board/power.kicad_sch (KiCad schematic)
At the start: 33 parts, among them Q1 DMN2400UFB-7, U2 TPS82084, U3 LT8645S, U4 TPS82084, U5 TPS82084, U6 XT30

Commit message: Updated the domcumentation
Parts:
- added D308: LED, LED_SMD:LED_0603_1608Metric, symbol Device:LED
- added R13: 280R, Resistor_SMD:R_0402_1005Metric, symbol Device:R
Connections:
- net +5V: now also R13.1
- net GND: now also Q1.2 (S)
- net PG_3V3: now also Q1.1 (G)
- net at Q1.3 (D): now also D308.1 (K)
- new net: D308.2 (A), R13.2
Other:
- moved on the sheet: Q1

Commit message: Commited Schematic Changes
Parts:
- added C69, C70, C71: 100u, Capacitor_SMD:CP_Elec_8x6.5, symbol Device:C_Polarized
- C11, C12: value 0.47u -> 470n
Connections:
- net +1V0: now also C69.1
- net +1V8: now also C70.1
- net +3V3: now also C71.1
- net GND: now also C69.2, C70.2, C71.2
Other:
- moved on the sheet: C1, C10, C11, C12, C13, C8, C9, D301, D308, L4, Q1, R13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

Commit message: Commited Schematic Changes
Parts:
- D301: footprint Diode_SMD:D_0402_1005Metric -> (none)
Other:
- moved on the sheet: C1, C10, C11, C12, C13, C2, C3, C4, C5, C6, C69, C7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

Commit message: Updated schematic diagram with configuration
Parts:
- L4: footprint Inductor_SMD:L_Coilcraft_XAL6060-XXX -> Inductor_SMD:L_Coilcraft_XAL6030-XXX
Other:
- moved on the sheet: C1, C10, C11, C12, C13, C8, C9, D301, D308, L4, Q1, R13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

Commit message: Added USB hub symbol
Parts:
- renumbered C13 to C1, C1 to C10, C4 to C11, C5 to C12, C70 to C13, C6 to C14, C7 to C15, C71 to C16, C12 to C2, C11 to C3, C10 to C4, C9 to C5, C8 to C6, C2 to C7, C3 to C8, C69 to C9, D308 to D1, D301 to D2, L4 to L1, R7 to R1, R1 to R3, R8 to R4, R3 to R5, R9 to R6, R4 to R7, R5 to R8, R6 to R9, U2 to U1, U3 to U2, U4 to U3, U5 to U4, U6 to U5

Commit message: Updated the schematic design - Fix the XC7A35T-CPG236 outline issue
Other:
- moved on the sheet: C1, C10, C2, C3, C4, C5, C6, D1, D2, L1, Q1, R1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

Commit message: Finished schematic design - preparation for review
Parts:
- D2: footprint (none) -> Diode_THT:D_DO-201AE_P15.24mm_Horizontal
Changed lines of the file:
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@@
 			)
 		)
-		(property "Datasheet" "https://jlcpcb.com/partdetail/Coilcraft-XGL6030222MEC/C3911448"
+		(property "Datasheet" "~"
 			(at 116.84 71.12 0)
 			(effects
@@
 			)
 		)
-		(property "Footprint" ""
+		(property "Footprint" "Diode_THT:D_DO-201AE_P15.24mm_Horizontal"
 			(at 62.23 140.97 0)
 			(effects
@@
 			)
 		)
-		(property "Datasheet" ""
+		(property "Datasheet" "https://www.vishay.com/docs/88301/15ke.pdf"
 			(at 67.31 139.7 0)
 			(effects
@@
 			)
 		)
-		(property "Description" ""
+		(property "Description" "1500W unidirectional TVS diode, DO-201AE"
 			(at 67.31 140.97 0)
 			(effects

Commit message: Finished DRC check. Moving to schematic review
Parts:
- removed U2: LT8645S, Custom_VoxLink_Footprints:LT8645S, symbol Custom_VoxLink_Symbols:LT8645S
- added U102: LT8645S, Custom_VoxLink_Footprints:LQFN-32-6EP_6x4mm_P0.5mm_EP1.355x1.125mm, symbol Custom_VoxLink_Symbols:LT8645S
- renumbered C7 to C101, C8 to C102, C9 to C103, C1 to C104, C2 to C105, C3 to C106, C4 to C107, C5 to C108, C6 to C109, C10 to C110, C11 to C111, C12 to C112, C13 to C113, C14 to C114, C15 to C115, C16 to C116, D1 to D101, D2 to D102, L1 to L101, Q1 to Q101, R2 to R101, R3 to R102, R5 to R103, R1 to R104, R4 to R105, R6 to R106, R7 to R107, R8 to R108, R9 to R109, R13 to R110, R10 to R111, R11 to R112, R12 to R113, U1 to U101, U3 to U103, U4 to U104, U5 to U105
Connections:
- net +5V: now also U101.4 (VIN), U103.4 (VIN), U104.4 (VIN), U102.1 (BIAS)
- net FB_5V0: now also U102.32 (FB)
- net GND: now also U101.6 (GND), U101.9 (GND), U103.6 (GND), U103.9 (GND), U104.6 (GND), U104.9 (GND), U102.10 (GND), U102.17 (GND), U102.18 (GND), U102.19 (GND), U102.33 (GND), U102.34 (GND), U102.35 (GND), U102.36 (GND), U102.37 (GND), U102.38 (GND), U102.8 (GND), U102.9 (GND)
- net SW_5V0: now also U102.12 (SW), U102.13 (SW), U102.14 (SW), U102.15 (SW), U102.16 (SW)
- net TR/SS: now also U102.29 (TR/SS)
- net VIN: now also C104.1, C105.1, C106.1, U102.21 (VIN), U102.22 (VIN), U102.23 (VIN), U102.25 (EN/UV), U102.4 (VIN), U102.5 (VIN), U102.6 (VIN)
- net at R106.1: now also U102.26 (RT)
- new net: U102.20 (NC), U102.24 (NC), U102.3 (NC), U102.7 (NC)
- no-connect marks 0 -> 7
