File: Hardware/Controller_Board/power.kicad_sch (KiCad schematic)
At the start: 38 parts, among them Q101 DMN2400UFB-7, U101 TPS82084, U102 LT8645S, U103 TPS82084, U104 TPS82084, U105 XT30

Commit message: Finished the schematic review
Parts:
- removed D102: TVS, Diode_THT:D_DO-201AE_P15.24mm_Horizontal, symbol Diode:1.5KExxA
- added C104: 10u, Capacitor_SMD:C_1210_3225Metric, symbol Device:C
- added D101: TVS/Zener, Diode_SMD:D_0603_1608Metric, symbol Device:D_Zener
- added D103: D_TVS, Diode_SMD:D_0402_1005Metric, symbol Device:D_TVS
- added R105: 1R, Resistor_SMD:R_0603_1608Metric, symbol Device:R
- added U103: TDS5311P, Package_DFN_QFN:DFN-6-1EP_2x2mm_P0.65mm_EP1x1.6mm, symbol Custom_VoxLink_Symbols:TDS5311P
- C103: footprint Capacitor_SMD:CP_Elec_8x6.5 -> Capacitor_SMD:CP_Elec_5x5.9
- C105: renamed from C104; footprint Capacitor_SMD:C_0805_2012Metric -> Capacitor_SMD:C_1210_3225Metric
- C106: renamed from C105; value 470n -> 100n; footprint Capacitor_SMD:C_0402_1005Metric -> Capacitor_SMD:C_0805_2012Metric
- C107: renamed from C106; value 470n -> 100n; footprint Capacitor_SMD:C_0402_1005Metric -> Capacitor_SMD:C_0805_2012Metric
- C109: renamed from C108; footprint Capacitor_SMD:CP_Elec_8x6.5 -> Capacitor_SMD:CP_Elec_5x5.9
- C111: renamed from C110; value 100n -> 10n; now fitted
- C114: renamed from C113; footprint Capacitor_SMD:CP_Elec_8x6.5 -> Capacitor_SMD:CP_Elec_5x5.9
- C117: renamed from C116; footprint Capacitor_SMD:CP_Elec_8x6.5 -> Capacitor_SMD:CP_Elec_5x5.9
- renumbered C107 to C108, C109 to C110, C111 to C112, C112 to C113, C114 to C115, C115 to C116, D101 to D102, R105 to R106, R106 to R107, R107 to R108, R108 to R109, R109 to R110, R110 to R111, R111 to R112, R112 to R113, R113 to R114, U103 to U104, U104 to U105, U105 to U106
Connections:
- net GND: now also U106.1 (GND), D101.2 (A), D103.1 (A1), R105.2, U103.4 (GND), U103.5 (GND), U103.6 (GND), U103.7 (GND); no longer U106.2 (GND)
- net VIN: now also U106.2 (VIN), C104.1, D101.1 (K), D103.2 (A2), U103.1 (VIN), U103.2 (VIN), U103.3 (VIN); no longer U106.1 (VIN)
- new net: C104.2, R105.1
Other:
- note added: "10mA through the LED"
- note added: "5ms soft-start"
- note added: "MAX VIN is 48V!"
- note removed: "Check the inrush current on the 10u cap!"
- moved on the sheet: C105, C106, C107, C108, C109, C110, L101, R104, R106, R107, U102

Commit message: Updated the documentation + minor scheme changes - Documented the schematic design - Added zener diode from USB VBUS to 5V
Parts:
- D103: value D_TVS -> TVS
Changed lines of the file:
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@@
 			)
 		)
-		(property "Value" "D_TVS"
+		(property "Value" "TVS"
 			(at 69.342 142.24 90)
 			(effects

Commit message: Started schematic rework and the PCB design
Connections:
- net GND: now also U102.39 (GND), U102.40 (GND), U102.41 (GND), U102.42 (GND)
Changed lines of the file:
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@@
 		(pin "30"
+		)
+		(pin "42"
+		)
+		(pin "41"
+		)
+		(pin "39"
+		)
+		(pin "40"
 		)
 		(instances

Commit message: Advanced PCB design: Advanced power routing
Parts:
- removed C103, C109, C114, C117: 100u, Capacitor_SMD:CP_Elec_5x5.9, symbol Device:C_Polarized
- added C109, C114, C117, C118, C119, C120, C121, C122, C123, C124, C125, C126, C127, C128, C129, C130: 100u, Capacitor_SMD:C_1206_3216Metric, symbol Device:C
- C101, C112, C115: value 10u -> 22u; footprint Capacitor_SMD:C_0805_2012Metric -> Capacitor_SMD:C_0603_1608Metric
- C102, C113, C116: footprint Capacitor_SMD:C_1210_3225Metric -> Capacitor_SMD:C_0603_1608Metric
- C104, C105: footprint Capacitor_SMD:C_1210_3225Metric -> Capacitor_SMD:C_1206_3216Metric
- C108: footprint Capacitor_SMD:C_1210_3225Metric -> Capacitor_SMD:C_0805_2012Metric
Connections:
- net +1V0: now also C117.1, C118.1
- net +1V8: now also C119.1, C120.1
- net +3V3: now also C121.1, C122.1
- net +5V: now also C109.1, C114.1, C123.1, C124.1, C125.1, C126.1, C127.1, C128.1, C129.1, C130.1
- net GND: now also C109.2, C114.2, C117.2, C118.2, C119.2, C120.2, C121.2, C122.2, C123.2, C124.2, C125.2, C126.2, C127.2, C128.2, C129.2, C130.2

Commit message: Advanced PCB Design: Routing Power + UVLO
Parts:
- removed D101: TVS/Zener, Diode_SMD:D_0603_1608Metric, symbol Device:D_Zener
- removed D103: TVS, Diode_SMD:D_0402_1005Metric, symbol Device:D_TVS
- added C131, C132: 22u, Capacitor_SMD:C_0603_1608Metric, symbol Device:C
- added C133, C134: 100u, Capacitor_SMD:C_1206_3216Metric, symbol Device:C
- added C135, C136: 100n, Capacitor_SMD:C_0805_2012Metric, symbol Device:C
- added Q2: Si7252ADP, Package_SO:PowerPAK_SO-8_Dual, symbol Transistor_FET:Q_Dual_NMOS_S1G1S2G2D2D1
- added R115: 499k, Resistor_SMD:R_0402_1005Metric, symbol Device:R
- added R116: 156.3k, Resistor_SMD:R_0402_1005Metric, symbol Device:R
- added R117: 50k, Resistor_SMD:R_0402_1005Metric, symbol Device:R
- added R118, R119, R120, R121, R122: 41.2k, Resistor_SMD:R_0402_1005Metric, symbol Device:R
- added U1: LTC4368, Package_DFN_QFN:DFN-10-1EP_3x3mm_P0.5mm_EP1.65x2.38mm, symbol Custom_VoxLink_Symbols:LTC4368
- added U107: TPS82084, Package_LGA:Texas_SIL0008C_MicroSiP-8-1EP_2.8x3mm_P0.65mm_EP1.1x1.9mm, symbol Custom_VoxLink_Symbols:TPS82084
- R113: value 156.3k -> 106.3k
Connections:
- net +3V3: now also C132.1, C133.1, C134.1, R116.1, U107.8 (VOUT); no longer C116.1, C121.1, C122.1, R113.1, U105.8 (VOUT)
- net +5V: now also C131.1, R115.1, U107.3 (VIN), U107.4 (VIN)
- net FB_3V3: now also R116.2, R117.1, U107.7 (FB); no longer R113.2, R114.1, U105.7 (FB)
- net GND: now also C131.2, C132.2, C133.2, C134.2, C135.2, C136.2, R117.2, R121.2, U1. (RETRY), U107.5 (GND), U107.6 (GND), U107.9 (GND)
- net PG_3V3: now also R115.2, U107.2 (PG); no longer R112.2, U105.2 (PG)
- net VIN: now also C136.1, Q2.5 (D), R120.1, U1. (RETRY); no longer C105.1, C106.1, C107.1, U102.21 (VIN), U102.22 (VIN), U102.23 (VIN), U102.25 (EN/UV), U102.4 (VIN), U102.5 (VIN), U102.6 (VIN)
- new net: R119.1, R120.2, U1. (RETRY)
- new net: R118.1, R119.2, U1. (RETRY)
- new net: R118.2, R121.1, U1. (RETRY)
- new net: C135.1, R122.2
- new net: Q2.1 (S), Q2.3 (S)
- new net +2V5: C116.1, C121.1, C122.1, R113.1, U105.8 (VOUT)
- new net FB_2V5: R113.2, R114.1, U105.7 (FB)
- new net PG_2V5: R112.2, U105.2 (PG), U107.1 (EN)
- new net UVLO_GATE: Q2.2 (G), Q2.4 (G), R122.1, U1. (RETRY)
- new net VREG_IN: C105.1, C106.1, C107.1, Q2.6 (D), U1. (RETRY), U102.21 (VIN), U102.22 (VIN), U102.23 (VIN), U102.25 (EN/UV), U102.4 (VIN), U102.5 (VIN), U102.6 (VIN)
- no-connect marks 7 -> 9
Other:
- note added: "Place at Ethernet connectors"
- moved on the sheet: C101, C102, C104, C105, C106, C107, C108, C109, C110, C111, C112, C113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

Commit message: Finished PCB Design - WARNING MORE CHANGES NEEDED! The main decision to be made is, whether to increase the layer count to 8 layers, and make the P7 and P8 permamently on 3V3
Parts:
- removed C104: 10u, Capacitor_SMD:C_1206_3216Metric, symbol Device:C
- removed C135, C136: 100n, Capacitor_SMD:C_0805_2012Metric, symbol Device:C
- removed Q2: Si7252ADP, Package_SO:PowerPAK_SO-8_Dual, symbol Transistor_FET:Q_Dual_NMOS_S1G1S2G2D2D1
- removed R105: 1R, Resistor_SMD:R_0603_1608Metric, symbol Device:R
- removed R118, R119, R120, R121, R122: 41.2k, Resistor_SMD:R_0402_1005Metric, symbol Device:R
- removed U1: LTC4368, Package_DFN_QFN:DFN-10-1EP_3x3mm_P0.5mm_EP1.65x2.38mm, symbol Custom_VoxLink_Symbols:LTC4368
- removed U103: TDS5311P, Package_DFN_QFN:DFN-6-1EP_2x2mm_P0.65mm_EP1x1.6mm, symbol Custom_VoxLink_Symbols:TDS5311P
- removed U106: XT30, Connector_AMASS:AMASS_XT30PW-M_1x02_P2.50mm_Horizontal, symbol Custom_VoxLink_Symbols:Conn_XT
- renumbered C101 to C201, C102 to C202, C117 to C203, C118 to C204, C129 to C205, C130 to C206, C127 to C207, C128 to C208, C125 to C209, C126 to C210, C123 to C211, C124 to C212, C112 to C213, C113 to C214, C119 to C215, C120 to C216, C108 to C217, C109 to C218, C114 to C219, C105 to C220, C106 to C221, C107 to C222, C110 to C223, C111 to C224, C115 to C225, C116 to C226, C121 to C227, C122 to C228, C131 to C229, C132 to C230, C133 to C231, C134 to C232, D102 to D201, L101 to L201, Q101 to Q201, R101 to R201, R102 to R202, R103 to R203, R108 to R204, R109 to R205, R104 to R206, R110 to R207, R106 to R208, R107 to R209, R112 to R210, R113 to R211, R114 to R212, R111 to R213, R115 to R214, R116 to R215, R117 to R216, U101 to U201, U104 to U202, U102 to U203, U105 to U204, U107 to U205
Connections:
- no-connect marks 9 -> 7
Other:
- note added: "MAX VIN is 48V! MAX CURRENT IS 3A!"
- note added: "Power [2]"
- note removed: "MAX VIN is 48V!"
- note removed: "Power [1]"
- moved on the sheet: C201, C202, C203, C204, C205, C206, C207, C208, C209, C210, C211, C212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

Commit message: Finished procuring almost all boards - CHANGED XDC IN XILINX FOR TESTING!! - Programmer needed
Parts:
- C201, C202, C213, C214, C225, C226, C229, C230: LCSC (none) -> C5116073; Manufacturer (none) -> Murata
- C203, C204, C205, C206, C207, C208, C209, C210, C211, C212, C215, C216, C218, C219, C227, C228, C231, C232: LCSC (none) -> C883598; Manufacturer (none) -> Murata
- C217: LCSC (none) -> C86816; Manufacturer (none) -> Murata
- C220: value 10u -> 4.7u; LCSC (none) -> C2997285; Manufacturer (none) -> Murata
- C221, C222: LCSC (none) -> C85866; Manufacturer (none) -> Murata
- C223: LCSC (none) -> C88886; Manufacturer (none) -> Murata
- C224: LCSC (none) -> C77019; Manufacturer (none) -> Murata
- D201: LCSC (none) -> C18198801; Manufacturer (none) -> Broadcom
- L201: LCSC (none) -> C3911448; Manufacturer (none) -> Coilcraft
- R201, R204, R210, R214: LCSC (none) -> C482187; Manufacturer (none) -> Vishay
- R202: value 12.5k -> 12.4k; LCSC (none) -> C1730790; Manufacturer (none) -> Vishay
- R203, R207, R212, R216: value 50k -> 49.9k; LCSC (none) -> C350874; Manufacturer (none) -> Vishay
- R205: value 62.5k -> 61.9k; LCSC (none) -> C4023393; Manufacturer (none) -> Vishay
- R206: LCSC (none) -> C4334825; Manufacturer (none) -> Vishay
- R208: LCSC (none) -> C2092035; Manufacturer (none) -> Vishay
- R209: LCSC (none) -> C844310; Manufacturer (none) -> Vishay
- R211: value 106.3k -> 154k; LCSC (none) -> C2085327; Manufacturer (none) -> Vishay
- R213: LCSC (none) -> C4193696; Manufacturer (none) -> Vishay
- R215: value 156.3k -> 154k; LCSC (none) -> C2085327; Manufacturer (none) -> Vishay
- U201, U202, U204, U205: LCSC (none) -> C468248; Manufacturer (none) -> TI
- U203: LCSC (none) -> C674140; Manufacturer (none) -> ADI
Other:
- note added: "WARNING! In the current version, the IO supply is 3V3! Net +2V5 is present to allow LVDS operation. For 2V5 operation, please put closest to 106.3kOhm resistor as R211!"
