File: Hardware/Controller_Board/power.kicad_sch (KiCad schematic)
At the start: 56 parts, among them Q201 DMN2400UFB-7, U201 TPS82084, U202 TPS82084, U203 LT8645S, U204 TPS82084, U205 TPS82084

Commit message: Finished PCB design and Review + Procured Boards
Parts:
- Q201: LCSC (none) -> C154757
Changed lines of the file:
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@@
 			)
 		)
-		(property "LCSC" ""
+		(property "LCSC" "C154757"
 			(at 41.91 162.56 0)
 			(hide yes)
