File: Hardware/Controller_Board/fpga_power.kicad_sch (KiCad schematic)
At the start: 58 parts, among them U201 XC7A35T-CPG236

Commit message: Started schematic rework and the PCB design
Parts:
- removed C201: 100n, Capacitor_SMD:C_0402_1005Metric, symbol Device:C
- removed C202: 10p, Capacitor_SMD:C_0402_1005Metric, symbol Device:C
- removed C203, C204, C207, C208, C209, C210, C211, C212, C221, C222, C223, C224, C225, C226, C229, C230, C231, C232, C233, C234, C237, C238, C239, C240, C241, C242, C247, C248, C249, C250, C251, C252, C253, C254: 100n, Capacitor_SMD:C_0201_0603Metric, symbol Device:C
- removed C205, C213, C214, C215, C218, C219, C220, C228, C235, C243, C246, C255: 1u, Capacitor_SMD:C_0402_1005Metric, symbol Device:C
- removed C206, C216, C217, C227, C236, C244, C245, C256: 10u, Capacitor_SMD:C_0805_2012Metric, symbol Device:C
- removed FB201: 600R/100MHz, Inductor_SMD:L_0402_1005Metric, symbol Device:FerriteBead
- removed U201: XC7A35T-CPG236, Package_BGA:Xilinx_CPG236, symbol Custom_VoxLink_Symbols:XC7A35T-CPG236
- added C257, C258, C261, C262, C263, C264, C265, C266, C269, C270, C271, C272, C273, C274, C277, C280, C281, C282, C283, C284, C285, C288, C289, C290, C291, C292, C293, C298, C299, C300, C304, C305, C306, C313, C314, C315, C316, C317, C318, C319, C320, C321, C322, C323, C324: 100n, Capacitor_SMD:C_0201_0603Metric, symbol Device:C
- added C259, C267, C275, C278, C286, C294, C297, C307, C310, C311, C312: 1u, Capacitor_SMD:C_0402_1005Metric, symbol Device:C
- added C260, C268, C276, C279, C287, C295, C296, C308, C309: 10u, Capacitor_SMD:C_0805_2012Metric, symbol Device:C
- added C325: 100n, Capacitor_SMD:C_0402_1005Metric, symbol Device:C
- added C326: 10p, Capacitor_SMD:C_0402_1005Metric, symbol Device:C
- added FB202: 600R/100MHz, Inductor_SMD:L_0402_1005Metric, symbol Device:FerriteBead
- added U202: XC7A35T-CSG324, Package_BGA:Xilinx_CSG324, symbol Custom_VoxLink_Symbols:XC7A35T-CSG324
Connections:
- net +1V0: now also C296.1, C297.1, C298.1, C299.1, C309.1, C310.1, C311.1, C312.1, C313.1, C314.1, C315.1, C316.1, C317.1, C318.1, C319.1, C320.1, C321.1, C322.1, C323.1, C324.1, U202.F10 (VCCBRAM), U202.F8 (VCCINT), U202.G11 (VCCBRAM), U202.G7 (VCCINT), U202.G9 (VCCINT), U202.H8 (VCCINT), U202.J11 (VCCINT), U202.J7 (VCCINT), U202.K8 (VCCINT), U202.L11 (VCCINT), U202.L7 (VCCINT), U202.M10 (VCCINT), U202.M8 (VCCINT), U202.N11 (VCCINT), U202.N7 (VCCINT), U202.N9 (VCCINT)
- net +1V8: now also C300.1, C304.1, C305.1, C306.1, C307.1, C308.1, FB202.1, U202.E8 (VCCBATT_0), U202.F12 (VCCAUX), U202.H12 (VCCAUX), U202.K12 (VCCAUX), U202.M12 (VCCAUX)
- net +3V3: now also C257.1, C258.1, C259.1, C260.1, C261.1, C262.1, C263.1, C264.1, C265.1, C266.1, C267.1, C268.1, C269.1, C270.1, C271.1, C272.1, C273.1, C274.1, C275.1, C276.1, C277.1, C278.1, C279.1, C280.1, C281.1, C282.1, C283.1, C284.1, C285.1, C286.1, C287.1, C288.1, C289.1, C290.1, C291.1, C292.1, C293.1, C294.1, C295.1, U202.A17 (VCCO_15), U202.A7 (VCCO_35), U202.B10 (VCCO_16), U202.C13 (VCCO_15), U202.C3 (VCCO_35), U202.D16 (VCCO_15), U202.D6 (VCCO_35), U202.F2 (VCCO_35), U202.G15 (VCCO_15), U202.G5 (VCCO_35), U202.H18 (VCCO_15), U202.J1 (VCCO_35), U202.K14 (VCCO_15), U202.K4 (VCCO_34), U202.L17 (VCCO_14), U202.N13 (VCCO_14), U202.N3 (VCCO_34), U202.P16 (VCCO_14), U202.P6 (VCCO_34), U202.R9 (VCCO_0), U202.T12 (VCCO_14), U202.T2 (VCCO_34), U202.U15 (VCCO_14), U202.U5 (VCCO_34), U202.V18 (VCCO_14), U202.V8 (VCCO_34)
- net GND: now also C257.2, C258.2, C259.2, C260.2, C261.2, C262.2, C263.2, C264.2, C265.2, C266.2, C267.2, C268.2, C269.2, C270.2, C271.2, C272.2, C273.2, C274.2, C275.2, C276.2, C277.2, C278.2, C279.2, C280.2, C281.2, C282.2, C283.2, C284.2, C285.2, C286.2, C287.2, C288.2, C289.2, C290.2, C291.2, C292.2, C293.2, C294.2, C295.2, C296.2, C297.2, C298.2, C299.2, C300.2, C304.2, C305.2, C306.2, C307.2, C308.2, C309.2, C310.2, C311.2, C312.2, C313.2, C314.2, C315.2, C316.2, C317.2, C318.2, C319.2, C320.2, C321.2, C322.2, C323.2, C324.2, C325.2, C326.2, U202.A12 (GND), U202.A2 (GND), U202.B15 (GND), U202.B5 (GND), U202.C18 (GND), U202.C8 (GND), U202.D1 (GND), U202.D11 (GND), U202.E14 (GND), U202.E4 (GND), U202.F11 (GND), U202.F17 (GND), U202.F7 (GND), U202.F9 (GND), U202.G10 (GND), U202.G12 (GND), U202.G8 (GND), U202.H11 (GND), U202.H13 (GND), U202.H3 (GND), U202.H7 (GND), U202.H9 (GNDADC_0), U202.J12 (GND), U202.J16 (GND), U202.J6 (GND), U202.J8 (GND), U202.K11 (GND), U202.K7 (GND), U202.L12 (GND), U202.L2 (GND), U202.L8 (GND), U202.M11 (GND), U202.M15 (GND), U202.M5 (GND), U202.M7 (GND), U202.M9 (GND), U202.N10 (GND), U202.N12 (GND), U202.N18 (GND), U202.N8 (GND), U202.P1 (GND), U202.R14 (GND), U202.R4 (GND), U202.T17 (GND), U202.T7 (GND), U202.U10 (GND), U202.V13 (GND), U202.V3 (GND)
- new net: C325.1, C326.1, FB202.2, U202.H10 (VCCADC_0)

Commit message: Commit before upgrading to KiCad 10.0
Parts:
- removed C259, C267, C275, C278, C286, C294, C297, C307, C310, C311, C312: 1u, Capacitor_SMD:C_0402_1005Metric, symbol Device:C
- added C220, C221: 100n, Capacitor_SMD:C_0201_0603Metric, symbol Device:C
- C205: renamed from C260; footprint Capacitor_SMD:C_0805_2012Metric -> Capacitor_SMD:C_0603_1608Metric
- C206: renamed from C309; footprint Capacitor_SMD:C_0805_2012Metric -> Capacitor_SMD:C_0603_1608Metric
- C219: renamed from C268; footprint Capacitor_SMD:C_0805_2012Metric -> Capacitor_SMD:C_0603_1608Metric
- C234: renamed from C276; footprint Capacitor_SMD:C_0805_2012Metric -> Capacitor_SMD:C_0603_1608Metric
- C237: renamed from C308; footprint Capacitor_SMD:C_0805_2012Metric -> Capacitor_SMD:C_0603_1608Metric
- C248: renamed from C287; footprint Capacitor_SMD:C_0805_2012Metric -> Capacitor_SMD:C_0603_1608Metric
- C249: renamed from C296; footprint Capacitor_SMD:C_0805_2012Metric -> Capacitor_SMD:C_0603_1608Metric
- C258: renamed from C295; footprint Capacitor_SMD:C_0805_2012Metric -> Capacitor_SMD:C_0603_1608Metric
- renumbered C325 to C201, C326 to C202, C257 to C203, C258 to C204, C313 to C207, C314 to C208, C315 to C209, C316 to C210, C317 to C211, C318 to C212, C261 to C213, C262 to C214, C263 to C215, C264 to C216, C265 to C217, C266 to C218, C319 to C222, C320 to C223, C321 to C224, C322 to C225, C323 to C226, C324 to C227, C269 to C228, C270 to C229, C271 to C230, C272 to C231, C273 to C232, C274 to C233, C277 to C235, C279 to C236, C306 to C238, C305 to C239, C304 to C240, C300 to C241, C280 to C242, C281 to C243, C282 to C244, C283 to C245, C284 to C246, C285 to C247, C298 to C250, C299 to C251, C288 to C252, C289 to C253, C290 to C254, C291 to C255, C292 to C256, C293 to C257, FB202 to FB201, U202 to U201
Connections:
- net +1V0: now also C220.1, C221.1
- net GND: now also C220.2, C221.2
Other:
- moved on the sheet: C205, C206, C219, C234, C236, C237, C248, C249, C258

Commit message: Advanced PCB design: Routed FTDIs + SPI Flash
Parts:
- removed C228: 100n, Capacitor_SMD:C_0201_0603Metric, symbol Device:C
Changed lines of the file:
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@@
 	)
 	(junction
-		(at 185.42 85.09)
-		(diameter 0)
-		(color 0 0 0 0)
-	)
-	(junction
 		(at 76.2 107.95)
 		(diameter 0)
@@
 	(wire
 		(pts
-			(xy 185.42 86.36) (xy 185.42 85.09)
-		)
-		(stroke
-			(width 0)
-			(type default)
-		)
-	)
-	(wire
-		(pts
 			(xy 66.04 67.31) (xy 55.88 67.31)
 		)
@@
 	(wire
 		(pts
-			(xy 185.42 85.09) (xy 195.58 85.09)
-		)
-		(stroke
-			(width 0)
-			(type default)
-		)
-	)
-	(wire
-		(pts
 			(xy 236.22 120.65) (xy 246.38 120.65)
 		)
@@
 	(wire
 		(pts
-			(xy 173.99 85.09) (xy 185.42 85.09)
+			(xy 173.99 85.09) (xy 195.58 85.09)
 		)
 		(stroke
@@
 	)
 	(symbol
-		(lib_id "Device:C")
-		(at 185.42 90.17 0)
-		(mirror y)
-		(unit 1)
-		(body_style 1)
-		(exclude_from_sim no)
-		(in_bom yes)
-		(on_board yes)
-		(in_pos_files yes)
-		(dnp no)
-		(property "Reference" "C228"
-			(at 182.88 88.9 0)
-			(show_name no)
-			(do_not_autoplace no)
-			(effects
-				(font
-					(size 1.27 1.27)
-				)
-				(justify left)
-			)
-		)
-		(property "Value" "100n"
-			(at 182.88 91.44 0)
-			(show_name no)
-			(do_not_autoplace no)
-			(effects
-				(font
-					(size 1.27 1.27)
-				)
-				(justify left)
-			)
-		)
-		(property "Footprint" "Capacitor_SMD:C_0201_0603Metric"
-			(at 184.4548 93.98 0)
-			(hide yes)
-			(show_name no)
-			(do_not_autoplace no)
-			(effects
-				(font
-					(size 1.27 1.27)
-				)
-			)
-		)
-		(property "Datasheet" ""
-			(at 185.42 90.17 0)
-			(hide yes)
-			(show_name no)
-			(do_not_autoplace no)
-			(effects
-				(font
-					(size 1.27 1.27)
-				)
-			)
-		)
-		(property "Description" "Unpolarized capacitor"
-			(at 185.42 90.17 0)
-			(hide yes)
-			(show_name no)
-			(do_not_autoplace no)
-			(effects
-				(font
-					(size 1.27 1.27)
-				)
-			)
-		)
-		(pin "2"
-		)
-		(pin "1"
-		)
-		(instances
-			(project "Controller_Board"
-				(path "/4e6e1af1-ede9-4a56-9d5f-a8dfd7fbcf8d/77637722-5c93-4eaa-a1cc-47897016a2a9"
-					(reference "C228")
-					(unit 1)
-				)
-			)
-		)
-	)
-	(symbol
 		(lib_id "power:GND")
 		(at 106.68 76.2 0)
@@
 					(unit 1)
 				)
-			)
-		)
-	)
-	(symbol
-		(lib_id "power:GND")
-		(at 185.42 93.98 0)
-		(unit 1)
-		(body_style 1)
-		(exclude_from_sim no)
-		(in_bom yes)
-		(on_board yes)
-		(in_pos_files yes)
-		(dnp no)
-		(property "Reference" "#PWR0234"
-			(at 185.42 100.33 0)
-			(hide yes)
-			(show_name no)
-			(do_not_autoplace no)
-			(effects
-				(font
-					(size 1.27 1.27)
-				)
-			)
-		)
-		(property "Value" "GND"
-			(at 185.42 97.536 0)
-			(hide yes)
-			(show_name no)
-			(do_not_autoplace no)
-			(effects
-				(font
-					(size 1.27 1.27)
-				)
-			)
-		)
-		(property "Footprint" ""
-			(at 185.42 93.98 0)
-			(hide yes)
-			(show_name no)
-			(do_not_autoplace no)
-			(effects
-				(font
-					(size 1.27 1.27)
-				)
-			)
-		)
-		(property "Datasheet" ""
-			(at 185.42 93.98 0)
-			(hide yes)
-			(show_name no)
-			(do_not_autoplace no)
-			(effects
-				(font
-					(size 1.27 1.27)
-				)
-			)
-		)
-		(property "Description" "Power symbol creates a global label with name \"GND\" , ground"
-			(at 185.42 93.98 0)
-			(hide yes)
-			(show_name no)
-			(do_not_autoplace no)
-			(effects
-				(font
-					(size 1.27 1.27)
-				)
-			)
-		)
-		(pin "1"
-		)
-		(instances
-			(project "Controller_Board"
-				(path "/4e6e1af1-ede9-4a56-9d5f-a8dfd7fbcf8d/77637722-5c93-4eaa-a1cc-47897016a2a9"
-					(reference "#PWR0234")
-					(unit 1)
-				)

Commit message: Advanced PCB design - Routed FTDI chips + USB HUB
Parts:
- removed C202: 10p, Capacitor_SMD:C_0402_1005Metric, symbol Device:C
- C201: footprint Capacitor_SMD:C_0402_1005Metric -> Capacitor_SMD:C_0201_0603Metric
- FB201: footprint Inductor_SMD:L_0402_1005Metric -> Inductor_SMD:L_0201_0603Metric
Changed lines of the file:
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@@
 	)
 	(junction
-		(at 116.84 49.53)
-		(diameter 0)
-		(color 0 0 0 0)
-	)
-	(junction
 		(at 185.42 102.87)
 		(diameter 0)
@@
 	(wire
 		(pts
-			(xy 116.84 49.53) (xy 128.27 49.53)
+			(xy 111.76 49.53) (xy 128.27 49.53)
 		)
 		(stroke
@@
 	(wire
 		(pts
-			(xy 111.76 49.53) (xy 116.84 49.53)
-		)
-		(stroke
-			(width 0)
-			(type default)
-		)
-	)
-	(wire
-		(pts
 			(xy 173.99 138.43) (xy 173.99 140.97)
 		)
@@
 	(wire
 		(pts
-			(xy 116.84 49.53) (xy 116.84 50.8)
-		)
-		(stroke
-			(width 0)
-			(type default)
-		)
-	)
-	(wire
-		(pts
 			(xy 66.04 67.31) (xy 55.88 67.31)
 		)
@@
 			)
 		)
-		(property "Footprint" "Capacitor_SMD:C_0402_1005Metric"
+		(property "Footprint" "Capacitor_SMD:C_0201_0603Metric"
 			(at 105.7148 58.42 0)
 			(hide yes)
@@
 			)
 		)
-		(property "Footprint" "Inductor_SMD:L_0402_1005Metric"
+		(property "Footprint" "Inductor_SMD:L_0201_0603Metric"
 			(at 97.79 51.308 90)
 			(hide yes)
@@
 	)
 	(symbol
-		(lib_id "Device:C")
-		(at 116.84 54.61 0)
-		(mirror y)
-		(unit 1)
-		(body_style 1)
-		(exclude_from_sim no)
-		(in_bom yes)
-		(on_board yes)
-		(in_pos_files yes)
-		(dnp no)
-		(property "Reference" "C202"
-			(at 114.3 53.34 0)
-			(show_name no)
-			(do_not_autoplace no)
-			(effects
-				(font
-					(size 1.27 1.27)
-				)
-				(justify left)
-			)
-		)
-		(property "Value" "10p"
-			(at 114.3 55.88 0)
-			(show_name no)
-			(do_not_autoplace no)
-			(effects
-				(font
-					(size 1.27 1.27)
-				)
-				(justify left)
-			)
-		)
-		(property "Footprint" "Capacitor_SMD:C_0402_1005Metric"
-			(at 115.8748 58.42 0)
-			(hide yes)
-			(show_name no)
-			(do_not_autoplace no)
-			(effects
-				(font
-					(size 1.27 1.27)
-				)
-			)
-		)
-		(property "Datasheet" ""
-			(at 116.84 54.61 0)
-			(hide yes)
-			(show_name no)
-			(do_not_autoplace no)
-			(effects
-				(font
-					(size 1.27 1.27)
-				)
-			)
-		)
-		(property "Description" "Unpolarized capacitor"
-			(at 116.84 54.61 0)
-			(hide yes)
-			(show_name no)
-			(do_not_autoplace no)
-			(effects
-				(font
-					(size 1.27 1.27)
-				)
-			)
-		)
-		(pin "2"
-		)
-		(pin "1"
-		)
-		(instances
-			(project "Controller_Board"
-				(path "/4e6e1af1-ede9-4a56-9d5f-a8dfd7fbcf8d/77637722-5c93-4eaa-a1cc-47897016a2a9"
-					(reference "C202")
-					(unit 1)
-				)
-			)
-		)
-	)
-	(symbol
 		(lib_id "power:GND")
 		(at 185.42 76.2 0)
@@
 					(unit 1)
 				)
-			)
-		)
-	)
-	(symbol
-		(lib_id "power:GND")
-		(at 116.84 58.42 0)
-		(unit 1)
-		(body_style 1)
-		(exclude_from_sim no)
-		(in_bom yes)
-		(on_board yes)
-		(in_pos_files yes)
-		(dnp no)
-		(property "Reference" "#PWR0204"
-			(at 116.84 64.77 0)
-			(hide yes)
-			(show_name no)
-			(do_not_autoplace no)
-			(effects
-				(font
-					(size 1.27 1.27)
-				)
-			)
-		)
-		(property "Value" "GND"
-			(at 116.84 61.976 0)
-			(hide yes)
-			(show_name no)
-			(do_not_autoplace no)
-			(effects
-				(font
-					(size 1.27 1.27)
-				)
-			)
-		)
-		(property "Footprint" ""
-			(at 116.84 58.42 0)
-			(hide yes)
-			(show_name no)
-			(do_not_autoplace no)
-			(effects
-				(font
-					(size 1.27 1.27)
-				)
-			)
-		)
-		(property "Datasheet" ""
-			(at 116.84 58.42 0)
-			(hide yes)
-			(show_name no)
-			(do_not_autoplace no)
-			(effects
-				(font
-					(size 1.27 1.27)
-				)
-			)
-		)
-		(property "Description" "Power symbol creates a global label with name \"GND\" , ground"
-			(at 116.84 58.42 0)
-			(hide yes)
-			(show_name no)
-			(do_not_autoplace no)
-			(effects
-				(font
-					(size 1.27 1.27)
-				)
-			)
-		)
-		(pin "1"
-		)
-		(instances
-			(project "Controller_Board"
-				(path "/4e6e1af1-ede9-4a56-9d5f-a8dfd7fbcf8d/77637722-5c93-4eaa-a1cc-47897016a2a9"
-					(reference "#PWR0204")
-					(unit 1)
-				)

Commit message: Advanced PCB design: Advanced power routing
Parts:
- removed C204: 100n, Capacitor_SMD:C_0201_0603Metric, symbol Device:C
- C236: footprint Capacitor_SMD:C_0805_2012Metric -> Capacitor_SMD:C_0603_1608Metric
Other:
- moved on the sheet: C205
Changed lines of the file:
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@@
 	)
 	(junction
-		(at 195.58 49.53)
-		(diameter 0)
-		(color 0 0 0 0)
-	)
-	(junction
 		(at 116.84 107.95)
 		(diameter 0)
@@
 	)
 	(junction
-		(at 205.74 49.53)
+		(at 195.58 49.53)
 		(diameter 0)
 		(color 0 0 0 0)
@@
 	)
 	(junction
+		(at 185.42 49.53)
+		(diameter 0)
+		(color 0 0 0 0)
+	)
+	(junction
 		(at 127 110.49)
 		(diameter 0)
@@
 	)
 	(junction
-		(at 185.42 49.53)
-		(diameter 0)
-		(color 0 0 0 0)
-	)
-	(junction
 		(at 127 81.28)
 		(diameter 0)
@@
 	(wire
 		(pts
-			(xy 195.58 49.53) (xy 195.58 50.8)
-		)
-		(stroke
-			(width 0)
-			(type default)
-		)
-	)
-	(wire
-		(pts
 			(xy 127 82.55) (xy 127 85.09)
 		)
@@
 	(wire
 		(pts
-			(xy 205.74 48.26) (xy 205.74 49.53)
+			(xy 195.58 48.26) (xy 195.58 49.53)
 		)
 		(stroke
@@
 	(wire
 		(pts
-			(xy 195.58 49.53) (xy 205.74 49.53)
-		)
-		(stroke
-			(width 0)
-			(type default)
-		)
-	)
-	(wire
-		(pts
 			(xy 55.88 66.04) (xy 55.88 67.31)
 		)
@@
 	(wire
 		(pts
-			(xy 205.74 49.53) (xy 205.74 50.8)
+			(xy 195.58 49.53) (xy 195.58 50.8)
 		)
 		(stroke
@@
 	(symbol
 		(lib_id "power:+3V3")
-		(at 205.74 48.26 0)
+		(at 195.58 48.26 0)
 		(unit 1)
 		(body_style 1)
@@
 		(dnp no)
 		(property "Reference" "#PWR0202"
-			(at 205.74 52.07 0)
+			(at 195.58 52.07 0)
 			(hide yes)
 			(show_name no)
@@
 		)
 		(property "Value" "+3V3"
-			(at 205.74 44.704 0)
+			(at 195.58 44.704 0)
 			(show_name no)
 			(do_not_autoplace no)
@@
 		)
 		(property "Footprint" ""
-			(at 205.74 48.26 0)
+			(at 195.58 48.26 0)
 			(hide yes)
 			(show_name no)
@@
 		)
 		(property "Datasheet" ""
-			(at 205.74 48.26 0)
+			(at 195.58 48.26 0)
 			(hide yes)
 			(show_name no)
@@
 		)
 		(property "Description" "Power symbol creates a global label with name \"+3V3\""
-			(at 205.74 48.26 0)
+			(at 195.58 48.26 0)
 			(hide yes)
 			(show_name no)
@@
 	(symbol
 		(lib_id "Device:C")
-		(at 205.74 54.61 0)
+		(at 195.58 54.61 0)
 		(mirror y)
 		(unit 1)
@@
 		(dnp no)
 		(property "Reference" "C205"
-			(at 203.2 53.34 0)
+			(at 193.04 53.34 0)
 			(show_name no)
 			(do_not_autoplace no)
@@
 		)
 		(property "Value" "10u"
-			(at 203.2 55.88 0)
+			(at 193.04 55.88 0)
 			(show_name no)
 			(do_not_autoplace no)
@@
 		)
 		(property "Footprint" "Capacitor_SMD:C_0603_1608Metric"
-			(at 204.7748 58.42 0)
+			(at 194.6148 58.42 0)
 			(hide yes)
 			(show_name no)
@@
 		)
 		(property "Datasheet" ""
-			(at 205.74 54.61 0)
+			(at 195.58 54.61 0)
 			(hide yes)
 			(show_name no)
@@
 		)
 		(property "Description" "Unpolarized capacitor"
-			(at 205.74 54.61 0)
+			(at 195.58 54.61 0)
 			(hide yes)
 			(show_name no)
@@
 	)
 	(symbol
-		(lib_id "power:GND")
-		(at 195.58 58.42 0)
-		(unit 1)
-		(body_style 1)
-		(exclude_from_sim no)
-		(in_bom yes)
-		(on_board yes)
-		(in_pos_files yes)
-		(dnp no)
-		(property "Reference" "#PWR0206"
-			(at 195.58 64.77 0)
-			(hide yes)
-			(show_name no)
-			(do_not_autoplace no)
-			(effects
-				(font
-					(size 1.27 1.27)
-				)
-			)
-		)
-		(property "Value" "GND"
-			(at 195.58 61.976 0)
-			(hide yes)
-			(show_name no)
-			(do_not_autoplace no)
-			(effects
-				(font
-					(size 1.27 1.27)
-				)
-			)
-		)
-		(property "Footprint" ""
-			(at 195.58 58.42 0)
-			(hide yes)
-			(show_name no)
-			(do_not_autoplace no)
-			(effects
-				(font
-					(size 1.27 1.27)
-				)
-			)
-		)
-		(property "Datasheet" ""
-			(at 195.58 58.42 0)
-			(hide yes)
-			(show_name no)
-			(do_not_autoplace no)
-			(effects
-				(font
-					(size 1.27 1.27)
-				)
-			)
-		)
-		(property "Description" "Power symbol creates a global label with name \"GND\" , ground"
-			(at 195.58 58.42 0)
-			(hide yes)
-			(show_name no)
-			(do_not_autoplace no)
-			(effects
-				(font
-					(size 1.27 1.27)
-				)
-			)
-		)
-		(pin "1"
-		)
-		(instances
-			(project "Controller_Board"
-				(path "/4e6e1af1-ede9-4a56-9d5f-a8dfd7fbcf8d/77637722-5c93-4eaa-a1cc-47897016a2a9"
-					(reference "#PWR0206")
-					(unit 1)
-				)
-			)
-		)
-	)
-	(symbol
 		(lib_id "Device:C")
 		(at 106.68 54.61 0)
@@
 			)
 		)
-		(property "Footprint" "Capacitor_SMD:C_0805_2012Metric"
+		(property "Footprint" "Capacitor_SMD:C_0603_1608Metric"
 			(at 194.6148 111.76 0)
 			(hide yes)
@@
 	(symbol
 		(lib_id "Device:C")
-		(at 195.58 54.61 0)
-		(mirror y)
-		(unit 1)
-		(body_style 1)
-		(exclude_from_sim no)
-		(in_bom yes)
-		(on_board yes)
-		(in_pos_files yes)
-		(dnp no)
-		(property "Reference" "C204"
-			(at 193.04 53.34 0)
-			(show_name no)
-			(do_not_autoplace no)
-			(effects
-				(font
-					(size 1.27 1.27)
-				)
-				(justify left)
-			)
-		)
-		(property "Value" "100n"
-			(at 193.04 55.88 0)
-			(show_name no)
-			(do_not_autoplace no)
-			(effects
-				(font
-					(size 1.27 1.27)
-				)
-				(justify left)
-			)
-		)
-		(property "Footprint" "Capacitor_SMD:C_0201_0603Metric"
-			(at 194.6148 58.42 0)
-			(hide yes)
-			(show_name no)
-			(do_not_autoplace no)
-			(effects
-				(font
-					(size 1.27 1.27)
-				)
-			)
-		)
-		(property "Datasheet" ""
-			(at 195.58 54.61 0)
-			(hide yes)
-			(show_name no)
-			(do_not_autoplace no)
-			(effects
-				(font
-					(size 1.27 1.27)
-				)
-			)
-		)
-		(property "Description" "Unpolarized capacitor"
-			(at 195.58 54.61 0)
-			(hide yes)
-			(show_name no)
-			(do_not_autoplace no)
-			(effects
-				(font
-					(size 1.27 1.27)
-				)
-			)
-		)
-		(pin "2"
-		)
-		(pin "1"
-		)
-		(instances
-			(project "Controller_Board"
-				(path "/4e6e1af1-ede9-4a56-9d5f-a8dfd7fbcf8d/77637722-5c93-4eaa-a1cc-47897016a2a9"
-					(reference "C204")
-					(unit 1)
-				)
-			)
-		)
-	)
-	(symbol
-		(lib_id "Device:C")
 		(at 215.9 143.51 0)
 		(mirror y)
@@
 	(symbol
 		(lib_id "power:GND")
-		(at 205.74 58.42 0)
+		(at 195.58 58.42 0)
 		(unit 1)
 		(body_style 1)
@@
 		(dnp no)
 		(property "Reference" "#PWR0207"
-			(at 205.74 64.77 0)
+			(at 195.58 64.77 0)
 			(hide yes)
 			(show_name no)
@@
 		)
 		(property "Value" "GND"
-			(at 205.74 61.976 0)
+			(at 195.58 61.976 0)
 			(hide yes)
 			(show_name no)
@@
 		)
 		(property "Footprint" ""
-			(at 205.74 58.42 0)
+			(at 195.58 58.42 0)
 			(hide yes)
 			(show_name no)
@@
 		)
 		(property "Datasheet" ""
-			(at 205.74 58.42 0)
+			(at 195.58 58.42 0)
 			(hide yes)
 			(show_name no)
@@
 		)
 		(property "Description" "Power symbol creates a global label with name \"GND\" , ground"
-			(at 205.74 58.42 0)
+			(at 195.58 58.42 0)
 			(hide yes)
 			(show_name no)

Commit message: Advanced PCB Design: Routing Power + UVLO
Connections:
- net +3V3 renamed +2V5
Other:
- moved on the sheet: C201, C203, C205, C206, C207, C208, C209, C210, C211, C212, C213, C214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

Commit message: Finished PCB Design - WARNING MORE CHANGES NEEDED! The main decision to be made is, whether to increase the layer count to 8 layers, and make the P7 and P8 permamently on 3V3
Parts:
- renumbered C201 to C301, C203 to C302, C205 to C303, C206 to C304, C207 to C305, C208 to C306, C209 to C307, C210 to C308, C211 to C309, C212 to C310, C213 to C311, C214 to C312, C215 to C313, C216 to C314, C217 to C315, C218 to C316, C219 to C317, C220 to C318, C221 to C319, C222 to C320, C223 to C321, C224 to C322, C225 to C323, C226 to C324, C227 to C325, C229 to C326, C230 to C327, C231 to C328, C232 to C329, C233 to C330, C234 to C331, C235 to C332, C236 to C333, C237 to C334, C238 to C335, C239 to C336, C240 to C337, C241 to C338, C242 to C339, C243 to C340, C244 to C341, C245 to C342, C246 to C343, C247 to C344, C248 to C345, C249 to C346, C250 to C347, C251 to C348, C252 to C349, C253 to C350, C254 to C351, C255 to C352, C256 to C353, C257 to C354, C258 to C355, FB201 to FB301, U201 to U301
Other:
- note added: "FPGA Power [3]"
- note removed: "FPGA Power [2]"
