File: Hardware/Controller_Board/fpga_power.kicad_sch (KiCad schematic)
At the start: 57 parts, among them U301 XC7A35T-CSG324

Commit message: Finished procuring almost all boards - CHANGED XDC IN XILINX FOR TESTING!! - Programmer needed
Parts:
- C301, C302, C305, C306, C307, C308, C309, C310, C311, C312, C313, C314, C315, C316, C318, C319, C320, C321, C322, C323, C324, C325, C326, C327, C328, C329, C330, C332, C335, C336, C337, C338, C339, C340, C341, C342, C343, C344, C347, C348, C349, C350, C351, C352, C353, C354: LCSC (none) -> C668346; Manufacturer (none) -> Murata
- C303, C304, C317, C331, C333, C334, C346: LCSC (none) -> C194427; Manufacturer (none) -> Murata
- C345: renamed from C355; LCSC (none) -> C194427; Manufacturer (none) -> Murata
- C355: renamed from C345; LCSC (none) -> C194427; Manufacturer (none) -> Murata
- FB301: LCSC (none) -> C237542; Manufacturer (none) -> Murata
- U301: LCSC (none) -> C1521726; Manufacturer (none) -> Xilinx
Connections:
- net +2V5: no longer C349.1, C350.1, C351.1, C352.1, C353.1, C354.1, C355.1, U301.A7 (VCCO_35), U301.C3 (VCCO_35), U301.D6 (VCCO_35), U301.F2 (VCCO_35), U301.G5 (VCCO_35), U301.J1 (VCCO_35)
- new net +3V3: C349.1, C350.1, C351.1, C352.1, C353.1, C354.1, C355.1, U301.A7 (VCCO_35), U301.C3 (VCCO_35), U301.D6 (VCCO_35), U301.F2 (VCCO_35), U301.G5 (VCCO_35), U301.J1 (VCCO_35)
Other:
- note added: "WARNING! BANK 35 is ALWAYS connected to +3V3! Do not plug LVDS devices into BANK 35 ports!"
- moved on the sheet: C345, C355
