File: Hardware/Controller_Board/fpga_config.kicad_sch (KiCad schematic)
At the start: 13 parts, among them U1 XC7A35T-CPG236, U7 IS25LP256D

Commit message: Added new sheets to the schematic
Parts:
- added C304: 1u, Capacitor_SMD:C_0402_1005Metric, symbol Device:C
- added D1: LED, LED_SMD:LED_0603_1608Metric, symbol Device:LED
- added R22, R23: 200R, Resistor_SMD:R_0402_1005Metric, symbol Device:R
- added R24, R25: 4.7k, symbol Device:R
- added SW301: Reset, Button_Switch_SMD:SW_Push_SPST_NO_Alps_SKRK, symbol Switch:SW_Push
Connections:
- net AGND is gone; now on net GND: U1.A12 (VP_0), U1.A13 (VREFN_0), U1.B12 (VREFP_0), U1.B13 (VN_0)
- net +3V3: now also R22.1, R24.1, R25.1
- net FPGA_RST: now also C304.1, R25.2, SW301.1
- net GND: now also C304.2, R23.2, SW301.2
- net FPGA_INIT: now reaches U1.U11 (INIT_B_0)
- net FPGA_INIT: now also R24.2
- net FPGA_DONE: now reaches U1.U12 (DONE_0)
- net FPGA_DONE: now also D1.2 (A), R22.2
- new net: D1.1 (K), R23.1
Other:
- note added: "Additionally, there is a delay to even start the spi communication after booting the FPGA up, so we're in the clear."
- note added: "Capacitor charge time is 4.7ms"
- note added: "Connect to ground for on-chip XADC reference (UG480)"
- note added: "Dedicated analog input. Connect to GND if not used (UG480)"
- note added: "FPGA Config [5]"
- note added: "FPGA Manual Reset"
- note added: "HIGH to set JTAG to 3.3V/2.5V operation (UG470)"
- note added: "If the LED shines, the device has been configured properly!"
- note added: "Maximum power-up time delay for Flash instruction readiness is 10ms. According to the DS181 AMD datasheet, the minimum FPGA Power-On Reset TPOR is also 10ms. By implementing a capacitor on the PROGRAM_B pin of the FPGA, the startup sequence is intentionally delayed to ensure a safe margin where the Flash initializes prior to the FPGA."
- note added: "Thermal diode Connect to GND id not used"
- note added: "This configuration makes the FPGA boot from SPI"
- note added: "UG470 Datasheet"
- note removed: "This makes the FPGA boot from SPI"
- moved on the sheet: C73, R14, R19, R20, R21, U7

Commit message: Added USB hub symbol
Parts:
- renumbered C304 to C74, D1 to D3, R22 to R14, R21 to R15, R20 to R16, R23 to R17, R24 to R18, R14 to R20, R25 to R21, R15 to R22, R16 to R23, R17 to R24, R18 to R25, Re to Re1, Re1 to Re2, SW301 to SW1, U1 to U6

Commit message: Updated the schematic design - Fix the XC7A35T-CPG236 outline issue
Other:
- note added: "FPGA Config [3]"
- note removed: "FPGA Config [5]"
Changed lines of the file:
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@@
 		)
 	)
-	(text "FPGA Config [5]"
+	(text "FPGA Config [3]"
 		(exclude_from_sim no)
 		(at 15.494 18.796 0)

Commit message: Fixed the bug in the FPGA symbol I have unchecked these boxes in the symbol properties and settings for the individual shapes -All units are interchangeable -Common to all units
Changed lines of the file:
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@@
 		(pin "U11"
+		)
+		(pin "C7"
 		)
 		(instances

Commit message: Finished schematic design - preparation for review
Parts:
- added C303: 100n, Capacitor_SMD:C_0402_1005Metric, symbol Device:C
- added R302: 22R, Resistor_SMD:R_0402_1005Metric, symbol Device:R
- added unit 7 of U6
- added unit 3 of U6
- added Y301: 12MHz, Oscillator:Oscillator_SMD_Abracon_ASCO-4Pin_1.6x1.2mm, symbol Oscillator:ASCO
Connections:
- net GND: now also C303.2, U6.A4 (MGTPRXN0_216), U6.A6 (MGTPRXN1_216), U6.B4 (MGTPRXP0_216), U6.B6 (MGTPRXP1_216), U6.C7 (MGTRREF_216), Y301.2 (GND)
- net TCK: now also U6.C8 (TCK_0); no longer U6.W8 (TDO_0)
- net TDI_FPGA: now also U6.W10 (TDI_0); no longer U6.W9 (TMS_0)
- net TDO_FPGA: now also U6.W8 (TDO_0); no longer U6.C8 (TCK_0)
- net TMS: now also U6.W9 (TMS_0); no longer U6.W10 (TDI_0)
- new net 12MHZ_CLK: R302.1, U6.P3 (IO_L12N_T1_MRCC_35)
- new net OSC_OUT: R302.2, Y301.3 (OUT)
- new net P5_L1: U6.G3 (IO_L1P_T0_AD4P_35)
- new net P5_L2: U6.G2 (IO_L1N_T0_AD4N_35)
- new net P6_L1: U6.H2 (IO_L2P_T0_AD12P_35)
- new net P6_L2: U6.J2 (IO_L2N_T0_AD12N_35)
- new net P7_L1: U6.H1 (IO_L3P_T0_DQS_AD5P_35)
- new net P7_L2: U6.J1 (IO_L3N_T0_DQS_AD5N_35)
- new net P8_L1: U6.K2 (IO_L5P_T0_AD13P_35)
- new net P8_L2: U6.L2 (IO_L5N_T0_AD13N_35)
- new net P9_L1: U6.L1 (IO_L6N_T0_VREF_35)
- new net P9_L2: U6.J3 (IO_L7P_T1_AD6P_35)
- new net VCCIO2: C303.1, Y301.1 (Tri-State), Y301.4 (VDD)
- no-connect marks 0 -> 17
Other:
- moved on the sheet: C73, C74, D3, R14, R15, R16, R17, R18, R19, R20, R21, SW1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

Commit message: Finished DRC check. Moving to schematic review
Parts:
- R302: renamed from R15; footprint (none) -> Resistor_SMD:R_0402_1005Metric
- R304: renamed from R16; footprint (none) -> Resistor_SMD:R_0402_1005Metric
- R305: renamed from R18; footprint (none) -> Resistor_SMD:R_0402_1005Metric
- R306: renamed from R21; footprint (none) -> Resistor_SMD:R_0402_1005Metric
- R307: renamed from R19; footprint (none) -> Resistor_SMD:R_0402_1005Metric
- R308: renamed from R20; footprint (none) -> Resistor_SMD:R_0402_1005Metric
- R309: renamed from R22; value R -> 100R; footprint (none) -> Resistor_SMD:R_0402_1005Metric
- R310: renamed from R23; value R -> 100R; footprint (none) -> Resistor_SMD:R_0402_1005Metric
- R311: renamed from R24; value R -> 100R; footprint (none) -> Resistor_SMD:R_0402_1005Metric
- R312: renamed from R25; value R -> 100R; footprint (none) -> Resistor_SMD:R_0402_1005Metric
- Re301: renamed from Re1; footprint (none) -> Resistor_SMD:R_0402_1005Metric
- Re302: renamed from Re2; footprint (none) -> Resistor_SMD:R_0402_1005Metric
- renumbered C74 to C301, C73 to C302, D3 to D301, R14 to R301, R17 to R303, R302 to R313, SW1 to SW301, U6 to U201, U7 to U301
Connections:
- net VCCIO2 is gone; now on net +3V3: C303.1, Y301.1 (Tri-State), Y301.4 (VDD)
- net TDI_FPGA renamed TDI
- net TDO_FPGA renamed TDO

Commit message: Finished the schematic review
Parts:
- removed R310, R311, R312: 100R, Resistor_SMD:R_0402_1005Metric, symbol Device:R
- added R304: 4.7k, Resistor_SMD:R_0402_1005Metric, symbol Device:R
- added TP301: N3, TestPoint:TestPoint_Pad_D1.0mm, symbol Connector:TestPoint
- added TP302: M2, TestPoint:TestPoint_Pad_D1.0mm, symbol Connector:TestPoint
- added TP303: M3, TestPoint:TestPoint_Pad_D1.0mm, symbol Connector:TestPoint
- added TP304: L3, TestPoint:TestPoint_Pad_D1.0mm, symbol Connector:TestPoint
- added TP305: K3, TestPoint:TestPoint_Pad_D1.0mm, symbol Connector:TestPoint
- R302: renamed from R303; value 200R -> 100R
- R305: renamed from R304; value 1k -> 4.7k
- R308, R309: value 100R -> 4.7k
- Re301, Re302: value 1k -> 4.7k
- renumbered R302 to R303, R305 to R306, R306 to R307, R307 to R310, R313 to R311
Connections:
- net NHL_FLASH is gone; now on net NHL_FPGA: U301.7 (NHOLD)
- net NWP_FLASH is gone; now on net NWP_FPGA: U301.3 (NWP)
- net SDO_FLASH is gone; now on net SDO_FPGA: U301.2 (SDO)
- net +3V3: now also R308.1, R309.1, R304.1
- net FPGA_DONE: now also R302.1; no longer D301.2 (A)
- net GND: now also D301.1 (K); no longer R302.2
- net NHL_FPGA: now also R308.2
- net NWP_FPGA: now also R309.2
- net P7_L1: now also U201.K2 (IO_L5P_T0_AD13P_35); no longer U201.H1 (IO_L3P_T0_DQS_AD5P_35)
- net P7_L2: now also U201.L2 (IO_L5N_T0_AD13N_35); no longer U201.J1 (IO_L3N_T0_DQS_AD5N_35)
- net P8_L1: now also U201.L1 (IO_L6N_T0_VREF_35); no longer U201.K2 (IO_L5P_T0_AD13P_35)
- net P8_L2: now also U201.J3 (IO_L7P_T1_AD6P_35); no longer U201.L2 (IO_L5N_T0_AD13N_35)
- net P9_L1: now also U201.K3 (IO_L7N_T1_AD6N_35); no longer U201.L1 (IO_L6N_T0_VREF_35)
- net P9_L2: now also U201.L3 (IO_L8P_T1_AD14P_35); no longer U201.J3 (IO_L7P_T1_AD6P_35)
- net SCK_FPGA: now also U201.E19 (IO_L3N_T0_DQS_EMCCLK_14), U301.6 (SCK); no longer R308.1
- net SDI_FPGA: now also U301.5 (SDI); no longer R309.1
- net at U201.M1 (IO_L9N_T1_DQS_AD7N_35): now also TP303.1
- net at U201.M2 (IO_L9P_T1_DQS_AD7P_35): now also TP304.1
- net at U201.M3 (IO_L8N_T1_AD14N_35): now also TP305.1
- net at U201.N1 (IO_L10N_T1_AD15N_35): now also TP301.1
- net at U201.N2 (IO_L10P_T1_AD15P_35): now also TP302.1
- removed net P5_L1: U201.G3 (IO_L1P_T0_AD4P_35)
- removed net P5_L2: U201.G2 (IO_L1N_T0_AD4N_35)
- removed net P6_L1: U201.H2 (IO_L2P_T0_AD12P_35)
- removed net P6_L2: U201.J2 (IO_L2N_T0_AD12N_35)
- removed net SCK_FLASH: R308.2, U301.6 (SCK)
- removed net SDI_FLASH: R309.2, U301.5 (SDI)
- new net: R304.2, U201.E18 (IO_L3P_T0_DQS_PUDC_B_14)
- new net: D301.2 (A), R302.2
- no-connect marks 17 -> 10
Other:
- note added: "For FLASH config outside bootloader mode"
- note added: "HIGH to disable internal pullups during startup"
- note added: "Since we're not using XADC, we tie ADCGND to GND (for VP_0 and VN_0)"
- note added: "Test Points"
- moved on the sheet: C302, D301, R302, R310, U301

Commit message: Started schematic rework and the PCB design
Parts:
- removed U201: XC7A35T-CPG236, Package_BGA:Xilinx_CPG236, symbol Custom_VoxLink_Symbols:XC7A35T-CPG236
- added U302: XC7A35T-CSG324, Package_BGA:Xilinx_CSG324, symbol Custom_VoxLink_Symbols:XC7A35T-CSG324
Connections:
- net FPGA_DONE: now also U302.P10 (DONE_0)
- net FPGA_INIT: now also U302.P7 (INIT_B_0)
- net FPGA_RST: now also U302.P9 (PROGRAM_B_0)
- net GND: now also U302.J10 (VP_0), U302.J9 (VREFN_0), U302.K10 (VREFP_0), U302.K9 (VN_0), U302.L10 (DXP_0), U302.L9 (DXN_0)
- net MODE0: now also U302.P12 (M0_0)
- net MODE1: now also U302.P13 (M1_0)
- net MODE2: now also U302.P11 (M2_0)
- net NCS_FPGA: now also U302.L13 (IO_L6P_T0_FCS_B_14)
- net NHL_FPGA: now also U302.M14 (IO_L2N_T0_D03_14)
- net NWP_FPGA: now also U302.L14 (IO_L2P_T0_D02_14)
- net SCK_FPGA: now also U302.E9 (CCLK_0), U302.L16 (IO_L3N_T0_DQS_EMCCLK_14)
- net SDI_FPGA: now also U302.K17 (IO_L1P_T0_D00_MOSI_14)
- net SDO_FPGA: now also U302.K18 (IO_L1N_T0_D01_DIN_14)
- net TCK: now also U302.E10 (TCK_0)
- net TDI: now also U302.E11 (TDI_0)
- net TDO: now also U302.E13 (TDO_0)
- net TMS: now also U302.E12 (TMS_0)
- net at R304.2: now also U302.L15 (IO_L3P_T0_DQS_PUDC_B_14)
- net at R303.2: now also U302.P8 (CFGBVS_0)
- no-connect marks 10 -> 2
Other:
- note added: "Connect to MRCC!!!!!!"
