File: Hardware/Controller_Board/fpga_config.kicad_sch (KiCad schematic)
At the start: 26 parts, among them SW301 Reset, U301 IS25LP256D, U302 XC7A35T-CSG324, Y301 12MHz

Commit message: Commit before upgrading to KiCad 10.0
Parts:
- removed unit 3 of U302
- removed unit 7 of U302
- removed unit 4 of U302
- removed unit 6 of U302
- renumbered U302 to U201
Connections:
- net 12MHZ_CLK: now also U201.C10 (IO_L13N_T2_MRCC_16)
- net at TP305.1: now also U201.D9 (IO_L6N_T0_VREF_16)
- net at U201.A8 (IO_L12N_T1_MRCC_16): now also TP301.1
- net at U201.B8 (IO_L12P_T1_MRCC_16): now also TP302.1
- net at U201.B9 (IO_L11N_T1_SRCC_16): now also TP303.1
- net at U201.C9 (IO_L11P_T1_SRCC_16): now also TP304.1
- no-connect marks 2 -> 4
Other:
- note removed: "Connect to MRCC!!!!!!"
- moved on the sheet: TP301, TP302, TP303, TP304, TP305, U201E

Commit message: Advanced PCB design: Routed FTDIs + SPI Flash
Parts:
- R303, R304, R305, R306, Re301, Re302: footprint Resistor_SMD:R_0402_1005Metric -> Resistor_SMD:R_0201_0603Metric
Changed lines of the file:
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@@
 			)
 		)
-		(property "Footprint" "Resistor_SMD:R_0402_1005Metric"
+		(property "Footprint" "Resistor_SMD:R_0201_0603Metric"
 			(at 115.57 75.438 90)
 			(hide yes)
@@
 			)
 		)
-		(property "Footprint" "Resistor_SMD:R_0402_1005Metric"
+		(property "Footprint" "Resistor_SMD:R_0201_0603Metric"
 			(at 115.57 70.358 90)
 			(hide yes)
@@
 			)
 		)
-		(property "Footprint" "Resistor_SMD:R_0402_1005Metric"
+		(property "Footprint" "Resistor_SMD:R_0201_0603Metric"
 			(at 60.96 62.738 90)
 			(hide yes)
@@
 			)
 		)
-		(property "Footprint" "Resistor_SMD:R_0402_1005Metric"
+		(property "Footprint" "Resistor_SMD:R_0201_0603Metric"
 			(at 115.57 72.898 90)
 			(hide yes)
@@
 			)
 		)
-		(property "Footprint" "Resistor_SMD:R_0402_1005Metric"
+		(property "Footprint" "Resistor_SMD:R_0201_0603Metric"
 			(at 60.96 55.118 90)
 			(hide yes)
@@
 			)
 		)
-		(property "Footprint" "Resistor_SMD:R_0402_1005Metric"
+		(property "Footprint" "Resistor_SMD:R_0201_0603Metric"
 			(at 122.428 86.36 90)
 			(hide yes)

Commit message: Advanced PCB design - Routed FTDI chips + USB HUB
Parts:
- U301: footprint Package_SON:WSON-8-1EP_8x6mm_P1.27mm_EP3.4x4.3mm -> Custom_VoxLink_Footprints:WSON-8-1EP_8.0x6.0mm_P1.27mm_EP4.7x4.6mm
Changed lines of the file:
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@@
 			)
 		)
-		(property "Footprint" "Package_SON:WSON-8-1EP_8x6mm_P1.27mm_EP3.4x4.3mm"
+		(property "Footprint" "Custom_VoxLink_Footprints:WSON-8-1EP_8.0x6.0mm_P1.27mm_EP4.7x4.6mm"
 			(at 161.29 104.14 0)
 			(hide yes)

Commit message: Advanced PCB design: Advanced power routing
Parts:
- removed TP303: M3, TestPoint:TestPoint_Pad_D1.0mm, symbol Connector:TestPoint
- removed TP304: L3, TestPoint:TestPoint_Pad_D1.0mm, symbol Connector:TestPoint
- removed TP305: K3, TestPoint:TestPoint_Pad_D1.0mm, symbol Connector:TestPoint
Connections:
- no-connect marks 4 -> 7
Other:
- moved on the sheet: TP301, TP302

Commit message: Advanced PCB Design: Routing Power + UVLO
Connections:
- net +3V3 renamed +2V5
Other:
- note added: "Select a 2V5 variant!"

Commit message: Finished PCB Design - WARNING MORE CHANGES NEEDED! The main decision to be made is, whether to increase the layer count to 8 layers, and make the P7 and P8 permamently on 3V3
Parts:
- renumbered C301 to C401, C302 to C402, C303 to C403, D301 to D401, R301 to R401, R302 to R402, R303 to R403, R304 to R404, R305 to R405, R306 to R406, R307 to R407, R308 to R408, R309 to R409, R310 to R410, R311 to R411, Re301 to Re401, Re302 to Re402, SW301 to SW401, TP301 to TP401, TP302 to TP402, U201 to U301, U301 to U401, Y301 to Y401
Connections:
- net at U301.A9 (IO_L14N_T2_SRCC_16): now also TP402.1
- net at U301.B8 (IO_L12P_T1_MRCC_16): no longer TP402.1
Other:
- note added: "FPGA Config [4]"
- note removed: "FPGA Config [3]"
- moved on the sheet: TP401, TP402

Commit message: Finished procuring almost all boards - CHANGED XDC IN XILINX FOR TESTING!! - Programmer needed
Parts:
- C401: LCSC (none) -> C528974; Manufacturer (none) -> Murata
- C402, C403: LCSC (none) -> C77020; Manufacturer (none) -> Murata
- D401: LCSC (none) -> C18198801; Manufacturer (none) -> Broadcom
- R401: LCSC (none) -> C482094; Manufacturer (none) -> Vishay
- R402: LCSC (none) -> C844502; Manufacturer (none) -> Vishay
- R403, R404, R405, R406, Re401, Re402: LCSC (none) -> C3000902; Manufacturer (none) -> Vishay
- R407, R408, R409, R410: LCSC (none) -> C482193; Manufacturer (none) -> Vishay
- R411: LCSC (none) -> C482106; Manufacturer (none) -> Vishay
- SW401: LCSC (none) -> C202388; Manufacturer (none) -> Alps
- TP401: renamed from TP402; now left out of the parts list
- TP402: renamed from TP401; now left out of the parts list
- U301: LCSC (none) -> C1521726; Manufacturer (none) -> Xilinx
- U401: LCSC (none) -> C1350139; Manufacturer (none) -> ISSI
- Y401: footprint Oscillator:Oscillator_SMD_Abracon_ASCO-4Pin_1.6x1.2mm -> Crystal:Crystal_SMD_2520-4Pin_2.5x2.0mm; LCSC (none) -> C17361989
Other:
- note removed: "Select a 2V5 variant!"
