File: Hardware/Controller_Board/fpga_config.kicad_sch (KiCad schematic)
At the start: 23 parts, among them SW401 Reset, U301 XC7A35T-CSG324, U401 IS25LP256D, Y401 12MHz

Commit message: Finished PCB design and Review + Procured Boards
Connections:
- net 12MHZ_CLK: now also U301.C11 (IO_L13P_T2_MRCC_16); no longer U301.C10 (IO_L13N_T2_MRCC_16)
Changed lines of the file:
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@@
 	)
 	(no_connect
-		(at 96.52 166.37)
+		(at 96.52 168.91)
 	)
 	(wire
@@
 	(global_label "12MHZ_CLK"
 		(shape input)
-		(at 96.52 168.91 180)
+		(at 96.52 166.37 180)
 		(fields_autoplaced yes)
 		(effects
@@
 		)
 		(property "Intersheetrefs" "${INTERSHEET_REFS}"
-			(at 82.5887 168.91 0)
+			(at 82.5887 166.37 0)
 			(hide yes)
 			(show_name no)
