File: Hardware/Controller_Board/connectivity.kicad_sch (KiCad schematic)
At the start: 0 parts

Commit message: Updated the schematic design - Fix the XC7A35T-CPG236 outline issue
Parts:
- added U14, U16, U17, U22, U25, U28, U31, U34, U37: RJ45, Custom_VoxLink_Footprints:TE_RJ45, symbol Custom_VoxLink_Symbols:RJ45_LED
- added U15, U27, U33: TPD4E02B04, Package_SON:USON-10_2.5x1.0mm_P0.5mm, symbol Custom_VoxLink_Symbols:TPD4E02B04DQA_Tall
- added U18, U19, U20, U21, U23, U24, U26, U29, U30, U32, U39, U501: TPD4E02B04, Package_SON:USON-10_2.5x1.0mm_P0.5mm, symbol Custom_VoxLink_Symbols:TPD4E02B04DQA
Connections:
- new net: U16.1 (RX), U20.2 (IN)
- new net: U16.2 (~{RX}), U20.1 (IN)
- new net: U15.4 (IN), U16.4 (CLK)
- new net: U15.5 (IN), U16.5 (~{CLK})
- new net: U16.7 (~{TX}), U20.4 (IN)
- new net: U16.8 (TX), U20.5 (IN)
- new net: U17.1 (RX), U19.5 (IN)
- new net: U17.2 (~{RX}), U19.4 (IN)
- new net: U17.4 (CLK), U18.5 (IN)
- new net: U17.5 (~{CLK}), U18.4 (IN)
- new net: U17.7 (~{TX}), U18.1 (IN)
- new net: U17.8 (TX), U18.2 (IN)
- new net: U22.1 (RX), U27.1 (IN)
- new net: U22.2 (~{RX}), U27.2 (IN)
- new net: U22.4 (CLK), U23.5 (IN)
- new net: U22.5 (~{CLK}), U23.4 (IN)
- new net: U22.7 (~{TX}), U23.1 (IN)
- new net: U22.8 (TX), U23.2 (IN)
- new net: U31.7 (~{TX}), U32.1 (IN)
- new net: U31.8 (TX), U32.2 (IN)
- new net: U31.5 (~{CLK}), U32.4 (IN)
- new net: U31.4 (CLK), U32.5 (IN)
- new net: U24.1 (IN), U25.2 (~{RX})
- new net: U24.2 (IN), U25.1 (RX)
- new net: U24.4 (IN), U25.7 (~{TX})
- new net: U24.5 (IN), U25.8 (TX)
- new net: U28.2 (~{RX}), U30.4 (IN)
- new net: U28.1 (RX), U30.5 (IN)
- new net: U28.7 (~{TX}), U29.1 (IN)
- new net: U28.8 (TX), U29.2 (IN)
- new net: U28.5 (~{CLK}), U29.4 (IN)
- new net: U28.4 (CLK), U29.5 (IN)
- new net: U14.1 (RX), U15.1 (IN)
- new net: U14.2 (~{RX}), U15.2 (IN)
- new net: U25.4 (CLK), U27.4 (IN)
- new net: U25.5 (~{CLK}), U27.5 (IN)
- new net: U14.7 (~{TX}), U501.1 (IN)
- new net: U14.8 (TX), U501.2 (IN)
- new net: U14.5 (~{CLK}), U501.4 (IN)
- new net: U14.4 (CLK), U501.5 (IN)
- new net: U26.1 (IN), U34.2 (~{RX})
- new net: U26.2 (IN), U34.1 (RX)
- new net: U26.4 (IN), U34.7 (~{TX})
- new net: U26.5 (IN), U34.8 (TX)
- new net: U31.1 (RX), U33.1 (IN)
- new net: U31.2 (~{RX}), U33.2 (IN)
- new net: U33.4 (IN), U34.4 (CLK)
- new net: U33.5 (IN), U34.5 (~{CLK})
- new net: U37.2 (~{RX}), U39.4 (IN)
- new net: U37.1 (RX), U39.5 (IN)
- new net: U21.1 (IN), U37.7 (~{TX})
- new net: U21.2 (IN), U37.8 (TX)
- new net: U21.4 (IN), U37.5 (~{CLK})
- new net: U21.5 (IN), U37.4 (CLK)
- new net +5V: U14.3 (VCC), U16.3 (VCC), U17.3 (VCC), U22.3 (VCC), U25.3 (VCC), U28.3 (VCC), U31.3 (VCC), U34.3 (VCC), U37.3 (VCC)
- new net GND: U14.13 (SHD), U14.14 (SHD), U14.6 (GND), U15.3 (GND), U15.8 (NC), U16.13 (SHD), U16.14 (SHD), U16.6 (GND), U17.13 (SHD), U17.14 (SHD), U17.6 (GND), U18.3 (GND), U18.8 (NC), U19.3 (GND), U19.8 (NC), U20.3 (GND), U20.8 (NC), U21.3 (GND), U21.8 (NC), U22.13 (SHD), U22.14 (SHD), U22.6 (GND), U23.3 (GND), U23.8 (NC), U24.3 (GND), U24.8 (NC), U25.13 (SHD), U25.14 (SHD), U25.6 (GND), U26.3 (GND), U26.8 (NC), U27.3 (GND), U27.8 (NC), U28.13 (SHD), U28.14 (SHD), U28.6 (GND), U29.3 (GND), U29.8 (NC), U30.3 (GND), U30.8 (NC), U31.13 (SHD), U31.14 (SHD), U31.6 (GND), U32.3 (GND), U32.8 (NC), U33.3 (GND), U33.8 (NC), U34.13 (SHD), U34.14 (SHD), U34.6 (GND), U37.13 (SHD), U37.14 (SHD), U37.6 (GND), U39.3 (GND), U39.8 (NC), U501.3 (GND), U501.8 (NC)
- no-connect marks 0 -> 12
Other:
- note added: "Connectivity [7]"
- title: (none) -> Connectivity

Commit message: Finished schematic design - preparation for review
Parts:
- added R49, R50, R51, R52, R53, R54, R55, R56, R57, R58, R59, R60, R61, R62, R63, R64, R65, R66: 1k, Resistor_SMD:R_0402_1005Metric, symbol Device:R
- added U6: XC7A35T-CPG236, Package_BGA:Xilinx_CPG236, symbol Custom_VoxLink_Symbols:XC7A35T-CPG236
Connections:
- net GND: now also U14.10 (LED2), U14.12 (LED4), U16.10 (LED2), U16.12 (LED4), U17.10 (LED2), U17.12 (LED4), U22.10 (LED2), U22.12 (LED4), U25.10 (LED2), U25.12 (LED4), U28.10 (LED2), U28.12 (LED4), U31.10 (LED2), U31.12 (LED4), U34.10 (LED2), U34.12 (LED4), U37.10 (LED2), U37.12 (LED4)
- net P2_RX_P: now reaches U16.1 (RX), U20.2 (IN)
- net P2_RX_P: now also U20.9 (NC), U6.N18 (IO_L9P_T1_DQS_14)
- net at U16.11 (LED3): now also R52.2
- net P2_RX_N: now reaches U16.2 (~{RX}), U20.1 (IN)
- net P2_RX_N: now also U20.10 (NC), U6.N19 (IO_L9N_T1_DQS_D13_14)
- net P2_CLK_P: now reaches U15.4 (IN), U16.4 (CLK)
- net P2_CLK_P: now also U15.7 (NC), U6.J17 (IO_L7P_T1_D09_14)
- net P2_CLK_N: now reaches U15.5 (IN), U16.5 (~{CLK})
- net P2_CLK_N: now also U15.6 (NC), U6.J18 (IO_L7N_T1_D10_14)
- net P2_TX_N: now reaches U16.7 (~{TX}), U20.4 (IN)
- net P2_TX_N: now also U20.7 (NC), U6.K18 (IO_L8N_T1_D12_14)
- net P2_TX_P: now reaches U16.8 (TX), U20.5 (IN)
- net P2_TX_P: now also U20.6 (NC), U6.L18 (IO_L8P_T1_D11_14)
- net at U16.9 (LED1): now also R51.2
- net P3_RX_P: now reaches U17.1 (RX), U19.5 (IN)
- net P3_RX_P: now also U19.6 (NC), U6.L17 (IO_L12P_T1_MRCC_14)
- net at U17.11 (LED3): now also R54.2
- net P3_RX_N: now reaches U17.2 (~{RX}), U19.4 (IN)
- net P3_RX_N: now also U19.7 (NC), U6.K17 (IO_L12N_T1_MRCC_14)
- net P3_CLK_P: now reaches U17.4 (CLK), U18.5 (IN)
- net P3_CLK_P: now also U18.6 (NC), U6.P19 (IO_L10P_T1_D14_14)
- net P3_CLK_N: now reaches U17.5 (~{CLK}), U18.4 (IN)
- net P3_CLK_N: now also U18.7 (NC), U6.R19 (IO_L10N_T1_D15_14)
- net P3_TX_N: now reaches U17.7 (~{TX}), U18.1 (IN)
- net P3_TX_N: now also U18.10 (NC), U6.M19 (IO_L11N_T1_SRCC_14)
- net P3_TX_P: now reaches U17.8 (TX), U18.2 (IN)
- net P3_TX_P: now also U18.9 (NC), U6.M18 (IO_L11P_T1_SRCC_14)
- net at U17.9 (LED1): now also R53.2
- net P4_RX_P: now reaches U22.1 (RX), U27.1 (IN)
- net P4_RX_P: now also U27.10 (NC), U6.U19 (IO_L15P_T2_DQS_RDWR_B_14)
- net at U22.11 (LED3): now also R56.2
- net P4_RX_N: now reaches U22.2 (~{RX}), U27.2 (IN)
- net P4_RX_N: now also U27.9 (NC), U6.V19 (IO_L15N_T2_DQS_DOUT_CSO_B_14)
- net P4_CLK_P: now reaches U22.4 (CLK), U23.5 (IN)
- net P4_CLK_P: now also U23.6 (NC), U6.N17 (IO_L13P_T2_MRCC_14)
- net P4_CLK_N: now reaches U22.5 (~{CLK}), U23.4 (IN)
- net P4_CLK_N: now also U23.7 (NC), U6.P17 (IO_L13N_T2_MRCC_14)
- net P4_TX_N: now reaches U22.7 (~{TX}), U23.1 (IN)
- net P4_TX_N: now also U23.10 (NC), U6.R18 (IO_L14N_T2_SRCC_14)
- net P4_TX_P: now reaches U22.8 (TX), U23.2 (IN)
- net P4_TX_P: now also U23.9 (NC), U6.P18 (IO_L14P_T2_SRCC_14)
- net at U22.9 (LED1): now also R55.2
- net P7_TX_N: now reaches U31.7 (~{TX}), U32.1 (IN)
- net P7_TX_N: now also U32.10 (NC), U6.U16 (IO_L23N_T3_A02_D18_14)
- net P7_TX_P: now reaches U31.8 (TX), U32.2 (IN)
- net P7_TX_P: now also U32.9 (NC), U6.U15 (IO_L23P_T3_A03_D19_14)
- net P7_CLK_N: now reaches U31.5 (~{CLK}), U32.4 (IN)
- net P7_CLK_N: now also U32.7 (NC), U6.W14 (IO_L22N_T3_A04_D20_14)
- net P7_CLK_P: now reaches U31.4 (CLK), U32.5 (IN)
- net P7_CLK_P: now also U32.6 (NC), U6.W13 (IO_L22P_T3_A05_D21_14)
- net P5_RX_N: now reaches U24.1 (IN), U25.2 (~{RX})
- net P5_RX_N: now also U24.10 (NC), U6.U18 (IO_L18N_T2_A11_D27_14)
- net P5_RX_P: now reaches U24.2 (IN), U25.1 (RX)
- net P5_RX_P: now also U24.9 (NC), U6.U17 (IO_L18P_T2_A12_D28_14)
- net P5_TX_N: now reaches U24.4 (IN), U25.7 (~{TX})
- net P5_TX_N: now also U24.7 (NC), U6.T18 (IO_L17N_T2_A13_D29_14)
- net P5_TX_P: now reaches U24.5 (IN), U25.8 (TX)
- net P5_TX_P: now also U24.6 (NC), U6.T17 (IO_L17P_T2_A14_D30_14)
- net P6_RX_N: now reaches U28.2 (~{RX}), U30.4 (IN)
- net P6_RX_N: now also U30.7 (NC), U6.W15 (IO_L21N_T3_DQS_A06_D22_14)
- net P6_RX_P: now reaches U28.1 (RX), U30.5 (IN)
- net P6_RX_P: now also U30.6 (NC), U6.V15 (IO_L21P_T3_DQS_14)
- net P6_TX_N: now reaches U28.7 (~{TX}), U29.1 (IN)
- net P6_TX_N: now also U29.10 (NC), U6.W17 (IO_L20N_T3_A07_D23_14)
- net P6_TX_P: now reaches U28.8 (TX), U29.2 (IN)
- net P6_TX_P: now also U29.9 (NC), U6.W16 (IO_L20P_T3_A08_D24_14)
- net P6_CLK_N: now reaches U28.5 (~{CLK}), U29.4 (IN)
- net P6_CLK_N: now also U29.7 (NC), U6.V17 (IO_L19N_T3_A09_D25_VREF_14)
- net P6_CLK_P: now reaches U28.4 (CLK), U29.5 (IN)
- net P6_CLK_P: now also U29.6 (NC), U6.V16 (IO_L19P_T3_A10_D26_14)
- net P1_RX_P: now reaches U14.1 (RX), U15.1 (IN)
- net P1_RX_P: now also U15.10 (NC), U6.H17 (IO_L5P_T0_D06_14)
- net P1_RX_N: now reaches U14.2 (~{RX}), U15.2 (IN)
- net P1_RX_N: now also U15.9 (NC), U6.G17 (IO_L5N_T0_D07_14)
- net P5_CLK_P: now reaches U25.4 (CLK), U27.4 (IN)
- net P5_CLK_P: now also U27.7 (NC), U6.W18 (IO_L16P_T2_CSI_B_14)
- net P5_CLK_N: now reaches U25.5 (~{CLK}), U27.5 (IN)
- net P5_CLK_N: now also U27.6 (NC), U6.W19 (IO_L16N_T2_A15_D31_14)
- net P1_TX_N: now reaches U14.7 (~{TX}), U501.1 (IN)
- net P1_TX_N: now also U501.10 (NC), U6.G19 (IO_L4N_T0_D05_14)
- net P1_TX_P: now reaches U14.8 (TX), U501.2 (IN)
- net P1_TX_P: now also U501.9 (NC), U6.H19 (IO_L4P_T0_D04_14)
- net P1_CLK_N: now reaches U14.5 (~{CLK}), U501.4 (IN)
- net P1_CLK_N: now also U501.7 (NC), U6.E19 (IO_L3N_T0_DQS_EMCCLK_14)
- net P1_CLK_P: now reaches U14.4 (CLK), U501.5 (IN)
- net P1_CLK_P: now also U501.6 (NC), U6.E18 (IO_L3P_T0_DQS_PUDC_B_14)
- net at U28.11 (LED3): now also R60.2
- net at U28.9 (LED1): now also R59.2
- net at U14.11 (LED3): now also R50.2
- net at U14.9 (LED1): now also R49.2
- net P8_RX_N: now reaches U26.1 (IN), U34.2 (~{RX})
- net P8_RX_N: now also U26.10 (NC), U6.A17 (IO_L12N_T1_MRCC_16)
- net P8_RX_P: now reaches U26.2 (IN), U34.1 (RX)
- net P8_RX_P: now also U26.9 (NC), U6.A16 (IO_L12P_T1_MRCC_16)
- net P8_TX_N: now reaches U26.4 (IN), U34.7 (~{TX})
- net P8_TX_N: now also U26.7 (NC), U6.B15 (IO_L11N_T1_SRCC_16)
- net P8_TX_P: now reaches U26.5 (IN), U34.8 (TX)
- net P8_TX_P: now also U26.6 (NC), U6.C15 (IO_L11P_T1_SRCC_16)
- net P7_RX_P: now reaches U31.1 (RX), U33.1 (IN)
- net P7_RX_P: now also U33.10 (NC), U6.V13 (IO_L24P_T3_A01_D17_14)
- net P7_RX_N: now reaches U31.2 (~{RX}), U33.2 (IN)
- net P7_RX_N: now also U33.9 (NC), U6.V14 (IO_L24N_T3_A00_D16_14)
- net P8_CLK_P: now reaches U33.4 (IN), U34.4 (CLK)
- net P8_CLK_P: now also U33.7 (NC), U6.A14 (IO_L6P_T0_16)
- net P8_CLK_N: now reaches U33.5 (IN), U34.5 (~{CLK})
- net P8_CLK_N: now also U33.6 (NC), U6.A15 (IO_L6N_T0_VREF_16)
- net P9_RX_N: now reaches U37.2 (~{RX}), U39.4 (IN)
- net P9_RX_N: now also U39.7 (NC), U6.A18 (IO_L19N_T3_VREF_16)
- net P9_RX_P: now reaches U37.1 (RX), U39.5 (IN)
- net P9_RX_P: now also U39.6 (NC), U6.B18 (IO_L19P_T3_16)
- net at U31.11 (LED3): now also R62.2
- net at U31.9 (LED1): now also R61.2
- net P9_TX_N: now reaches U21.1 (IN), U37.7 (~{TX})
- net P9_TX_N: now also U21.10 (NC), U6.B17 (IO_L14N_T2_SRCC_16)
- net P9_TX_P: now reaches U21.2 (IN), U37.8 (TX)
- net P9_TX_P: now also U21.9 (NC), U6.C17 (IO_L14P_T2_SRCC_16)
- net P9_CLK_N: now reaches U21.4 (IN), U37.5 (~{CLK})
- net P9_CLK_N: now also U21.7 (NC), U6.B16 (IO_L13N_T2_MRCC_16)
- net P9_CLK_P: now reaches U21.5 (IN), U37.4 (CLK)
- net P9_CLK_P: now also U21.6 (NC), U6.C16 (IO_L13P_T2_MRCC_16)
- net at U34.11 (LED3): now also R64.2
- net at U34.9 (LED1): now also R63.2
- net at U25.11 (LED3): now also R58.2
- net at U25.9 (LED1): now also R57.2
- net at U37.11 (LED3): now also R66.2
- net at U37.9 (LED1): now also R65.2
- new net P1_L1: R49.1
- new net P1_L2: R50.1
- new net P2_L1: R51.1
- new net P2_L2: R52.1
- new net P3_L1: R53.1
- new net P3_L2: R54.1
- new net P4_L1: R55.1
- new net P4_L2: R56.1
- new net P5_L1: R57.1
- new net P5_L2: R58.1
- new net P6_L1: R59.1
- new net P6_L2: R60.1
- new net P7_L1: R61.1
- new net P7_L2: R62.1
- new net P8_L1: R63.1
- new net P8_L2: R64.1
- new net P9_L1: R65.1
- new net P9_L2: R66.1
- no-connect marks 12 -> 15
Other:
- moved on the sheet: U14, U16, U17, U18, U19, U21, U22, U23, U25, U28, U29, U30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

Commit message: Finished DRC check. Moving to schematic review
Parts:
- renumbered R49 to R701, R55 to R702, R61 to R703, R50 to R704, R56 to R705, R62 to R706, R51 to R707, R57 to R708, R63 to R709, R52 to R710, R58 to R711, R64 to R712, R53 to R713, R59 to R714, R65 to R715, R54 to R716, R60 to R717, R66 to R718, U6 to U201, U14 to U701, U22 to U702, U31 to U703, U501 to U704, U23 to U705, U32 to U706, U15 to U707, U27 to U708, U33 to U709, U16 to U710, U25 to U711, U34 to U712, U20 to U713, U24 to U714, U26 to U715, U17 to U716, U28 to U717, U37 to U718, U18 to U719, U29 to U720, U21 to U721, U19 to U722, U30 to U723, U39 to U724

Commit message: Finished the schematic review
Parts:
- added unit 8 of U201
- renumbered U722 to U723, U723 to U724, U724 to U725
Connections:
- net P1_CLK_N: now also U201.G2 (IO_L1N_T0_AD4N_35); no longer U201.E19 (IO_L3N_T0_DQS_EMCCLK_14)
- net P1_CLK_P: now also U201.G3 (IO_L1P_T0_AD4P_35); no longer U201.E18 (IO_L3P_T0_DQS_PUDC_B_14)
- net P1_RX_N: now also U201.J1 (IO_L3N_T0_DQS_AD5N_35); no longer U201.G17 (IO_L5N_T0_D07_14)
- net P1_RX_P: now also U201.H1 (IO_L3P_T0_DQS_AD5P_35); no longer U201.H17 (IO_L5P_T0_D06_14)
- net P1_TX_N: now also U201.J2 (IO_L2N_T0_AD12N_35); no longer U201.G19 (IO_L4N_T0_D05_14)
- net P1_TX_P: now also U201.H2 (IO_L2P_T0_AD12P_35); no longer U201.H19 (IO_L4P_T0_D04_14)
- net P5_L1: now also U201.H19 (IO_L4P_T0_D04_14)
- net P5_L2: now also U201.G19 (IO_L4N_T0_D05_14)
- net P6_L1: now also U201.H17 (IO_L5P_T0_D06_14)
- net P6_L2: now also U201.G17 (IO_L5N_T0_D07_14)
Other:
- moved on the sheet: R701, R702, R703, R704, R705, R706, R707, R708, R709, R710, R711, R712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

Commit message: Updated the documentation + minor scheme changes - Documented the schematic design - Added zener diode from USB VBUS to 5V
Parts:
- renumbered U723 to U722, U724 to U723, U725 to U724
Changed lines of the file:
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@@
 		(on_board yes)
 		(dnp no)
-		(property "Reference" "U723"
+		(property "Reference" "U722"
 			(at 87.63 210.058 0)
 			(effects
@@
 			(project "Controller_Board"
 				(path "/4e6e1af1-ede9-4a56-9d5f-a8dfd7fbcf8d/9851e49e-1b9b-43e7-98e9-5307aaba6efe"
-					(reference "U723")
+					(reference "U722")
 					(unit 1)
 				)
@@
 		(on_board yes)
 		(dnp no)
-		(property "Reference" "U724"
+		(property "Reference" "U723"
 			(at 162.56 210.058 0)
 			(effects
@@
 			(project "Controller_Board"
 				(path "/4e6e1af1-ede9-4a56-9d5f-a8dfd7fbcf8d/9851e49e-1b9b-43e7-98e9-5307aaba6efe"
-					(reference "U724")
+					(reference "U723")
 					(unit 1)
 				)
@@
 		(on_board yes)
 		(dnp no)
-		(property "Reference" "U725"
+		(property "Reference" "U724"
 			(at 237.49 210.058 0)
 			(effects
@@
 			(project "Controller_Board"
 				(path "/4e6e1af1-ede9-4a56-9d5f-a8dfd7fbcf8d/9851e49e-1b9b-43e7-98e9-5307aaba6efe"
-					(reference "U725")
+					(reference "U724")
 					(unit 1)
 				)

Commit message: Started schematic rework and the PCB design
Connections:
- net P1_CLK_N: now also U201.W17 (IO_L20N_T3_A07_D23_14); no longer U201.G2 (IO_L1N_T0_AD4N_35)
- net P1_CLK_P: now also U201.W16 (IO_L20P_T3_A08_D24_14); no longer U201.G3 (IO_L1P_T0_AD4P_35)
- net P1_RX_N: now also U201.V17 (IO_L19N_T3_A09_D25_VREF_14); no longer U201.J1 (IO_L3N_T0_DQS_AD5N_35)
- net P1_RX_P: now also U201.V16 (IO_L19P_T3_A10_D26_14); no longer U201.H1 (IO_L3P_T0_DQS_AD5P_35)
- net P1_TX_N: now also U201.W15 (IO_L21N_T3_DQS_A06_D22_14); no longer U201.J2 (IO_L2N_T0_AD12N_35)
- net P1_TX_P: now also U201.V15 (IO_L21P_T3_DQS_14); no longer U201.H2 (IO_L2P_T0_AD12P_35)
- net P3_CLK_N: now also U201.A15 (IO_L6N_T0_VREF_16); no longer U201.R19 (IO_L10N_T1_D15_14)
- net P3_CLK_P: now also U201.A14 (IO_L6P_T0_16); no longer U201.P19 (IO_L10P_T1_D14_14)
- net P3_RX_N: now also U201.A17 (IO_L12N_T1_MRCC_16); no longer U201.K17 (IO_L12N_T1_MRCC_14)
- net P3_RX_P: now also U201.A16 (IO_L12P_T1_MRCC_16); no longer U201.L17 (IO_L12P_T1_MRCC_14)
- net P3_TX_N: now also U201.B15 (IO_L11N_T1_SRCC_16); no longer U201.M19 (IO_L11N_T1_SRCC_14)
- net P3_TX_P: now also U201.C15 (IO_L11P_T1_SRCC_16); no longer U201.M18 (IO_L11P_T1_SRCC_14)
- net P5_CLK_N: now also U201.R19 (IO_L10N_T1_D15_14); no longer U201.W19 (IO_L16N_T2_A15_D31_14)
- net P5_CLK_P: now also U201.P19 (IO_L10P_T1_D14_14); no longer U201.W18 (IO_L16P_T2_CSI_B_14)
- net P5_RX_N: now also U201.K17 (IO_L12N_T1_MRCC_14); no longer U201.U18 (IO_L18N_T2_A11_D27_14)
- net P5_RX_P: now also U201.L17 (IO_L12P_T1_MRCC_14); no longer U201.U17 (IO_L18P_T2_A12_D28_14)
- net P5_TX_N: now also U201.M19 (IO_L11N_T1_SRCC_14); no longer U201.T18 (IO_L17N_T2_A13_D29_14)
- net P5_TX_P: now also U201.M18 (IO_L11P_T1_SRCC_14); no longer U201.T17 (IO_L17P_T2_A14_D30_14)
- net P6_CLK_N: now also U201.W19 (IO_L16N_T2_A15_D31_14); no longer U201.V17 (IO_L19N_T3_A09_D25_VREF_14)
- net P6_CLK_P: now also U201.W18 (IO_L16P_T2_CSI_B_14); no longer U201.V16 (IO_L19P_T3_A10_D26_14)
- net P6_RX_N: now also U201.U18 (IO_L18N_T2_A11_D27_14); no longer U201.W15 (IO_L21N_T3_DQS_A06_D22_14)
- net P6_RX_P: now also U201.U17 (IO_L18P_T2_A12_D28_14); no longer U201.V15 (IO_L21P_T3_DQS_14)
- net P6_TX_N: now also U201.T18 (IO_L17N_T2_A13_D29_14); no longer U201.W17 (IO_L20N_T3_A07_D23_14)
- net P6_TX_P: now also U201.T17 (IO_L17P_T2_A14_D30_14); no longer U201.W16 (IO_L20P_T3_A08_D24_14)
- net P7_CLK_N: now also U201.G2 (IO_L1N_T0_AD4N_35); no longer U201.W14 (IO_L22N_T3_A04_D20_14)
- net P7_CLK_P: now also U201.G3 (IO_L1P_T0_AD4P_35); no longer U201.W13 (IO_L22P_T3_A05_D21_14)
- net P7_RX_N: now also U201.J1 (IO_L3N_T0_DQS_AD5N_35); no longer U201.V14 (IO_L24N_T3_A00_D16_14)
- net P7_RX_P: now also U201.H1 (IO_L3P_T0_DQS_AD5P_35); no longer U201.V13 (IO_L24P_T3_A01_D17_14)
- net P7_TX_N: now also U201.J2 (IO_L2N_T0_AD12N_35); no longer U201.U16 (IO_L23N_T3_A02_D18_14)
- net P7_TX_P: now also U201.H2 (IO_L2P_T0_AD12P_35); no longer U201.U15 (IO_L23P_T3_A03_D19_14)
- net P8_CLK_N: now also U201.W14 (IO_L22N_T3_A04_D20_14); no longer U201.A15 (IO_L6N_T0_VREF_16)
- net P8_CLK_P: now also U201.W13 (IO_L22P_T3_A05_D21_14); no longer U201.A14 (IO_L6P_T0_16)
- net P8_RX_N: now also U201.U16 (IO_L23N_T3_A02_D18_14); no longer U201.A17 (IO_L12N_T1_MRCC_16)
- net P8_RX_P: now also U201.U15 (IO_L23P_T3_A03_D19_14); no longer U201.A16 (IO_L12P_T1_MRCC_16)
- net P8_TX_N: now also U201.V14 (IO_L24N_T3_A00_D16_14); no longer U201.B15 (IO_L11N_T1_SRCC_16)
- net P8_TX_P: now also U201.V13 (IO_L24P_T3_A01_D17_14); no longer U201.C15 (IO_L11P_T1_SRCC_16)

Commit message: Commit before upgrading to KiCad 10.0
Parts:
- removed U201: XC7A35T-CPG236, Package_BGA:Xilinx_CPG236, symbol Custom_VoxLink_Symbols:XC7A35T-CPG236
- added U201: XC7A35T-CSG324, Package_BGA:Xilinx_CSG324, symbol Custom_VoxLink_Symbols:XC7A35T-CSG324
Connections:
- net P3_CLK_N: now also U201.U18 (IO_L17N_T2_A13_D29_14)
- net P3_CLK_P: now also U201.U17 (IO_L17P_T2_A14_D30_14)
- net P3_RX_N: now also U201.T18 (IO_L7N_T1_D10_14)
- net P3_RX_P: now also U201.R18 (IO_L7P_T1_D09_14)
- net P3_TX_N: now also U201.V17 (IO_L18N_T2_A11_D27_14)
- net P3_TX_P: now also U201.U16 (IO_L18P_T2_A12_D28_14)
- net P4_CLK_N: now also U201.V11 (IO_L21N_T3_DQS_A06_D22_14)
- net P4_CLK_P: now also U201.V10 (IO_L21P_T3_DQS_14)
- net P4_RX_N: now also U201.V12 (IO_L20N_T3_A07_D23_14)
- net P4_RX_P: now also U201.U12 (IO_L20P_T3_A08_D24_14)
- net P4_TX_N: now also U201.V9 (IO_L21N_T3_DQS_34)
- net P4_TX_P: now also U201.U9 (IO_L21P_T3_DQS_34)
- net P5_CLK_N: now also U201.V14 (IO_L22N_T3_A04_D20_14)
- net P5_CLK_P: now also U201.U14 (IO_L22P_T3_A05_D21_14)
- net P5_RX_N: now also U201.V16 (IO_L16N_T2_A15_D31_14)
- net P5_RX_P: now also U201.V15 (IO_L16P_T2_CSI_B_14)
- net P5_TX_N: now also U201.U13 (IO_L23N_T3_A02_D18_14)
- net P5_TX_P: now also U201.T13 (IO_L23P_T3_A03_D19_14)
- no-connect marks 15 -> 12
Other:
- moved on the sheet: R701, R702, R703, R704, R705, R706, R707, R708, R709, R710, R711, R712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

Commit message: Converted to 10.0 KiCad schematic + Began BGA fan
Connections:
- net P1_CLK_N: now also U201.V1 (IO_L7N_T1_34)
- net P1_CLK_P: now also U201.U1 (IO_L7P_T1_34)
- net P1_RX_N: now also U201.V2 (IO_L9N_T1_DQS_34)
- net P1_RX_P: now also U201.U2 (IO_L9P_T1_DQS_34)
- net P1_TX_N: now also U201.T1 (IO_L17N_T2_34)
- net P1_TX_P: now also U201.R1 (IO_L17P_T2_34)
- net P2_CLK_N: now also U201.G17 (IO_L18N_T2_A23_15)
- net P2_CLK_P: now also U201.H17 (IO_L18P_T2_A24_15)
- net P2_RX_N: now also U201.F18 (IO_L22N_T3_A16_15)
- net P2_RX_P: now also U201.G18 (IO_L22P_T3_A17_15)
- net P2_TX_N: now also U201.J18 (IO_L23N_T3_FWE_B_15)
- net P2_TX_P: now also U201.J17 (IO_L23P_T3_FOE_B_15)
- net P3_CLK_N: now also U201.P18 (IO_L9N_T1_DQS_D13_14); no longer U201.U18 (IO_L17N_T2_A13_D29_14)
- net P3_CLK_P: now also U201.N17 (IO_L9P_T1_DQS_14); no longer U201.U17 (IO_L17P_T2_A14_D30_14)
- net P3_RX_N: now also U201.M18 (IO_L4N_T0_D05_14); no longer U201.T18 (IO_L7N_T1_D10_14)
- net P3_RX_P: now also U201.L18 (IO_L4P_T0_D04_14); no longer U201.R18 (IO_L7P_T1_D09_14)
- net P3_TX_N: now also U201.T18 (IO_L7N_T1_D10_14); no longer U201.V17 (IO_L18N_T2_A11_D27_14)
- net P3_TX_P: now also U201.R18 (IO_L7P_T1_D09_14); no longer U201.U16 (IO_L18P_T2_A12_D28_14)
- net P4_CLK_N: now also U201.V12 (IO_L20N_T3_A07_D23_14); no longer U201.V11 (IO_L21N_T3_DQS_A06_D22_14)
- net P4_CLK_P: now also U201.U12 (IO_L20P_T3_A08_D24_14); no longer U201.V10 (IO_L21P_T3_DQS_14)
- net P4_RX_N: now also U201.V14 (IO_L22N_T3_A04_D20_14); no longer U201.V12 (IO_L20N_T3_A07_D23_14)
- net P4_RX_P: now also U201.U14 (IO_L22P_T3_A05_D21_14); no longer U201.U12 (IO_L20P_T3_A08_D24_14)
- net P4_TX_N: now also U201.V11 (IO_L21N_T3_DQS_A06_D22_14); no longer U201.V9 (IO_L21N_T3_DQS_34)
- net P4_TX_P: now also U201.V10 (IO_L21P_T3_DQS_14); no longer U201.U9 (IO_L21P_T3_DQS_34)
- net P5_CLK_N: now also U201.V17 (IO_L18N_T2_A11_D27_14); no longer U201.V14 (IO_L22N_T3_A04_D20_14)
- net P5_CLK_P: now also U201.U16 (IO_L18P_T2_A12_D28_14); no longer U201.U14 (IO_L22P_T3_A05_D21_14)
- net P5_RX_N: now also U201.U18 (IO_L17N_T2_A13_D29_14); no longer U201.V16 (IO_L16N_T2_A15_D31_14)
- net P5_RX_P: now also U201.U17 (IO_L17P_T2_A14_D30_14); no longer U201.V15 (IO_L16P_T2_CSI_B_14)
- net P5_TX_N: now also U201.V16 (IO_L16N_T2_A15_D31_14); no longer U201.U13 (IO_L23N_T3_A02_D18_14)
- net P5_TX_P: now also U201.V15 (IO_L16P_T2_CSI_B_14); no longer U201.T13 (IO_L23P_T3_A03_D19_14)
- net P6_CLK_N: now also U201.V6 (IO_L20N_T3_34)
- net P6_CLK_P: now also U201.V7 (IO_L20P_T3_34)
- net P6_RX_N: now also U201.V9 (IO_L21N_T3_DQS_34)
- net P6_RX_P: now also U201.U9 (IO_L21P_T3_DQS_34)
- net P6_TX_N: now also U201.V4 (IO_L10N_T1_34)
- net P6_TX_P: now also U201.V5 (IO_L10P_T1_34)
- net P7_CLK_N: now also U201.E1 (IO_L18N_T2_35)
- net P7_CLK_P: now also U201.F1 (IO_L18P_T2_35)
- net P7_RX_N: now also U201.G1 (IO_L17N_T2_35)
- net P7_RX_P: now also U201.H1 (IO_L17P_T2_35)
- net P7_TX_N: now also U201.C1 (IO_L16N_T2_35)
- net P7_TX_P: now also U201.C2 (IO_L16P_T2_35)
- net P8_CLK_N: now also U201.K1 (IO_L23N_T3_35)
- net P8_CLK_P: now also U201.K2 (IO_L23P_T3_35)
- net P8_RX_N: now also U201.M2 (IO_L4N_T0_34)
- net P8_RX_P: now also U201.M3 (IO_L4P_T0_34)
- net P8_TX_N: now also U201.J2 (IO_L22N_T3_35)
- net P8_TX_P: now also U201.J3 (IO_L22P_T3_35)
- net P9_CLK_N: now also U201.C17 (IO_L20N_T3_A19_15)
- net P9_CLK_P: now also U201.C16 (IO_L20P_T3_A20_15)
- net P9_RX_N: now also U201.A18 (IO_L10N_T1_AD11N_15)
- net P9_RX_P: now also U201.B18 (IO_L10P_T1_AD11P_15)
- net P9_TX_N: now also U201.D18 (IO_L21N_T3_DQS_A18_15)
- net P9_TX_P: now also U201.E18 (IO_L21P_T3_DQS_15)
