File: Hardware/Controller_Board/connectivity.kicad_sch (KiCad schematic)
At the start: 43 parts, among them U201 XC7A35T-CSG324, U701 RJ45, U702 RJ45, U703 RJ45, U704 TPD4E02B04, U705 TPD4E02B04, U706 TPD4E02B04, U707 TPD4E02B04, U708 TPD4E02B04, U709 TPD4E02B04, U710 RJ45, U711 RJ45, U712 RJ45, U713 TPD4E02B04, U714 TPD4E02B04, U715 TPD4E02B04, U716 RJ45, U717 RJ45, U718 RJ45, U719 TPD4E02B04, U720 TPD4E02B04, U721 TPD4E02B04, U722 TPD4E02B04, U723 TPD4E02B04, U724 TPD4E02B04

Commit message: Advanced PCB routing and reorganized FPGA traces
Parts:
- removed U707, U708, U709: TPD4E02B04, Package_SON:USON-10_2.5x1.0mm_P0.5mm, symbol Custom_VoxLink_Symbols:TPD4E02B04DQA_Tall
- added U725, U726, U727, U728, U729, U730: TPD4E02B04, Package_SON:USON-10_2.5x1.0mm_P0.5mm, symbol Custom_VoxLink_Symbols:TPD4E02B04DQA
Connections:
- net GND: now also U725.3 (GND), U725.8 (NC), U726.3 (GND), U726.8 (NC), U727.3 (GND), U727.8 (NC), U728.3 (GND), U728.8 (NC), U729.3 (GND), U729.8 (NC), U730.3 (GND), U730.8 (NC)
- net P1_CLK_N: now also U201.R2 (IO_L15N_T2_DQS_34); no longer U201.V1 (IO_L7N_T1_34)
- net P1_CLK_P: now also U201.P2 (IO_L15P_T2_DQS_34); no longer U201.U1 (IO_L7P_T1_34)
- net P1_RX_N: now also U201.V1 (IO_L7N_T1_34), U725.5 (IN), U725.6 (NC); no longer U201.V2 (IO_L9N_T1_DQS_34)
- net P1_RX_P: now also U201.U1 (IO_L7P_T1_34), U725.4 (IN), U725.7 (NC); no longer U201.U2 (IO_L9P_T1_DQS_34)
- net P1_TX_N: now also U201.N1 (IO_L3N_T0_DQS_34); no longer U201.T1 (IO_L17N_T2_34)
- net P1_TX_P: now also U201.N2 (IO_L3P_T0_DQS_34); no longer U201.R1 (IO_L17P_T2_34)
- net P2_CLK_N: now also U201.J18 (IO_L23N_T3_FWE_B_15), U726.1 (IN), U726.10 (NC); no longer U201.G17 (IO_L18N_T2_A23_15)
- net P2_CLK_P: now also U201.J17 (IO_L23P_T3_FOE_B_15), U726.2 (IN), U726.9 (NC); no longer U201.H17 (IO_L18P_T2_A24_15)
- net P2_RX_N: now also U201.G17 (IO_L18N_T2_A23_15); no longer U201.F18 (IO_L22N_T3_A16_15)
- net P2_RX_P: now also U201.H17 (IO_L18P_T2_A24_15); no longer U201.G18 (IO_L22P_T3_A17_15)
- net P2_TX_N: now also U201.M18 (IO_L4N_T0_D05_14); no longer U201.J18 (IO_L23N_T3_FWE_B_15)
- net P2_TX_P: now also U201.L18 (IO_L4P_T0_D04_14); no longer U201.J17 (IO_L23P_T3_FOE_B_15)
- net P3_CLK_N: now also U201.T18 (IO_L7N_T1_D10_14); no longer U201.P18 (IO_L9N_T1_DQS_D13_14)
- net P3_CLK_P: now also U201.R18 (IO_L7P_T1_D09_14); no longer U201.N17 (IO_L9P_T1_DQS_14)
- net P3_RX_N: now also U201.P18 (IO_L9N_T1_DQS_D13_14); no longer U201.M18 (IO_L4N_T0_D05_14)
- net P3_RX_P: now also U201.N17 (IO_L9P_T1_DQS_14); no longer U201.L18 (IO_L4P_T0_D04_14)
- net P3_TX_N: now also U201.U18 (IO_L17N_T2_A13_D29_14); no longer U201.T18 (IO_L7N_T1_D10_14)
- net P3_TX_P: now also U201.U17 (IO_L17P_T2_A14_D30_14); no longer U201.R18 (IO_L7P_T1_D09_14)
- net P4_CLK_N: now also U201.U11 (IO_L19N_T3_A09_D25_VREF_14); no longer U201.V12 (IO_L20N_T3_A07_D23_14)
- net P4_CLK_P: now also U201.T11 (IO_L19P_T3_A10_D26_14); no longer U201.U12 (IO_L20P_T3_A08_D24_14)
- net P4_RX_N: now also U201.V12 (IO_L20N_T3_A07_D23_14), U727.5 (IN), U727.6 (NC); no longer U201.V14 (IO_L22N_T3_A04_D20_14)
- net P4_RX_P: now also U201.U12 (IO_L20P_T3_A08_D24_14), U727.4 (IN), U727.7 (NC); no longer U201.U14 (IO_L22P_T3_A05_D21_14)
- net P4_TX_N: now also U201.V9 (IO_L21N_T3_DQS_34); no longer U201.V11 (IO_L21N_T3_DQS_A06_D22_14)
- net P4_TX_P: now also U201.U9 (IO_L21P_T3_DQS_34); no longer U201.V10 (IO_L21P_T3_DQS_14)
- net P5_CLK_N: now also U201.V16 (IO_L16N_T2_A15_D31_14), U728.1 (IN), U728.10 (NC); no longer U201.V17 (IO_L18N_T2_A11_D27_14)
- net P5_CLK_P: now also U201.V15 (IO_L16P_T2_CSI_B_14), U728.2 (IN), U728.9 (NC); no longer U201.U16 (IO_L18P_T2_A12_D28_14)
- net P5_RX_N: now also U201.V17 (IO_L18N_T2_A11_D27_14); no longer U201.U18 (IO_L17N_T2_A13_D29_14)
- net P5_RX_P: now also U201.U16 (IO_L18P_T2_A12_D28_14); no longer U201.U17 (IO_L17P_T2_A14_D30_14)
- net P5_TX_N: now also U201.V14 (IO_L22N_T3_A04_D20_14); no longer U201.V16 (IO_L16N_T2_A15_D31_14)
- net P5_TX_P: now also U201.U14 (IO_L22P_T3_A05_D21_14); no longer U201.V15 (IO_L16P_T2_CSI_B_14)
- net P6_CLK_N: now also U201.V4 (IO_L10N_T1_34); no longer U201.V6 (IO_L20N_T3_34)
- net P6_CLK_P: now also U201.V5 (IO_L10P_T1_34); no longer U201.V7 (IO_L20P_T3_34)
- net P6_RX_N: now also U201.V6 (IO_L20N_T3_34), U723.5 (IN), U723.6 (NC); no longer U201.V9 (IO_L21N_T3_DQS_34), U723.4 (IN), U723.7 (NC)
- net P6_RX_P: now also U201.V7 (IO_L20P_T3_34), U723.4 (IN), U723.7 (NC); no longer U201.U9 (IO_L21P_T3_DQS_34), U723.5 (IN), U723.6 (NC)
- net P6_TX_N: now also U201.V2 (IO_L9N_T1_DQS_34), U720.2 (IN), U720.9 (NC); no longer U201.V4 (IO_L10N_T1_34), U720.1 (IN), U720.10 (NC)
- net P6_TX_P: now also U201.U2 (IO_L9P_T1_DQS_34), U720.1 (IN), U720.10 (NC); no longer U201.V5 (IO_L10P_T1_34), U720.2 (IN), U720.9 (NC)
- net P7_RX_N: now also U729.4 (IN), U729.7 (NC)
- net P7_RX_P: now also U729.5 (IN), U729.6 (NC)
- net P8_CLK_N: now also U730.1 (IN), U730.10 (NC)
- net P8_CLK_P: now also U730.2 (IN), U730.9 (NC)
- no-connect marks 12 -> 36

Commit message: Commiting PCB design with 45 degree tracks
Connections:
- net P1_RX_N: now also U725.1 (IN), U725.10 (NC); no longer U725.5 (IN), U725.6 (NC)
- net P1_RX_P: now also U725.2 (IN), U725.9 (NC); no longer U725.4 (IN), U725.7 (NC)
- net P2_CLK_N: now also U713.2 (IN), U713.9 (NC); no longer U726.1 (IN), U726.10 (NC)
- net P2_CLK_P: now also U713.1 (IN), U713.10 (NC); no longer U726.2 (IN), U726.9 (NC)
- net P2_RX_N: now also U726.5 (IN), U726.6 (NC); no longer U713.1 (IN), U713.10 (NC)
- net P2_RX_P: now also U726.4 (IN), U726.7 (NC); no longer U713.2 (IN), U713.9 (NC)
- net P2_TX_N: now also U713.5 (IN), U713.6 (NC); no longer U713.4 (IN), U713.7 (NC)
- net P2_TX_P: now also U713.4 (IN), U713.7 (NC); no longer U713.5 (IN), U713.6 (NC)
- net P3_CLK_N: now also U719.2 (IN), U719.9 (NC); no longer U719.4 (IN), U719.7 (NC)
- net P3_CLK_P: now also U719.1 (IN), U719.10 (NC); no longer U719.5 (IN), U719.6 (NC)
- net P3_RX_N: now also U722.5 (IN), U722.6 (NC); no longer U722.4 (IN), U722.7 (NC)
- net P3_RX_P: now also U722.4 (IN), U722.7 (NC); no longer U722.5 (IN), U722.6 (NC)
- net P3_TX_N: now also U719.5 (IN), U719.6 (NC); no longer U719.1 (IN), U719.10 (NC)
- net P3_TX_P: now also U719.4 (IN), U719.7 (NC); no longer U719.2 (IN), U719.9 (NC)
- net P4_RX_N: now also U727.1 (IN), U727.10 (NC); no longer U727.5 (IN), U727.6 (NC)
- net P4_RX_P: now also U727.2 (IN), U727.9 (NC); no longer U727.4 (IN), U727.7 (NC)
- net P5_CLK_N: now also U714.4 (IN), U714.7 (NC); no longer U728.1 (IN), U728.10 (NC)
- net P5_CLK_P: now also U714.5 (IN), U714.6 (NC); no longer U728.2 (IN), U728.9 (NC)
- net P5_RX_N: now also U728.1 (IN), U728.10 (NC); no longer U714.1 (IN), U714.10 (NC)
- net P5_RX_P: now also U728.2 (IN), U728.9 (NC); no longer U714.2 (IN), U714.9 (NC)
- net P5_TX_N: now also U714.2 (IN), U714.9 (NC); no longer U714.4 (IN), U714.7 (NC)
- net P5_TX_P: now also U714.1 (IN), U714.10 (NC); no longer U714.5 (IN), U714.6 (NC)
- net P6_RX_N: now also U723.1 (IN), U723.10 (NC); no longer U723.5 (IN), U723.6 (NC)
- net P6_RX_P: now also U723.2 (IN), U723.9 (NC); no longer U723.4 (IN), U723.7 (NC)
- net P6_TX_N: now also U720.1 (IN), U720.10 (NC); no longer U720.2 (IN), U720.9 (NC)
- net P6_TX_P: now also U720.2 (IN), U720.9 (NC); no longer U720.1 (IN), U720.10 (NC)
- net P7_RX_N: now also U729.1 (IN), U729.10 (NC); no longer U729.4 (IN), U729.7 (NC)
- net P7_RX_P: now also U729.2 (IN), U729.9 (NC); no longer U729.5 (IN), U729.6 (NC)
- net P8_CLK_N: now also U730.4 (IN), U730.7 (NC); no longer U730.1 (IN), U730.10 (NC)
- net P8_CLK_P: now also U730.5 (IN), U730.6 (NC); no longer U730.2 (IN), U730.9 (NC)
- net P8_TX_N: now also U730.1 (IN), U730.10 (NC); no longer U715.4 (IN), U715.7 (NC)
- net P8_TX_P: now also U730.2 (IN), U730.9 (NC); no longer U715.5 (IN), U715.6 (NC)
- net P9_CLK_N: now also U724.5 (IN), U724.6 (NC); no longer U721.4 (IN), U721.7 (NC)
- net P9_CLK_P: now also U724.4 (IN), U724.7 (NC); no longer U721.5 (IN), U721.6 (NC)
- net P9_RX_N: now also U724.2 (IN), U724.9 (NC); no longer U724.4 (IN), U724.7 (NC)
- net P9_RX_P: now also U724.1 (IN), U724.10 (NC); no longer U724.5 (IN), U724.6 (NC)

Commit message: Advanced PCB design: Routed FTDIs + SPI Flash
Connections:
- net SERIAL_D2: now reaches U201.A1 (IO_L9N_T1_DQS_AD7N_35)
- net SERIAL_D5: now reaches U201.A3 (IO_L8N_T1_AD14N_35)
- net SERIAL_D7: now reaches U201.A4 (IO_L8P_T1_AD14P_35)
- net SERIAL_D8: now reaches U201.A5 (IO_L3N_T0_DQS_AD5N_35)
- net SERIAL_PWR#: now reaches U201.A6 (IO_L3P_T0_DQS_AD5P_35)
- net SERIAL_D1: now reaches U201.B1 (IO_L9P_T1_DQS_AD7P_35)
- net SERIAL_D3: now reaches U201.B2 (IO_L10N_T1_AD15N_35)
- net SERIAL_D4: now reaches U201.B3 (IO_L10P_T1_AD15P_35)
- net SERIAL_D6: now reaches U201.B4 (IO_L7N_T1_AD6N_35)
- net SERIAL_OE#: now reaches U201.B7 (IO_L2P_T0_AD12P_35)
- net SERIAL_SIWU#: now reaches U201.C4 (IO_L7P_T1_AD6P_35)
- net SERIAL_TXE#: now reaches U201.D2 (IO_L14N_T2_SRCC_35)
- net SERIAL_RXF#: now reaches U201.D3 (IO_L12N_T1_MRCC_35)
- net SERIAL_WR#: now reaches U201.D5 (IO_L11P_T1_SRCC_35)
- net SERIAL_RD#: now reaches U201.E2 (IO_L14P_T2_SRCC_35)
- net SERIAL_CLK: now reaches U201.E3 (IO_L12P_T1_MRCC_35)

Commit message: Advanced PCB design - Routed FTDI chips + USB HUB
Parts:
- added H1, H2, H3, H4: M3, MountingHole:MountingHole_3.2mm_M3_Pad_Via, symbol Mechanical:MountingHole_Pad
Connections:
- net GND: now also H1.1, H2.1, H3.1, H4.1
- net P1_L1: now also U201.U3 (IO_L8N_T1_34)
- net P1_L2: now also U201.U4 (IO_L8P_T1_34)
- net P2_L1: now also U201.R17 (IO_L12N_T1_MRCC_14)
- net P2_L2: now also U201.P17 (IO_L12P_T1_MRCC_14)
- net P3_L1: now also U201.R15 (IO_L13N_T2_MRCC_14)
- net P3_L2: now also U201.R16 (IO_L15P_T2_DQS_RDWR_B_14)
- net P4_L1: now also U201.T9 (IO_L24P_T3_A01_D17_14)
- net P4_L2: now also U201.T10 (IO_L24N_T3_A00_D16_14)
- net P5_L1: now also U201.T14 (IO_L14P_T2_SRCC_14)
- net P5_L2: now also U201.T15 (IO_L14N_T2_SRCC_14)
- net P6_L1: now also U201.U6 (IO_L22N_T3_34)
- net P6_L2: now also U201.U7 (IO_L22P_T3_34)
- net P7_L1: now also U201.L3 (IO_L2N_T0_34)
- net P7_L2: now also U201.K3 (IO_L2P_T0_34)
- net P8_L1: now also U201.P4 (IO_L14P_T2_SRCC_34)
- net P8_L2: now also U201.P5 (IO_L13N_T2_MRCC_34)
- net P9_L1: now also U201.A16 (IO_L8N_T1_AD10N_15)
- net P9_L2: now also U201.A15 (IO_L8P_T1_AD10P_15)

Commit message: Advanced PCB Design: Routing Power + UVLO
Parts:
- added D605, D606, D607, D608, D609, D610, D611, D612, D613: TVS, Diode_SMD:D_0402_1005Metric, symbol Device:D_TVS
Connections:
- net +5V: now also D605.2 (A2), D606.2 (A2), D607.2 (A2), D608.2 (A2), D609.2 (A2), D610.2 (A2), D611.2 (A2), D612.2 (A2), D613.2 (A2)
- net GND: now also D605.1 (A1), D606.1 (A1), D607.1 (A1), D608.1 (A1), D609.1 (A1), D610.1 (A1), D611.1 (A1), D612.1 (A1), D613.1 (A1)

Commit message: Finished PCB Design - WARNING MORE CHANGES NEEDED! The main decision to be made is, whether to increase the layer count to 8 layers, and make the P7 and P8 permamently on 3V3
Parts:
- renumbered D605 to D801, D606 to D802, D607 to D803, D608 to D804, D609 to D805, D610 to D806, D611 to D807, D612 to D808, D613 to D809, H1 to H801, H2 to H802, H3 to H803, H4 to H804, R701 to R801, R702 to R802, R703 to R803, R704 to R804, R705 to R805, R706 to R806, R707 to R807, R708 to R808, R709 to R809, R710 to R810, R711 to R811, R712 to R812, R713 to R813, R714 to R814, R715 to R815, R716 to R816, R717 to R817, R718 to R818, U201 to U301, U701 to U801, U702 to U802, U703 to U803, U704 to U804, U705 to U805, U706 to U806, U725 to U807, U727 to U808, U729 to U809, U710 to U810, U711 to U811, U712 to U812, U713 to U813, U714 to U814, U730 to U815, U726 to U816, U728 to U817, U715 to U818, U716 to U819, U717 to U820, U718 to U821, U719 to U822, U720 to U823, U724 to U824, U722 to U825, U723 to U826, U721 to U827
Connections:
- no-connect marks 36 -> 141
Other:
- note added: "Connectivity [8]"
- note added: "Please exuse this mess, I'll try to make this pretty later"
- note removed: "Connectivity [7]"
- moved on the sheet: D801, D802, D803, D804, D805, D806, D807, D808, D809, H801, H802, H803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

Commit message: Finished procuring almost all boards - CHANGED XDC IN XILINX FOR TESTING!! - Programmer needed
Parts:
- D801, D802, D803, D804, D805, D806, D807, D808, D809: LCSC (none) -> C1973340; Manufacturer (none) -> Littelfuse
- R801, R802, R803, R804, R805, R806, R807, R808, R809, R810, R811, R812, R813, R814, R815, R816, R817, R818: LCSC (none) -> C71623; Manufacturer (none) -> Vishay
- U301: LCSC (none) -> C1521726; Manufacturer (none) -> Xilinx
- U801, U802, U803, U810, U811, U812, U819, U820, U821: LCSC (none) -> C125068; Manufacturer (none) -> TE
- U804, U805, U806, U807, U808, U809, U813, U814, U815, U816, U817, U818, U822, U823, U824, U825, U826, U827: LCSC (none) -> C106794; Manufacturer (none) -> TI
Connections:
- net P8_RX_N: now also U301.H4 (IO_L21N_T3_DQS_35); no longer U301.M2 (IO_L4N_T0_34)
- net P8_RX_P: now also U301.J4 (IO_L21P_T3_DQS_35); no longer U301.M3 (IO_L4P_T0_34)
