File: Hardware/Controller_Board/usb.kicad_sch (KiCad schematic)
At the start: 0 parts

Commit message: Added USB hub symbol
Parts:
- added U12: ~, Package_DFN_QFN:QFN-36-1EP_6x6mm_P0.5mm_EP3.7x3.7mm, symbol Custom_VoxLink_Symbols:USB2512
Connections:
- new net: U12.18 (NC), U12.19 (NC), U12.20 (NC), U12.21 (NC), U12.6 (NC), U12.7 (NC), U12.8 (NC), U12.9 (NC)
- no-connect marks 0 -> 5
Other:
- note added: "Make it more pretty"
- note added: "OCS have internal pullup resistors Since we have non-removable devices we won't check the over-current"
Changed lines of the file:
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@@
 		(comment 1 "Designer: Michal Varsanyi")
 	)
+	(text "Make it more pretty"
+		(exclude_from_sim no)
+		(at 180.594 131.064 0)
+		(effects
+			(font
+				(size 1.27 1.27)
+			)
+		)
+	)
+	(text "OCS have internal pullup resistors\nSince we have non-removable devices\nwe won't check the over-current"
+		(exclude_from_sim no)
+		(at 90.17 98.298 0)
+		(effects
+			(font
+				(size 1.27 1.27)
+			)
+		)
+	)
+	(no_connect
+		(at 148.59 96.52)
+	)
+	(no_connect
+		(at 113.03 96.52)
+	)
+	(no_connect
+		(at 113.03 99.06)
+	)
+	(no_connect
+		(at 148.59 99.06)
+	)
+	(no_connect
+		(at 113.03 101.6)
+	)
+	(symbol
+		(lib_id "Custom_VoxLink_Symbols:USB2512")
+		(at 101.6 134.62 0)
+		(unit 1)
+		(exclude_from_sim no)
+		(in_bom yes)
+		(on_board yes)
+		(dnp no)
+		(fields_autoplaced yes)
+		(property "Reference" "U12"
+			(at 130.4133 130.81 0)
+			(effects
+				(font
+					(size 1.27 1.27)
+				)
+				(justify left)
+			)
+		)
+		(property "Value" "~"
+			(at 130.4133 133.35 0)
+			(effects
+				(font
+					(size 1.27 1.27)
+				)
+				(justify left)
+			)
+		)
+		(property "Footprint" "Package_DFN_QFN:QFN-36-1EP_6x6mm_P0.5mm_EP3.7x3.7mm"
+			(at 101.6 134.62 0)
+			(effects
+				(font
+					(size 1.27 1.27)
+				)
+				(hide yes)
+			)
+		)
+		(property "Datasheet" "https://www.mouser.sk/ProductDetail/Microchip-Technology/USB2532-1080AEN-TR?qs=3i1%252BhB2xfwnqLAgBp2F6Xg%3D%3D"
+			(at 101.6 134.62 0)
+			(effects
+				(font
+					(size 1.27 1.27)
+				)
+				(hide yes)
+			)
+		)
+		(property "Description" ""
+			(at 101.6 134.62 0)
+			(effects
+				(font
+					(size 1.27 1.27)
+				)
+				(hide yes)
+			)
+		)
+		(pin "24"
+		)
+		(pin "28"
+		)
+		(pin "22"
+		)
+		(pin ""
+		)
+		(pin ""
+		)
+		(pin "25"
+		)
+		(pin "21"
+		)
+		(pin "18"
+		)
+		(pin "7"
+		)
+		(pin "13"
+		)
+		(pin "17"
+		)
+		(pin "19"
+		)
+		(pin "27"
+		)
+		(pin "11"
+		)
+		(pin "6"
+		)
+		(pin "8"
+		)
+		(pin "20"
+		)
+		(pin "9"
+		)
+		(pin "14"
+		)
+		(pin "34"
+		)
+		(pin "32"
+		)
+		(pin "33"
+		)
+		(pin "4"
+		)
+		(pin "16"
+		)
+		(pin "12"
+		)
+		(pin "35"
+		)
+		(pin "1"
+		)
+		(pin "36"
+		)
+		(pin "2"
+		)
+		(pin "3"
+		)
+		(pin "5"
+		)
+		(pin "15"
+		)
+		(pin "29"
+		)
+		(pin "10"
+		)
+		(pin "37"
+		)
+		(pin "23"
+		)
+		(pin "26"
+		)
+		(instances
+			(project ""
+				(path "/4e6e1af1-ede9-4a56-9d5f-a8dfd7fbcf8d/6841ebe0-d0f7-414d-8e63-132e7a23cd7b"
+					(reference "U12")
+					(unit 1)
+				)
+			)
+		)
+	)
 )

Commit message: Updated the schematic design - Fix the XC7A35T-CPG236 outline issue
Parts:
- added C105, C106: 10p, Capacitor_SMD:C_0402_1005Metric, symbol Device:C
- added C107: 4u7, Capacitor_SMD:C_0402_1005Metric, symbol Device:C
- added C108, C109, C110, C111, C112, C113, C115, C117: 100n, Capacitor_SMD:C_0402_1005Metric, symbol Device:C
- added C114, C116: 10n, Capacitor_SMD:C_0402_1005Metric, symbol Device:C
- added D104: TVS, Diode_SMD:D_0402_1005Metric, symbol Diode:1.5KExxA
- added D105: LED, LED_SMD:LED_0603_1608Metric, symbol Device:LED
- added J103: USB_C_USB2.0, Connector_USB:USB_C_Receptacle_GCT_USB4105-xx-A_16P_TopMnt_Horizontal, symbol Connector:USB_C_Receptacle_USB2.0
- added R104, R105: 5k1, Resistor_SMD:R_0402_1005Metric, symbol Device:R
- added R107, R48: 1k, Resistor_SMD:R_0402_1005Metric, symbol Device:R
- added R40: 22R, Resistor_SMD:R_0402_1005Metric, symbol Device:R
- added R41: 12k, Resistor_SMD:R_0402_1005Metric, symbol Device:R
- added R42, R43, R44, R45, R46, R47: 100k, Resistor_SMD:R_0402_1005Metric, symbol Device:R
- added U13: ESD122, symbol Custom_VoxLink_Symbols:ESD122
- added Y3: 24MHz, Crystal:Crystal_SMD_2520-4Pin_2.5x2.0mm, symbol Device:Crystal_GND24
- U12: value ~ -> USB2512B
Connections:
- net USB_UP_D-: now reaches U12. (USBUP_D-)
- net USB_UP_D-: now also J103.A7 (D-), J103.B7 (D-), U13.2 (1)
- net JTAG_D-: now reaches U12.1 (USBDP_D1-)
- net +3V3: now reaches U12.10 (VDDA33)
- net +3V3: now also U12.15 (VDD33), U12.23 (VDD33), U12.29 (VDDA33), U12.36 (VDDA33), U12.5 (VDDA33), C107.1, C108.1, C109.1, C110.1, C111.1, C112.1, C113.1, R47.2, R48.1
- net GND: now reaches U12.11 (TEST)
- net GND: now also U12.37 (EP), C105.2, C106.2, C107.2, C108.2, C109.2, C110.2, C111.2, C112.2, C113.2, C114.2, C115.2, C116.2, C117.2, D104.2 (A2), D105.1 (K), J103.A1 (GND), J103.A12 (GND), J103.B1 (GND), J103.B12 (GND), R104.1, R105.1, R41.1, R43.1, R44.1, R45.1, R46.1, U13.1 (G), Y3.2, Y3.4
- net at U12.14 (CRFILT): now also C116.1, C117.1
- net JTAG_D+: now reaches U12.2 (USBDP_D1+)
- net at U12.22 (NON_REM1): now also R47.1
- net at U12.24 (CFG_SEL0): now also R44.2
- net at U12.25 (CFG_SEL1): now also R45.2
- net at U12.26 (NRESET): now also R48.2
- net at U12.27 (VBUS_DET): now also R42.1, R43.2
- net at U12.28 (NON_REM0): now also R46.2
- net SERIAL_D-: now reaches U12.3 (USBDP_D2-)
- net OSC_OUT: now reaches U12.32 (XTALOUT)
- net OSC_OUT: now also R40.1
- net OSC_IN: now reaches U12.33 (XTALIN)
- net OSC_IN: now also C105.1, Y3.1
- net at U12.34 (PLLFILT): now also C114.1, C115.1
- net at U12.35 (RBIAS): now also R41.2
- net SERIAL_D+: now reaches U12.4 (USBDP_D2+)
- new net: D105.2 (A), R107.1
- new net: C106.1, R40.2, Y3.3
- new net: J103.A5 (CC1), R104.2
- new net: J103.B5 (CC2), R105.2
- new net USB_UP_D+: J103.A6 (D+), J103.B6 (D+), U12. (USBUP_D-), U13.3 (2)
- new net VBUS: D104.1 (A1), J103.A4 (VBUS), J103.A9 (VBUS), J103.B4 (VBUS), J103.B9 (VBUS), R107.2, R42.2
- no-connect marks 5 -> 8
Other:
- note added: "(10pF Load Capacitance - 5pF Stray Capacitance) * 2 = 10pF Load Capacitors"
- note added: "NON_REM[1:0] = 10 : ports 1 and 2 are non-removable"
- note added: "USB [6]"
- note removed: "Make it more pretty"

Commit message: Finished schematic design - preparation for review
Parts:
- D104: footprint Diode_SMD:D_0402_1005Metric -> Diode_THT:D_DO-201AE_P15.24mm_Horizontal

Commit message: Finished DRC check. Moving to schematic review
Parts:
- removed J103: USB_C_USB2.0, Connector_USB:USB_C_Receptacle_GCT_USB4105-xx-A_16P_TopMnt_Horizontal, symbol Connector:USB_C_Receptacle_USB2.0
- added J601: USB-C, Connector_USB:USB_C_Receptacle_GCT_USB4105-xx-A_16P_TopMnt_Horizontal, symbol Custom_VoxLink_Symbols:USB-C_2.0
- renumbered C107 to C601, C108 to C602, C109 to C603, C110 to C604, C111 to C605, C112 to C606, C113 to C607, C114 to C608, C115 to C609, C116 to C610, C117 to C611, C105 to C612, C106 to C613, D104 to D601, D105 to D602, R107 to R601, R104 to R602, R105 to R603, R48 to R604, R41 to R605, R47 to R606, R44 to R607, R45 to R608, R46 to R609, R42 to R610, R40 to R611, R43 to R612, U13 to U601, U12 to U602, Y3 to Y601
Connections:
- net GND: now also J601.A1 (GND), J601.A12 (GND), J601.B1 (GND), J601.B12 (GND)
- net USB_UP_D+: now also U602.31 (USBUP_D+), J601.A6 (D+), J601.B6 (D+); no longer U602. (USBUP_D-)
- net USB_UP_D-: now also U602.30 (USBUP_D-), J601.A7 (D-), J601.B7 (D-); no longer U602. (USBUP_D-)
- net VBUS: now also J601.A4 (VBUS), J601.A9 (VBUS), J601.B4 (VBUS), J601.B9 (VBUS)
- net at R602.2: now also J601.A5 (CC1)
- net at R603.2: now also J601.B5 (CC2)

Commit message: Finished the schematic review
Parts:
- removed D601: TVS, Diode_THT:D_DO-201AE_P15.24mm_Horizontal, symbol Diode:1.5KExxA
- added C608: 100n, Capacitor_SMD:C_0402_1005Metric, symbol Device:C
- added D601: D_TVS, Diode_SMD:D_0402_1005Metric, symbol Device:D_TVS
- C601: value 4u7 -> 10u; footprint Capacitor_SMD:C_0402_1005Metric -> Capacitor_SMD:C_0805_2012Metric
- U601: footprint (none) -> Amass_XT60:CONN_XT60PW-M_AMA
- renumbered C608 to C609, C609 to C610, C610 to C611, C611 to C612, C612 to C613, C613 to C614
Connections:
- net GND: now also C608.2, D601.1 (A1)
- net VBUS: now also D601.2 (A2)
- net at R604.2, U602.26 (NRESET): now also C608.1

Commit message: Updated the documentation + minor scheme changes - Documented the schematic design - Added zener diode from USB VBUS to 5V
Parts:
- added D601: Schottky, Diode_SMD:D_SOD-323F, symbol Device:D_Schottky
- D602: renamed from D601; value D_TVS -> TVS
- renumbered D602 to D603
Connections:
- net VBUS: now also D601.2 (A)
- new net +5V: D601.1 (K)

Commit message: Started schematic rework and the PCB design
Parts:
- U601: footprint Amass_XT60:CONN_XT60PW-M_AMA -> Custom_VoxLink_Footprints:X2SON-3
Changed lines of the file:
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@@
 			)
 		)
-		(property "Footprint" "Amass_XT60:CONN_XT60PW-M_AMA"
+		(property "Footprint" "Custom_VoxLink_Footprints:X2SON-3"
 			(at 80.01 90.17 0)
 			(effects

Commit message: Converted to 10.0 KiCad schematic + Began BGA fan
Parts:
- removed Y601: 24MHz, Crystal:Crystal_SMD_2520-4Pin_2.5x2.0mm, symbol Device:Crystal_GND24
- added Y1: 24MHz, Crystal:Crystal_SMD_2520-4Pin_2.5x2.0mm, symbol Device:Crystal_GND24
Connections:
- net GND: now also Y1.2 (G), Y1.4 (G)
- net OSC_IN: now also Y1.1
- net at C614.1, R611.2: now also Y1.3
