File: Hardware/Controller_Board/usb.kicad_sch (KiCad schematic)
At the start: 33 parts, among them J601 USB-C, U601 ESD122, U602 USB2512B, Y1 24MHz

Commit message: Advanced PCB design - Routed FTDI chips + USB HUB
Parts:
- added D604: TVS, Diode_SMD:D_0402_1005Metric, symbol Device:D_TVS
Connections:
- net GND: now also D604.1 (A1)
- net JTAG_D+: now also U602.4 (USBDP_D2+); no longer U602.2 (USBDP_D1+)
- net JTAG_D-: now also U602.3 (USBDP_D2-); no longer U602.1 (USBDP_D1-)
- net SERIAL_D+: now also U602.2 (USBDP_D1+); no longer U602.4 (USBDP_D2+)
- net SERIAL_D-: now also U602.1 (USBDP_D1-); no longer U602.3 (USBDP_D2-)
- net VBUS: now also D604.2 (A2)

Commit message: Finished PCB Design - WARNING MORE CHANGES NEEDED! The main decision to be made is, whether to increase the layer count to 8 layers, and make the P7 and P8 permamently on 3V3
Parts:
- renumbered C601 to C701, C602 to C702, C603 to C703, C604 to C704, C605 to C705, C606 to C706, C607 to C707, C608 to C708, C609 to C709, C610 to C710, C611 to C711, C612 to C712, C613 to C713, C614 to C714, D601 to D701, D604 to D702, D602 to D703, D603 to D704, J601 to J701, R601 to R701, R602 to R702, R603 to R703, R604 to R704, R605 to R705, R606 to R706, R607 to R707, R608 to R708, R609 to R709, R610 to R710, R611 to R711, R612 to R712, U601 to U701, U602 to U702, Y1 to Y701
Other:
- note added: "USB [7]"
- note removed: "USB [6]"

Commit message: Finished procuring almost all boards - CHANGED XDC IN XILINX FOR TESTING!! - Programmer needed
Parts:
- C701: LCSC (none) -> C237493; Manufacturer (none) -> Murata
- C702, C703, C704, C705, C706, C707, C708, C710, C712: LCSC (none) -> C77020; Manufacturer (none) -> Murata
- C709, C711: LCSC (none) -> C77019; Manufacturer (none) -> Murata
- C713, C714: LCSC (none) -> C76946; Manufacturer (none) -> Murata
- D701: LCSC (none) -> C5636538; Manufacturer (none) -> Toshiba
- D702, D703: LCSC (none) -> C1973340; Manufacturer (none) -> Littelfuse
- D704: LCSC (none) -> C18198801; Manufacturer (none) -> Broadcom
- J701: LCSC (none) -> C5184243; Manufacturer (none) -> GCT
- R701, R704: LCSC (none) -> C71623; Manufacturer (none) -> Vishay
- R702, R703: LCSC (none) -> C482289; Manufacturer (none) -> Vishay
- R705: LCSC (none) -> C481938; Manufacturer (none) -> Vishay
- R706, R707, R708, R709, R710, R712: LCSC (none) -> C481918; Manufacturer (none) -> Vishay
- R711: LCSC (none) -> C482106; Manufacturer (none) -> Vishay
- U701: LCSC (none) -> C544474; Manufacturer (none) -> TI
- U702: LCSC (none) -> C144303; Manufacturer (none) -> Microchip
- Y701: LCSC (none) -> C6941895; Manufacturer (none) -> ECS

Commit message: Finished PCB design and Review + Procured Boards
Parts:
- D701: LCSC C5636538 -> C456093; Manufacturer Toshiba -> Nexperia
Changed lines of the file:
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@@
 			)
 		)
-		(property "Datasheet" "https://www.lcsc.com/product-detail/C5636538.html?s_z=n_CUHS20S30%252CH3F"
+		(property "Datasheet" "https://www.lcsc.com/product-detail/C456093.html?s_z=n_PMEG3020EJ%252C115"
 			(at 92.71 62.23 0)
 			(hide yes)
@@
 			)
 		)
-		(property "LCSC" "C5636538"
+		(property "LCSC" "C456093"
 			(at 92.71 62.23 0)
 			(hide yes)
@@
 			)
 		)
-		(property "Manufacturer" "Toshiba"
+		(property "Manufacturer" "Nexperia"
 			(at 92.71 62.23 0)
 			(hide yes)
