File: Hardware/Controller_Board/serial.kicad_sch (KiCad schematic)
At the start: 0 parts

Commit message: Added USB hub symbol
Parts:
- added C100, C90, C98: 4u7, Capacitor_SMD:C_0402_1005Metric, symbol Device:C
- added C101, C102, C91, C92, C93, C94, C95, C96, C97, C99: 100n, Capacitor_SMD:C_0402_1005Metric, symbol Device:C
- added C103, C104: 10p, Capacitor_SMD:C_0402_1005Metric, symbol Device:C
- added FB4, FB5: 600R, Inductor_SMD:L_0402_1005Metric, symbol Device:FerriteBead
- added R33: 1k, Resistor_SMD:R_0402_1005Metric, symbol Device:R
- added R34: 12k, Resistor_SMD:R_0402_1005Metric, symbol Device:R
- added R35, R36, R37: 10k, Resistor_SMD:R_0402_1005Metric, symbol Device:R
- added R38: 2k2, Resistor_SMD:R_0402_1005Metric, symbol Device:R
- added R39: 22R, Resistor_SMD:R_0402_1005Metric, symbol Device:R
- added U10: FT232H, Package_DFN_QFN:QFN-48-1EP_8x8mm_P0.5mm_EP6.2x6.2mm, symbol Custom_VoxLink_Symbols:FT232H
- added U11: 93LC56B, Package_DFN_QFN:TDFN-8-1EP_3x2mm_P0.5mm_EP1.3x1.4mm, symbol Custom_VoxLink_Symbols:93LC56B
- added Y2: 12MHz, Crystal:Crystal_SMD_2520-4Pin_2.5x2.0mm, symbol Device:Crystal_GND24
Connections:
- new net: R35.1, R38.1, U11.4 (DO)
- new net: C97.1, U10.37 (VCCA)
- new net: C96.1, U10.38 (VCCCORE)
- new net: R33.2, U10.34 (~{RESET})
- new net: R34.2, U10.5 (REF)
- new net: C104.1, R39.2, Y2.3
- new net +3V3: C102.1, C90.1, C91.1, C92.1, C93.1, C94.1, C95.1, FB4.2, FB5.2, R33.1, R35.2, R36.2, R37.2, U10.12 (VCCIO), U10.24 (VCCIO), U10.39 (VCCD), U10.40 (VREGIN), U10.46 (VCCIO), U11.6 (ORG), U11.8 (VCC)
- new net +3V3_VPHY: C98.1, C99.1, FB4.1, U10.3 (VPHY)
- new net +3V3_VPLL: C100.1, C101.1, FB5.1, U10.8 (VPLL)
- new net EECLK: R37.1, U10.44 (EECLK), U11.2 (CLK)
- new net EECS: R36.1, U10.45 (EECS), U11.1 (CS)
- new net EEDATA: R38.2, U10.43 (EEDATA), U11.3 (DI)
- new net FTDI_USB_D+: U10.7 (DP)
- new net FTDI_USB_D-: U10.6 (DM)
- new net GND: C100.2, C101.2, C102.2, C103.2, C104.2, C90.2, C91.2, C92.2, C93.2, C94.2, C95.2, C96.2, C97.2, C98.2, C99.2, R34.1, U10.10 (GND), U10.11 (GND), U10.22 (GND), U10.23 (GND), U10.35 (GND), U10.36 (GND), U10.4 (AGND), U10.41 (AGND), U10.42 (TEST), U10.47 (GND), U10.48 (GND), U10.49 (EP), U10.9 (AGND), U11.5 (VSS), U11.9 (EP), Y2.2, Y2.4
- new net OSC_IN: C103.1, U10.1 (XCSI), Y2.1
- new net OSC_OUT: R39.1, U10.2 (XCSO)
- no-connect marks 0 -> 15
Other:
- note added: "(10pF Load Capacitance - 5pF Stray Capacitance) * 2 = 10pF Load Capacitors"
- note added: "Ferrite beads must be rated at least for 600mA"
- note added: "JTAG [3]"
- note added: "VREGIN = 5V -> VCCD = 3.3V OUTPUT VREGIN = 3.3V -> VCCD = 3.3V INPUT"

Commit message: Updated the schematic design - Fix the XC7A35T-CPG236 outline issue
Connections:
- net FTDI_USB_D+ renamed SERIAL_D+
- net FTDI_USB_D- renamed SERIAL_D-
Other:
- note added: "Serial [5]"
- note removed: "JTAG [3]"
Changed lines of the file:
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@@
 		)
 	)
-	(text "JTAG [3]"
+	(text "Serial [5]"
 		(exclude_from_sim no)
-		(at 51.816 25.4 0)
+		(at 15.494 18.796 0)
 		(effects
 			(font
@@
 				(color 132 0 0 1)
 			)
+			(justify left top)
 		)
 	)
@@
 		)
 	)
-	(global_label "FTDI_USB_D-"
+	(global_label "SERIAL_D-"
 		(shape input)
 		(at 179.07 76.2 180)
@@
 		)
 		(property "Intersheetrefs" "${INTERSHEET_REFS}"
-			(at 163.5662 76.2 0)
+			(at 165.9248 76.2 0)
 			(effects
 				(font
@@
 		)
 	)
-	(global_label "FTDI_USB_D+"
+	(global_label "SERIAL_D+"
 		(shape input)
 		(at 179.07 78.74 180)
@@
 		)
 		(property "Intersheetrefs" "${INTERSHEET_REFS}"
-			(at 163.5662 78.74 0)
+			(at 165.9248 78.74 0)
 			(effects
 				(font

Commit message: Finished schematic design - preparation for review
Parts:
- added U6: XC7A35T-CPG236, Package_BGA:Xilinx_CPG236, symbol Custom_VoxLink_Symbols:XC7A35T-CPG236
Connections:
- net SERIAL_D1: now reaches U10.13 (ADBUS0)
- net SERIAL_D1: now also U6.R2 (IO_L1P_T0_34)
- net SERIAL_D2: now reaches U10.14 (ADBUS1)
- net SERIAL_D2: now also U6.T2 (IO_L1N_T0_34)
- net SERIAL_D3: now reaches U10.15 (ADBUS2)
- net SERIAL_D3: now also U6.R3 (IO_L2P_T0_34)
- net SERIAL_D4: now reaches U10.16 (ADBUS3)
- net SERIAL_D4: now also U6.T3 (IO_L2N_T0_34)
- net SERIAL_D5: now reaches U10.17 (ADBUS4)
- net SERIAL_D5: now also U6.T1 (IO_L3P_T0_DQS_34)
- net SERIAL_D6: now reaches U10.18 (ADBUS5)
- net SERIAL_D6: now also U6.U1 (IO_L3N_T0_DQS_34)
- net SERIAL_D7: now reaches U10.19 (ADBUS6)
- net SERIAL_D7: now also U6.V2 (IO_L5P_T0_34)
- net SERIAL_D8: now reaches U10.20 (ADBUS7)
- net SERIAL_D8: now also U6.W2 (IO_L5N_T0_34)
- net SERIAL_RXF#: now reaches U10.21 (ACBUS0)
- net SERIAL_RXF#: now also U6.V3 (IO_L6P_T0_34)
- net SERIAL_TXE#: now reaches U10.25 (ACBUS1)
- net SERIAL_TXE#: now also U6.W3 (IO_L6N_T0_VREF_34)
- net SERIAL_RD#: now reaches U10.26 (ACBUS2)
- net SERIAL_RD#: now also U6.U3 (IO_L9P_T1_DQS_34)
- net SERIAL_WR#: now reaches U10.27 (ACBUS3)
- net SERIAL_WR#: now also U6.U2 (IO_L9N_T1_DQS_34)
- net SERIAL_SIWU#: now reaches U10.28 (ACBUS4)
- net SERIAL_SIWU#: now also U6.U4 (IO_L11P_T1_SRCC_34)
- net SERIAL_IO: now reaches U10.29 (ACBUS5)
- net SERIAL_IO: now also U6.V4 (IO_L11N_T1_SRCC_34)
- net SERIAL_CLK: now reaches U10.30 (ACBUS6)
- net SERIAL_CLK: now also U6.W5 (IO_L12P_T1_MRCC_34)
- net SERIAL_OE#: now reaches U10.31 (ACBUS7)
- net SERIAL_OE#: now also U6.W4 (IO_L12N_T1_MRCC_34)
- new net P1_L2: U6.W6 (IO_L13N_T2_MRCC_34)
- new net P2_L1: U6.U8 (IO_L14P_T2_SRCC_34)
- new net P2_L2: U6.V8 (IO_L14N_T2_SRCC_34)
- new net P3_L1: U6.U5 (IO_L16P_T2_34)
- new net P3_L2: U6.V5 (IO_L16N_T2_34)
- new net P4_L1: U6.U7 (IO_L19P_T3_34)
- new net P4_L2: U6.V7 (IO_L19N_T3_VREF_34)
- no-connect marks 15 -> 3
Other:
- moved on the sheet: C100, C101, C102, C103, C104, C90, C91, C92, C93, C94, C95, C96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

Commit message: Finished DRC check. Moving to schematic review
Parts:
- renumbered C90 to C501, C91 to C502, C92 to C503, C93 to C504, C94 to C505, C95 to C506, C96 to C507, C97 to C508, C98 to C509, C99 to C510, C100 to C511, C101 to C512, C102 to C513, C103 to C514, C104 to C515, FB4 to FB501, FB5 to FB502, R33 to R501, R34 to R502, R35 to R503, R36 to R504, R37 to R505, R38 to R506, R39 to R507, U6 to U201, U10 to U501, U11 to U502, Y2 to Y501
Connections:
- net P1_L1: now also U201.W7 (IO_L13P_T2_MRCC_34)

Commit message: Finished the schematic review
Parts:
- added C512: 10u, Capacitor_SMD:C_0805_2012Metric, symbol Device:C
- C501, C509: value 4u7 -> 10u; footprint Capacitor_SMD:C_0402_1005Metric -> Capacitor_SMD:C_0805_2012Metric
- C511: value 4u7 -> 100n
- R503, R504, R505: value 10k -> 12k
- renumbered C512 to C513, C513 to C514, C514 to C515, C515 to C516
Connections:
- net GND: now also C512.2
- net SERIAL_CLK: now also U201.W4 (IO_L12N_T1_MRCC_34), U501.29 (ACBUS5); no longer U201.W5 (IO_L12P_T1_MRCC_34), U501.30 (ACBUS6)
- net SERIAL_OE#: now also U201.W5 (IO_L12P_T1_MRCC_34), U501.30 (ACBUS6); no longer U201.W4 (IO_L12N_T1_MRCC_34), U501.31 (ACBUS7)
- net at R501.2, U501.34 (~{RESET}): now also C511.1
- net +3V3_VPHY renamed +3V3_VPHY_SER
- net +3V3_VPLL renamed +3V3_VPLL_SER
- net +3V3_VPLL_SER: now also C512.1; no longer C511.1
- net SERIAL_IO renamed SERIAL_PWR#
- net SERIAL_PWR#: now also U501.31 (ACBUS7); no longer U501.29 (ACBUS5)
Other:
- note added: "RJ45 LEDs"

Commit message: Commit before upgrading to KiCad 10.0
Parts:
- removed U201: XC7A35T-CPG236, Package_BGA:Xilinx_CPG236, symbol Custom_VoxLink_Symbols:XC7A35T-CPG236
Other:
- note removed: "RJ45 LEDs"
- note removed: "VREGIN = 5V -> VCCD = 3.3V OUTPUT VREGIN = 3.3V -> VCCD = 3.3V INPUT"

Commit message: Converted to 10.0 KiCad schematic + Began BGA fan
Parts:
- removed Y501: 12MHz, Crystal:Crystal_SMD_2520-4Pin_2.5x2.0mm, symbol Device:Crystal_GND24
- added Y2: 12MHz, Crystal:Crystal_SMD_2520-4Pin_2.5x2.0mm, symbol Device:Crystal_GND24
Connections:
- net GND: now also Y2.2 (G), Y2.4 (G)
- net OSC_IN: now also Y2.1
- net at C516.1, R507.2: now also Y2.3
