File: Hardware/Controller_Board/jtag.kicad_sch (KiCad schematic)
At the start: 28 parts, among them U201 FT2232HQ, U202 93LC56B, Y201 12MHz

Commit message: Added new sheets to the schematic
Parts:
- removed C213, C214: 100n, Capacitor_SMD:C_0402_1005Metric, symbol Device:C
- removed U201: FT2232HQ, Package_DFN_QFN:QFN-64-1EP_9x9mm_P0.5mm_EP4.35x4.35mm, symbol Interface_USB:FT2232HQ
- added C74: 100n, Capacitor_SMD:C_0402_1005Metric, symbol Device:C
- added U8: FT232H, Package_DFN_QFN:QFN-48-1EP_8x8mm_P0.5mm_EP6.2x6.2mm, symbol Custom_VoxLink_Symbols:FT232H
- C72: value 4u7 -> 100n
Connections:
- net +3V3: now also C72.1, U8.12 (VCCIO), U8.24 (VCCIO), U8.39 (VCCD), U8.40 (VREGIN), U8.46 (VCCIO)
- net +3V3_VPHY: now also U8.3 (VPHY)
- net +3V3_VPLL: now also U8.8 (VPLL)
- net EECLK: now also U8.44 (EECLK)
- net EECS: now also U8.45 (EECS)
- net EEDATA: now also U8.43 (EEDATA)
- net FTDI_USB_D+: now also U8.7 (DP)
- net FTDI_USB_D-: now also U8.6 (DM)
- net GND: now also C74.2, U8.10 (GND), U8.11 (GND), U8.22 (GND), U8.23 (GND), U8.35 (GND), U8.36 (GND), U8.4 (AGND), U8.41 (AGND), U8.42 (TEST), U8.47 (GND), U8.48 (GND), U8.49 (EP), U8.9 (AGND)
- net OSC_IN: now also U8.1 (XCSI)
- net OSC_OUT: now also U8.2 (XCSO)
- net TCK: now also U8.13 (ADBUS0)
- net TDI_FPGA: now also U8.14 (ADBUS1)
- net TDO_FPGA: now also U8.15 (ADBUS2)
- net TMS: now also U8.16 (ADBUS3)
- net at R207.2: now also U8.34 (~{RESET})
- net at R206.2: now also U8.5 (REF)
- net +1V8_FTDI: no longer names the net of C215.1
- net +1V8_FTDI: now also U8.38 (VCCCORE); no longer C72.1
- new net: C74.1, U8.37 (VCCA)
- no-connect marks 30 -> 15
Other:
- note added: "JTAG [3]"
- note added: "VREGIN = 5V -> VCCD = 3.3V OUTPUT VREGIN = 3.3V -> VCCD = 3.3V INPUT"
- note removed: "FTDI [3]"
- title: (none) -> JTAG
- moved on the sheet: C215

Commit message: Added USB hub symbol
Parts:
- renumbered C207 to C75, C208 to C76, C209 to C77, C210 to C78, C211 to C79, C72 to C80, C215 to C81, C74 to C82, C201 to C83, C202 to C84, C203 to C85, C204 to C86, C216 to C87, C205 to C88, C206 to C89, FB201 to FB2, FB202 to FB3, R207 to R26, R206 to R27, R205 to R28, R203 to R29, R204 to R30, R202 to R31, R201 to R32, U202 to U9, Y201 to Y1

Commit message: Updated the schematic design - Fix the XC7A35T-CPG236 outline issue
Connections:
- net FTDI_USB_D+ renamed JTAG_D+
- net FTDI_USB_D- renamed JTAG_D-
Other:
- note added: "JTAG [4]"
- note removed: "JTAG [3]"
Changed lines of the file:
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@@
 		)
 	)
-	(text "JTAG [3]"
+	(text "JTAG [4]"
 		(exclude_from_sim no)
-		(at 51.816 25.4 0)
+		(at 15.494 18.796 0)
 		(effects
 			(font
@@
 				(color 132 0 0 1)
 			)
+			(justify left top)
 		)
 	)
@@
 		)
 	)
-	(global_label "FTDI_USB_D-"
+	(global_label "JTAG_D-"
 		(shape input)
 		(at 179.07 76.2 180)
@@
 		)
 		(property "Intersheetrefs" "${INTERSHEET_REFS}"
-			(at 163.5662 76.2 0)
+			(at 167.981 76.2 0)
 			(effects
 				(font
@@
 		)
 	)
-	(global_label "FTDI_USB_D+"
+	(global_label "JTAG_D+"
 		(shape input)
 		(at 179.07 78.74 180)
@@
 		)
 		(property "Intersheetrefs" "${INTERSHEET_REFS}"
-			(at 163.5662 78.74 0)
+			(at 167.981 78.74 0)
 			(effects
 				(font

Commit message: Finished DRC check. Moving to schematic review
Parts:
- renumbered C75 to C401, C76 to C402, C77 to C403, C78 to C404, C79 to C405, C80 to C406, C81 to C407, C82 to C408, C83 to C409, C84 to C410, C85 to C411, C86 to C412, C87 to C413, C88 to C414, C89 to C415, FB2 to FB401, FB3 to FB402, R26 to R401, R27 to R402, R28 to R403, R29 to R404, R30 to R405, R31 to R406, R32 to R407, U8 to U401, U9 to U402, Y1 to Y401
Connections:
- net TDI_FPGA renamed TDI
- net TDO_FPGA renamed TDO
Other:
- note removed: "WE HAVE TO CHECK THE TDI/TDO CONNECTIONS!"

Commit message: Finished the schematic review
Parts:
- added C412: 10u, Capacitor_SMD:C_0805_2012Metric, symbol Device:C
- C401, C409: value 4u7 -> 10u; footprint Capacitor_SMD:C_0402_1005Metric -> Capacitor_SMD:C_0805_2012Metric
- C411: value 4u7 -> 100n
- R403, R404, R405: value 10k -> 12k
- U402: Distributor Link https://www.mouser.sk/ProductDetail/Microchip-Technology/93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 -> (none)
- renumbered C412 to C413, C413 to C414, C414 to C415, C415 to C416
Connections:
- net GND: now also C412.2
- net at R401.2, U401.34 (~{RESET}): now also C411.1
- net +3V3_VPHY renamed +3V3_VPHY_JTAG
- net +3V3_VPLL renamed +3V3_VPLL_JTAG
- net +3V3_VPLL_JTAG: now also C412.1; no longer C411.1
Other:
- moved on the sheet: R401, R402

Commit message: Converted to 10.0 KiCad schematic + Began BGA fan
Parts:
- removed Y401: 12MHz, Crystal:Crystal_SMD_2520-4Pin_2.5x2.0mm, symbol Device:Crystal_GND24
- added Y3: 12MHz, Crystal:Crystal_SMD_2520-4Pin_2.5x2.0mm, symbol Device:Crystal_GND24
Connections:
- net GND: now also Y3.2 (G), Y3.4 (G)
- net OSC_IN: now also Y3.1
- net at C416.1, R407.2: now also Y3.3

Commit message: Advanced PCB design - Routed FTDI chips + USB HUB
Parts:
- removed C406: 100n, Capacitor_SMD:C_0402_1005Metric, symbol Device:C
- C409, C412: footprint Capacitor_SMD:C_0805_2012Metric -> Capacitor_SMD:C_0603_1608Metric
Changed lines of the file:
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@@
 		)
 	)
-	(text_box "FTDI USB-to-UART"
+	(text_box "FTDI USB-to-JTAG"
 		(exclude_from_sim no)
 		(at 106.045 20.32 0)
@@
 	)
 	(junction
-		(at 154.94 36.83)
-		(diameter 0)
-		(color 0 0 0 0)
-	)
-	(junction
 		(at 114.3 36.83)
 		(diameter 0)
@@
 	(wire
 		(pts
-			(xy 154.94 36.83) (xy 165.1 36.83)
-		)
-		(stroke
-			(width 0)
-			(type default)
-		)
-	)
-	(wire
-		(pts
 			(xy 62.23 72.39) (xy 68.58 72.39)
 		)
@@
 	(wire
 		(pts
-			(xy 165.1 36.83) (xy 165.1 38.1)
-		)
-		(stroke
-			(width 0)
-			(type default)
-		)
-	)
-	(wire
-		(pts
 			(xy 219.71 43.18) (xy 219.71 41.91)
 		)
@@
 	)
 	(symbol
-		(lib_id "Device:C")
-		(at 165.1 41.91 0)
-		(mirror y)
-		(unit 1)
-		(body_style 1)
-		(exclude_from_sim no)
-		(in_bom yes)
-		(on_board yes)
-		(in_pos_files yes)
-		(dnp no)
-		(property "Reference" "C406"
-			(at 162.814 40.894 0)
-			(show_name no)
-			(do_not_autoplace no)
-			(effects
-				(font
-					(size 1.27 1.27)
-				)
-				(justify left)
-			)
-		)
-		(property "Value" "100n"
-			(at 162.814 42.926 0)
-			(show_name no)
-			(do_not_autoplace no)
-			(effects
-				(font
-					(size 1.27 1.27)
-				)
-				(justify left)
-			)
-		)
-		(property "Footprint" "Capacitor_SMD:C_0402_1005Metric"
-			(at 164.1348 45.72 0)
-			(hide yes)
-			(show_name no)
-			(do_not_autoplace no)
-			(effects
-				(font
-					(size 1.27 1.27)
-				)
-			)
-		)
-		(property "Datasheet" ""
-			(at 165.1 41.91 0)
-			(hide yes)
-			(show_name no)
-			(do_not_autoplace no)
-			(effects
-				(font
-					(size 1.27 1.27)
-				)
-			)
-		)
-		(property "Description" "Unpolarized capacitor"
-			(at 165.1 41.91 0)
-			(hide yes)
-			(show_name no)
-			(do_not_autoplace no)
-			(effects
-				(font
-					(size 1.27 1.27)
-				)
-			)
-		)
-		(pin "1"
-		)
-		(pin "2"
-		)
-		(instances
-			(project "Controller_Board"
-				(path "/4e6e1af1-ede9-4a56-9d5f-a8dfd7fbcf8d/cd46e716-e63c-4118-a3e6-5dedd1612b37"
-					(reference "C406")
-					(unit 1)
-				)
-			)
-		)
-	)
-	(symbol
 		(lib_id "power:GND")
 		(at 114.3 45.72 0)
@@
 			)
 		)
-		(property "Footprint" "Capacitor_SMD:C_0805_2012Metric"
+		(property "Footprint" "Capacitor_SMD:C_0603_1608Metric"
 			(at 54.9148 104.14 0)
 			(hide yes)
@@
 			)
 		)
-		(property "Footprint" "Capacitor_SMD:C_0805_2012Metric"
+		(property "Footprint" "Capacitor_SMD:C_0603_1608Metric"
 			(at 54.9148 82.55 0)
 			(hide yes)
@@
 					(unit 1)
 				)
-			)
-		)
-	)
-	(symbol
-		(lib_id "power:GND")
-		(at 165.1 45.72 0)
-		(mirror y)
-		(unit 1)
-		(body_style 1)
-		(exclude_from_sim no)
-		(in_bom yes)
-		(on_board yes)
-		(in_pos_files yes)
-		(dnp no)
-		(property "Reference" "#PWR0410"
-			(at 165.1 52.07 0)
-			(hide yes)
-			(show_name no)
-			(do_not_autoplace no)
-			(effects
-				(font
-					(size 1.27 1.27)
-				)
-			)
-		)
-		(property "Value" "GND"
-			(at 165.1 49.53 0)
-			(hide yes)
-			(show_name no)
-			(do_not_autoplace no)
-			(effects
-				(font
-					(size 1.27 1.27)
-				)
-			)
-		)
-		(property "Footprint" ""
-			(at 165.1 45.72 0)
-			(hide yes)
-			(show_name no)
-			(do_not_autoplace no)
-			(effects
-				(font
-					(size 1.27 1.27)
-				)
-			)
-		)
-		(property "Datasheet" ""
-			(at 165.1 45.72 0)
-			(hide yes)
-			(show_name no)
-			(do_not_autoplace no)
-			(effects
-				(font
-					(size 1.27 1.27)
-				)
-			)
-		)
-		(property "Description" "Power symbol creates a global label with name \"GND\" , ground"
-			(at 165.1 45.72 0)
-			(hide yes)
-			(show_name no)
-			(do_not_autoplace no)
-			(effects
-				(font
-					(size 1.27 1.27)
-				)
-			)
-		)
-		(pin "1"
-		)
-		(instances
-			(project "Controller_Board"
-				(path "/4e6e1af1-ede9-4a56-9d5f-a8dfd7fbcf8d/cd46e716-e63c-4118-a3e6-5dedd1612b37"
-					(reference "#PWR0410")
-					(unit 1)
-				)
