File: Hardware/Controller_Board/jtag.kicad_sch (KiCad schematic)
At the start: 27 parts, among them U401 FT232H, U402 93LC56B, Y3 12MHz

Commit message: Advanced PCB Design: Routing Power + UVLO
Connections:
- net +3V3: no longer C403.1, C404.1, C405.1, U401.12 (VCCIO), U401.24 (VCCIO), U401.39 (VCCD), U401.46 (VCCIO)
- new net +2V5: C403.1, C404.1, C405.1, U401.12 (VCCIO), U401.24 (VCCIO), U401.46 (VCCIO)
- no-connect marks 15 -> 16

Commit message: Finished PCB Design - WARNING MORE CHANGES NEEDED! The main decision to be made is, whether to increase the layer count to 8 layers, and make the P7 and P8 permamently on 3V3
Parts:
- renumbered C401 to C501, C402 to C502, C403 to C503, C404 to C504, C405 to C505, C407 to C506, C408 to C507, C409 to C508, C410 to C509, C411 to C510, C412 to C511, C413 to C512, C414 to C513, C415 to C514, C416 to C515, FB401 to FB501, FB402 to FB502, R401 to R501, R402 to R502, R403 to R503, R404 to R504, R405 to R505, R406 to R506, R407 to R507, U401 to U501, U402 to U502, Y3 to Y501
Other:
- note added: "JTAG [5]"
- note removed: "JTAG [4]"

Commit message: Finished procuring almost all boards - CHANGED XDC IN XILINX FOR TESTING!! - Programmer needed
Parts:
- added U501: SN74AXC4T774, Package_DFN_QFN:UQFN-16_1.8x2.6mm_P0.4mm, symbol Custom_VoxLink_Symbols:SN74AXC4T774
- C501: LCSC (none) -> C237493; Manufacturer (none) -> Murata
- C502, C503, C504, C505, C506, C507, C509, C510, C512, C513: LCSC (none) -> C77020; Manufacturer (none) -> Murata
- C508, C511: LCSC (none) -> C194427; Manufacturer (none) -> Murata
- C514, C515: LCSC (none) -> C76946; Manufacturer (none) -> Murata
- FB501, FB502: LCSC (none) -> C160977; Manufacturer (none) -> Murata
- R501: LCSC (none) -> C71623; Manufacturer (none) -> Vishay
- R502, R503, R504, R505: LCSC (none) -> C481938; Manufacturer (none) -> Vishay
- R506: LCSC (none) -> C82680; Manufacturer (none) -> Vishay
- R507: LCSC (none) -> C482106; Manufacturer (none) -> Vishay
- U502: renamed from U501; LCSC (none) -> C82158; Manufacturer (none) -> FTDI
- U503: renamed from U502; LCSC (none) -> C616589; Manufacturer (none) -> Microchip
- Y501: LCSC (none) -> C6372529; Manufacturer (none) -> ECS
Connections:
- net +2V5: now also U501.13 (VCCB); no longer C503.1, C504.1, C505.1, U502.12 (VCCIO), U502.24 (VCCIO), U502.46 (VCCIO)
- net +3V3: now also C503.1, C504.1, C505.1, U502.12 (VCCIO), U502.24 (VCCIO), U502.46 (VCCIO), U501.14 (VCCA), U501.15 (DIR1), U501.5 (DIR3), U501.6 (DIR4)
- net GND: now also U501.16 (DIR2), U501.7 (~{OE}), U501.8 (GND)
- net TCK: now also U501.9 (B4); no longer U502.13 (ADBUS0)
- net TDI: now also U501.10 (B3); no longer U502.14 (ADBUS1)
- net TDO: now also U501.11 (B2); no longer U502.15 (ADBUS2)
- net TMS: now also U501.12 (B1); no longer U502.16 (ADBUS3)
- new net FTDI_TCK: U501.4 (A4), U502.13 (ADBUS0)
- new net FTDI_TDI: U501.3 (A3), U502.14 (ADBUS1)
- new net FTDI_TDO: U501.2 (A2), U502.15 (ADBUS2)
- new net FTDI_TMS: U501.1 (A1), U502.16 (ADBUS3)
Other:
- note added: "DIR = HIGH: data A to B DIR = LOW: data B to A"
