File: Hardware/Controller_Board/Controller_Board.kicad_sch (KiCad schematic)
At the start: 1 part, among them U1 XC7A35T-CPG236

Commit message: Updated the domcumentation
Other:
- added sheet FTDI (ftdi.kicad_sch)
Changed lines of the file:
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@@
+		)
+	)
+	(sheet
+		(at 86.36 -78.74)
+		(size 45.72 30.48)
+		(exclude_from_sim no)
+		(in_bom yes)
+		(on_board yes)
+		(dnp no)
+		(fields_autoplaced yes)
+		(stroke
+			(width 0.1524)
+			(type solid)
+		)
+		(fill
+			(color 0 0 0 0.0000)
+		)
+		(property "Sheetname" "FTDI"
+			(at 86.36 -79.4516 0)
+			(effects
+				(font
+					(size 1.27 1.27)
+				)
+				(justify left bottom)
+			)
+		)
+		(property "Sheetfile" "ftdi.kicad_sch"
+			(at 86.36 -47.6754 0)
+			(effects
+				(font
+					(size 1.27 1.27)
+				)
+				(justify left top)
+			)
+		)
+		(instances
+			(project "Controller_Board"
+				(path "/4e6e1af1-ede9-4a56-9d5f-a8dfd7fbcf8d"
+					(page "3")
+				)
+			)
 		)
 	)

Commit message: Commited Schematic Changes
Parts:
- removed U1: XC7A35T-CPG236, Package_BGA:Xilinx_CPG236, symbol FPGA_Xilinx_Artix7:XC7A35T-CPG236
Other:
- added sheet FPGA Power (fpga_power.kicad_sch)
- company: (none) -> Czech Technical University in Prague
- title: (none) -> Root

Commit message: Updated schematic diagram with configuration
Other:
- sheet FPGA Power renamed FPGA_Power
- added sheet Connectivity (connectivity.kicad_sch)
- added sheet FPGA_Config (fpga_config.kicad_sch)
Changed lines of the file:
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@@
+	)
+	(sheet
+		(at 170.18 86.36)
+		(size 35.56 25.4)
+		(exclude_from_sim no)
+		(in_bom yes)
+		(on_board yes)
+		(dnp no)
+		(fields_autoplaced yes)
+		(stroke
+			(width 0.1524)
+			(type solid)
+		)
+		(fill
+			(color 0 0 0 0.0000)
+		)
+		(property "Sheetname" "FPGA_Config"
+			(at 170.18 85.6484 0)
+			(effects
+				(font
+					(size 1.27 1.27)
+				)
+				(justify left bottom)
+			)
+		)
+		(property "Sheetfile" "fpga_config.kicad_sch"
+			(at 170.18 112.3446 0)
+			(effects
+				(font
+					(size 1.27 1.27)
+				)
+				(justify left top)
+			)
+		)
+		(instances
+			(project "Controller_Board"
+				(path "/4e6e1af1-ede9-4a56-9d5f-a8dfd7fbcf8d"
+					(page "5")
+				)
+			)
+		)
 	)
 	(sheet
@@
 			(color 0 0 0 0.0000)
 		)
-		(property "Sheetname" "FPGA Power"
+		(property "Sheetname" "FPGA_Power"
 			(at 128.27 64.0584 0)
 			(effects
@@
 	)
 	(sheet
-		(at 86.36 -78.74)
+		(at 231.14 86.36)
+		(size 44.45 30.48)
+		(exclude_from_sim no)
+		(in_bom yes)
+		(on_board yes)
+		(dnp no)
+		(fields_autoplaced yes)
+		(stroke
+			(width 0.1524)
+			(type solid)
+		)
+		(fill
+			(color 0 0 0 0.0000)
+		)
+		(property "Sheetname" "Connectivity"
+			(at 231.14 85.6484 0)
+			(effects
+				(font
+					(size 1.27 1.27)
+				)
+				(justify left bottom)
+			)
+		)
+		(property "Sheetfile" "connectivity.kicad_sch"
+			(at 231.14 117.4246 0)
+			(effects
+				(font
+					(size 1.27 1.27)
+				)
+				(justify left top)
+			)
+		)
+		(instances
+			(project "Controller_Board"
+				(path "/4e6e1af1-ede9-4a56-9d5f-a8dfd7fbcf8d"
+					(page "6")
+				)
+			)
+		)
+	)
+	(sheet
+		(at 213.36 35.56)
 		(size 45.72 30.48)
 		(exclude_from_sim no)
@@
 		)
 		(property "Sheetname" "FTDI"
-			(at 86.36 -79.4516 0)
+			(at 213.36 34.8484 0)
 			(effects
 				(font
@@
 		)
 		(property "Sheetfile" "ftdi.kicad_sch"
-			(at 86.36 -47.6754 0)
+			(at 213.36 66.6246 0)
 			(effects
 				(font

Commit message: Added new sheets to the schematic
Other:
- sheet FTDI renamed JTAG
- added sheet Serial (serial.kicad_sch)
- added sheet USB (usb.kicad_sch)
- sheet JTAG: file ftdi.kicad_sch -> jtag.kicad_sch
Changed lines of the file:
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@@
+			(project "Controller_Board"
+				(path "/4e6e1af1-ede9-4a56-9d5f-a8dfd7fbcf8d"
+					(page "3")
+				)
+			)
+		)
+	)
+	(sheet
+		(at 123.19 121.92)
+		(size 45.72 26.67)
+		(exclude_from_sim no)
+		(in_bom yes)
+		(on_board yes)
+		(dnp no)
+		(fields_autoplaced yes)
+		(stroke
+			(width 0.1524)
+			(type solid)
+		)
+		(fill
+			(color 0 0 0 0.0000)
+		)
+		(property "Sheetname" "Serial"
+			(at 123.19 121.2084 0)
+			(effects
+				(font
+					(size 1.27 1.27)
+				)
+				(justify left bottom)
+			)
+		)
+		(property "Sheetfile" "serial.kicad_sch"
+			(at 123.19 149.1746 0)
+			(effects
+				(font
+					(size 1.27 1.27)
+				)
+				(justify left top)
+			)
+		)
+		(instances
 			(project "Controller_Board"
 				(path "/4e6e1af1-ede9-4a56-9d5f-a8dfd7fbcf8d"
@@
 	)
 	(sheet
+		(at 41.91 128.27)
+		(size 49.53 35.56)
+		(exclude_from_sim no)
+		(in_bom yes)
+		(on_board yes)
+		(dnp no)
+		(fields_autoplaced yes)
+		(stroke
+			(width 0.1524)
+			(type solid)
+		)
+		(fill
+			(color 0 0 0 0.0000)
+		)
+		(property "Sheetname" "USB"
+			(at 41.91 127.5584 0)
+			(effects
+				(font
+					(size 1.27 1.27)
+				)
+				(justify left bottom)
+			)
+		)
+		(property "Sheetfile" "usb.kicad_sch"
+			(at 41.91 164.4146 0)
+			(effects
+				(font
+					(size 1.27 1.27)
+				)
+				(justify left top)
+			)
+		)
+		(instances
+			(project "Controller_Board"
+				(path "/4e6e1af1-ede9-4a56-9d5f-a8dfd7fbcf8d"
+					(page "6")
+				)
+			)
+		)
+	)
+	(sheet
 		(at 128.27 64.77)
 		(size 48.26 30.48)
@@
 			(project "Controller_Board"
 				(path "/4e6e1af1-ede9-4a56-9d5f-a8dfd7fbcf8d"
-					(page "6")
+					(page "7")
 				)
 			)
@@
 			(color 0 0 0 0.0000)
 		)
-		(property "Sheetname" "FTDI"
+		(property "Sheetname" "JTAG"
 			(at 213.36 34.8484 0)
 			(effects
@@
 			)
 		)
-		(property "Sheetfile" "ftdi.kicad_sch"
+		(property "Sheetfile" "jtag.kicad_sch"
 			(at 213.36 66.6246 0)
 			(effects
@@
 			(project "Controller_Board"
 				(path "/4e6e1af1-ede9-4a56-9d5f-a8dfd7fbcf8d"
-					(page "3")
-				)
-			)
+					(page "4")
+				)
+			)

Commit message: Updated the schematic design - Fix the XC7A35T-CPG236 outline issue
Other:
- note added: "Technical Sheet Only! Please refer to the subsequent sheets for schematic"
Changed lines of the file:
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@@
 		(comment 1 "Designer: Michal Varsanyi")
 	)
+	(text "Technical Sheet Only!\nPlease refer to the subsequent sheets for schematic"
+		(exclude_from_sim no)
+		(at 147.32 46.99 0)
+		(effects
+			(font
+				(size 2.54 2.54)
+				(thickness 0.508)
+				(bold yes)
+			)
+		)
+	)
 	(text "Root [0]"
 		(exclude_from_sim no)
-		(at 16.764 20.066 0)
+		(at 16.51 20.32 0)
 		(effects
 			(font
@@
 	)
 	(sheet
-		(at 170.18 86.36)
-		(size 35.56 25.4)
+		(at 180.34 57.15)
+		(size 50.8 34.29)
 		(exclude_from_sim no)
 		(in_bom yes)
@@
 		)
 		(property "Sheetname" "FPGA_Config"
-			(at 170.18 85.6484 0)
+			(at 180.34 56.4384 0)
 			(effects
 				(font
@@
 		)
 		(property "Sheetfile" "fpga_config.kicad_sch"
-			(at 170.18 112.3446 0)
+			(at 180.34 92.0246 0)
 			(effects
 				(font
@@
 	)
 	(sheet
-		(at 123.19 121.92)
-		(size 45.72 26.67)
+		(at 123.19 99.06)
+		(size 50.8 34.29)
 		(exclude_from_sim no)
 		(in_bom yes)
@@
 		)
 		(property "Sheetname" "Serial"
-			(at 123.19 121.2084 0)
+			(at 123.19 98.3484 0)
 			(effects
 				(font
@@
 		)
 		(property "Sheetfile" "serial.kicad_sch"
-			(at 123.19 149.1746 0)
+			(at 123.19 133.9346 0)
 			(effects
 				(font
@@
 	)
 	(sheet
-		(at 59.69 74.93)
-		(size 50.8 27.305)
+		(at 66.04 57.15)
+		(size 50.8 34.29)
 		(exclude_from_sim no)
 		(in_bom yes)
@@
 		)
 		(property "Sheetname" "Power"
-			(at 59.69 74.2184 0)
+			(at 66.04 56.4384 0)
 			(effects
 				(font
@@
 		)
 		(property "Sheetfile" "power.kicad_sch"
-			(at 59.69 102.8196 0)
+			(at 66.04 92.0246 0)
 			(effects
 				(font
@@
 	)
 	(sheet
-		(at 41.91 128.27)
-		(size 49.53 35.56)
+		(at 180.34 99.06)
+		(size 50.8 34.29)
 		(exclude_from_sim no)
 		(in_bom yes)
@@
 		)
 		(property "Sheetname" "USB"
-			(at 41.91 127.5584 0)
+			(at 180.34 98.3484 0)
 			(effects
 				(font
@@
 		)
 		(property "Sheetfile" "usb.kicad_sch"
-			(at 41.91 164.4146 0)
+			(at 180.34 133.9346 0)
 			(effects
 				(font
@@
 	)
 	(sheet
-		(at 128.27 64.77)
-		(size 48.26 30.48)
+		(at 123.19 57.15)
+		(size 50.8 34.29)
 		(exclude_from_sim no)
 		(in_bom yes)
@@
 		)
 		(property "Sheetname" "FPGA_Power"
-			(at 128.27 64.0584 0)
+			(at 123.19 56.4384 0)
 			(effects
 				(font
@@
 		)
 		(property "Sheetfile" "fpga_power.kicad_sch"
-			(at 128.27 95.8346 0)
+			(at 123.19 92.0246 0)
 			(effects
 				(font
@@
 	)
 	(sheet
-		(at 231.14 86.36)
-		(size 44.45 30.48)
+		(at 66.04 140.97)
+		(size 50.8 34.29)
 		(exclude_from_sim no)
 		(in_bom yes)
@@
 		)
 		(property "Sheetname" "Connectivity"
-			(at 231.14 85.6484 0)
+			(at 66.04 140.2584 0)
 			(effects
 				(font
@@
 		)
 		(property "Sheetfile" "connectivity.kicad_sch"
-			(at 231.14 117.4246 0)
+			(at 66.04 175.8446 0)
 			(effects
 				(font
@@
 	)
 	(sheet
-		(at 213.36 35.56)
-		(size 45.72 30.48)
+		(at 66.04 99.06)
+		(size 50.8 34.29)
 		(exclude_from_sim no)
 		(in_bom yes)
@@
 		)
 		(property "Sheetname" "JTAG"
-			(at 213.36 34.8484 0)
+			(at 66.04 98.3484 0)
 			(effects
 				(font
@@
 		)
 		(property "Sheetfile" "jtag.kicad_sch"
-			(at 213.36 66.6246 0)
-			(effects
-				(font
+			(at 66.04 133.9346 0)
+			(effects
+				(font

Commit message: Finished PCB Design - WARNING MORE CHANGES NEEDED! The main decision to be made is, whether to increase the layer count to 8 layers, and make the P7 and P8 permamently on 3V3
Other:
- added sheet Input (voltage_input.kicad_sch)
Changed lines of the file:
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@@
 			(project "Controller_Board"
 				(path "/4e6e1af1-ede9-4a56-9d5f-a8dfd7fbcf8d"
-					(page "3")
+					(page "4")
 				)
 			)
@@
 			(project "Controller_Board"
 				(path "/4e6e1af1-ede9-4a56-9d5f-a8dfd7fbcf8d"
-					(page "5")
+					(page "6")
 				)
 			)
@@
 			(project "Controller_Board"
 				(path "/4e6e1af1-ede9-4a56-9d5f-a8dfd7fbcf8d"
-					(page "1")
+					(page "2")
 				)
 			)
@@
 			(project "Controller_Board"
 				(path "/4e6e1af1-ede9-4a56-9d5f-a8dfd7fbcf8d"
-					(page "6")
+					(page "7")
 				)
 			)
@@
 			(project "Controller_Board"
 				(path "/4e6e1af1-ede9-4a56-9d5f-a8dfd7fbcf8d"
-					(page "2")
+					(page "3")
 				)
 			)
@@
 			(project "Controller_Board"
 				(path "/4e6e1af1-ede9-4a56-9d5f-a8dfd7fbcf8d"
-					(page "7")
+					(page "8")
 				)
 			)
@@
 			(project "Controller_Board"
 				(path "/4e6e1af1-ede9-4a56-9d5f-a8dfd7fbcf8d"
-					(page "4")
-				)
-			)
+					(page "5")
+				)
+			)
+		)
+	)
+	(sheet
+		(at 123.19 140.97)
+		(size 50.8 34.29)
+		(exclude_from_sim no)
+		(in_bom yes)
+		(on_board yes)
+		(dnp no)
+		(fields_autoplaced yes)
+		(stroke
+			(width 0.1524)
+			(type solid)
+		)
+		(fill
+			(color 0 0 0 0)
+		)
+		(property "Sheetname" "Input"
+			(at 123.19 140.2584 0)
+			(show_name no)
+			(do_not_autoplace no)
+			(effects
+				(font
+					(size 1.27 1.27)
+				)
+				(justify left bottom)
+			)
+		)
+		(property "Sheetfile" "voltage_input.kicad_sch"
+			(at 123.19 175.8446 0)
+			(show_name no)
+			(do_not_autoplace no)
+			(effects
+				(font
+					(size 1.27 1.27)
+				)
+				(justify left top)
+			)
+		)
+		(instances
+			(project "Controller_Board"
+				(path "/4e6e1af1-ede9-4a56-9d5f-a8dfd7fbcf8d"
+					(page "1")
+				)
+			)
