File: Hardware/Controller_Board/voltage_input.kicad_sch (KiCad schematic)
At the start: 15 parts, among them Q101 Si7252ADP, U101 TDS5311P, U102 LTC4368, U103 XT30

Commit message: Finished procuring almost all boards - CHANGED XDC IN XILINX FOR TESTING!! - Programmer needed
Parts:
- C101: value 10u -> 4.7u; LCSC (none) -> C2997285; Manufacturer (none) -> Murata
- C102: LCSC (none) -> C85866; Manufacturer (none) -> Murata
- C103: LCSC (none) -> C77019; Manufacturer (none) -> Murata
- C104: LCSC (none) -> C77020; Manufacturer (none) -> Murata
- Q101: LCSC (none) -> C3289528; Manufacturer (none) -> Vishay
- R101: value 15mOhm 1/2W -> 17mOhm 1/2W; LCSC (none) -> C201283; Manufacturer (none) -> Walter
- R102: LCSC (none) -> C445774; Manufacturer (none) -> Panasonic
- R103: LCSC (none) -> C482106; Manufacturer (none) -> Vishay
- R104, R105: LCSC (none) -> C2076674; Manufacturer (none) -> Vishay
- R106: value 277k -> 280k; LCSC (none) -> C4198226; Manufacturer (none) -> Vishay
- R107: value 23k -> 23.2k; LCSC (none) -> C2076557; Manufacturer (none) -> Vishay
- U101: LCSC (none) -> C9900267203; Manufacturer (none) -> Semtech
- U102: LCSC (none) -> C688380; Manufacturer (none) -> ADI
- U103: LCSC (none) -> C431092; Manufacturer (none) -> Amass
Connections:
- net SENSE: now also Q101.6 (D); no longer Q101.6 (D)
- net VIN: now also Q101.5 (D); no longer Q101.5 (D)
Other:
- note added: "2.94A Current Limit"
- note removed: "3.33A Current Limit"
- note removed: "Maybe connect the P8_RX J4 and H4 and use the Bank 35 at 3V3"

Commit message: Finished PCB design and Review + Procured Boards
Parts:
- R103: LCSC C482106 -> C482105
Changed lines of the file:
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@@
 			)
 		)
-		(property "Datasheet" "https://www.lcsc.com/product-detail/C482106.html"
+		(property "Datasheet" "https://www.lcsc.com/product-detail/C482105.html"
 			(at 123.19 81.28 0)
 			(hide yes)
@@
 			)
 		)
-		(property "LCSC" "C482106"
+		(property "LCSC" "C482105"
 			(at 123.19 81.28 0)
 			(hide yes)
