File: Hardware/Core_Module/Connectivity.kicad_sch (KiCad schematic)
At the start: 30 parts, among them J201 Connector_Left, J202 Connector_Bottom, J203 Connector_Right, J205 Connector_Top

Commit message: Generated manufacturing files for Module boards
Parts:
- D201, D202, D203, D204, D205, D206, D207, D208, D209, D210, D211, D212, D213, D215, D216, D217, D218, D219, D220, D221, D222, D223, D224, D225, D226: LCSC (none) -> C2939949; Manufacturer (none) -> Infineon
- D214: value (none) -> TVS; LCSC (none) -> C2939949; Manufacturer (none) -> Infineon
- J201, J202, J203, J205: Manufacturer (none) -> Connfly; now left out of the parts list
