File: Hardware/Core_Module/Core_Module.kicad_pcb (KiCad board)
At the start: 6 copper layers, 13 x 13 mm, 53 parts, among them J201 Connector_Left, J202 Connector_Bottom, J203 Connector_Right, U101 TPS7A20L_1V2, U102 ICE40UL1K-CM36AI, U103 TPS7A20L_2V2, U104 TPS7A20L_3V3, U105 N25Q032A, Y101 12MHz

Commit message: Commit with restored changes after KiCad crash
Parts:
- removed C102, C106, C111: 4u7, Capacitor_SMD:C_0603_1608Metric
- removed R102: 10k, Resistor_SMD:R_0201_0603Metric
- added J205: Connector_Top, Custom_VoxLink_Footprints:6-Pin_Casselated_Edge, F.Cu at (148.8, 84.8)
- C104, C105, C108, C109, C114, C115: footprint Capacitor_SMD:C_0402_1005Metric -> Capacitor_SMD:C_0201_0603Metric
- C110: footprint Capacitor_SMD:C_0603_1608Metric -> Capacitor_SMD:C_0201_0603Metric
- U103: value TPS7A20L_2V2 -> TPS7A20L_2V5
- moved R103 1.21 mm to (144.3, 86.9)
- moved R106 1.15 mm to (145.0, 86.9)
- moved D101 0.65 mm to (143.8, 85.5)
- moved D102 0.65 mm to (144.5, 85.5)
- moved C110 0.39 mm to (145.7, 88.2)
- moved C108 0.28 mm to (152.4, 88.3)
- moved C107 0.22 mm to (147.7, 90.2)
- moved R101 0.22 mm to (146.9, 90.2)
- moved U103 0.21 mm to (151.3, 88.3)
- moved U104 0.21 mm to (149.1, 88.3)
- moved C104 0.21 mm to (147.9, 88.2)
- moved U101 0.21 mm to (146.8, 88.3)
- moved C101 0.20 mm to (145.2, 92.5)
- moved C103 0.20 mm to (145.2, 94.2)
- moved C112 0.20 mm to (148.9, 94.4)
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Connections:
- C110 pad 2: Net-(C110-Pad2) -> GND
Routing:
- net GND: track 4.37 -> 2.99 mm, vias 39 -> 36
- net Net-(C110-Pad2): track 1.32 -> 0.00 mm
- net +3V3: track 3.13 -> 1.90 mm
- net Net-(D101-A): track 0.70 -> 1.62 mm
- net /FPGA/LED: track 7.95 -> 8.81 mm
- net +1V2_CORE: track 2.35 -> 3.14 mm
- net /FPGA/CDONE: track 10.8 -> 11.5 mm, vias 6 -> 7

Commit message: Wrapping up for today. Almost reworked core module
Routing:
- net IOB_7B_G5: track 3.43 -> 16.8 mm
- net /FPGA/FLASH_SCK: track 2.49 -> 12.8 mm, vias 0 -> 3
- net /FPGA/FLASH_~{CS}: track 5.11 -> 14.0 mm, vias 0 -> 1
- net /FPGA/FLASH_MISO: track 7.78 -> 15.8 mm, vias 2 -> 3
- net /FPGA/FLASH_MOSI: track 4.60 -> 10.2 mm, vias 0 -> 1
- net /FPGA/CDONE: track 11.5 -> 12.7 mm
- net /FPGA/FLASH_~{HOLD}: track 3.81 -> 4.59 mm, vias 0 -> 1
- net GND: track 2.99 -> 3.49 mm

Commit message: Finished Lattice Core, waiting for PCB Review
Parts:
- added D221: TVS, Custom_VoxLink_Footprints:WLL-2-3, F.Cu at (145.8, 86.8)
- added D222: TVS, Custom_VoxLink_Footprints:WLL-2-3, F.Cu at (153.6, 86.3)
- added D223: TVS, Custom_VoxLink_Footprints:WLL-2-3, F.Cu at (152.4, 86.8)
- added D224: TVS, Custom_VoxLink_Footprints:WLL-2-3, F.Cu at (150.2, 86.8)
- added D225: TVS, Custom_VoxLink_Footprints:WLL-2-3, F.Cu at (148.0, 86.8)
- added D226: TVS, Custom_VoxLink_Footprints:WLL-2-3, F.Cu at (145.2, 85.9)
- moved R103 0.35 mm to (144.3, 87.2)
- moved R106 0.35 mm to (145.0, 87.2)
Connections:
- D102 pad 2: /FPGA/CDONE -> CDONE
- D220 pad 2: ~{CRESET} -> IOT_18B
- J201 pad 1: ~{CRESET} -> IOT_18B
- J205 pad 1: unconnected-(J205-Pin_1-Pad1) -> FLASH_~{CS}
- J205 pad 2: unconnected-(J205-Pin_2-Pad2) -> FLASH_MISO
- J205 pad 3: unconnected-(J205-Pin_3-Pad3) -> FLASH_SCK
- J205 pad 4: unconnected-(J205-Pin_4-Pad4) -> FLASH_MOSI
- J205 pad 5: unconnected-(J205-Pin_5-Pad5) -> CDONE
- J205 pad 6: unconnected-(J205-Pin_6-Pad6) -> ~{CRESET}
- R106 pad 2: /FPGA/CDONE -> CDONE
- U102 pad B5: unconnected-(U102C-IOT_18B-PadB5) -> IOT_18B
- U102 pad D5: /FPGA/CDONE -> CDONE
- U102 pad E5: /FPGA/FLASH_MISO -> FLASH_MISO
- U102 pad E6: /FPGA/FLASH_SCK -> FLASH_SCK
- U102 pad F5: /FPGA/FLASH_~{CS} -> FLASH_~{CS}
- U102 pad F6: /FPGA/FLASH_MOSI -> FLASH_MOSI
- U105 pad 1: /FPGA/FLASH_~{CS} -> FLASH_~{CS}
- U105 pad 2: /FPGA/FLASH_MISO -> FLASH_MISO
- U105 pad 5: /FPGA/FLASH_MOSI -> FLASH_MOSI
- U105 pad 6: /FPGA/FLASH_SCK -> FLASH_SCK
Routing:
- net FLASH_MISO: track 0.00 -> 16.9 mm, vias 0 -> 4
- net FLASH_~{CS}: track 0.00 -> 15.9 mm, vias 0 -> 2
- net /FPGA/FLASH_MISO: track 15.8 -> 0.00 mm, vias 3 -> 0
- net CDONE: track 0.00 -> 14.8 mm, vias 0 -> 6
- net FLASH_SCK: track 0.00 -> 14.3 mm, vias 0 -> 4
- net /FPGA/FLASH_~{CS}: track 14.0 -> 0.00 mm, vias 1 -> 0
- net IOT_18B: track 0.00 -> 13.4 mm, vias 0 -> 4
- net IOB_7B_G5: track 16.8 -> 3.43 mm
- net /FPGA/FLASH_SCK: track 12.8 -> 0.00 mm, vias 3 -> 0
- net /FPGA/CDONE: track 12.7 -> 0.00 mm, vias 7 -> 0
- net FLASH_MOSI: track 0.00 -> 12.7 mm, vias 0 -> 2
- net ~{CRESET}: track 6.71 -> 18.9 mm
- net /FPGA/FLASH_MOSI: track 10.2 -> 0.00 mm, vias 1 -> 0
- net IOB_4A: track 4.39 -> 3.18 mm
- net Net-(D101-A): track 1.62 -> 2.35 mm
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
Commit message: Advanced Intel Core Module Development
Connections:
- net I2C_SCL renamed IOT_22B_G0
- net I2C_SDA renamed IOB_3B_G6
- net I2C_~{RST} renamed IOT_21A_G1
