File: Hardware/Core_Module/Core_Module.kicad_pcb (KiCad board)
At the start: 6 copper layers, 13 x 13 mm, 56 parts, among them J201 Connector_Left, J202 Connector_Bottom, J203 Connector_Right, J205 Connector_Top, U101 TPS7A20L_1V2, U102 ICE40UL1K-CM36AI, U103 TPS7A20L_2V5, U104 TPS7A20L_3V3, U105 N25Q032A, Y101 12MHz

Commit message: Generated manufacturing files for Module boards
Other:
- board text added: "iCE40-UL"

Commit message: Finished procuring almost all boards - CHANGED XDC IN XILINX FOR TESTING!! - Programmer needed
Parts:
- C110: value 10u -> 2.2u
- D214: value ~ -> TVS
- R103, R106: value 510R -> 499R
- U105: value N25Q032A -> W25Q32JV
Changed lines of the file:
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@@
 		(capping no)
 		(filling no)
-		(zone_defaults)
 		(pcbplotparams
 			(layerselection 0x00000000_00000000_55555555_5755f5ff)
@@
 			)
 		)
-		(property "Value" "~"
+		(property "Value" "TVS"
 			(at 0 1 0)
 			(unlocked yes)
@@
 			)
 		)
-		(attr through_hole)
+		(attr through_hole exclude_from_bom)
 		(duplicate_pad_numbers_are_jumpers no)
 		(fp_line
@@
 			)
 		)
-		(property "Value" "510R"
+		(property "Value" "499R"
 			(at 0 1.05 90)
 			(layer "F.Fab")
@@
 			)
 		)
-		(property "Value" "N25Q032A"
+		(property "Value" "W25Q32JV"
 			(at 0 3 180)
 			(unlocked yes)
@@
 			)
 		)
-		(attr through_hole)
+		(attr through_hole exclude_from_bom)
 		(duplicate_pad_numbers_are_jumpers no)
 		(fp_line
@@
 			)
 		)
-		(attr through_hole)
+		(attr through_hole exclude_from_bom)
 		(duplicate_pad_numbers_are_jumpers no)
 		(fp_line
@@
 			)
 		)
-		(property "Value" "10u"
+		(property "Value" "2.2u"
 			(at 0 1.05 90)
 			(layer "F.Fab")
@@
 			)
 		)
-		(attr through_hole)
+		(attr through_hole exclude_from_bom)
 		(duplicate_pad_numbers_are_jumpers no)
 		(fp_line
@@
 			)
 		)
-		(property "Value" "510R"
+		(property "Value" "499R"
 			(at 0 1.05 90)
 			(layer "F.Fab")
