File: Hardware/Core_Module/fpga.kicad_sch (KiCad schematic)
At the start: 26 parts, among them U101 TPS7A20L_1V2, U102 ICE40UL1K-CM36AI, U103 TPS7A20L_2V5, U104 TPS7A20L_3V3, U105 N25Q032A, Y101 12MHz

Commit message: Generated manufacturing files for Module boards
Parts:
- C101, C103, C107, C112, C113, C116: LCSC (none) -> C668346; Manufacturer (none) -> Murata
- C104, C105, C108, C109, C114, C115: LCSC (none) -> C335102; Manufacturer (none) -> Murata
- C110: value 10u -> 2.2u; LCSC (none) -> C335106; Manufacturer (none) -> Murata
- D101: LCSC (none) -> C5846955; Manufacturer (none) -> Kingbright
- D102: LCSC (none) -> C4153580; Manufacturer (none) -> Kingbright
- R101: LCSC (none) -> C3009113; Manufacturer (none) -> Vishay
- R103, R106: value 510R -> 499R; LCSC (none) -> C2094902; Manufacturer (none) -> Vishay
- R104, R105: LCSC (none) -> C844303; Manufacturer (none) -> Vishay
- U101: LCSC (none) -> C30875939; Manufacturer (none) -> TI
- U102: LCSC (none) -> C1519040; Manufacturer (none) -> Lattice
- U103: LCSC (none) -> C41487851; Manufacturer (none) -> TI
- U104: LCSC (none) -> C22445532; Manufacturer (none) -> TI
- U105: value N25Q032A -> W25Q32JV; LCSC (none) -> C2999380; Manufacturer (none) -> Winbond
- Y101: LCSC (none) -> SMD1612-4P; Manufacturer (none) -> Abracon
Other:
- note added: "No room for larger bulk capacitors"
- moved on the sheet: C110

Commit message: Finished PCB design and Review + Procured Boards
Other:
- note added: "INCLUDE A PULLUP ON ~{CRESET} IN NEXT REVISION!"
Changed lines of the file:
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@@
+		)
+	)
+	(text "INCLUDE A PULLUP ON\n~{CRESET} IN NEXT REVISION!"
+		(exclude_from_sim no)
+		(at 98.806 172.212 0)
+		(effects
+			(font
+				(size 1.27 1.27)
+				(thickness 0.254)
+				(bold yes)
+				(color 255 0 0 1)
+			)
 		)
 	)
