File: Hardware/Core_Module_Intel/Core_Module_Intel.kicad_sch (KiCad schematic)
At the start: 6 parts, among them U101 TPS7A20L_1V2, U103 TPS7A20L_2V5

Commit message: Advanced Intel Core Module Development
Parts:
- added C110, C111, C112, C113, C116, C117: 100n, Capacitor_SMD:C_0402_1005Metric, symbol Device:C
- added D101, D102: LED, LED_SMD:LED_0201_0603Metric, symbol Device:LED
- added J201: Connector_Left, Custom_VoxLink_Footprints:7-Pin_Casselated_Edge, symbol Connector:Conn_01x07_Socket
- added J202: Connector_Bottom, Custom_VoxLink_Footprints:7-Pin_Casselated_Edge, symbol Connector:Conn_01x07_Socket
- added J203: Connector_Right, Custom_VoxLink_Footprints:7-Pin_Casselated_Edge, symbol Connector:Conn_01x07_Socket
- added J205: Connector_Top, Custom_VoxLink_Footprints:6-Pin_Casselated_Edge, symbol Connector:Conn_01x06_Socket
- added R103, R106: 510R, Resistor_SMD:R_0201_0603Metric, symbol Device:R
- added R2, R3, R4, R5: 10k, Resistor_SMD:R_0402_1005Metric, symbol Device:R
- added R6, R7: 100R, Resistor_SMD:R_0402_1005Metric, symbol Device:R
- added U1: 10M02DCV36C8G, Custom_VoxLink_Footprints:10M02DCV36C8G, symbol Custom_VoxLink_Symbols:10M02DCV36C8G
Connections:
- net +1V2_CORE: now also C110.1, C111.1, U1.B1 (VCC), U1.F5 (VCC)
- net +5V: now also J201.6 (Pin_6)
- net GND: now also C110.2, C111.2, C112.2, C113.2, C116.2, C117.2, D101.1 (K), D102.1 (K), J201.1 (Pin_1), J201.7 (Pin_7), J202.3 (Pin_3), U1.B3 (GND), U1.F1 (GND), U1.F6 (GND)
- net +2V5_NVCM renamed +2V5
- net +2V5: now also C112.1, C113.1, C116.1, C117.1, R106.1, R2.1, R3.1, R4.1, R5.1, U1.A1 (VCCA3), U1.A6 (VCCA2), U1.C4 (VCCIO_1_2_8), U1.D4 (VCCIO_3_5_6)
- new net: R5.2, U1.B2 (NSTATUS)
- new net: R3.2, U1.A2 (CONFIG_DONE)
- new net: R4.2, U1.A4 (NCONFIG)
- new net: R2.2, U1.C2 (JTAGEN)
- new net: D101.2 (A), R103.2
- new net: D102.2 (A), R106.2
- new net CDONE: J205.5 (Pin_5)
- new net IN_CLK_N: J202.5 (Pin_5), R6.2, U1.E6 (DIFFOUT_R10n)
- new net IN_CLK_P: J202.4 (Pin_4), R6.1, U1.D6 (DIFFOUT_R10p)
- new net IN_DATA_N: J201.3 (Pin_3), R7.2, U1.C6 (DIFFOUT_R12n)
- new net IN_DATA_P: J201.2 (Pin_2), R7.1, U1.D5 (DIFFOUT_R12p)
- new net LED: R103.1
- new net NRST: U1.A5 (DEV_CLRN)
- new net OUT_CLK_N: J202.2 (Pin_2), U1.F2 (DIFFOUT_B1n)
- new net OUT_CLK_P: J202.1 (Pin_1), U1.F3 (DIFFOUT_B1p)
- new net OUT_DATA_N: J202.7 (Pin_7), U1.E3 (DIFFOUT_B7n)
- new net OUT_DATA_P: J202.6 (Pin_6), U1.F4 (DIFFOUT_B7p)
- new net TCK: J205.3 (Pin_3), U1.D3 (TCK)
- new net TDI: J205.4 (Pin_4), U1.C1 (TDI)
- new net TDO: J205.2 (Pin_2), U1.D2 (TDO)
- new net TMS: J205.1 (Pin_1), U1.C3 (TMS)
- new net ~{CRESET}: J205.6 (Pin_6)
- no-connect marks 0 -> 2
Other:
- note added: "Input from transmit of the master"
- note added: "Output to receive of the master"
