File: Hardware/Sensor_Module/connectivity.kicad_sch (KiCad schematic)
At the start: 14 parts, among them J1 Connector_Left, J2 Connector_Right

Commit message: Generated manufacturing files for Module boards
Parts:
- D10, D11, D12, D13, D2, D3, D4, D5, D6, D7, D8, D9: LCSC (none) -> C2939949; Manufacturer (none) -> Infineon
- J1, J2: Manufacturer (none) -> Connfly; now left out of the parts list
