File: Hardware/Sensor_Module/sensor.kicad_sch (KiCad schematic)
At the start: 20 parts, among them U1 BNO086, U2 TPS7A20L_3V3, Y1 32.768 kHz

Commit message: Generated manufacturing files for Module boards
Parts:
- C1, C2, C5: LCSC (none) -> C77020; Manufacturer (none) -> Murata
- C3, C4: value 1u -> 4.7u; LCSC (none) -> C2858031; Manufacturer (none) -> Murata
- C6, C7: LCSC (none) -> C2169087; Manufacturer (none) -> Murata
- D1: LCSC (none) -> C7466700; Manufacturer (none) -> Broadcom
- R1, R2, R5, R6: LCSC (none) -> C482193; Manufacturer (none) -> Vishay
- R3, R4, R8: LCSC (none) -> C71617; Manufacturer (none) -> Vishay
- R7: LCSC (none) -> C482201; Manufacturer (none) -> Vishay
- R9: LCSC (none) -> C482106; Manufacturer (none) -> Vishay
- U1: LCSC (none) -> C5264422; Manufacturer (none) -> CEVA
- U2: LCSC (none) -> C22445532; Manufacturer (none) -> TI
- Y1: LCSC (none) -> C5154201; Manufacturer (none) -> Epson
