File: Hardware/Sensor_Module/Sensor_Module.kicad_pcb (KiCad board)
At the start: 4 copper layers, 13 x 13 mm, 34 parts, among them J1 Connector_Left, J2 Connector_Right, U1 BNO086, U2 TPS7A20L_3V3, Y1 32.768 kHz

Commit message: Generated manufacturing files for Module boards
Parts:
- moved D2 0.36 mm to (144.3, 88.3), turned to 180 degrees
Routing:
- net +5V: track 3.07 -> 2.02 mm
- net GND: track 23.3 -> 23.2 mm, vias 24 -> 23
Changed lines of the file:
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@@
 			(usegerberattributes yes)
 			(usegerberadvancedattributes yes)
-			(creategerberjobfile yes)
+			(creategerberjobfile no)
 			(dashed_line_dash_ratio 12)
 			(dashed_line_gap_ratio 3)
@@
 			(plotframeref no)
 			(mode 1)
-			(useauxorigin no)
+			(useauxorigin yes)
 			(pdf_front_fp_property_popups yes)
 			(pdf_back_fp_property_popups yes)
@@
 			(plotpadnumbers no)
 			(hidednponfab no)
-			(sketchdnponfab yes)
-			(crossoutdnponfab yes)
+			(sketchdnponfab no)
+			(crossoutdnponfab no)
 			(subtractmaskfromsilk no)
 			(outputformat 1)
 			(mirror no)
-			(drillshape 1)
+			(drillshape 0)
 			(scaleselection 1)
-			(outputdirectory "")
+			(outputdirectory "gerber/")
 		)
 	)
@@
 		(fp_poly
 			(pts
-				(xy -0.85 -0.35) (xy -0.95 -0.45) (xy -0.95 -0.25)
+				(xy -0.8 -0.35) (xy -0.90018 -0.45) (xy -0.9 -0.25)
 			)
 			(stroke
@@
 	(footprint "Custom_VoxLink_Footprints:WLL-2-3"
 		(layer "F.Cu")
-		(at 144.3 88.71)
+		(at 144.3 88.35 180)
 		(property "Reference" "D2"
-			(at 0 -0.5 0)
+			(at 0 -0.5 180)
 			(unlocked yes)
 			(layer "F.SilkS")
@@
 		)
 		(property "Value" "TVS"
-			(at 0 1 0)
+			(at 0 1 180)
 			(unlocked yes)
 			(layer "F.Fab")
@@
 		)
 		(property "Datasheet" ""
-			(at 0 0 0)
+			(at 0 0 180)
 			(unlocked yes)
 			(layer "F.Fab")
@@
 		)
 		(property "Description" ""
-			(at 0 0 0)
+			(at 0 0 180)
 			(unlocked yes)
 			(layer "F.Fab")
@@
 		(duplicate_pad_numbers_are_jumpers no)
 		(fp_line
-			(start -0.25 -0.55)
+			(start 0.25 0.2)
 			(end -0.25 0.2)
 			(stroke
@@
 		)
 		(fp_line
-			(start -0.25 -0.55)
-			(end 0.25 -0.55)
+			(start 0.25 -0.55)
+			(end 0.25 0.2)
 			(stroke
 				(width 0.05)
@@
 		)
 		(fp_line
-			(start 0.25 -0.55)
-			(end 0.25 0.2)
+			(start -0.25 -0.55)
+			(end 0.25 -0.55)
 			(stroke
 				(width 0.05)
@@
 		)
 		(fp_line
-			(start 0.25 0.2)
+			(start -0.25 -0.55)
 			(end -0.25 0.2)
 			(stroke
@@
 		)
 		(fp_text user "${REFERENCE}"
-			(at 0 2.5 0)
+			(at 0 2.5 180)
 			(unlocked yes)
 			(layer "F.Fab")
@@
 		)
 		(pad "1" smd rect
-			(at 0 -0.36)
+			(at 0 -0.36 180)
 			(size 0.24 0.17)
 			(layers "F.Cu" "F.Mask" "F.Paste")
@@
 		)
 		(pad "2" smd rect
-			(at 0 0)
+			(at 0 0 180)
 			(size 0.24 0.17)
 			(layers "F.Cu" "F.Mask" "F.Paste")
@@
 		(fp_poly
 			(pts
-				(xy -2.7 -1.684671) (xy -2.903219 -1.494671) (xy -2.903219 -1.854671)
+				(xy -2.75 -1.65) (xy -2.95 -1.85) (xy -2.95 -1.45)
 			)
 			(stroke
@@
 		(duplicate_pad_numbers_are_jumpers no)
 		(fp_line
-			(start -1 -0.3)
-			(end -1 0.3)
+			(start -0.95 -0.15)
+			(end -0.95 0.15)
 			(stroke
 				(width 0.1)
@@
 	(gr_text "BNO086"
 		(at 149 97.21 0)
-		(layer "F.SilkS")
+		(layer "F.SilkS" knockout)
 		(effects
 			(font
@@
 	)
 	(segment
+		(start 144.3 88.71)
+		(end 144.3 89.175)
+		(width 0.1)
+		(layer "F.Cu")
+		(net "GND")
+	)
+	(segment
 		(start 146.55 90.27)
 		(end 147.3375 90.27)
@@
 	)
 	(segment
-		(start 144.75 88.175)
-		(end 144.575 88.35)
-		(width 0.1)
-		(layer "F.Cu")
-		(net "GND")
-	)
-	(segment
 		(start 149.75 91.622)
 		(end 150.398 92.27)
@@
 		(net "GND")
 	)
-	(segment
-		(start 144.575 88.35)
-		(end 144.3 88.35)
-		(width 0.1)
-		(layer "F.Cu")
-		(net "GND")
-	)
 	(via
 		(at 149.75 90.95)
@@
 	)
 	(via
-		(at 144.75 88.175)
-		(size 0.45)
-		(drill 0.2)
-		(layers "F.Cu" "B.Cu")
-		(free yes)
-		(net "GND")
-	)
-	(via
 		(at 147.702678 88.025)
 		(size 0.45)
@@
 	)
 	(segment
-		(start 143.25 88.71)
-		(end 144.3 88.71)
-		(width 0.1)
-		(layer "F.Cu")
-		(net "+5V")
-	)
-	(segment
 		(start 144.467082 87.425)
 		(end 144.702678 87.425)
@@
 	)
 	(segment
-		(start 143.25 95.06)
-		(end 144.3 95.06)
+		(start 148.05 94.35)
+		(end 147.9 94.5)
 		(width 0.1)
 		(layer "F.Cu")
@@
 	)
 	(segment
-		(start 145.4 95.5)
-		(end 144.96 95.06)
+		(start 143.25 95.06)
+		(end 144.3 95.06)
 		(width 0.1)
 		(layer "F.Cu")
@@
 	)
 	(segment
-		(start 149.25 94.9075)
-		(end 149.25 94.697)
+		(start 149.0765 94.35)
+		(end 148.05 94.35)
 		(width 0.1)
 		(layer "F.Cu")
@@
 	)
 	(segment
-		(start 148.903 94.35)
-		(end 147.825 94.35)
+		(start 147.9 94.5)
+		(end 147.9 94.972)
 		(width 0.1)
 		(layer "F.Cu")
@@
 	)
 	(segment
-		(start 149.25 94.697)
-		(end 148.903 94.35)
+		(start 149.25 94.9075)
+		(end 149.25 94.5235)
 		(width 0.1)
 		(layer "F.Cu")
@@
 	)
 	(segment
-		(start 147.372 95.5)
-		(end 145.4 95.5)
+		(start 145.4 95.5)
+		(end 144.96 95.06)
 		(width 0.1)
 		(layer "F.Cu")
@@
 	)
 	(segment
-		(start 147.825 94.35)
-		(end 147.825 95.047)
+		(start 147.9 94.972)
+		(end 147.372 95.5)
 		(width 0.1)
 		(layer "F.Cu")
@@
 	)
 	(segment
-		(start 147.825 95.047)
-		(end 147.372 95.5)
+		(start 147.372 95.5)
+		(end 145.4 95.5)
+		(width 0.1)
+		(layer "F.Cu")
+		(net "~{H_CS}")
+	)
+	(segment
+		(start 149.25 94.5235)
+		(end 149.0765 94.35)
 		(width 0.1)
 		(layer "F.Cu")
@@
 	)
 	(zone
+		(net "+5V")
+		(layer "F.Cu")
+		(hatch edge 0.5)
+		(priority 2)
+		(connect_pads yes
+			(clearance 0.2)
+		)
+		(min_thickness 0.1)
+		(fill yes
+			(thermal_gap 0.2)
+			(thermal_bridge_width 0.1)
+			(island_removal_mode 0)
+		)
+		(polygon
+			(pts
+				(xy 144.45 88.5) (xy 145.8 87.15) (xy 144.401172 87.15) (xy 143.050326 88.499089)
+			)
+		)
+	)
+	(zone
 		(net "+3V3")
 		(layer "F.Cu")
@@
 		(layer "In1.Cu")
 		(hatch edge 0.5)
-		(connect_pads
+		(connect_pads yes
 			(clearance 0.2)
 		)

Commit message: Finished procuring almost all boards - CHANGED XDC IN XILINX FOR TESTING!! - Programmer needed
Parts:
- C3, C4: value 1u -> 4.7u
Routing:
- added copper zone on In2.Cu, net GND
Changed lines of the file:
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@@
 			)
 		)
-		(property "Value" "1u"
+		(property "Value" "4.7u"
 			(at 0 1.16 90)
 			(layer "F.Fab")
@@
 			)
 		)
-		(attr smd)
+		(attr smd exclude_from_bom)
 		(duplicate_pad_numbers_are_jumpers no)
 		(fp_line
@@
 			)
 		)
-		(attr smd)
+		(attr smd exclude_from_bom)
 		(duplicate_pad_numbers_are_jumpers no)
 		(fp_line
@@
 			)
 		)
-		(property "Value" "1u"
+		(property "Value" "4.7u"
 			(at 0 1.16 90)
 			(layer "F.Fab")
@@
 		(layer "F.SilkS")
 	)
-	(gr_rect
-		(start 143.8 84.86)
-		(end 144.7 85.72)
-		(stroke
-			(width 0)
-			(type solid)
-		)
-		(fill yes)
-		(layer "F.SilkS")
-	)
 	(gr_line
 		(start 152.309485 96.429125)
@@
 	)
 	(gr_text "PWR"
-		(at 145.75 85.35 0)
+		(at 145.95 85.35 0)
 		(layer "F.SilkS" knockout)
 		(effects
@@
 			(polygon
 				(pts
-					(xy 145.045515 84.938528) (xy 145.090554 84.949236) (xy 145.128958 84.966206) (xy 145.161778 84.989275)
-					(xy 145.188193 85.018515) (xy 145.207771 85.05519) (xy 145.220353 85.100952) (xy 145.224908 85.158022)
-					(xy 145.220146 85.221059) (xy 145.207254 85.26956) (xy 145.187656 85.30659) (xy 145.161778 85.334463)
-					(xy 145.129264 85.355815) (xy 145.089432 85.37193) (xy 145.040792 85.382341) (xy 144.981533 85.386096)
-					(xy 144.831848 85.386096) (xy 144.831848 85.6405) (xy 144.685541 85.6405) (xy 144.685541 85.265733)
-					(xy 144.831848 85.265733) (xy 144.969095 85.265733) (xy 145.002924 85.262541) (xy 145.029399 85.25376)
-					(xy 145.050134 85.240002) (xy 145.065454 85.220879) (xy 145.075377 85.194514) (xy 145.079071 85.158492)
-					(xy 145.075326 85.122477) (xy 145.065374 85.096856) (xy 145.050134 85.078906) (xy 145.02955 85.066244)
-					(xy 145.003077 85.058081) (xy 144.969095 85.055098) (xy 144.831848 85.055098) (xy 144.831848 85.265733)
-					(xy 144.685541 85.265733) (xy 144.685541 84.934735) (xy 144.992517 84.934735)
+					(xy 145.245515 84.938528) (xy 145.290554 84.949236) (xy 145.328958 84.966206) (xy 145.361778 84.989275)
+					(xy 145.388193 85.018515) (xy 145.407771 85.05519) (xy 145.420353 85.100952) (xy 145.424908 85.158022)
+					(xy 145.420146 85.221059) (xy 145.407254 85.26956) (xy 145.387656 85.30659) (xy 145.361778 85.334463)
+					(xy 145.329264 85.355815) (xy 145.289432 85.37193) (xy 145.240792 85.382341) (xy 145.181533 85.386096)
+					(xy 145.031848 85.386096) (xy 145.031848 85.6405) (xy 144.885541 85.6405) (xy 144.885541 85.265733)
+					(xy 145.031848 85.265733) (xy 145.169095 85.265733) (xy 145.202924 85.262541) (xy 145.229399 85.25376)
+					(xy 145.250134 85.240002) (xy 145.265454 85.220879) (xy 145.275377 85.194514) (xy 145.279071 85.158492)
+					(xy 145.275326 85.122477) (xy 145.265374 85.096856) (xy 145.250134 85.078906) (xy 145.22955 85.066244)
+					(xy 145.203077 85.058081) (xy 145.169095 85.055098) (xy 145.031848 85.055098) (xy 145.031848 85.265733)
+					(xy 144.885541 85.265733) (xy 144.885541 84.934735) (xy 145.192517 84.934735)
 				)
 			)
 			(polygon
 				(pts
-					(xy 145.431397 84.934735) (xy 145.524662 85.338866) (xy 145.544708 85.451364) (xy 145.565267 85.341259)
-					(xy 145.644682 84.934735) (xy 145.800094 84.934735) (xy 145.883741 85.338866) (xy 145.905283 85.451364)
-					(xy 145.926783 85.34314) (xy 146.020987 84.934735) (xy 146.170672 84.934735) (xy 145.972218 85.6405)
-					(xy 145.831638 85.6405) (xy 145.746538 85.227778) (xy 145.721662 85.091301) (xy 145.696786 85.227778)
-					(xy 145.611685 85.6405) (xy 145.474909 85.6405) (xy 145.275045 84.934735)
+					(xy 145.631397 84.934735) (xy 145.724662 85.338866) (xy 145.744708 85.451364) (xy 145.765267 85.341259)
+					(xy 145.844682 84.934735) (xy 146.000094 84.934735) (xy 146.083741 85.338866) (xy 146.105283 85.451364)
+					(xy 146.126783 85.34314) (xy 146.220987 84.934735) (xy 146.370672 84.934735) (xy 146.172218 85.6405)
+					(xy 146.031638 85.6405) (xy 145.946538 85.227778) (xy 145.921662 85.091301) (xy 145.896786 85.227778)
+					(xy 145.811685 85.6405) (xy 145.674909 85.6405) (xy 145.475045 84.934735)
 				)
 			)
 			(polygon
 				(pts
-					(xy 146.658564 84.937842) (xy 146.695747 84.944216) (xy 146.72299 84.952944) (xy 146.759951 84.973691)
-					(xy 146.790694 85.002269) (xy 146.811258 85.030518) (xy 146.827025 85.061638) (xy 146.836917 85.095702)
-					(xy 146.840404 85.135882) (xy 146.837655 85.168805) (xy 146.829322 85.201627) (xy 146.815058 85.234745)
-					(xy 146.794855 85.26359) (xy 146.767405 85.286381) (xy 146.731368 85.303475) (xy 146.761879 85.319208)
-					(xy 146.784451 85.337857) (xy 146.80044 85.359468) (xy 146.810818 85.384648) (xy 146.818025 85.420386)
-					(xy 146.820785 85.469829) (xy 146.820785 85.517187) (xy 146.821998 85.56159) (xy 146.824632 85.582669)
-					(xy 146.834395 85.606629) (xy 146.851389 85.622804) (xy 146.851389 85.6405) (xy 146.689309 85.6405)
-					(xy 146.679735 85.602715) (xy 146.673537 85.542021) (xy 146.672554 85.476539) (xy 146.668571 85.431886)
-					(xy 146.659812 85.403607) (xy 146.647934 85.386695) (xy 146.630448 85.375423) (xy 146.602347 85.367401)
-					(xy 146.559244 85.364212) (xy 146.407166 85.364212) (xy 146.407166 85.6405) (xy 146.263252 85.6405)
-					(xy 146.263252 85.246585) (xy 146.407166 85.246585) (xy 146.574033 85.246585) (xy 146.620476 85.243201)
-					(xy 146.648661 85.234959) (xy 146.667525 85.222674) (xy 146.680975 85.205951) (xy 146.689518 85.183862)
-					(xy 146.692643 85.154731) (xy 146.689529 85.122792) (xy 146.681088 85.098757) (xy 146.668017 85.080766)
-					(xy 146.650072 85.067665) (xy 146.622893 85.058737) (xy 146.57835 85.055098) (xy 146.407166 85.055098)
-					(xy 146.407166 85.246585) (xy 146.263252 85.246585) (xy 146.263252 84.934735) (xy 146.608953 84.934735)
+					(xy 146.858564 84.937842) (xy 146.895747 84.944216) (xy 146.92299 84.952944) (xy 146.959951 84.973691)
+					(xy 146.990694 85.002269) (xy 147.011258 85.030518) (xy 147.027025 85.061638) (xy 147.036917 85.095702)
+					(xy 147.040404 85.135882) (xy 147.037655 85.168805) (xy 147.029322 85.201627) (xy 147.015058 85.234745)
+					(xy 146.994855 85.26359) (xy 146.967405 85.286381) (xy 146.931368 85.303475) (xy 146.961879 85.319208)
+					(xy 146.984451 85.337857) (xy 147.00044 85.359468) (xy 147.010818 85.384648) (xy 147.018025 85.420386)
+					(xy 147.020785 85.469829) (xy 147.020785 85.517187) (xy 147.021998 85.56159) (xy 147.024632 85.582669)
+					(xy 147.034395 85.606629) (xy 147.051389 85.622804) (xy 147.051389 85.6405) (xy 146.889309 85.6405)
+					(xy 146.879735 85.602715) (xy 146.873537 85.542021) (xy 146.872554 85.476539) (xy 146.868571 85.431886)
+					(xy 146.859812 85.403607) (xy 146.847934 85.386695) (xy 146.830448 85.375423) (xy 146.802347 85.367401)
+					(xy 146.759244 85.364212) (xy 146.607166 85.364212) (xy 146.607166 85.6405) (xy 146.463252 85.6405)
+					(xy 146.463252 85.246585) (xy 146.607166 85.246585) (xy 146.774033 85.246585) (xy 146.820476 85.243201)
+					(xy 146.848661 85.234959) (xy 146.867525 85.222674) (xy 146.880975 85.205951) (xy 146.889518 85.183862)
+					(xy 146.892643 85.154731) (xy 146.889529 85.122792) (xy 146.881088 85.098757) (xy 146.868017 85.080766)
+					(xy 146.850072 85.067665) (xy 146.822893 85.058737) (xy 146.77835 85.055098) (xy 146.607166 85.055098)
+					(xy 146.607166 85.246585) (xy 146.463252 85.246585) (xy 146.463252 84.934735) (xy 146.808953 84.934735)
 				)
 			)
@@
 	(zone
 		(net "GND")
-		(layer "In1.Cu")
+		(layers "In1.Cu" "In2.Cu")
 		(hatch edge 0.5)
 		(connect_pads yes
