File: Hardware/Shell_Module_BUS/Shell_Module_BUS.kicad_pcb (KiCad board)
At the start: 4 copper layers, 54 x 29.5 mm, 6 parts, among them J1 PicoBlade, J2 RJ45_Output, U1 VoxLink_Core_Module, U2 VoxLink_BNO086_Module

Commit message: Finished procuring almost all boards - CHANGED XDC IN XILINX FOR TESTING!! - Programmer needed
Parts:
- added C1: 10u, Capacitor_SMD:C_1206_3216Metric, B.Cu at (92.7, 65.1)
- added R1: 1R, Resistor_SMD:R_0603_1608Metric, B.Cu at (92.7, 61.2)
Routing:
- net Net-(C1-Pad2): track 0.00 -> 1.52 mm
- net GND: track 0.00 -> 0.77 mm, vias 0 -> 1

Commit message: Finished PCB design and Review + Procured Boards
Parts:
- added C304: 1u, Capacitor_SMD:C_0603_1608Metric, B.Cu at (109.0, 71.1)
- added R2: 10k, Resistor_SMD:R_0603_1608Metric, B.Cu at (114.7, 61.6)
- added SW301: Reset, Button_Switch_THT:SW_TH_Tactile_Omron_B3F-102x, B.Cu at (107.5, 63.4)
Connections:
- U1 pad 1: unconnected-(U1-NRESET-Pad1) -> /NRESET
- U2 pad 9: unconnected-(U2-+3V3-Pad9) -> +3V3
Routing:
- net /NRESET: track 0.00 -> 25.2 mm, vias 0 -> 1
- net /TX_N: track 45.2 -> 58.7 mm
- net /TX_P: track 45.6 -> 58.7 mm
- net /RX_P: track 46.0 -> 58.8 mm
- net /RX_N: track 48.9 -> 58.8 mm
- net /CLK_N: track 55.2 -> 58.9 mm
- net GND: track 0.77 -> 2.50 mm
- net +3V3: track 0.00 -> 1.58 mm
- net +5V: track 56.8 -> 57.5 mm
Other:
- board text added: "RST"
