File: Hardware/Shell_Module_BUS/Shell_Module_BUS.kicad_sch (KiCad schematic)
At the start: 6 parts, among them J1 PicoBlade, J2 RJ45_Output, U1 VoxLink_Core_Module, U2 VoxLink_BNO086_Module

Commit message: Finished procuring almost all boards - CHANGED XDC IN XILINX FOR TESTING!! - Programmer needed
Parts:
- added C1: 10u, Capacitor_SMD:C_1206_3216Metric, symbol Device:C
- added R1: 1R, Resistor_SMD:R_0603_1608Metric, symbol Device:R
Connections:
- net +5V: now also C1.1
- net GND: now also R1.2
- new net: C1.2, R1.1

Commit message: Finished PCB design and Review + Procured Boards
Parts:
- added C304: 1u, Capacitor_SMD:C_0603_1608Metric, symbol Device:C
- added R2: 10k, Resistor_SMD:R_0603_1608Metric, symbol Device:R
- added SW301: Reset, Button_Switch_THT:SW_TH_Tactile_Omron_B3F-102x, symbol Switch:SW_Push
- C1: LCSC (none) -> C77092
- J1, J2, U1, U2: now left out of the parts list
- R1: LCSC (none) -> C445774
Connections:
- net GND: now also C304.2, SW301.2
- net +3V3: now reaches U2.9 (+3V3)
- net +3V3: now also R2.1
- net NRESET: now reaches U1.1 (NRESET)
- net NRESET: now also C304.1, R2.2, SW301.1
- no-connect marks 22 -> 20
Other:
- note added: "FPGA Manual Reset"
