File: Hardware/Shell_Module_DAISY/Shell_Module_DAISY.kicad_pcb (KiCad board)
At the start: 4 copper layers, 54 x 29.5 mm, 6 parts, among them J1 PicoBlade, J2 RJ45_Output, U1 VoxLink_Core_Module, U2 VoxLink_BNO086_Module

Commit message: Finished PCB design and Review + Procured Boards
Parts:
- added C1: 10u, Capacitor_SMD:C_1206_3216Metric, B.Cu at (111.9, 87.5)
- added C304: 1u, Capacitor_SMD:C_0805_2012Metric, B.Cu at (128.5, 93.5)
- added R1: 1R, Resistor_SMD:R_0603_1608Metric, B.Cu at (111.9, 83.8)
- added R2: 10k, Resistor_SMD:R_0603_1608Metric, B.Cu at (134.0, 84.1)
- added SW301: Reset, Button_Switch_THT:SW_TH_Tactile_Omron_B3F-102x, B.Cu at (126.8, 85.8)
Connections:
- U1 pad 1: unconnected-(U1-NRESET-Pad1) -> /NRESET
- U2 pad 9: unconnected-(U2-+3V3-Pad9) -> +3.3V
Routing:
- net /NRESET: track 0.00 -> 25.2 mm
- net /OUT_RX_N: track 32.9 -> 42.8 mm
- net /OUT_RX_P: track 34.8 -> 42.9 mm
- net /OUT_CLK_N: track 39.0 -> 42.9 mm
- net GND: track 0.00 -> 2.42 mm, vias 0 -> 1
- net +3.3V: track 0.00 -> 1.53 mm
- net Net-(C1-Pad2): track 0.00 -> 1.50 mm
- net /TX_P: track 45.7 -> 47.2 mm
- net +5V: track 56.8 -> 57.5 mm
- net /OUT_CLK_P: track 42.3 -> 43.0 mm
Other:
- board text added: "RST"
